Commit message: No comments

File: hyq_description/robots/hyq_gazebo.urdf.xacro (robot description, xacro)
@@ -78,5 +78,5 @@
 		name="ptu"
 		parent="trunk">
-		<origin xyz="0.693327 -0.015447 0.119533" rpy="-0.013127 0.574478 -0.007748"/>
+		<origin xyz="0.693327 -0.015447 0.119533" rpy="-0.013127 0.754478 -0.007748"/> <!-- <origin xyz="0.693327 -0.015447 0.119533" rpy="-0.013127 0.754478 -0.007748"/>-->
 	</xacro:ptu_d46>
 	<!-- Asus Xtion Pro -->
