Commit message: Added new files for the description of the PTU unit. Cleaded unuseful files

File: hyq_description/robots/hyq.urdf.xacro (robot description, xacro)
@@ -14,4 +14,5 @@
 	<xacro:include filename="$(find hyq_description)/urdfs/sensors/velodyne.urdf.xacro"/>
 	<xacro:include filename="$(find hyq_description)/urdfs/sensors/kinect.urdf.xacro"/>
+	<xacro:include filename="$(find hyq_description)/urdfs/sensors/ptu_d46.urdf.xacro"/>
 	<!-- generic simulator_gazebo plugins for starting mechanism control, ros time -->
 	<xacro:include filename="$(find hyq_description)/gazebo/gazebo.urdf.xacro"/>
@@ -47,13 +48,16 @@
 		<origin xyz="0.3 0.0 0.095" rpy="0.0 ${-PI} 0.0"/>
 	</xacro:microstrain_3dmgx325_imu>
+	<!-- PTU unit -->
+	<xacro:ptu_d46 name="ptu" parent="trunk" >
+		<origin xyz="0.63 0.0 0.095" rpy="0.0 0.0 0.0"/>
+	</xacro:ptu_d46>
 	<!-- Asus Xtion Pro -->
-	<xacro:asus_xtion_camera name="head_mount" parent="trunk">
-		<origin xyz="0.63 0.0 0.095" rpy="0.0 0.0 0.0"/>
-	</xacro:asus_xtion_camera>
-<!-- rpy="0.0 1.2 0.0" -->
+<!--	<xacro:asus_xtion_camera name="head_mount" parent="trunk">
+		<origin xyz="0.63 0.0 0.095" rpy="0.0 ${PI/6} 0.0"/>
+	</xacro:asus_xtion_camera>--> <!-- <origin xyz="0.63 0.0 0.095" rpy="0.0 0.0 0.0"/> --> <!-- ptu_mount_link -->
 	<!-- Velodyne -->
-	<xacro:velodyne name="trunk_mount" parent="trunk">
+<!--	<xacro:velodyne name="trunk_mount" parent="trunk">
 		<origin xyz="0.39 0.0 0.269" rpy="0.0 0.0 0.0"/>
-	</xacro:velodyne>
+	</xacro:velodyne> -->
 	<!-- Kinect mount -->
 <!--	<xacro:kinect_camera name="head_mount" parent="trunk">

File: hyq_description/urdfs/common.xacro (robot description, xacro)
@@ -43,5 +43,12 @@
 	<property name="ixy_lower" value="-0.0"/>
 	<property name="ixz_lower" value="-0.0"/>
-	 <property name="iyz_lower" value="0.0"/>
+	<property name="iyz_lower" value="0.0"/>
+	<!-- PTU unit -->
+	<property name="pan_velocity" value="1.0" />
+	<property name="pan_range" value="2.775" />
+	<property name="tilt_velocity" value="1.0" />
+	<property name="tilt_up_range" value="0.52" />
+	<property name="tilt_down_range" value="0.82" />
+	<property name="joint_effort" value="30" />
 	<!-- Asus Xtion Camera Location (Nominally 0) -->
 	<property name="asus_xtion_x" value="0.009"/>

Commit message: Cleaned unuseful files

File: hyq_description/robots/hyq.urdf.xacro (robot description, xacro)
@@ -53,7 +53,7 @@
 	</xacro:ptu_d46>
 	<!-- Asus Xtion Pro -->
-<!--	<xacro:asus_xtion_camera name="head_mount" parent="trunk">
-		<origin xyz="0.63 0.0 0.095" rpy="0.0 ${PI/6} 0.0"/>
-	</xacro:asus_xtion_camera>--> <!-- <origin xyz="0.63 0.0 0.095" rpy="0.0 0.0 0.0"/> --> <!-- ptu_mount_link -->
+	<xacro:asus_xtion_camera name="head_mount" parent="ptu_mount_link">
+		<origin xyz="0.0 0.0 0.0" rpy="0.0 0.0 0.0"/>
+	</xacro:asus_xtion_camera> <!-- <origin xyz="0.63 0.0 0.095" rpy="0.0 ${PI/6} 0.0"/> --> <!-- ptu_mount_link -->
 	<!-- Velodyne -->
 <!--	<xacro:velodyne name="trunk_mount" parent="trunk">

Commit message: Added new file for the description of the bumblebee stereo camera

File: hyq_description/robots/hyq.urdf.xacro (robot description, xacro)
@@ -15,4 +15,5 @@
 	<xacro:include filename="$(find hyq_description)/urdfs/sensors/kinect.urdf.xacro"/>
 	<xacro:include filename="$(find hyq_description)/urdfs/sensors/ptu_d46.urdf.xacro"/>
+	<xacro:include filename="$(find hyq_description)/urdfs/sensors/bumblebee.urdf.xacro"/>
 	<!-- generic simulator_gazebo plugins for starting mechanism control, ros time -->
 	<xacro:include filename="$(find hyq_description)/gazebo/gazebo.urdf.xacro"/>
@@ -29,38 +30,79 @@
 	<xacro:hyq_trunk name="base" />
 	<!-- LF leg -->
-	<xacro:hyq_leg name="lf" parent="trunk" reflect_hip="1" reflect_upper="1" reflect_front="1">
-		<origin xyz="${d_fh/2} ${d_lr/2} 0.0" rpy="0.0 ${PI/2} ${PI}"/>
+	<xacro:hyq_leg
+		name="lf"
+		parent="trunk"
+		reflect_hip="1"
+		reflect_upper="1"
+		reflect_front="1">
+		<origin xyz="${d_fh/2} ${d_lr/2} 0" rpy="0 ${PI/2} ${PI}"/>
 	</xacro:hyq_leg>
 	<!-- RF leg -->
-	<xacro:hyq_leg name="rf" parent="trunk" reflect_hip="-1" reflect_upper="-1" reflect_front="1">
-		<origin xyz="${d_fh/2} ${-d_lr/2} 0.0" rpy="0.0 ${PI/2} 0.0"/>
+	<xacro:hyq_leg
+		name="rf"
+		parent="trunk"
+		reflect_hip="-1"
+		reflect_upper="-1"
+		reflect_front="1">
+		<origin xyz="${d_fh/2} ${-d_lr/2} 0" rpy="0 ${PI/2} 0"/>
 	</xacro:hyq_leg>
 	<!-- LH leg -->
-	<xacro:hyq_leg name="lh" parent="trunk" reflect_hip="-1" reflect_upper="1" reflect_front="-1">
-		<origin xyz="${-d_fh/2} ${d_lr/2} 0.0" rpy="0.0 ${PI/2} ${PI}"/>
+	<xacro:hyq_leg
+		name="lh"
+		parent="trunk"
+		reflect_hip="-1"
+		reflect_upper="1"
+		reflect_front="-1">
+		<origin xyz="${-d_fh/2} ${d_lr/2} 0" rpy="0 ${PI/2} ${PI}"/>
 	</xacro:hyq_leg>
 	<!-- RH leg -->
-	<xacro:hyq_leg name="rh" parent="trunk" reflect_hip="1" reflect_upper="-1" reflect_front="-1">
-		<origin xyz="${-d_fh/2} ${-d_lr/2} 0.0" rpy="0.0 ${PI/2} 0.0"/>
+	<xacro:hyq_leg
+		name="rh"
+		parent="trunk"
+		reflect_hip="1"
+		reflect_upper="-1"
+		reflect_front="-1">
+		<origin xyz="${-d_fh/2} ${-d_lr/2} 0" rpy="0 ${PI/2} 0"/>
 	</xacro:hyq_leg>
 	<!-- IMU runk -->
-	<xacro:microstrain_3dmgx325_imu parent="trunk" imu_name="3dmgx325_trunk_imu" imu_topic="trunk_imu/data" update_rate="100.0" stdev="0.00017">
-		<origin xyz="0.3 0.0 0.095" rpy="0.0 ${-PI} 0.0"/>
+	<xacro:microstrain_3dmgx325_imu
+		parent="trunk"
+		imu_name="3dmgx325_trunk_imu"
+		imu_topic="trunk_imu/data"
+		update_rate="100.0"
+		stdev="0.00017">
+		<origin xyz="0.3 0 0.095" rpy="0 ${-PI} 0"/>
 	</xacro:microstrain_3dmgx325_imu>
 	<!-- PTU unit -->
-	<xacro:ptu_d46 name="ptu" parent="trunk" >
-		<origin xyz="0.63 0.0 0.095" rpy="0.0 0.0 0.0"/>
-	</xacro:ptu_d46>
+<!--	<xacro:ptu_d46
+		name="ptu"
+		parent="trunk">
+		<origin xyz="0.63 0 0.095" rpy="0 0 0"/>
+	</xacro:ptu_d46>-->
 	<!-- Asus Xtion Pro -->
-	<xacro:asus_xtion_camera name="head_mount" parent="ptu_mount_link">
-		<origin xyz="0.0 0.0 0.0" rpy="0.0 0.0 0.0"/>
-	</xacro:asus_xtion_camera> <!-- <origin xyz="0.63 0.0 0.095" rpy="0.0 ${PI/6} 0.0"/> --> <!-- ptu_mount_link -->
+	<xacro:asus_xtion_camera
+		name="head_mount"
+		parent="trunk">
+		<origin xyz="0.63 0 0.095" rpy="0 ${PI/6} 0"/>
+	</xacro:asus_xtion_camera> <!-- <origin xyz="0.63 0 0.095" rpy="0 ${PI/6} 0"/> --> <!-- ptu_mount_link -->
 	<!-- Velodyne -->
-<!--	<xacro:velodyne name="trunk_mount" parent="trunk">
-		<origin xyz="0.39 0.0 0.269" rpy="0.0 0.0 0.0"/>
+<!--	<xacro:velodyne
+		name="trunk_mount"
+		parent="trunk">
+		<origin xyz="0.39 0 0.269" rpy="0 0 0"/>
 	</xacro:velodyne> -->
 	<!-- Kinect mount -->
-<!--	<xacro:kinect_camera name="head_mount" parent="trunk">
-		<origin xyz="0.63 0.0 0.095" rpy="0.0 0.0 0.0"/>
+<!--	<xacro:kinect_camera
+		name="head_mount"
+		parent="trunk">
+		<origin xyz="0.63 0 0.095" rpy="0 0 0"/>
 	</xacro:kinect_camera>-->
+	<!-- Bumblebee -->
+<!--	<xacro:bumblebee_66
+		parent_link="ptu_mount_link"
+		xyz="0 0 0"
+		rpy="${PI/2} 0 ${PI/2}"
+		ns="bumblebee"
+		frame_prefix="bumblebee_"
+		high_res="false"/>--> <!-- xyz="0.63 0 0.095" rpy="0 0 0" -->
 </robot>

File: hyq_description/urdfs/common.xacro (robot description, xacro)
@@ -67,4 +67,9 @@
 	<property name="kinect_pitch" value="0.0"/>
 	<property name="kinect_yaw" value="${-PI/2}"/>
+	<!-- Bumblebee mass and lengths for computing inertia tensor -->
+	<property name="b2mass" value="0.342"/>
+	<property name="b2lx" value="0.157"/>
+	<property name="b2ly" value="0.036"/>
+	<property name="b2lz" value="0.0474"/>
 	<!-- Velodyne Lidar Location (Nominally 0) -->
 	<property name="velodyne_x" value="0.0"/>

Commit message: Cleaned up the description of the robot and made corections to play with both the real robot and the gazeebo simulator.

File: hyq_description/robots/hyq.urdf.xacro (robot description, xacro)
@@ -65,5 +65,5 @@
 		<origin xyz="${-d_fh/2} ${-d_lr/2} 0" rpy="0 ${PI/2} 0"/>
 	</xacro:hyq_leg>
-	<!-- IMU runk -->
+	<!-- IMU trunk -->
 	<xacro:microstrain_3dmgx325_imu
 		parent="trunk"
@@ -87,9 +87,9 @@
 	</xacro:asus_xtion_camera> <!-- <origin xyz="0.63 0 0.095" rpy="0 ${PI/6} 0"/> --> <!-- ptu_mount_link -->
 	<!-- Velodyne -->
-<!--	<xacro:velodyne
+	<xacro:velodyne
 		name="trunk_mount"
 		parent="trunk">
 		<origin xyz="0.39 0 0.269" rpy="0 0 0"/>
-	</xacro:velodyne> -->
+	</xacro:velodyne>
 	<!-- Kinect mount -->
 <!--	<xacro:kinect_camera

File: hyq_description/urdfs/common.xacro (robot description, xacro)
@@ -8,7 +8,7 @@
 	<property name="d_p1p2" value="0.35"/>
 	<!-- Initial joint positions -->
-	<property name="haa_pos0" value="-0.3"/>
-	<property name="hfe_pos0" value="0.6"/>
-	<property name="kfe_pos0" value="-1.4"/>
+	<property name="haa_pos0" value="0.0"/>
+	<property name="hfe_pos0" value="0.0"/>
+	<property name="kfe_pos0" value="0.0"/>
 	<!-- Inertial values -->
 	<!-- Trunk with hydraulic system -->
@@ -53,6 +53,6 @@
 	<!-- Asus Xtion Camera Location (Nominally 0) -->
 	<property name="asus_xtion_x" value="0.009"/>
-	<property name="asus_xtion_ir_y" value="0.0285"/>
-	<property name="asus_xtion_rgb_y" value="0.0185"/>
+	<property name="asus_xtion_depth_y" value="0.049"/>
+	<property name="asus_xtion_rgb_y" value="0.022"/>
 	<property name="asus_xtion_z" value="0.035"/>
 	<property name="asus_xtion_roll" value="${-PI/2}"/>

File: hyq_description/urdfs/leg/leg.urdf.xacro (robot description, xacro)
@@ -8,5 +8,5 @@
 	<xacro:macro name="hyq_leg" params="name parent *origin reflect_hip reflect_upper reflect_front">
 		<!-- Joints -->
-		<!-- Fake joint -->
+		<!-- Fake joint
 		<joint name="${name}_haa_fake_joint" type="fixed">
 			<insert_block name="origin"/>
@@ -14,8 +14,11 @@
 			<child  link="${name}_haa_fake"/>
 		</joint>
+		-->
 		<!-- Hip joint assembly -->
 		<joint name="${name}_haa_joint" type="revolute">
-			<origin xyz="0.0 0.0 0.0" rpy="0.0 0.0 ${haa_pos0}"/>
-			<parent link="${name}_haa_fake"/>
+		<!--	<origin xyz="0.0 0.0 0.0" rpy="0.0 0.0 ${haa_pos0}"/>
+			<parent link="${name}_haa_fake"/>-->
+			<insert_block name="origin"/>
+			<parent link="${parent}"/>
 			<child  link="${name}_hip_assembly"/>
 			<limit effort="200.0" velocity="1000.0" lower="${-PI/2-haa_pos0}" upper="${PI/6-haa_pos0}"/>
@@ -51,5 +54,5 @@
 		</joint>
 		<!-- Links -->
-		<!-- Fake hip assembly link -->
+		<!-- Fake hip assembly link
 		<link name="${name}_haa_fake">
 			<inertial>
@@ -59,4 +62,5 @@
 			</inertial>
 		</link>
+		-->
 		<!-- Hip assembly link -->
 		<link name="${name}_hip_assembly">

File: hyq_description/urdfs/sensors/asus_xtion.gazebo.xacro (robot description, xacro)
@@ -1,7 +1,7 @@
 <?xml version="1.0"?>
 <root xmlns:xacro="http://ros.org/wiki/xacro">
-	<xacro:macro name="asus_xtion_ir_sensor" params="link_name frame_name camera_name">
+	<xacro:macro name="asus_xtion_depth_sensor" params="link_name frame_name camera_name">
 		<gazebo reference="${link_name}">
-			<sensor type="depth" name="${link_name}_ir_sensor">
+			<sensor type="depth" name="${link_name}_depth_sensor">
 				<always_on>true</always_on>
 				<update_rate>1.0</update_rate>
@@ -88,86 +88,3 @@
 		</gazebo>
 	</xacro:macro>
-<!--
-	<xacro:macro name="prosilica_cam" params="link_name frame_name camera_name ">
-		<gazebo reference="${link_name}">
-			<sensor type="camera" name="${link_name}_sensor">
-				<always_on>true</always_on>
-				<update_rate>1.0</update_rate>
-				<camera>
-					<horizontal_fov>${64.2*M_PI/180.0}</horizontal_fov>
-					<image>
-						<format>R8G8B8</format>
-						<width>320</width>
-						<height>240</height>
-					</image>
-					<clip>
-						<near>0.1</near>
-						<far>100</far>
-					</clip>
-				</camera>
-				<plugin name="${link_name}_controller" filename="libgazebo_ros_prosilica.so">
-					<alwaysOn>true</alwaysOn>
-					<updateRate>1.0</updateRate>
-					<cameraName>${camera_name}_1mb</cameraName>
-					<imageTopicName>image_raw</imageTopicName>
-					<cameraInfoTopicName>camera_info</cameraInfoTopicName>
-					<depthImageTopicName>depth/image_raw</depthImageTopicName>
-					<depthImageCameraInfoTopicName>depth/camera_info</depthImageCameraInfoTopicName>
-					<pollServiceName>request_image</pollServiceName>
-					<pointCloudTopicName>points</pointCloudTopicName>
-					<frameName>${frame_name}</frameName>
-					<pointCloudCutoff>0.4</pointCloudCutoff>
-					<distortionK1>0.0</distortionK1>
-					<distortionK2>0.0</distortionK2>
-					<distortionK3>0.0</distortionK3>
-					<distortionT1>0.0</distortionT1>
-					<distortionT2>0.0</distortionT2>
-					<CxPrime>0</CxPrime>
-					<Cx>0</Cx>
-					<Cy>0</Cy>
-					<focalLength>0</focalLength>
-					<hackBaseline>0</hackBaseline>
-				</plugin>
-			</sensor>
-			<sensor type="depth" name="${link_name}_sim_pcd_sensor">
-				<always_on>true</always_on>
-				<update_rate>1.0</update_rate>
-				<camera>
-					<horizontal_fov>${64.2*PI/180.0}</horizontal_fov>
-					<image>
-						<format>R8G8B8</format>
-						<width>320</width>
-						<height>240</height>
-					</image>
-					<clip>
-						<near>0.1</near>
-						<far>100</far>
-					</clip>
-				</camera>
-				<plugin name="${link_name}_sim_pcd_controller" filename="libgazebo_ros_openni_kinect.so">
-					<alwaysOn>true</alwaysOn>
-					<updateRate>1.0</updateRate>
-					<cameraName>${camera_name}_1mb_sim_pcd</cameraName>
-					<imageTopicName>image_raw</imageTopicName>
-					<depthImageTopicName>depth/image_raw</depthImageTopicName>
-					<depthImageCameraInfoTopicName>depth/camera_info</depthImageCameraInfoTopicName>
-					<cameraInfoTopicName>camera_info</cameraInfoTopicName>
-					<pointCloudTopicName>points</pointCloudTopicName>
-					<frameName>${frame_name}</frameName>
-					<pointCloudCutoff>0.4</pointCloudCutoff>
-					<distortionK1>0.00000001</distortionK1>
-					<distortionK2>0.00000001</distortionK2>
-					<distortionK3>0.00000001</distortionK3>
-					<distortionT1>0.00000001</distortionT1>
-					<distortionT2>0.00000001</distortionT2>
-					<CxPrime>0</CxPrime>
-					<Cx>0</Cx>
-					<Cy>0</Cy>
-					<focalLength>0</focalLength>
-					<hackBaseline>0</hackBaseline>
-				</plugin>
-			</sensor>
-			<material value="Gazebo/Red" />
-		</gazebo>
-	</xacro:macro>-->
 </root>

File: hyq_description/urdfs/sensors/asus_xtion.urdf.xacro (robot description, xacro)
@@ -12,14 +12,14 @@
 		</joint>
 		<!-- asus ir sensor physical attachment -->
-		<joint name="${name}_asus_xtion_ir_joint" type="fixed">
-			<origin xyz="${asus_xtion_x} -${asus_xtion_ir_y} ${asus_xtion_z}" rpy="0.0 0.0 0.0"/>
+		<joint name="${name}_asus_xtion_depth_joint" type="fixed">
+			<origin xyz="${asus_xtion_x} ${asus_xtion_depth_y} ${asus_xtion_z}" rpy="0.0 0.0 0.0"/>
 			<parent link="${name}_asus_xtion_link"/>
-			<child link="${name}_asus_xtion_ir_link"/>
+			<child link="${name}_asus_xtion_depth_frame"/>
 		</joint>
 		<!-- asus xtion ir sensor frame -->
-		<joint name="${name}_asus_xtion_ir_optical_frame_joint" type="fixed">
+		<joint name="${name}_asus_xtion_depth_optical_frame_joint" type="fixed">
 			<origin xyz="0 0 0"	rpy="${asus_xtion_roll} ${asus_xtion_pitch} ${asus_xtion_yaw}"/>
-			<parent link="${name}_asus_xtion_ir_link"/>
-			<child link="${name}_asus_xtion_ir_optical_frame"/>
+			<parent link="${name}_asus_xtion_depth_frame"/>
+			<child link="${name}_asus_xtion_depth_optical_frame"/>
 		</joint>
 		<!-- asus_xtion rgb sensor physical attachment -->
@@ -27,25 +27,12 @@
 			<origin xyz="${asus_xtion_x} ${asus_xtion_rgb_y} ${asus_xtion_z}" rpy="0.0 0.0 0.0"/>
 			<parent link="${name}_asus_xtion_link"/>
-			<child link="${name}_asus_xtion_rgb_link"/>
+			<child link="${name}_asus_xtion_rgb_frame"/>
 		</joint>
 		<!-- asus xtion rgb sensor frame -->
 		<joint name="${name}_asus_xtion_rgb_optical_frame_joint" type="fixed">
 			<origin xyz="0 0 0"	rpy="${asus_xtion_roll} ${asus_xtion_pitch} ${asus_xtion_yaw}"/>
-			<parent link="${name}_asus_xtion_rgb_link"/>
+			<parent link="${name}_asus_xtion_rgb_frame"/>
 			<child link="${name}_asus_xtion_rgb_optical_frame"/>
 		</joint>
-		<!-- prosilica sensor physical attachment -->
-<!--		<joint name="${name}_asus_xtion_prosilica_joint" type="fixed">
-			<origin xyz="${asus_xtion_x} ${asus_xtion_rgb_y} ${asus_xtion_z}" rpy="0.0 0.0 0.0"/>
-			<parent link="${name}_link"/>
-			<child link="${name}_prosilica_link"/>
-		</joint>-->
-		<!-- prosilica sensor frame -->
-<!--		<joint name="${name}_prosilica_optical_frame_joint" type="fixed">
-			<origin xyz="${cal_high_def_x} ${cal_high_def_y} ${cal_high_def_z}"
-					rpy="${-PI/2+cal_high_def_roll} ${0.0+cal_high_def_pitch} ${-PI/2+cal_high_def_yaw}" />
-			<parent link="${name}_prosilica_link"/>
-			<child link="${name}_prosilica_optical_frame"/>
-		</joint>-->
 		<!-- Links -->
 		<link name="${name}_asus_xtion_link">
@@ -64,13 +51,13 @@
 				</material>
 			</visual>
-			<collision>
-				<origin xyz="0.0 0.0 0.0" rpy="0.0 0.0 0.0"/>
-				<geometry>
-					<sphere radius="0.0005"/>
-				</geometry>
-			</collision>
+	<collision>
+		<origin xyz="0.0 0.0 ${asus_xtion_z}" rpy="0 0 0" />
+		<geometry>
+			<box size="0.05 .18 0.035" />
+		</geometry>
+	</collision>
 		</link>
 		<!-- ir sensor link -->
-		<link name="${name}_asus_xtion_ir_link">
+		<link name="${name}_asus_xtion_depth_frame">
 			<inertial>
 				<mass value="0.1" />
@@ -92,7 +79,7 @@
 		</link>
 		<!-- ir optical sensor link -->
-		<link name="${name}_asus_xtion_ir_optical_frame"/>
+		<link name="${name}_asus_xtion_depth_optical_frame"/>
 		<!-- rgb sensor link -->
-		<link name="${name}_asus_xtion_rgb_link" >
+		<link name="${name}_asus_xtion_rgb_frame" >
 			<inertial>
 				<mass value="0.1" />
@@ -116,6 +103,6 @@
 		<link name="${name}_asus_xtion_rgb_optical_frame"/>
 	<!-- gazebo extensions -->
-	<xacro:asus_xtion_ir_sensor link_name="${name}_asus_xtion_ir_link" frame_name="${name}_asus_xtion_ir_optical_frame" camera_name="${name}_asus_xtion" />
-	<xacro:asus_xtion_rgb_sensor link_name="${name}_asus_xtion_rgb_link" frame_name="${name}_asus_xtion_rgb_optical_frame" camera_name="${name}_asus_xtion" />
+	<xacro:asus_xtion_depth_sensor link_name="${name}_asus_xtion_depth_frame" frame_name="${name}_asus_xtion_depth_optical_frame" camera_name="${name}_asus_xtion" />
+	<xacro:asus_xtion_rgb_sensor link_name="${name}_asus_xtion_rgb_frame" frame_name="${name}_asus_xtion_rgb_optical_frame" camera_name="${name}_asus_xtion" />
 	</xacro:macro>
 </root>

File: hyq_description/urdfs/sensors/velodyne.urdf.xacro (robot description, xacro)
@@ -9,20 +9,14 @@
 			<insert_block name="origin"/>
 			<parent link="${parent}"/>
-			<child link="${name}_velodyne_link"/>
+			<child link="${name}_velodyne_frame"/>
 		</joint>
-		<!-- velodyne sensor physical attachment -->
-		<joint name="${name}_velodyne_sensor_joint" type="fixed">
+		<!-- velodyne sensor optical frame -->
+		<joint name="${name}_velodyne_optical_frame_joint" type="fixed">
 			<origin xyz="${velodyne_x} ${velodyne_y} ${velodyne_z}" rpy="0.0 0.0 0.0"/>
-			<parent link="${name}_velodyne_link"/>
-			<child link="${name}_velodyne_sensor_link"/>
-		</joint>
-		<!-- velodyne sensor frame -->
-		<joint name="${name}_velodyne_optical_frame_joint" type="fixed">
-			<origin xyz="0 0 0"	rpy="0 0 0"/>
-			<parent link="${name}_velodyne_sensor_link"/>
-			<child link="${name}_velodyne_sensor_optical_frame"/>
+			<parent link="${name}_velodyne_frame"/>
+			<child link="${name}_velodyne_optical_frame"/>
 		</joint>
 		<!-- Links -->
-		<link name="${name}_velodyne_link">
+		<link name="${name}_velodyne_frame">
 			<inertial>
 				<mass value="0.1"/>
@@ -42,32 +36,12 @@
 				<origin xyz="0.0 0.0 0.0" rpy="0.0 0.0 0.0"/>
 				<geometry>
-					<sphere radius="0.0005"/>
-				</geometry>
-			</collision>
-		</link>
-		<!-- velodyne sensor link -->
-		<link name="${name}_velodyne_sensor_link">
-			<inertial>
-				<mass value="0.1" />
-				<origin xyz="0.0 0.0 0.0" rpy="0.0 0.0 0.0"/>
-				<inertia ixx="0.01" ixy="0.0" ixz="0.0" iyy="0.01" iyz="0.0" izz="0.01"/>
-			</inertial>
-			<visual>
-				<origin xyz="0.0 0.0 0.0" rpy="0.0 0.0 0.0"/>
-				<geometry>
-					<sphere radius="0.0005"/>
-				</geometry>
-			</visual>
-			<collision>
-				<origin xyz="0.0 0.0 0.0" rpy="0.0 0.0 0.0"/>
-				<geometry>
-					<sphere radius="0.0005"/>
+					<box size="0.1 0.18 0.1" />
 				</geometry>
 			</collision>
 		</link>
 		<!-- rgb optical sensor link -->
-		<link name="${name}_velodyne_sensor_optical_frame"/>
+		<link name="${name}_velodyne_optical_frame"/>
 	<!-- gazebo extensions -->
-	<xacro:velodyne_sensor link_name="${name}_velodyne_sensor_link" frame_name="${name}_velodyne_sensor_optical_frame" lidar_name="${name}_velodyne" />
+	<xacro:velodyne_sensor link_name="${name}_velodyne_optical_frame" frame_name="${name}_velodyne_frame" lidar_name="${name}_velodyne" />
 	</xacro:macro>
 </root>

File: hyq_description/urdfs/trunk/trunk.urdf.xacro (robot description, xacro)
@@ -10,5 +10,5 @@
 			<origin xyz="0.0 0.0 0.0" rpy="0.0 0.0 0.0"/>
 			<!--<origin xyz="0.0 0.0 -0.49"  rpy="3.1416 0.0 0.0" />-->
-			<parent link="${name}_footprint"/>
+			<parent link="${name}_link"/>
 			<child link="trunk"/>
 		</joint>
@@ -27,5 +27,5 @@
 		<!-- Links -->
 		<!-- Footprint link -->
-		<link name="${name}_footprint">
+		<link name="${name}_link">
 			<visual>
 				<geometry>
