Commit message: corrected errors in stereo camera model

File: hyq_description/robots/hyq.urdf.xacro (robot description, xacro)
@@ -75,34 +75,16 @@
 	</xacro:microstrain_3dmgx325_imu>
 	<!-- PTU unit -->
-<!--	<xacro:ptu_d46
+	<xacro:ptu_d46
 		name="ptu"
 		parent="trunk">
 		<origin xyz="0.63 0 0.095" rpy="0 0 0"/>
-	</xacro:ptu_d46>-->
-	<!-- Asus Xtion Pro -->
-	<xacro:asus_xtion_camera
-		name="head_mount"
-		parent="trunk">
-		<origin xyz="0.63 0 0.095" rpy="0 ${PI/6} 0"/>
-	</xacro:asus_xtion_camera> <!-- <origin xyz="0.63 0 0.095" rpy="0 ${PI/6} 0"/> --> <!-- ptu_mount_link -->
-	<!-- Velodyne -->
-	<xacro:velodyne
-		name="trunk_mount"
-		parent="trunk">
-		<origin xyz="0.39 0 0.269" rpy="0 0 0"/>
-	</xacro:velodyne>
-	<!-- Kinect mount -->
-<!--	<xacro:kinect_camera
-		name="head_mount"
-		parent="trunk">
-		<origin xyz="0.63 0 0.095" rpy="0 0 0"/>
-	</xacro:kinect_camera>-->
+	</xacro:ptu_d46>
 	<!-- Bumblebee -->
-<!--	<xacro:bumblebee_66
+	<xacro:bumblebee_97
 		parent_link="ptu_mount_link"
 		xyz="0 0 0"
-		rpy="${PI/2} 0 ${PI/2}"
+		rpy="0 0 0"
 		ns="bumblebee"
 		frame_prefix="bumblebee_"
-		high_res="false"/>--> <!-- xyz="0.63 0 0.095" rpy="0 0 0" -->
+		high_res="false"/><!-- xyz="0.63 0 0.095" rpy="0 0 0" -->
 </robot>

File: hyq_description/urdfs/common.xacro (robot description, xacro)
@@ -8,7 +8,7 @@
 	<property name="d_p1p2" value="0.35"/>
 	<!-- Initial joint positions -->
-	<property name="haa_pos0" value="0.0"/>
-	<property name="hfe_pos0" value="0.0"/>
-	<property name="kfe_pos0" value="0.0"/>
+	<property name="haa_pos0" value="-0.8"/>
+	<property name="hfe_pos0" value="0.6"/>
+	<property name="kfe_pos0" value="-1.4"/>
 	<!-- Inertial values -->
 	<!-- Trunk with hydraulic system -->

File: hyq_description/urdfs/sensors/bumblebee.urdf.xacro (robot description, xacro)
@@ -11,9 +11,10 @@
 			<parent link="${frame_prefix}mount_link"/>
 			<child link="${frame_prefix}optical_frame"/>
-			<origin xyz="0 0 0" rpy="0 0 0"/>
+			<!--<origin xyz="0 0 0" rpy="0 0 0"/>-->
+			<origin xyz="0 -0.06 0.00" rpy="-${PI/2} 0 -${PI/2}"/>
 		</joint>
 		<link name="${frame_prefix}mount_link">
 			<visual>
-				<origin xyz="0 0 0" rpy="0 0 0"/>
+				<origin xyz="0 0 0" rpy="${PI/2} 0 ${PI/2}"/>
 				<geometry>
 					<mesh filename="package://hyq_description/meshes/sensors/bumblebee.dae"/>
@@ -21,5 +22,5 @@
 			</visual>
 			<collision>
-				<origin xyz="0 0 0" rpy="0 0 0"/>
+				<origin xyz="0 0 0" rpy="${PI/2} 0 ${PI/2}"/>
 				<geometry>
 					<mesh filename="package://hyq_description/meshes/sensors/bumblebee.dae"/>
@@ -42,6 +43,6 @@
 		<xacro:if value="${high_res}">
 			<xacro:stereo_camera
-				reference="${frame_prefix}optical_frame"
-				frame_id="${frame_prefix}optical_frame"
+				reference="${frame_prefix}mount_link"
+				frame_id="${frame_prefix}mount_link"
 				ns="${ns}"
 				hfov="${hfov}"
@@ -54,6 +55,6 @@
 		<xacro:unless value="${high_res}">
 			<xacro:stereo_camera
-				reference="${frame_prefix}optical_frame"
-				frame_id="${frame_prefix}optical_frame"
+				reference="${frame_prefix}mount_link"
+				frame_id="${frame_prefix}mount_link"
 				ns="${ns}"
 				hfov="${hfov}"

File: hyq_description/urdfs/sensors/ptu_d46.transmission.xacro (robot description, xacro)
@@ -5,5 +5,5 @@
 		<transmission name="${name}_pan_trans">
 			<type>transmission_interface/SimpleTransmission</type>
-			<joint name="${name}_pan_joint"/>
+			<joint name="${name}_pan"/>
 			<actuator name="${name}_pan_motor">
 				<hardwareInterface>EffortJointInterface</hardwareInterface>
@@ -14,5 +14,5 @@
 		<transmission name="${name}_tilt_trans">
 			<type>transmission_interface/SimpleTransmission</type>
-			<joint name="${name}_tilt_joint"/>
+			<joint name="${name}_tilt"/>
 			<actuator name="${name}_tilt_motor">
 				<hardwareInterface>EffortJointInterface</hardwareInterface>

File: hyq_description/urdfs/sensors/ptu_d46.urdf.xacro (robot description, xacro)
@@ -101,5 +101,5 @@
 			<origin xyz="0 0 0" rpy="-${PI/2} 0 0"/>
 			<child link="${name}_tilted_link"/>
-			<axis xyz="0 1 0"/>
+			<axis xyz="0 1 0"/> <!-- 0 1 0-->
 			<limit lower="${-tilt_down_range}" upper="${tilt_up_range}" effort="${joint_effort}" velocity="${tilt_velocity}"/>
 		</joint>

File: hyq_description/urdfs/sensors/stereo_camera.gazebo.xacro (robot description, xacro)
@@ -6,5 +6,5 @@
 				<update_rate>${update_rate}</update_rate>
 				<camera name="left">
-					<pose>${baseline / 2.0} 0 0 0 1.5707 1.5707</pose>
+					<pose> 0 ${baseline / 2.0} 0 0 0 0</pose>
 					<horizontal_fov>${hfov}</horizontal_fov>
 					<image>
@@ -24,5 +24,5 @@
 				</camera>
 				<camera name="right">
-					<pose>${-baseline / 2.0} 0 0 0 1.5707 1.5707</pose>
+					<pose> 0 ${-baseline / 2.0} 0 0 0 0</pose>
 					<horizontal_fov>${hfov}</horizontal_fov>
 					<image>

Commit message: ptu rotated 30 degrees looking down

File: hyq_description/robots/hyq.urdf.xacro (robot description, xacro)
@@ -78,5 +78,5 @@
 		name="ptu"
 		parent="trunk">
-		<origin xyz="0.63 0 0.095" rpy="0 0 0"/>
+		<origin xyz="0.63 0 0.095" rpy="0 ${PI/6} 0"/>
 	</xacro:ptu_d46>
 	<!-- Bumblebee -->

Commit message: The last comments

File: hyq_description/robots/hyq.urdf.xacro (robot description, xacro)
@@ -31,5 +31,5 @@
 	<!-- LF leg -->
 	<xacro:hyq_leg
-		name="lf"
+		name="LF"
 		parent="trunk"
 		reflect_hip="1"
@@ -40,5 +40,5 @@
 	<!-- RF leg -->
 	<xacro:hyq_leg
-		name="rf"
+		name="RF"
 		parent="trunk"
 		reflect_hip="-1"
@@ -49,5 +49,5 @@
 	<!-- LH leg -->
 	<xacro:hyq_leg
-		name="lh"
+		name="LH"
 		parent="trunk"
 		reflect_hip="-1"
@@ -58,5 +58,5 @@
 	<!-- RH leg -->
 	<xacro:hyq_leg
-		name="rh"
+		name="RH"
 		parent="trunk"
 		reflect_hip="1"
@@ -74,22 +74,16 @@
 		<origin xyz="0.3 0 0.095" rpy="0 ${-PI} 0"/>
 	</xacro:microstrain_3dmgx325_imu>
-	<!-- PTU unit -->
-<!--	<xacro:ptu_d46
-		name="ptu"
-		parent="trunk">
-		<origin xyz="0.63 0 0.095" rpy="0 0 0"/>
-	</xacro:ptu_d46>-->
-	<!-- Asus Xtion Pro -->
-	<xacro:asus_xtion_camera
+<!-- Asus Xtion Pro -->
+<!--	<xacro:asus_xtion_camera
 		name="head_mount"
 		parent="trunk">
 		<origin xyz="0.63 0 0.095" rpy="0 ${PI/6} 0"/>
-	</xacro:asus_xtion_camera> <!-- <origin xyz="0.63 0 0.095" rpy="0 ${PI/6} 0"/> --> <!-- ptu_mount_link -->
+	</xacro:asus_xtion_camera> --> <!-- <origin xyz="0.63 0 0.095" rpy="0 ${PI/6} 0"/> --> <!-- ptu_mount_link -->
 	<!-- Velodyne -->
-	<xacro:velodyne
+<!--	<xacro:velodyne
 		name="trunk_mount"
 		parent="trunk">
 		<origin xyz="0.39 0 0.269" rpy="0 0 0"/>
-	</xacro:velodyne>
+	</xacro:velodyne>-->
 	<!-- Kinect mount -->
 <!--	<xacro:kinect_camera
@@ -98,11 +92,17 @@
 		<origin xyz="0.63 0 0.095" rpy="0 0 0"/>
 	</xacro:kinect_camera>-->
+	<!-- PTU unit -->
+	<xacro:ptu_d46
+		name="ptu"
+		parent="trunk">
+		<origin xyz="0.6357 0.04397 0.08809" rpy="-0.041779 0.31978 -0.061764"/>
+	</xacro:ptu_d46>
 	<!-- Bumblebee -->
-<!--	<xacro:bumblebee_66
+	<xacro:bumblebee_97
 		parent_link="ptu_mount_link"
 		xyz="0 0 0"
-		rpy="${PI/2} 0 ${PI/2}"
+		rpy="0 0 0"
 		ns="bumblebee"
 		frame_prefix="bumblebee_"
-		high_res="false"/>--> <!-- xyz="0.63 0 0.095" rpy="0 0 0" -->
+		high_res="false"/> <!-- xyz="0.63 0 0.095" rpy="0 0 0" -->
 </robot>

File: hyq_description/urdfs/common.xacro (robot description, xacro)
@@ -8,7 +8,7 @@
 	<property name="d_p1p2" value="0.35"/>
 	<!-- Initial joint positions -->
-	<property name="haa_pos0" value="0.0"/>
-	<property name="hfe_pos0" value="0.0"/>
-	<property name="kfe_pos0" value="0.0"/>
+	<property name="haa_pos0" value="0"/>
+	<property name="hfe_pos0" value="0"/>
+	<property name="kfe_pos0" value="0"/>
 	<!-- Inertial values -->
 	<!-- Trunk with hydraulic system -->

File: hyq_description/urdfs/leg/leg.transmission.xacro (robot description, xacro)
@@ -5,5 +5,5 @@
 		<transmission name="${name}_haa_trans">
 			<type>transmission_interface/SimpleTransmission</type>
-			<joint name="${name}_haa_joint"/>
+			<joint name="${name}_HAA"/>
 			<actuator name="${name}_haa_motor">
 				<hardwareInterface>EffortJointInterface</hardwareInterface>
@@ -14,5 +14,5 @@
 		<transmission name="${name}_hfe_upper_trans">
 			<type>transmission_interface/SimpleTransmission</type>
-			<joint name="${name}_hfe_joint"/>
+			<joint name="${name}_HFE"/>
 			<actuator name="${name}_hfe_motor">
 				<hardwareInterface>EffortJointInterface</hardwareInterface>
@@ -23,5 +23,5 @@
 		<transmission name="${name}_kfe_trans">
 			<type>transmission_interface/SimpleTransmission</type>
-			<joint name="${name}_kfe_joint"/>
+			<joint name="${name}_KFE"/>
 			<actuator name="${name}_hfe_motor">
 				<hardwareInterface>EffortJointInterface</hardwareInterface>

File: hyq_description/urdfs/leg/leg.urdf.xacro (robot description, xacro)
@@ -13,10 +13,9 @@
 			<parent link="${parent}"/>
 			<child  link="${name}_haa_fake"/>
-		</joint>
-		-->
+		</joint>-->
 		<!-- Hip joint assembly -->
-		<joint name="${name}_haa_joint" type="revolute">
-		<!--	<origin xyz="0.0 0.0 0.0" rpy="0.0 0.0 ${haa_pos0}"/>
-			<parent link="${name}_haa_fake"/>-->
+		<joint name="${name}_HAA" type="revolute">
+			<origin xyz="0.0 0.0 0.0" rpy="0.0 0.0 ${haa_pos0}"/>
+			<!--<parent link="${name}_haa_fake"/>-->
 			<insert_block name="origin"/>
 			<parent link="${parent}"/>
@@ -28,5 +27,5 @@
 		</joint>
 		<!-- Upper leg joint -->
-		<joint name="${name}_hfe_joint" type="revolute">
+		<joint name="${name}_HFE" type="revolute">
 			<origin xyz="${d_tbb} 0.0 0.0" rpy="${reflect_upper*PI/2} ${-reflect_hip*hfe_pos0} 0.0"/>
 			<parent link="${name}_hip_assembly"/>
@@ -38,5 +37,5 @@
 		</joint>
 		<!-- Lower leg joint -->
-		<joint name="${name}_kfe_joint" type="revolute">
+		<joint name="${name}_KFE" type="revolute">
 			<origin xyz="${d_p1p2} 0.0 0.0" rpy="0.0 0.0 ${reflect_front*kfe_pos0}"/>
 			<parent link="${name}_upper_leg"/>

Commit message: Fixed the naming of joint according to our convention Fixed the haa transfromation as a "bug" has creeped in while I was away

File: hyq_description/robots/hyq.urdf.xacro (robot description, xacro)
@@ -31,5 +31,5 @@
 	<!-- LF leg -->
 	<xacro:hyq_leg
-		name="LF"
+		name="lf"
 		parent="trunk"
 		reflect_hip="1"
@@ -40,5 +40,5 @@
 	<!-- RF leg -->
 	<xacro:hyq_leg
-		name="RF"
+		name="rf"
 		parent="trunk"
 		reflect_hip="-1"
@@ -49,5 +49,5 @@
 	<!-- LH leg -->
 	<xacro:hyq_leg
-		name="LH"
+		name="lh"
 		parent="trunk"
 		reflect_hip="-1"
@@ -58,5 +58,5 @@
 	<!-- RH leg -->
 	<xacro:hyq_leg
-		name="RH"
+		name="rh"
 		parent="trunk"
 		reflect_hip="1"

File: hyq_description/urdfs/leg/leg.transmission.xacro (robot description, xacro)
@@ -5,5 +5,5 @@
 		<transmission name="${name}_haa_trans">
 			<type>transmission_interface/SimpleTransmission</type>
-			<joint name="${name}_HAA"/>
+			<joint name="${name}_haa"/>
 			<actuator name="${name}_haa_motor">
 				<hardwareInterface>EffortJointInterface</hardwareInterface>
@@ -14,5 +14,5 @@
 		<transmission name="${name}_hfe_upper_trans">
 			<type>transmission_interface/SimpleTransmission</type>
-			<joint name="${name}_HFE"/>
+			<joint name="${name}_hfe"/>
 			<actuator name="${name}_hfe_motor">
 				<hardwareInterface>EffortJointInterface</hardwareInterface>
@@ -23,6 +23,6 @@
 		<transmission name="${name}_kfe_trans">
 			<type>transmission_interface/SimpleTransmission</type>
-			<joint name="${name}_KFE"/>
-			<actuator name="${name}_hfe_motor">
+			<joint name="${name}_kfe"/>
+			<actuator name="${name}_kfe_motor">
 				<hardwareInterface>EffortJointInterface</hardwareInterface>
 				<mechanicalReduction>1</mechanicalReduction>

File: hyq_description/urdfs/leg/leg.urdf.xacro (robot description, xacro)
@@ -15,7 +15,7 @@
 		</joint>-->
 		<!-- Hip joint assembly -->
-		<joint name="${name}_HAA" type="revolute">
-			<origin xyz="0.0 0.0 0.0" rpy="0.0 0.0 ${haa_pos0}"/>
-			<!--<parent link="${name}_haa_fake"/>-->
+		<joint name="${name}_haa_joint" type="revolute">
+			<!--<origin xyz="0.0 0.0 0.0" rpy="0.0 0.0 ${haa_pos0}"/>
+			<parent link="${name}_haa_fake"/>-->
 			<insert_block name="origin"/>
 			<parent link="${parent}"/>
@@ -27,5 +27,5 @@
 		</joint>
 		<!-- Upper leg joint -->
-		<joint name="${name}_HFE" type="revolute">
+		<joint name="${name}_hfe_joint" type="revolute">
 			<origin xyz="${d_tbb} 0.0 0.0" rpy="${reflect_upper*PI/2} ${-reflect_hip*hfe_pos0} 0.0"/>
 			<parent link="${name}_hip_assembly"/>
@@ -37,5 +37,5 @@
 		</joint>
 		<!-- Lower leg joint -->
-		<joint name="${name}_KFE" type="revolute">
+		<joint name="${name}_kfe_joint" type="revolute">
 			<origin xyz="${d_p1p2} 0.0 0.0" rpy="0.0 0.0 ${reflect_front*kfe_pos0}"/>
 			<parent link="${name}_upper_leg"/>

Commit message: corrected PTU transforms, bumblebee transform and PTU mount position (with calibration made by Jesus

File: hyq_description/robots/hyq.urdf.xacro (robot description, xacro)
@@ -31,5 +31,5 @@
 	<!-- LF leg -->
 	<xacro:hyq_leg
-		name="lf"
+		name="LF"
 		parent="trunk"
 		reflect_hip="1"
@@ -40,5 +40,5 @@
 	<!-- RF leg -->
 	<xacro:hyq_leg
-		name="rf"
+		name="RF"
 		parent="trunk"
 		reflect_hip="-1"
@@ -49,5 +49,5 @@
 	<!-- LH leg -->
 	<xacro:hyq_leg
-		name="lh"
+		name="LH"
 		parent="trunk"
 		reflect_hip="-1"
@@ -58,5 +58,5 @@
 	<!-- RH leg -->
 	<xacro:hyq_leg
-		name="rh"
+		name="RH"
 		parent="trunk"
 		reflect_hip="1"
@@ -78,5 +78,5 @@
 		name="ptu"
 		parent="trunk">
-		<origin xyz="0.63 0 0.095" rpy="0 ${PI/6} 0"/>
+		<origin xyz="0.684637 -0.024200 0.051570" rpy="0.071069 0.619695 0.020771"/>
 	</xacro:ptu_d46>
 	<!-- Bumblebee -->
@@ -87,4 +87,4 @@
 		ns="bumblebee"
 		frame_prefix="bumblebee_"
-		high_res="false"/><!-- xyz="0.63 0 0.095" rpy="0 0 0" -->
+		high_res="false"/> <!-- xyz="0.63 0 0.095" rpy="0 0 0" -->
 </robot>

Commit message: Corrections to urdf and gazebo descriptions

File: hyq_description/robots/hyq.urdf.xacro (robot description, xacro)
@@ -80,4 +80,9 @@
 		<origin xyz="0.63 0 0.095" rpy="0 ${PI/6} 0"/>
 	</xacro:asus_xtion_camera> --> <!-- <origin xyz="0.63 0 0.095" rpy="0 ${PI/6} 0"/> --> <!-- ptu_mount_link -->
+	<xacro:asus_xtion_camera
+		name="head_mount"
+		parent="ptu_mount_link">
+		<origin xyz="0.0 0 0.04" rpy="0 0 0"/>
+	</xacro:asus_xtion_camera>
 	<!-- Velodyne -->
 <!--	<xacro:velodyne
@@ -96,5 +101,6 @@
 		name="ptu"
 		parent="trunk">
-		<origin xyz="0.6357 0.04397 0.08809" rpy="-0.041779 0.31978 -0.061764"/>
+<!-- 		<origin xyz="0.6357 0.04397 0.08809" rpy="-0.041779 0.31978 -0.061764"/> -->
+		<origin xyz="0.684637 -0.024200 0.051570" rpy="0.071069 0.619695 0.020771"/>
 	</xacro:ptu_d46>
 	<!-- Bumblebee -->

File: hyq_description/urdfs/leg/leg.transmission.xacro (robot description, xacro)
@@ -5,5 +5,5 @@
 		<transmission name="${name}_haa_trans">
 			<type>transmission_interface/SimpleTransmission</type>
-			<joint name="${name}_haa"/>
+			<joint name="${name}_haa_joint"/>
 			<actuator name="${name}_haa_motor">
 				<hardwareInterface>EffortJointInterface</hardwareInterface>
@@ -14,5 +14,5 @@
 		<transmission name="${name}_hfe_upper_trans">
 			<type>transmission_interface/SimpleTransmission</type>
-			<joint name="${name}_hfe"/>
+			<joint name="${name}_hfe_joint"/>
 			<actuator name="${name}_hfe_motor">
 				<hardwareInterface>EffortJointInterface</hardwareInterface>
@@ -23,5 +23,5 @@
 		<transmission name="${name}_kfe_trans">
 			<type>transmission_interface/SimpleTransmission</type>
-			<joint name="${name}_kfe"/>
+			<joint name="${name}_kfe_joint"/>
 			<actuator name="${name}_kfe_motor">
 				<hardwareInterface>EffortJointInterface</hardwareInterface>

Commit message: Revert "Merge branch 'vision'"
This reverts commit 5c0a77c8d8353eb73e90cf3b4bbb1ce35fa5ef09, reversing
changes made to 05308aa2998ee2cb23c12dafeba2a5d9e08b7dea.

File: hyq_description/robots/hyq.urdf.xacro (robot description, xacro)
@@ -74,30 +74,33 @@
 		<origin xyz="0.3 0 0.095" rpy="0 ${-PI} 0"/>
 	</xacro:microstrain_3dmgx325_imu>
-	<!-- Asus Xtion Pro -->
+<!-- Asus Xtion Pro -->
+<!--	<xacro:asus_xtion_camera
+		name="head_mount"
+		parent="trunk">
+		<origin xyz="0.63 0 0.095" rpy="0 ${PI/6} 0"/>
+	</xacro:asus_xtion_camera> --> <!-- <origin xyz="0.63 0 0.095" rpy="0 ${PI/6} 0"/> --> <!-- ptu_mount_link -->
 	<xacro:asus_xtion_camera
 		name="head_mount"
 		parent="ptu_mount_link">
-		<origin xyz="0.0 0 0.015" rpy="0 0 0"/>
-<!-- The vertical offset between the middle of xtion and the middle of bumblebee is 5 cm-->
-<!-- but since bumblebee_mount_link is computed in the middle of the camera and the xtion on its base instead -->
-<!-- we have 5 cm - 3.5 cm (vertical distance between xtion optical frame and base) = 1.5 cm -->
+		<origin xyz="0.0 0 0.04" rpy="0 0 0"/>
 	</xacro:asus_xtion_camera>
 	<!-- Velodyne -->
-	<!--xacro:velodyne
+<!--	<xacro:velodyne
 		name="trunk_mount"
 		parent="trunk">
 		<origin xyz="0.39 0 0.269" rpy="0 0 0"/>
-	</xacro:velodyne-->
-	<!-- Kinect --> <!-- is no more used, but we keep it for compatibilty -->
-	<!--xacro:kinect_camera
+	</xacro:velodyne>-->
+	<!-- Kinect mount -->
+<!--	<xacro:kinect_camera
 		name="head_mount"
 		parent="trunk">
 		<origin xyz="0.63 0 0.095" rpy="0 0 0"/>
-	</xacro:kinect_camera-->
+	</xacro:kinect_camera>-->
 	<!-- PTU unit -->
 	<xacro:ptu_d46
 		name="ptu"
 		parent="trunk">
-		<origin xyz="0.693327 -0.015447 0.119533" rpy="-0.013127 0.574478 -0.007748"/>
+<!-- 		<origin xyz="0.6357 0.04397 0.08809" rpy="-0.041779 0.31978 -0.061764"/> -->
+		<origin xyz="0.684637 -0.024200 0.051570" rpy="0.071069 0.619695 0.020771"/>
 	</xacro:ptu_d46>
 	<!-- Bumblebee -->
@@ -108,4 +111,4 @@
 		ns="bumblebee"
 		frame_prefix="bumblebee_"
-		high_res="false"/>
+		high_res="false"/> <!-- xyz="0.63 0 0.095" rpy="0 0 0" -->
 </robot>

File: hyq_description/urdfs/sensors/bumblebee.urdf.xacro (robot description, xacro)
@@ -11,9 +11,9 @@
 			<parent link="${frame_prefix}mount_link"/>
 			<child link="${frame_prefix}optical_frame"/>
-			<origin xyz="0 -0.06 0.00" rpy="-${PI/2} 0 -${PI/2}"/>
+			<origin xyz="0 0 0" rpy="0 0 0"/>
 		</joint>
 		<link name="${frame_prefix}mount_link">
 			<visual>
-				<origin xyz="0 0 0" rpy="${PI/2} 0 ${PI/2}"/>
+				<origin xyz="0 0 0" rpy="0 0 0"/>
 				<geometry>
 					<mesh filename="package://hyq_description/meshes/sensors/bumblebee.dae"/>
@@ -21,5 +21,5 @@
 			</visual>
 			<collision>
-				<origin xyz="0 0 0" rpy="${PI/2} 0 ${PI/2}"/>
+				<origin xyz="0 0 0" rpy="0 0 0"/>
 				<geometry>
 					<mesh filename="package://hyq_description/meshes/sensors/bumblebee.dae"/>
@@ -42,6 +42,6 @@
 		<xacro:if value="${high_res}">
 			<xacro:stereo_camera
-				reference="${frame_prefix}mount_link"
-				frame_id="${frame_prefix}mount_link"
+				reference="${frame_prefix}optical_frame"
+				frame_id="${frame_prefix}optical_frame"
 				ns="${ns}"
 				hfov="${hfov}"
@@ -54,6 +54,6 @@
 		<xacro:unless value="${high_res}">
 			<xacro:stereo_camera
-				reference="${frame_prefix}mount_link"
-				frame_id="${frame_prefix}mount_link"
+				reference="${frame_prefix}optical_frame"
+				frame_id="${frame_prefix}optical_frame"
 				ns="${ns}"
 				hfov="${hfov}"

File: hyq_description/urdfs/sensors/ptu_d46.urdf.xacro (robot description, xacro)
@@ -101,5 +101,5 @@
 			<origin xyz="0 0 0" rpy="-${PI/2} 0 0"/>
 			<child link="${name}_tilted_link"/>
-			<axis xyz="0 1 0"/> <!-- 0 1 0-->
+			<axis xyz="0 1 0"/>
 			<limit lower="${-tilt_down_range}" upper="${tilt_up_range}" effort="${joint_effort}" velocity="${tilt_velocity}"/>
 		</joint>

File: hyq_description/urdfs/sensors/stereo_camera.gazebo.xacro (robot description, xacro)
@@ -6,5 +6,5 @@
 				<update_rate>${update_rate}</update_rate>
 				<camera name="left">
-					<pose> 0 ${baseline / 2.0} 0 0 0 0</pose>
+					<pose>${baseline / 2.0} 0 0 0 1.5707 1.5707</pose>
 					<horizontal_fov>${hfov}</horizontal_fov>
 					<image>
@@ -24,5 +24,5 @@
 				</camera>
 				<camera name="right">
-					<pose> 0 ${-baseline / 2.0} 0 0 0 0</pose>
+					<pose>${-baseline / 2.0} 0 0 0 1.5707 1.5707</pose>
 					<horizontal_fov>${hfov}</horizontal_fov>
 					<image>

Commit message: Solved issue. I took the updated files from branch vision and I committed them inside master. Merging the other way round somehow overwrites my correct modifications to sensors files

File: hyq_description/robots/hyq.urdf.xacro (robot description, xacro)
@@ -31,5 +31,5 @@
 	<!-- LF leg -->
 	<xacro:hyq_leg
-		name="lf"
+		name="LF"
 		parent="trunk"
 		reflect_hip="1"
@@ -40,5 +40,5 @@
 	<!-- RF leg -->
 	<xacro:hyq_leg
-		name="rf"
+		name="RF"
 		parent="trunk"
 		reflect_hip="-1"
@@ -49,5 +49,5 @@
 	<!-- LH leg -->
 	<xacro:hyq_leg
-		name="lh"
+		name="LH"
 		parent="trunk"
 		reflect_hip="-1"
@@ -58,5 +58,5 @@
 	<!-- RH leg -->
 	<xacro:hyq_leg
-		name="rh"
+		name="RH"
 		parent="trunk"
 		reflect_hip="1"
@@ -74,32 +74,8 @@
 		<origin xyz="0.3 0 0.095" rpy="0 ${-PI} 0"/>
 	</xacro:microstrain_3dmgx325_imu>
-<!-- Asus Xtion Pro -->
-<!--	<xacro:asus_xtion_camera
-		name="head_mount"
-		parent="trunk">
-		<origin xyz="0.63 0 0.095" rpy="0 ${PI/6} 0"/>
-	</xacro:asus_xtion_camera> --> <!-- <origin xyz="0.63 0 0.095" rpy="0 ${PI/6} 0"/> --> <!-- ptu_mount_link -->
-	<xacro:asus_xtion_camera
-		name="head_mount"
-		parent="ptu_mount_link">
-		<origin xyz="0.0 0 0.04" rpy="0 0 0"/>
-	</xacro:asus_xtion_camera>
-	<!-- Velodyne -->
-<!--	<xacro:velodyne
-		name="trunk_mount"
-		parent="trunk">
-		<origin xyz="0.39 0 0.269" rpy="0 0 0"/>
-	</xacro:velodyne>-->
-	<!-- Kinect mount -->
-<!--	<xacro:kinect_camera
-		name="head_mount"
-		parent="trunk">
-		<origin xyz="0.63 0 0.095" rpy="0 0 0"/>
-	</xacro:kinect_camera>-->
 	<!-- PTU unit -->
 	<xacro:ptu_d46
 		name="ptu"
 		parent="trunk">
-<!-- 		<origin xyz="0.6357 0.04397 0.08809" rpy="-0.041779 0.31978 -0.061764"/> -->
 		<origin xyz="0.684637 -0.024200 0.051570" rpy="0.071069 0.619695 0.020771"/>
 	</xacro:ptu_d46>
