Commit message: I really hate git. Committing the most updated hyq model. Hope this is the last dirty fix.

File: hyq_description/robots/hyq.urdf.xacro (robot description, xacro)
@@ -31,5 +31,5 @@
 	<!-- LF leg -->
 	<xacro:hyq_leg
-		name="LF"
+		name="lf"
 		parent="trunk"
 		reflect_hip="1"
@@ -40,5 +40,5 @@
 	<!-- RF leg -->
 	<xacro:hyq_leg
-		name="RF"
+		name="rf"
 		parent="trunk"
 		reflect_hip="-1"
@@ -49,5 +49,5 @@
 	<!-- LH leg -->
 	<xacro:hyq_leg
-		name="LH"
+		name="lh"
 		parent="trunk"
 		reflect_hip="-1"
@@ -58,5 +58,5 @@
 	<!-- RH leg -->
 	<xacro:hyq_leg
-		name="RH"
+		name="rh"
 		parent="trunk"
 		reflect_hip="1"
@@ -74,9 +74,30 @@
 		<origin xyz="0.3 0 0.095" rpy="0 ${-PI} 0"/>
 	</xacro:microstrain_3dmgx325_imu>
+	<!-- Asus Xtion Pro -->
+	<xacro:asus_xtion_camera
+		name="head_mount"
+		parent="ptu_mount_link">
+		<origin xyz="0.0 0 0.015" rpy="0 0 0"/>
+<!-- The vertical offset between the middle of xtion and the middle of bumblebee is 5 cm-->
+<!-- but since bumblebee_mount_link is computed in the middle of the camera and the xtion on its base instead -->
+<!-- we have 5 cm - 3.5 cm (vertical distance between xtion optical frame and base) = 1.5 cm -->
+	</xacro:asus_xtion_camera>
+	<!-- Velodyne -->
+	<!--xacro:velodyne
+		name="trunk_mount"
+		parent="trunk">
+		<origin xyz="0.39 0 0.269" rpy="0 0 0"/>
+	</xacro:velodyne-->
+	<!-- Kinect --> <!-- is no more used, but we keep it for compatibilty -->
+	<!--xacro:kinect_camera
+		name="head_mount"
+		parent="trunk">
+		<origin xyz="0.63 0 0.095" rpy="0 0 0"/>
+	</xacro:kinect_camera-->
 	<!-- PTU unit -->
 	<xacro:ptu_d46
 		name="ptu"
 		parent="trunk">
-		<origin xyz="0.684637 -0.024200 0.051570" rpy="0.071069 0.619695 0.020771"/>
+		<origin xyz="0.693327 -0.015447 0.119533" rpy="-0.013127 0.574478 -0.007748"/>
 	</xacro:ptu_d46>
 	<!-- Bumblebee -->
@@ -87,4 +108,4 @@
 		ns="bumblebee"
 		frame_prefix="bumblebee_"
-		high_res="false"/> <!-- xyz="0.63 0 0.095" rpy="0 0 0" -->
+		high_res="false"/>
 </robot>

Commit message: Fixed the problem with the PTU joints. Added the bumblebee and velodyne for common simulations.

File: hyq_description/robots/hyq.urdf.xacro (robot description, xacro)
@@ -90,9 +90,9 @@
 	</xacro:asus_xtion_camera>
 	<!-- Velodyne -->
-	<!--xacro:velodyne
+	<xacro:velodyne
 		name="trunk_mount"
 		parent="trunk">
 		<origin xyz="0.39 0 0.269" rpy="0 0 0"/>
-	</xacro:velodyne-->
+	</xacro:velodyne>
 	<!-- Kinect --> <!-- is no more used, but we keep it for compatibilty -->
 	<!--xacro:kinect_camera

File: hyq_description/robots/hyq_gazebo.urdf.xacro (robot description, xacro)
@@ -85,14 +85,14 @@
 	<!-- we have 5 cm - 3.5 cm (vertical distance between xtion optical frame and base) = 1.5 cm -->
 	<xacro:asus_xtion_camera
-		name="head_mount_asus_xtion"
+		name="head_mount"
 		parent="ptu_mount_link">
 		<origin xyz="0.0 0 0.015" rpy="0 0 0"/>
 	</xacro:asus_xtion_camera>
 	<!-- Velodyne -->
-	<!--<xacro:velodyne
+	<xacro:velodyne
 		name="trunk_mount"
 		parent="trunk">
 		<origin xyz="0.39 0 0.269" rpy="0 0 0"/>
-	</xacro:velodyne-->
+	</xacro:velodyne>
 	<!-- Kinect --> <!-- is no more used, but we keep it for compatibilty -->
 	<!--<xacro:kinect_camera
@@ -102,5 +102,5 @@
 	</xacro:kinect_camera-->
 	<!-- Bumblebee -->
-	<!--<xacro:bumblebee_97
+	<xacro:bumblebee_97
 		parent_link="ptu_mount_link"
 		xyz="0 0 0"
@@ -108,4 +108,4 @@
 		ns="bumblebee"
 		frame_prefix="bumblebee_"
-		high_res="false"/>-->
+		high_res="false"/>
 </robot>

File: hyq_description/urdfs/sensors/asus_xtion.urdf.xacro (robot description, xacro)
@@ -9,32 +9,32 @@
 			<insert_block name="origin"/>
 			<parent link="${parent}"/>
-			<child link="${name}_link"/>
+			<child link="${name}_asus_xtion_link"/>
 		</joint>
 		<!-- asus ir sensor physical attachment -->
-		<joint name="${name}_depth_joint" type="fixed">
+		<joint name="${name}_asus_xtion_depth_joint" type="fixed">
 			<origin xyz="${asus_xtion_x} ${asus_xtion_depth_y} ${asus_xtion_z}" rpy="0.0 0.0 0.0"/>
-			<parent link="${name}_link"/>
-			<child link="${name}_depth_frame"/>
+			<parent link="${name}_asus_xtion_link"/>
+			<child link="${name}_asus_xtion_depth_frame"/>
 		</joint>
 		<!-- asus xtion ir sensor frame -->
-		<joint name="${name}_depth_optical_frame_joint" type="fixed">
+		<joint name="${name}_asus_xtion_depth_optical_frame_joint" type="fixed">
 			<origin xyz="0 0 0"	rpy="${asus_xtion_roll} ${asus_xtion_pitch} ${asus_xtion_yaw}"/>
-			<parent link="${name}_depth_frame"/>
-			<child link="${name}_depth_optical_frame"/>
+			<parent link="${name}_asus_xtion_depth_frame"/>
+			<child link="${name}_asus_xtion_depth_optical_frame"/>
 		</joint>
 		<!-- asus_xtion rgb sensor physical attachment -->
-		<joint name="${name}_rgb_joint" type="fixed">
+		<joint name="${name}_asus_xtion_rgb_joint" type="fixed">
 			<origin xyz="${asus_xtion_x} ${asus_xtion_rgb_y} ${asus_xtion_z}" rpy="0.0 0.0 0.0"/>
-			<parent link="${name}_link"/>
-			<child link="${name}_rgb_frame"/>
+			<parent link="${name}_asus_xtion_link"/>
+			<child link="${name}_asus_xtion_rgb_frame"/>
 		</joint>
 		<!-- asus xtion rgb sensor frame -->
-		<joint name="${name}_rgb_optical_frame_joint" type="fixed">
+		<joint name="${name}_asus_xtion_rgb_optical_frame_joint" type="fixed">
 			<origin xyz="0 0 0"	rpy="${asus_xtion_roll} ${asus_xtion_pitch} ${asus_xtion_yaw}"/>
-			<parent link="${name}_rgb_frame"/>
-			<child link="${name}_rgb_optical_frame"/>
+			<parent link="${name}_asus_xtion_rgb_frame"/>
+			<child link="${name}_asus_xtion_rgb_optical_frame"/>
 		</joint>
 		<!-- Links -->
-		<link name="${name}_link">
+		<link name="${name}_asus_xtion_link">
 			<inertial>
 				<mass value="0.1"/>
@@ -59,5 +59,5 @@
 		</link>
 		<!-- ir sensor link -->
-		<link name="${name}_depth_frame">
+		<link name="${name}_asus_xtion_depth_frame">
 			<inertial>
 				<mass value="0.1" />
@@ -79,7 +79,7 @@
 		</link>
 		<!-- ir optical sensor link -->
-		<link name="${name}_depth_optical_frame"/>
+		<link name="${name}_asus_xtion_depth_optical_frame"/>
 		<!-- rgb sensor link -->
-		<link name="${name}_rgb_frame" >
+		<link name="${name}_asus_xtion_rgb_frame" >
 			<inertial>
 				<mass value="0.1" />
@@ -101,8 +101,8 @@
 		</link>
 		<!-- rgb optical sensor link -->
-		<link name="${name}_rgb_optical_frame"/>
+		<link name="${name}_asus_xtion_rgb_optical_frame"/>
 	<!-- gazebo extensions -->
-	<xacro:asus_xtion_depth_sensor link_name="${name}_depth_frame" frame_name="${name}_depth_optical_frame" camera_name="${name}" />
-	<xacro:asus_xtion_rgb_sensor link_name="${name}_rgb_frame" frame_name="${name}_rgb_optical_frame" camera_name="${name}" />
+	<xacro:asus_xtion_depth_sensor link_name="${name}_asus_xtion_depth_frame" frame_name="${name}_asus_xtion_depth_optical_frame" camera_name="${name}_asus_xtion" />
+	<xacro:asus_xtion_rgb_sensor link_name="${name}_asus_xtion_rgb_frame" frame_name="${name}_asus_xtion_rgb_optical_frame" camera_name="${name}_asus_xtion" />
 	</xacro:macro>
 </root>

File: hyq_description/urdfs/sensors/ptu_d46.urdf.xacro (robot description, xacro)
@@ -8,5 +8,5 @@
 				<origin xyz="0.0 0.0 0.0"/>
 				<mass value="0.65"/>
-				<inertia ixx="0.0" iyy="0.0" izz="0.0" ixy="0.0" ixz="0.0" iyz="0.0"/>
+				<inertia ixx="0.01" iyy="0.01" izz="0.01" ixy="0.0" ixz="0.0" iyz="0.0"/>
 			</inertial>
 			<visual>
@@ -66,5 +66,5 @@
 		</joint>
 		<!-- The pan joint -->
-		<joint name="${name}_pan" type="fixed">
+		<joint name="${name}_pan" type="revolute">
 			<origin xyz="0 0 0.066" rpy="-${PI/2} 0 0"/>
 			<parent link="${name}_pan_link"/>
@@ -74,5 +74,5 @@
 		</joint>
 		<!-- The tilt joint -->
-		<joint name="${name}_tilt" type="fixed">
+		<joint name="${name}_tilt" type="revolute">
 			<origin xyz="0 0 0" rpy="-${PI/2} 0 0"/>
 			<parent link="${name}_tilt_link"/>
@@ -94,5 +94,5 @@
 				<origin xyz="0.0 0.0 0.0"/>
 				<mass value="0.01"/>
-				<inertia ixx="0.0" iyy="0.0" izz="0.0" ixy="0.0" ixz="0.0" iyz="0.0"/>
+				<inertia ixx="0.01" iyy="0.01" izz="0.01" ixy="0.0" ixz="0.0" iyz="0.0"/>
 			</inertial>
 			<visual>
@@ -113,5 +113,5 @@
 				<origin xyz="0.0 0.0 0.0"/>
 				<mass value="0.01"/>
-				<inertia ixx="0.0" iyy="0.0" izz="0.0" ixy="0.0" ixz="0.0" iyz="0.0"/>
+				<inertia ixx="0.01" iyy="0.01" izz="0.01" ixy="0.0" ixz="0.0" iyz="0.0"/>
 			</inertial>
 			<visual>
@@ -132,5 +132,5 @@
 				<origin xyz="0.0 0.0 0.0"/>
 				<mass value="0.01"/>
-				<inertia ixx="0.0" iyy="0.0" izz="0.0" ixy="0.0" ixz="0.0" iyz="0.0"/>
+				<inertia ixx="0.01" iyy="0.01" izz="0.01" ixy="0.0" ixz="0.0" iyz="0.0"/>
 			</inertial>
 			<visual>
@@ -148,5 +148,5 @@
 		</link>
 		<!-- Extensions -->
-		<!--<xacro:ptu_transmission name="${name}"/>-->
+		<xacro:ptu_transmission name="${name}"/>
 	</xacro:macro>
 </robot>

File: hyq_description/urdfs/sensors/velodyne.urdf.xacro (robot description, xacro)
@@ -41,7 +41,13 @@
 		</link>
 		<!-- rgb optical sensor link -->
-		<link name="${name}_velodyne_optical_frame"/>
-	<!-- gazebo extensions -->
-	<xacro:velodyne_sensor link_name="${name}_velodyne_optical_frame" frame_name="${name}_velodyne_frame" lidar_name="${name}_velodyne" />
+		<link name="${name}_velodyne_optical_frame">
+			<inertial>
+				<mass value="0.1"/>
+				<origin xyz="0.0 0.0 0.0" rpy="0.0 0.0 0.0"/>
+				<inertia ixx="0.01" ixy="0.0" ixz="0.0" iyy="0.01" iyz="0.0" izz="0.01"/>
+			</inertial>
+		</link>
+		<!-- gazebo extensions -->
+		<xacro:velodyne_sensor link_name="${name}_velodyne_optical_frame" frame_name="${name}_velodyne_frame" lidar_name="${name}_velodyne" />
 	</xacro:macro>
 </root>

Commit message: Restablishing the old values. I need to calibrate the Asus Xtion camera.

File: hyq_description/robots/hyq.urdf.xacro (robot description, xacro)
@@ -87,5 +87,5 @@
 		name="head_mount"
 		parent="ptu_mount_link">
-		<origin xyz="0.0 0 0.015" rpy="0 0 0"/>
+		<origin xyz="0 0 0.015" rpy="0 0 0"/>
 	</xacro:asus_xtion_camera>
 	<!-- Velodyne -->

File: hyq_description/urdfs/sensors/asus_xtion.urdf.xacro (robot description, xacro)
@@ -43,5 +43,5 @@
 			</inertial>
 			<visual>
-				<origin xyz="-0.01 0.0 0.0" rpy="0.0 0.0 0.0"/>
+				<origin xyz="0.0 0.0 0.0" rpy="0.0 0.0 0.0"/>
 				<geometry>
 					<mesh filename="package://hyq_description/meshes/sensors/asus_xtion.dae" scale="1 1 1" />

Commit message: Fixed the problem of dimension of Asion Xtion

File: hyq_description/robots/hyq.urdf.xacro (robot description, xacro)
@@ -81,11 +81,8 @@
 	</xacro:ptu_d46>
 	<!-- Asus Xtion Pro -->
-	<!-- The vertical offset between the middle of xtion and the middle of bumblebee is 5 cm-->
-	<!-- but since bumblebee_mount_link is computed in the middle of the camera and the xtion on its base instead -->
-	<!-- we have 5 cm - 3.5 cm (vertical distance between xtion optical frame and base) = 1.5 cm -->
 	<xacro:asus_xtion_camera
 		name="head_mount"
 		parent="ptu_mount_link">
-		<origin xyz="0 0 0.015" rpy="0 0 0"/>
+		<origin xyz="0 0 0.036" rpy="0 0 0"/>
 	</xacro:asus_xtion_camera>
 	<!-- Velodyne -->
@@ -104,5 +101,5 @@
 	<xacro:bumblebee_97
 		parent_link="ptu_mount_link"
-		xyz="0 0 0"
+		xyz="0 0 0.018"
 		rpy="0 0 0"
 		ns="bumblebee"

Commit message: Added the vislab sensor description

File: hyq_description/robots/hyq.urdf.xacro (robot description, xacro)
@@ -16,4 +16,5 @@
 	<xacro:include filename="$(find hyq_description)/urdfs/sensors/ptu_d46.urdf.xacro"/>
 	<xacro:include filename="$(find hyq_description)/urdfs/sensors/bumblebee.urdf.xacro"/>
+	<xacro:include filename="$(find hyq_description)/urdfs/sensors/vislab_3dve.urdf.xacro"/>
 	<!-- generic simulator_gazebo plugins for starting mechanism control, ros time -->
 	<xacro:include filename="$(find hyq_description)/gazebo/gazebo.urdf.xacro"/>
@@ -84,5 +85,5 @@
 		name="head_mount"
 		parent="ptu_mount_link">
-		<origin xyz="0 0 0.036" rpy="0 0 0"/>
+		<origin xyz="0 0 0.050" rpy="0 0 0"/><!--<origin xyz="0 0 0.036" rpy="0 0 0"/> with Bumblebee setup -->
 	</xacro:asus_xtion_camera>
 	<!-- Velodyne -->
@@ -99,5 +100,5 @@
 	</xacro:kinect_camera-->
 	<!-- Bumblebee -->
-	<xacro:bumblebee_97
+<!--	<xacro:bumblebee_97
 		parent_link="ptu_mount_link"
 		xyz="0 0 0.018"
@@ -105,4 +106,10 @@
 		ns="bumblebee"
 		frame_prefix="bumblebee_"
+		high_res="false"/>-->
+	<xacro:vislab_3dve_72
+		name="vislab_3dve"
+		parent="ptu_mount_link"
+		xyz="0 0 0.025"
+		rpy="0 0 0"
 		high_res="false"/>
 </robot>

Commit message: Fixed the position of the Asus Xtion for Vislab camera

File: hyq_description/robots/hyq.urdf.xacro (robot description, xacro)
@@ -85,5 +85,5 @@
 		name="head_mount"
 		parent="ptu_mount_link">
-		<origin xyz="0 0 0.050" rpy="0 0 0"/><!--<origin xyz="0 0 0.036" rpy="0 0 0"/> with Bumblebee setup -->
+		<origin xyz="0 0 0.04397" rpy="0 0 0"/><!--<origin xyz="0 0 0.036" rpy="0 0 0"/> with Bumblebee setup -->
 	</xacro:asus_xtion_camera>
 	<!-- Velodyne -->

Commit message: Changed the position of the Asus sensor to the real one. In the past, I put a wrong value because the ptu wasn't calibrate

File: hyq_description/robots/hyq.urdf.xacro (robot description, xacro)
@@ -82,8 +82,10 @@
 	</xacro:ptu_d46>
 	<!-- Asus Xtion Pro -->
+	<!--<origin xyz="0 0 0.036" rpy="0 0 0"/> with Bumblebee setup -->
+	<!--<origin xyz="0 0 0.04397" rpy="0 0 0"/> with Vislab setup -->
 	<xacro:asus_xtion_camera
 		name="head_mount"
 		parent="ptu_mount_link">
-		<origin xyz="0 0 0.04397" rpy="0 0 0"/><!--<origin xyz="0 0 0.036" rpy="0 0 0"/> with Bumblebee setup -->
+		<origin xyz="0 0 0.036" rpy="0 0 0"/>
 	</xacro:asus_xtion_camera>
 	<!-- Velodyne -->
@@ -100,5 +102,5 @@
 	</xacro:kinect_camera-->
 	<!-- Bumblebee -->
-<!--	<xacro:bumblebee_97
+	<xacro:bumblebee_97
 		parent_link="ptu_mount_link"
 		xyz="0 0 0.018"
@@ -106,10 +108,10 @@
 		ns="bumblebee"
 		frame_prefix="bumblebee_"
-		high_res="false"/>-->
-	<xacro:vislab_3dve_72
+		high_res="false"/>
+<!--	<xacro:vislab_3dve_72
 		name="vislab_3dve"
 		parent="ptu_mount_link"
 		xyz="0 0 0.025"
 		rpy="0 0 0"
-		high_res="false"/>
+		high_res="false"/>-->
 </robot>

File: hyq_description/urdfs/common.xacro (robot description, xacro)
@@ -53,7 +53,7 @@
 	<!-- Asus Xtion Camera Location (Nominally 0) -->
 	<property name="asus_xtion_x" value="0.0"/>
-	<property name="asus_xtion_depth_y" value="0.069"/>
-	<property name="asus_xtion_rgb_y" value="0.049"/>
-	<property name="asus_xtion_z" value="0.03"/>
+	<property name="asus_xtion_depth_y" value="0.045"/><!-- 0.069 -->
+	<property name="asus_xtion_rgb_y" value="0.01875"/><!-- 0.049 -->
+	<property name="asus_xtion_z" value="0.035"/>
 	<property name="asus_xtion_roll" value="${-PI/2}"/>
 	<property name="asus_xtion_pitch" value="0.0"/>

File: hyq_description/urdfs/sensors/asus_xtion.urdf.xacro (robot description, xacro)
@@ -9,10 +9,10 @@
 			<insert_block name="origin"/>
 			<parent link="${parent}"/>
-			<child link="${name}_asus_xtion_link"/>
+			<child link="${name}_asus_xtion_mount_link"/>
 		</joint>
 		<!-- asus ir sensor physical attachment -->
 		<joint name="${name}_asus_xtion_depth_joint" type="fixed">
 			<origin xyz="${asus_xtion_x} ${asus_xtion_depth_y} ${asus_xtion_z}" rpy="0.0 0.0 0.0"/>
-			<parent link="${name}_asus_xtion_link"/>
+			<parent link="${name}_asus_xtion_mount_link"/>
 			<child link="${name}_asus_xtion_depth_frame"/>
 		</joint>
@@ -26,5 +26,5 @@
 		<joint name="${name}_asus_xtion_rgb_joint" type="fixed">
 			<origin xyz="${asus_xtion_x} ${asus_xtion_rgb_y} ${asus_xtion_z}" rpy="0.0 0.0 0.0"/>
-			<parent link="${name}_asus_xtion_link"/>
+			<parent link="${name}_asus_xtion_mount_link"/>
 			<child link="${name}_asus_xtion_rgb_frame"/>
 		</joint>
@@ -36,5 +36,5 @@
 		</joint>
 		<!-- Links -->
-		<link name="${name}_asus_xtion_link">
+		<link name="${name}_asus_xtion_mount_link">
 			<inertial>
 				<mass value="0.1"/>
@@ -43,5 +43,5 @@
 			</inertial>
 			<visual>
-				<origin xyz="-0.015 0.0 0.0" rpy="0.0 0.0 0.0"/>
+				<origin xyz="0 0 0" rpy="0 0 0"/>
 				<geometry>
 					<mesh filename="package://hyq_description/meshes/sensors/asus_xtion.dae" scale="1 1 1" />

Commit message: Improved the calibration values of PTU. I used the new values from Stephane, and I modified a bit in order to get better results; this was tested using Asus Xtion and Bumblebee cameras. The Stephane's values are commented inside the code. Added a vicon marker link in order to use the original vicon_bridge code. I realized that Jesus's values are not complitly well, so I modified a bit!

File: hyq_description/robots/hyq.urdf.xacro (robot description, xacro)
@@ -17,4 +17,5 @@
 	<xacro:include filename="$(find hyq_description)/urdfs/sensors/bumblebee.urdf.xacro"/>
 	<xacro:include filename="$(find hyq_description)/urdfs/sensors/vislab_3dve.urdf.xacro"/>
+	<xacro:include filename="$(find hyq_description)/urdfs/sensors/vicon.urdf.xacro"/>
 	<!-- generic simulator_gazebo plugins for starting mechanism control, ros time -->
 	<xacro:include filename="$(find hyq_description)/gazebo/gazebo.urdf.xacro"/>
@@ -75,18 +76,4 @@
 		<origin xyz="0.3 0 0.095" rpy="0 ${-PI} 0"/>
 	</xacro:microstrain_3dmgx325_imu>
-	<!-- PTU unit -->
-	<xacro:ptu_d46
-		name="ptu"
-		parent="trunk">
-		<origin xyz="0.693327 -0.015447 0.119533" rpy="-0.013127 0.574478 -0.007748"/>
-	</xacro:ptu_d46>
-	<!-- Asus Xtion Pro -->
-	<!--<origin xyz="0 0 0.036" rpy="0 0 0"/> with Bumblebee setup -->
-	<!--<origin xyz="0 0 0.04397" rpy="0 0 0"/> with Vislab setup -->
-	<xacro:asus_xtion_camera
-		name="head_mount"
-		parent="ptu_mount_link">
-		<origin xyz="0 0 0.036" rpy="0 0 0"/>
-	</xacro:asus_xtion_camera>
 	<!-- Velodyne -->
 	<xacro:velodyne
@@ -95,4 +82,19 @@
 		<origin xyz="0.39 0 0.269" rpy="0 0 0"/>
 	</xacro:velodyne>
+	<!-- PTU unit -->
+	<xacro:ptu_d46
+		name="ptu"
+		parent="trunk">
+		<origin xyz="0.657353 0.015447 0.119533" rpy="-0.013127 0.569257 -0.007748"/>
+<!--		<origin xyz="0.667353 -0.010101 0.160544" rpy="0.043239 0.569257 0.041771"/>-->
+	</xacro:ptu_d46>
+	<!-- Asus Xtion Pro -->
+	<!--<origin xyz="0 0.005 0.036" rpy="0 0 0"/> with Bumblebee setup -->
+	<!--<origin xyz="0 0 0.04397" rpy="0 0 0"/> with Vislab setup -->
+	<xacro:asus_xtion_camera
+		name="head_mount"
+		parent="ptu_mount_link">
+		<origin xyz="0 0.005 0.036" rpy="0 0 0"/>
+	</xacro:asus_xtion_camera>
 	<!-- Kinect --> <!-- is no more used, but we keep it for compatibilty -->
 	<!--xacro:kinect_camera
@@ -115,3 +117,6 @@
 		rpy="0 0 0"
 		high_res="false"/>-->
+		<xacro:vicon parent="base_link">
+			<origin xyz="0.443 0.191 0.276" rpy="0 0 0"/>
+		</xacro:vicon>
 </robot>

File: hyq_description/urdfs/common.xacro (robot description, xacro)
@@ -52,7 +52,7 @@
 	<property name="joint_effort" value="30" />
 	<!-- Asus Xtion Camera Location (Nominally 0) -->
-	<property name="asus_xtion_x" value="0.0"/>
-	<property name="asus_xtion_depth_y" value="0.045"/><!-- 0.069 -->
-	<property name="asus_xtion_rgb_y" value="0.01875"/><!-- 0.049 -->
+	<property name="asus_xtion_x" value="0.009"/>
+	<property name="asus_xtion_depth_y" value="0.045"/>
+	<property name="asus_xtion_rgb_y" value="0.01875"/>
 	<property name="asus_xtion_z" value="0.035"/>
 	<property name="asus_xtion_roll" value="${-PI/2}"/>

File: hyq_description/urdfs/common_gazebo.xacro (robot description, xacro)
@@ -53,6 +53,6 @@
 	<!-- Asus Xtion Camera Location (Nominally 0) -->
 	<property name="asus_xtion_x" value="0.009"/>
-	<property name="asus_xtion_depth_y" value="0.049"/>
-	<property name="asus_xtion_rgb_y" value="0.022"/>
+	<property name="asus_xtion_depth_y" value="0.045"/>
+	<property name="asus_xtion_rgb_y" value="0.01875"/>
 	<property name="asus_xtion_z" value="0.035"/>
 	<property name="asus_xtion_roll" value="${-PI/2}"/>

File: hyq_description/urdfs/sensors/asus_xtion.urdf.xacro (robot description, xacro)
@@ -13,5 +13,5 @@
 		<!-- asus ir sensor physical attachment -->
 		<joint name="${name}_asus_xtion_depth_joint" type="fixed">
-			<origin xyz="${asus_xtion_x} ${asus_xtion_depth_y} ${asus_xtion_z}" rpy="0.0 0.0 0.0"/>
+			<origin xyz="${asus_xtion_x} ${asus_xtion_depth_y} ${asus_xtion_z}" rpy="0 0 0"/>
 			<parent link="${name}_asus_xtion_mount_link"/>
 			<child link="${name}_asus_xtion_depth_frame"/>
@@ -25,5 +25,5 @@
 		<!-- asus_xtion rgb sensor physical attachment -->
 		<joint name="${name}_asus_xtion_rgb_joint" type="fixed">
-			<origin xyz="${asus_xtion_x} ${asus_xtion_rgb_y} ${asus_xtion_z}" rpy="0.0 0.0 0.0"/>
+			<origin xyz="${asus_xtion_x} ${asus_xtion_rgb_y} ${asus_xtion_z}" rpy="0 0 0"/>
 			<parent link="${name}_asus_xtion_mount_link"/>
 			<child link="${name}_asus_xtion_rgb_frame"/>
@@ -39,5 +39,5 @@
 			<inertial>
 				<mass value="0.1"/>
-				<origin xyz="0.0 0.0 0.0" rpy="0.0 0.0 0.0"/>
+				<origin xyz="0 0 0" rpy="0 0 0"/>
 				<inertia ixx="0.01" ixy="0.0" ixz="0.0" iyy="0.01" iyz="0.0" izz="0.01"/>
 			</inertial>
@@ -52,5 +52,5 @@
 			</visual>
 			<collision>
-				<origin xyz="0.0 0.0 ${asus_xtion_z}" rpy="0 0 0" />
+				<origin xyz="0 0 ${asus_xtion_z}" rpy="0 0 0" />
 				<geometry>
 					<box size="0.05 .18 0.035" />
@@ -62,9 +62,9 @@
 			<inertial>
 				<mass value="0.1" />
-				<origin xyz="0.0 0.0 0.0" rpy="0.0 0.0 0.0"/>
+				<origin xyz="0 0 0" rpy="0 0 0"/>
 				<inertia ixx="0.01" ixy="0.0" ixz="0.0" iyy="0.01" iyz="0.0" izz="0.01"/>
 			</inertial>
 			<visual>
-				<origin xyz="0.0 0.0 0.0" rpy="0.0 0.0 0.0"/>
+				<origin xyz="0 0 0" rpy="0 0 0"/>
 				<geometry>
 					<sphere radius="0.0005"/>
@@ -72,5 +72,5 @@
 			</visual>
 			<collision>
-				<origin xyz="0.0 0.0 0.0" rpy="0.0 0.0 0.0"/>
+				<origin xyz="0 0 0" rpy="0 0 0"/>
 				<geometry>
 					<sphere radius="0.0005"/>
@@ -84,9 +84,9 @@
 			<inertial>
 				<mass value="0.1" />
-				<origin xyz="0.0 0.0 0.0" rpy="0.0 0.0 0.0"/>
+				<origin xyz="0 0 0" rpy="0 0 0"/>
 				<inertia ixx="0.01" ixy="0.0" ixz="0.0" iyy="0.01" iyz="0.0" izz="0.01" />
 			</inertial>
 			<visual>
-				<origin xyz="0.0 0.0 0.0" rpy="0.0 0.0 0.0"/>
+				<origin xyz="0 0 0" rpy="0 0 0"/>
 				<geometry>
 					<sphere radius="0.0005"/>
@@ -94,5 +94,5 @@
 			</visual>
 			<collision>
-				<origin xyz="0.0 0.0 0.0" rpy="0.0 0.0 0.0"/>
+				<origin xyz="0 0 0" rpy="0 0 0"/>
 				<geometry>
 					<sphere radius="0.0005"/>
