Commit message: Cleaned the code. Removed the vicon frame. It was a fail

File: hyq_description/robots/hyq.urdf.xacro (robot description, xacro)
@@ -3,10 +3,8 @@
 	<!-- The following included files set up definitions of parts of the robot body -->
 	<xacro:include filename="$(find hyq_description)/urdfs/common.xacro"/>
-	<!-- HyQ base -->
+	<!-- HyQ trunk -->
 	<xacro:include filename="$(find hyq_description)/urdfs/trunk/trunk.urdf.xacro"/>
 	<!-- HyQ legs -->
 	<xacro:include filename="$(find hyq_description)/urdfs/leg/leg.urdf.xacro"/>
-	<!-- HyQ torso -->
-<!--  <xacro:include filename="$(find hyq_model)/urdfs/torso/torso.urdf.xacro" />-->
 	<!-- HyQ sensors -->
 	<xacro:include filename="$(find hyq_description)/urdfs/sensors/microstrain_3dmgx325_imu.urdf.xacro"/>
@@ -17,5 +15,4 @@
 	<xacro:include filename="$(find hyq_description)/urdfs/sensors/bumblebee.urdf.xacro"/>
 	<xacro:include filename="$(find hyq_description)/urdfs/sensors/vislab_3dve.urdf.xacro"/>
-	<xacro:include filename="$(find hyq_description)/urdfs/sensors/vicon.urdf.xacro"/>
 	<!-- generic simulator_gazebo plugins for starting mechanism control, ros time -->
 	<xacro:include filename="$(find hyq_description)/gazebo/gazebo.urdf.xacro"/>
@@ -30,5 +27,7 @@
 	<!-- body -->
 	<!-- trunk -->
-	<xacro:hyq_trunk name="base" />
+	<xacro:hyq_trunk name="base">
+		<origin xyz="-0.443 -0.191 -0.276" rpy="0 0 0"/>
+	</xacro:hyq_trunk>
 	<!-- LF leg -->
 	<xacro:hyq_leg
@@ -117,6 +116,3 @@
 		rpy="0 0 0"
 		high_res="false"/>-->
-		<xacro:vicon parent="base_link">
-			<origin xyz="0.443 0.191 0.276" rpy="0 0 0"/>
-		</xacro:vicon>
 </robot>

File: hyq_description/urdfs/leg/leg.urdf.xacro (robot description, xacro)
@@ -16,5 +16,5 @@
 		<!-- Hip joint assembly -->
 		<joint name="${name}_haa_joint" type="revolute">
-			<origin xyz="0.0 0.0 0.0" rpy="0.0 0.0 ${haa_pos0}"/>
+			<origin xyz="0 0 0" rpy="0 0 ${haa_pos0}"/>
 			<parent link="${name}_assembly"/>
 			<!--<insert_block name="origin"/>-->
@@ -38,5 +38,5 @@
 		<!-- Lower leg joint -->
 		<joint name="${name}_kfe_joint" type="revolute">
-			<origin xyz="${d_p1p2} 0.0 0.0" rpy="0.0 0.0 ${reflect_front*kfe_pos0}"/>
+			<origin xyz="${d_p1p2} 0 0" rpy="0 0 ${reflect_front*kfe_pos0}"/>
 			<parent link="${name}_upper_leg"/>
 			<child  link="${name}_lower_leg"/>
@@ -48,5 +48,5 @@
 		</joint>
 		<joint name="${name}_foot_joint" type="fixed">
-			<origin xyz="0.34 0.0 0.0" rpy="${PI/2} 0.0 ${-PI/2}"/>
+			<origin xyz="0.34 0 0" rpy="${PI/2} 0 ${-PI/2}"/>
 			<parent link="${name}_lower_leg"/>
 			<child  link="${name}_foot"/>
@@ -56,5 +56,5 @@
 		<link name="${name}_assembly">
 			<inertial>
-				<origin xyz="0.0 0.0 0.0"/>
+				<origin xyz="0 0 0"/>
 				<mass value="0.01"/>
 				<inertia ixx="0.01" iyy="0.01" izz="0.01" ixy="0.0" ixz="0.0" iyz="0.0"/>
@@ -69,5 +69,5 @@
 			</inertial>
 			<visual>
-				<origin xyz="0.0 0.0 0.0" rpy="${(1-reflect_hip)*PI/2} 0.0 0.0"/>
+				<origin xyz="0 0 0" rpy="${(1-reflect_hip)*PI/2} 0 0"/>
 				<geometry>
 					<mesh filename="package://hyq_description/meshes/leg/hip.dae" scale="1 1 1"/>
@@ -75,5 +75,5 @@
 			</visual>
 			<collision>
-				<origin xyz="0.0 0.0 0.0" rpy="${(1-reflect_hip)*PI/2} 0.0 0.0"/>
+				<origin xyz="0 0 0" rpy="${(1-reflect_hip)*PI/2} 0 0"/>
 				<geometry>
 					<mesh filename="package://hyq_description/meshes/leg/hip.dae" scale="1 1 1"/>
@@ -84,10 +84,10 @@
 		<link name="${name}_upper_leg">
 			<inertial>
-				<origin xyz="0.14796 ${reflect_upper*0.02958} 0.0"/>
+				<origin xyz="0.14796 ${reflect_upper*0.02958} 0"/>
 				<mass value="${m_upper}"/>
 				<inertia ixx="${ixx_upper}" iyy="${iyy_upper}" izz="${izz_upper}" ixy="${ixy_upper}" ixz="${ixz_upper}" iyz="${iyz_upper}"/>
 			</inertial>
 			<visual>
-				<origin xyz="0.0 0.0 0.0" rpy="${(1-reflect_front)*PI/2} 0.0 0.0"/>
+				<origin xyz="0 0 0" rpy="${(1-reflect_front)*PI/2} 0 0"/>
 				<geometry>
 					<mesh filename="package://hyq_description/meshes/leg/upper.dae" scale="1 1 1"/>
@@ -95,5 +95,5 @@
 			</visual>
 			<collision>
-				<origin xyz="0.0 0.0 0.0" rpy="${(1-reflect_front)*PI/2} 0.0 0.0"/>
+				<origin xyz="0 0 0" rpy="${(1-reflect_front)*PI/2} 0 0"/>
 				<geometry>
 					<mesh filename="package://hyq_description/meshes/leg/upper.dae" scale="1 1 1"/>
@@ -123,5 +123,5 @@
 		<link name="${name}_foot">
 			<inertial>
-				<origin xyz="0.0 0.0 0.0"/>
+				<origin xyz="0 0 0"/>
 				<mass value="0.01"/>
 				<inertia ixx="0.0" iyy="0.0" izz="0.0" ixy="0.0" ixz="0.0" iyz="0.0"/>
@@ -134,5 +134,5 @@
 			</visual>-->
 			<collision>
-				<origin xyz="0.0 0.0 0.0" rpy="0.0 0.0 0.0"/>
+				<origin xyz="0 0 0" rpy="0 0 0"/>
 				<geometry>
 					<sphere radius="0.02175"/>

File: hyq_description/urdfs/sensors/bumblebee.urdf.xacro (robot description, xacro)
@@ -2,4 +2,6 @@
 <robot xmlns:xacro="http://www.ros.org/wiki/xacro">
 	<xacro:include filename="$(find hyq_description)/urdfs/sensors/stereo_camera.gazebo.xacro"/>
+	<!-- ================================ Bumblebee ============================== -->
+	<!-- The xacro macro xacro:bumblebee contains: camera, mount and optical frame -->
 	<xacro:macro name="bumblebee" params="parent_link xyz rpy ns frame_prefix high_res hfov">
 		<joint name="bumblebee_mount_joint" type="fixed">
@@ -12,5 +14,5 @@
 			<child link="${frame_prefix}optical_frame"/>
 			<!--<origin xyz="0 0 0" rpy="0 0 0"/>-->
-			<origin xyz="0 -0.06 0.00" rpy="-${PI/2} 0 -${PI/2}"/>
+			<origin xyz="0 -0.06 0" rpy="-${PI/2} 0 -${PI/2}"/>
 		</joint>
 		<link name="${frame_prefix}mount_link">

File: hyq_description/urdfs/sensors/microstrain_3dmgx325_imu.urdf.xacro (robot description, xacro)
@@ -2,4 +2,6 @@
 <robot xmlns:xacro="http://ros.org/wiki/xacro">
 	<xacro:include filename="$(find hyq_description)/urdfs/sensors/microstrain_3dmgx325_imu.gazebo.xacro"/>
+	<!-- ============================ IMU microstrain ============================== -->
+	<!-- The xacro macro xacro:microstrain_3dmgx325_imu: imu frame -->
 	<xacro:macro name="microstrain_3dmgx325_imu" params="parent *origin imu_name imu_topic update_rate stdev">
 		<!-- Joint -->

File: hyq_description/urdfs/sensors/velodyne.urdf.xacro (robot description, xacro)
@@ -1,4 +1,4 @@
 <?xml version="1.0"?>
-<root xmlns:xacro="http://www.ros.org/wiki/xacro">
+<robot xmlns:xacro="http://www.ros.org/wiki/xacro">
 	<xacro:include filename="$(find hyq_description)/urdfs/sensors/velodyne.gazebo.xacro" />
 	<!-- ===================================== VELODYNE ==================================== -->
@@ -25,5 +25,5 @@
 			</inertial>
 			<visual>
-				<origin xyz="0.0 0.0 0.0" rpy="0.0 0.0 0.0"/>
+				<origin xyz="0 0 0" rpy="0 0 0"/>
 				<geometry>
 					<mesh filename="package://hyq_description/meshes/sensors/velodyne_hdl32e.dae" scale="1 1 1" />
@@ -34,5 +34,5 @@
 			</visual>
 			<collision>
-				<origin xyz="0.0 0.0 0.0" rpy="0.0 0.0 0.0"/>
+				<origin xyz="0 0 0" rpy="0 0 0"/>
 				<geometry>
 					<box size="0.1 0.18 0.1" />
@@ -44,5 +44,5 @@
 			<inertial>
 				<mass value="0.1"/>
-				<origin xyz="0.0 0.0 0.0" rpy="0.0 0.0 0.0"/>
+				<origin xyz="0 0 0" rpy="0 0 0"/>
 				<inertia ixx="0.01" ixy="0.0" ixz="0.0" iyy="0.01" iyz="0.0" izz="0.01"/>
 			</inertial>
@@ -51,3 +51,3 @@
 		<xacro:velodyne_sensor link_name="${name}_velodyne_optical_frame" frame_name="${name}_velodyne_frame" lidar_name="${name}_velodyne" />
 	</xacro:macro>
-</root>
+</robot>

File: hyq_description/urdfs/sensors/vicon.urdf.xacro (robot description, xacro)
@@ -1,17 +1,17 @@
 <?xml version="1.0"?>
-<root xmlns:xacro="http://www.ros.org/wiki/xacro">
+<robot xmlns:xacro="http://www.ros.org/wiki/xacro">
 	<!-- ======================================= VICON MARKER ====================================== -->
 	<!-- The xacro macro xacro:vicon_marker contains: vicon marker link -->
-	<xacro:macro name="vicon" params="parent *origin">
+	<xacro:macro name="vicon" params="child *origin">
 		<!-- Joints -->
-		<joint name="vicon_maker_joint" type="fixed">
+		<joint name="vicon_maker_joint" type="floating">
 			<insert_block name="origin"/>
-			<parent link="${parent}"/>
-			<child link="vicon_marker_link"/>
+			<parent link="vicon_marker_link"/>
+			<child link="${child}"/>
 		</joint>
 		<!-- Links -->
 		<link name="vicon_marker_link">
 			<inertial>
-				<mass value="0.1"/>
+				<mass value="0.001"/>
 				<origin xyz="0 0 0" rpy="0 0 0"/>
 				<inertia ixx="0.01" ixy="0.0" ixz="0.0" iyy="0.01" iyz="0.0" izz="0.01"/>
@@ -33,4 +33,4 @@
 			</collision>
 		</link>
-		</xacro:macro>
-</root>
+	</xacro:macro>
+</robot>

File: hyq_description/urdfs/trunk/trunk.urdf.xacro (robot description, xacro)
@@ -7,7 +7,6 @@
 	<xacro:macro name="hyq_trunk" params="name">
 		<!-- Floating-base Joint -->
-		<joint name="floating_base" type="fixed">
-			<origin xyz="0.0 0.0 0.0" rpy="0.0 0.0 0.0"/>
-			<!--<origin xyz="0.0 0.0 -0.49"  rpy="3.1416 0.0 0.0" />-->
+		<joint name="floating_base" type="floating">
+			<origin xyz="0 0 0" rpy="0 0 0"/>
 			<parent link="${name}_link"/>
 			<child link="trunk"/>
