Commit message: Fixed a problem in the definition of the collision of hip and upper leg links. Added a sphere model for modeling a contact.

File: hyq_description/urdfs/common_gazebo.xacro (robot description, xacro)
@@ -8,5 +8,5 @@
 	<property name="d_p1p2" value="0.35"/>
 	<!-- Initial joint positions -->
-	<property name="haa_pos0" value="-0.3"/>
+	<property name="haa_pos0" value="-0.1"/>
 	<property name="hfe_pos0" value="0.6"/>
 	<property name="kfe_pos0" value="-1.4"/>

File: hyq_description/urdfs/leg/leg.urdf.xacro (robot description, xacro)
@@ -75,5 +75,5 @@
 			</visual>
 			<collision>
-				<origin xyz="0.0 0.0 0.0" rpy="${(1+reflect_hip)*PI/2} ${-reflect_hip*PI/2} 0.0"/>
+				<origin xyz="0.0 0.0 0.0" rpy="${(1-reflect_hip)*PI/2} 0.0 0.0"/>
 				<geometry>
 					<mesh filename="package://hyq_description/meshes/leg/hip.dae" scale="1 1 1"/>
@@ -95,5 +95,5 @@
 			</visual>
 			<collision>
-				<origin xyz="0.0 0.0 0.0" rpy="${(1+reflect_front)*PI/2} 0.0 0.0"/>
+				<origin xyz="0.0 0.0 0.0" rpy="${(1-reflect_front)*PI/2} 0.0 0.0"/>
 				<geometry>
 					<mesh filename="package://hyq_description/meshes/leg/upper.dae" scale="1 1 1"/>
@@ -127,4 +127,16 @@
 				<inertia ixx="0.0" iyy="0.0" izz="0.0" ixy="0.0" ixz="0.0" iyz="0.0"/>
 			</inertial>
+			<!--<visual>
+				<origin xyz="0.0 0.0 0.0" rpy="0.0 0.0 0.0"/>
+				<geometry>
+					<sphere radius="0.021"/>
+				</geometry>
+			</visual>-->
+			<collision>
+				<origin xyz="0.0 0.0 0.0" rpy="0.0 0.0 0.0"/>
+				<geometry>
+					<sphere radius="0.021"/>
+				</geometry>
+			</collision>
 		</link>
 		<!-- Extensions -->

Commit message: Changed the pose0 position according with the go0 joint position of HyQ. Improved the definition of the collision of the foot. Changed the initial z position.

File: hyq_description/urdfs/common_gazebo.xacro (robot description, xacro)
@@ -5,10 +5,10 @@
 	<property name="d_lr" value="0.414"/>
 	<property name="d_fh" value="0.747"/>
-	<property name="d_tbb" value="0.082"/>
+	<property name="d_tbb" value="0.0825"/>
 	<property name="d_p1p2" value="0.35"/>
 	<!-- Initial joint positions -->
-	<property name="haa_pos0" value="-0.1"/>
-	<property name="hfe_pos0" value="0.6"/>
-	<property name="kfe_pos0" value="-1.4"/>
+	<property name="haa_pos0" value="-0.2"/>
+	<property name="hfe_pos0" value="0.75"/>
+	<property name="kfe_pos0" value="-1.5"/>
 	<!-- Inertial values -->
 	<!-- Trunk with hydraulic system -->

File: hyq_description/urdfs/leg/leg.urdf.xacro (robot description, xacro)
@@ -48,5 +48,5 @@
 		</joint>
 		<joint name="${name}_foot_joint" type="fixed">
-			<origin xyz="0.35 0.0 0.0" rpy="0.0 0.0 0.0"/>
+			<origin xyz="0.34 0.0 0.0" rpy="0.0 0.0 0.0"/>
 			<parent link="${name}_lower_leg"/>
 			<child  link="${name}_foot"/>
@@ -136,5 +136,5 @@
 				<origin xyz="0.0 0.0 0.0" rpy="0.0 0.0 0.0"/>
 				<geometry>
-					<sphere radius="0.021"/>
+					<sphere radius="0.02175"/>
 				</geometry>
 			</collision>
