Commit message: Added a shift in the sensor reference system of Asus in order to get good result. Now, I don't know what is happening!

File: hyq_description/urdfs/common.xacro (robot description, xacro)
@@ -52,8 +52,8 @@
 	<property name="joint_effort" value="30" />
 	<!-- Asus Xtion Camera Location (Nominally 0) -->
-	<property name="asus_xtion_x" value="0.009"/>
-	<property name="asus_xtion_depth_y" value="0.049"/>
-	<property name="asus_xtion_rgb_y" value="0.022"/>
-	<property name="asus_xtion_z" value="0.035"/>
+	<property name="asus_xtion_x" value="0.0"/>
+	<property name="asus_xtion_depth_y" value="0.069"/>
+	<property name="asus_xtion_rgb_y" value="0.042"/>
+	<property name="asus_xtion_z" value="0.03"/>
 	<property name="asus_xtion_roll" value="${-PI/2}"/>
 	<property name="asus_xtion_pitch" value="0.0"/>

File: hyq_description/urdfs/leg/leg.urdf.xacro (robot description, xacro)
@@ -58,5 +58,5 @@
 				<origin xyz="0.0 0.0 0.0"/>
 				<mass value="0.01"/>
-				<inertia ixx="0.0" iyy="0.0" izz="0.0" ixy="0.0" ixz="0.0" iyz="0.0"/>
+				<inertia ixx="0.01" iyy="0.01" izz="0.01" ixy="0.0" ixz="0.0" iyz="0.0"/>
 			</inertial>
 		</link>

File: hyq_description/urdfs/sensors/asus_xtion.urdf.xacro (robot description, xacro)
@@ -51,10 +51,10 @@
 				</material>
 			</visual>
-	<collision>
-		<origin xyz="0.0 0.0 ${asus_xtion_z}" rpy="0 0 0" />
-		<geometry>
-			<box size="0.05 .18 0.035" />
-		</geometry>
-	</collision>
+			<collision>
+				<origin xyz="0.0 0.0 ${asus_xtion_z}" rpy="0 0 0" />
+				<geometry>
+					<box size="0.05 .18 0.035" />
+				</geometry>
+			</collision>
 		</link>
 		<!-- ir sensor link -->

Commit message: No comments

File: hyq_description/urdfs/common.xacro (robot description, xacro)
@@ -52,7 +52,7 @@
 	<property name="joint_effort" value="30" />
 	<!-- Asus Xtion Camera Location (Nominally 0) -->
-	<property name="asus_xtion_x" value="0.015"/>
+	<property name="asus_xtion_x" value="0.0"/>
 	<property name="asus_xtion_depth_y" value="0.069"/>
-	<property name="asus_xtion_rgb_y" value="0.042"/>
+	<property name="asus_xtion_rgb_y" value="0.049"/>
 	<property name="asus_xtion_z" value="0.03"/>
 	<property name="asus_xtion_roll" value="${-PI/2}"/>

File: hyq_description/urdfs/sensors/asus_xtion.urdf.xacro (robot description, xacro)
@@ -43,5 +43,5 @@
 			</inertial>
 			<visual>
-				<origin xyz="0.0 0.0 0.0" rpy="0.0 0.0 0.0"/>
+				<origin xyz="-0.015 0.0 0.0" rpy="0.0 0.0 0.0"/>
 				<geometry>
 					<mesh filename="package://hyq_description/meshes/sensors/asus_xtion.dae" scale="1 1 1" />
