Commit message: fixed pan axis

File: hyq_description/urdfs/sensors/ptu_d46.urdf.xacro (robot description, xacro)
@@ -52,39 +52,4 @@
 	</xacro:macro>
 	<xacro:macro name="ptu_d46" params="name parent *origin">
-		<joint name="${name}_joint" type="fixed">
-			<insert_block name="origin"/>
-			<parent link="${parent}"/>
-			<child link="${name}_base_link"/>
-		</joint>
-		<!-- There's an offset between the origin of the pan joint and the origin of
-        	 the overall device, which is between the mounting screws on its base. -->
-		<joint name="${name}_base" type="fixed">
-			<origin xyz="0 -0.011 0.022" rpy="0 0 0"/>
-			<parent link="${name}_base_link"/>
-			<child link="${name}_pan_link"/>
-		</joint>
-		<!-- The pan joint -->
-		<joint name="${name}_pan_joint" type="revolute">
-			<origin xyz="0 0 0.066" rpy="-${PI/2} 0 0"/>
-			<parent link="${name}_pan_link"/>
-			<!--<parent link="${name}_base_link"/>-->
-			<child link="${name}_tilt_link"/>
-			<axis xyz="0 1 0" rpy="0 0 0"/>
-			<limit lower="${-pan_range}" upper="${pan_range}" effort="${joint_effort}" velocity="${pan_velocity}"/>
-		</joint>
-		<!-- The tilt joint -->
-		<joint name="${name}_tilt_joint" type="revolute">
-			<origin xyz="0 0 0" rpy="-${PI/2} 0 0"/>
-			<parent link="${name}_tilt_link"/>
-			<child link="${name}_tilted_link"/>
-			<axis xyz="0 1 0"/>
-			<limit lower="${-tilt_down_range}" upper="${tilt_up_range}" effort="${joint_effort}" velocity="${tilt_velocity}"/>
-		</joint>
-		<!-- Fixed joint to provide a convenient attachment point for accessories. -->
-		<joint name="${name}_mount_joint" type="fixed">
-			<origin xyz="0 0 -0.03912" rpy="${PI} 0 0"/>
-			<parent link="${name}_tilted_link"/>
-			<child link="${name}_mount_link"/>
-		</joint>
 		<d46_stepper_module ptu_name="${name}" joint_name="pan" />
 		<d46_stepper_module ptu_name="${name}" joint_name="tilt" />
@@ -110,4 +75,39 @@
 			</inertial>
 		</link>
+		<joint name="${name}_joint" type="fixed">
+			<insert_block name="origin"/>
+			<parent link="${parent}"/>
+			<child link="${name}_base_link"/>
+		</joint>
+		<!-- There's an offset between the origin of the pan joint and the origin of
+        	 the overall device, which is between the mounting screws on its base. -->
+		<joint name="${name}_base" type="fixed">
+			<origin xyz="0 -0.011 0.022" rpy="0 0 0"/>
+			<parent link="${name}_base_link"/>
+			<child link="${name}_pan_link"/>
+		</joint>
+		<!-- The pan joint -->
+		<joint name="${name}_pan" type="revolute">
+			<origin xyz="0 0 0.066" rpy="-${PI/2} 0 0"/>
+			<parent link="${name}_pan_link"/>
+			<!--<parent link="${name}_base_link"/>-->
+			<child link="${name}_tilt_link"/>
+			<axis xyz="0 -1 0" rpy="0 0 0"/>
+			<limit lower="${-pan_range}" upper="${pan_range}" effort="${joint_effort}" velocity="${pan_velocity}"/>
+		</joint>
+		<!-- The tilt joint -->
+		<joint name="${name}_tilt" type="revolute">
+			<parent link="${name}_tilt_link"/>
+			<origin xyz="0 0 0" rpy="-${PI/2} 0 0"/>
+			<child link="${name}_tilted_link"/>
+			<axis xyz="0 1 0"/>
+			<limit lower="${-tilt_down_range}" upper="${tilt_up_range}" effort="${joint_effort}" velocity="${tilt_velocity}"/>
+		</joint>
+		<!-- Fixed joint to provide a convenient attachment point for accessories. -->
+		<joint name="${name}_mount" type="fixed">
+			<origin xyz="0 0 -0.03912" rpy="${PI} 0 0"/>
+			<parent link="${name}_tilted_link"/>
+			<child link="${name}_mount_link"/>
+		</joint>
 		<!-- Extensions -->
 		<xacro:ptu_transmission name="${name}"/>

Commit message: Improved the color of the meshes. Cleaned unuseful things in the trunk urdf file

File: hyq_description/urdfs/sensors/ptu_d46.urdf.xacro (robot description, xacro)
@@ -12,5 +12,5 @@
 			<visual>
 				<material name="ptu_body_color">
-					<color rgba="0.3 0.3 0.3 1.0"/>
+					<color rgba="0.28 0.28 0.28 1"/>
 				</material>
 				<geometry>
@@ -50,4 +50,7 @@
 			</collision>
 		</link>
+		<gazebo reference="${ptu_name}_${joint_name}_link">
+			<material>Gazebo/Grey</material>
+		</gazebo>
 	</xacro:macro>
 	<xacro:macro name="ptu_d46" params="name parent *origin">

File: hyq_description/urdfs/trunk/trunk.urdf.xacro (robot description, xacro)
@@ -20,7 +20,4 @@
 					<cylinder length="0.01" radius="0.01"/>
 				</geometry>
-				<material name="blue">
-					<color rgba="0 0 .8 1"/>
-				</material>
 			</visual>
 		</link>
@@ -42,7 +39,4 @@
 					<mesh filename="package://hyq_description/meshes/trunk/trunk_frame.dae" scale="1 1 1"/>
 				</geometry>
-				<material name="white">
-					<color rgba="1 1 1 1"/>
-				</material>
 			</visual>
 		</link>
