Commit message: Added an offset in the cad file of Asus Xtion for improving the visualization with scanning motion

File: hyq_description/urdfs/sensors/asus_xtion.urdf.xacro (robot description, xacro)
@@ -43,5 +43,5 @@
 			</inertial>
 			<visual>
-				<origin xyz="0.0 0.0 0.0" rpy="0.0 0.0 0.0"/>
+				<origin xyz="-0.01 0.0 0.0" rpy="0.0 0.0 0.0"/>
 				<geometry>
 					<mesh filename="package://hyq_description/meshes/sensors/asus_xtion.dae" scale="1 1 1" />
