Commit message: Added the hardwareInterface tag that is required for Indigo version.

File: hyq_description/urdfs/leg/leg.transmission.xacro (robot description, xacro)
@@ -5,5 +5,7 @@
 		<transmission name="${name}_haa_trans">
 			<type>transmission_interface/SimpleTransmission</type>
-			<joint name="${name}_haa_joint"/>
+			<joint name="${name}_haa_joint">
+				<hardwareInterface>EffortJointInterface</hardwareInterface>
+			</joint>
 			<actuator name="${name}_haa_motor">
 				<hardwareInterface>EffortJointInterface</hardwareInterface>
@@ -14,5 +16,7 @@
 		<transmission name="${name}_hfe_upper_trans">
 			<type>transmission_interface/SimpleTransmission</type>
-			<joint name="${name}_hfe_joint"/>
+			<joint name="${name}_hfe_joint">
+				<hardwareInterface>EffortJointInterface</hardwareInterface>
+			</joint>
 			<actuator name="${name}_hfe_motor">
 				<hardwareInterface>EffortJointInterface</hardwareInterface>
@@ -23,5 +27,7 @@
 		<transmission name="${name}_kfe_trans">
 			<type>transmission_interface/SimpleTransmission</type>
-			<joint name="${name}_kfe_joint"/>
+			<joint name="${name}_kfe_joint">
+				<hardwareInterface>EffortJointInterface</hardwareInterface>
+			</joint>
 			<actuator name="${name}_kfe_motor">
 				<hardwareInterface>EffortJointInterface</hardwareInterface>

File: hyq_description/urdfs/sensors/ptu_d46.transmission.xacro (robot description, xacro)
@@ -5,5 +5,7 @@
 		<transmission name="${name}_pan_trans">
 			<type>transmission_interface/SimpleTransmission</type>
-			<joint name="${name}_pan"/>
+			<joint name="${name}_pan">
+				<hardwareInterface>EffortJointInterface</hardwareInterface>
+			</joint>
 			<actuator name="${name}_pan_motor">
 				<hardwareInterface>EffortJointInterface</hardwareInterface>
@@ -14,5 +16,7 @@
 		<transmission name="${name}_tilt_trans">
 			<type>transmission_interface/SimpleTransmission</type>
-			<joint name="${name}_tilt"/>
+			<joint name="${name}_tilt">
+				<hardwareInterface>EffortJointInterface</hardwareInterface>
+			</joint>
 			<actuator name="${name}_tilt_motor">
 				<hardwareInterface>EffortJointInterface</hardwareInterface>
