Commit message: Removed the old convex hulls from the model

File: hyq_description/urdfs/leg/leg.urdf.xacro (robot description, xacro)
@@ -74,7 +74,7 @@
 			</visual>
 			<collision>
-				<origin xyz="0.0 0.0 0.0" rpy="${(1+reflect_hip)*PI/2} ${-reflect_hip*PI/2} 0.0"/>
+				<origin xyz="0.0 0.0 0.0" rpy="${(1-reflect_hip)*PI/2} 0.0 0.0"/>
 				<geometry>
-					<mesh filename="package://hyq_description/meshes/leg/hip_convex.dae" scale="0.001 0.001 0.001"/>
+					<mesh filename="package://hyq_description/meshes/leg/hip.dae" scale="1 1 1"/>
 				</geometry>
 			</collision>
@@ -95,7 +95,7 @@
 			</visual>
 			<collision>
-				<origin xyz="0.0 0.0 0.0" rpy="${(1+reflect_front)*PI/2} 0.0 0.0"/>
+				<origin xyz="0.0 0.0 0.0" rpy="${(1-reflect_front)*PI/2} 0.0 0.0"/>
 				<geometry>
-					<mesh filename="package://hyq_description/meshes/leg/upper_convex.dae" scale="0.001 0.001 0.001"/>
+					<mesh filename="package://hyq_description/meshes/leg/upper.dae" scale="1 1 1"/>
 				</geometry>
 			</collision>
@@ -116,5 +116,5 @@
 			<collision>
 				<geometry>
-					<mesh filename="package://hyq_description/meshes/leg/lower_convex.dae" scale="0.001 0.001 0.001"/>
+					<mesh filename="package://hyq_description/meshes/leg/lower.dae" scale="1 1 1"/>
 				</geometry>
 			</collision>

Commit message: Changed the orientation of the foot reference frame according to the group standard.

File: hyq_description/urdfs/leg/leg.urdf.xacro (robot description, xacro)
@@ -48,5 +48,5 @@
 		</joint>
 		<joint name="${name}_foot_joint" type="fixed">
-			<origin xyz="0.34 0.0 0.0" rpy="0.0 0.0 0.0"/>
+			<origin xyz="0.34 0.0 0.0" rpy="${PI/2} 0.0 ${-PI/2}"/>
 			<parent link="${name}_lower_leg"/>
 			<child  link="${name}_foot"/>

Commit message: now the foot frame is following the convention: x front, y left, z up when the leg is straight

File: hyq_description/urdfs/leg/leg.urdf.xacro (robot description, xacro)
@@ -48,5 +48,5 @@
 		</joint>
 		<joint name="${name}_foot_joint" type="fixed">
-			<origin xyz="0.35 0.0 0.0" rpy="0.0 0.0 0.0"/>
+			<origin xyz="0.35 0.0 0.0" rpy="${PI/2} 0.0 ${-PI/2}"/>
 			<parent link="${name}_lower_leg"/>
 			<child  link="${name}_foot"/>

Commit message: Added the real limitations of the joints

File: hyq_description/urdfs/leg/leg.urdf.xacro (robot description, xacro)
@@ -21,5 +21,5 @@
 			<!--<parent link="${parent}"/>-->
 			<child  link="${name}_hip_assembly"/>
-			<limit effort="200.0" velocity="1000.0" lower="${-PI/2-haa_pos0}" upper="${PI/6-haa_pos0}"/>
+			<limit effort="150.0" velocity="12.0" lower="${-PI/2-haa_pos0}" upper="${PI/6-haa_pos0}"/>
 			<axis xyz="0 0 1"/>
 			<dynamics damping="0.1" friction="0" />
@@ -31,5 +31,5 @@
 			<parent link="${name}_hip_assembly"/>
 			<child  link="${name}_upper_leg"/>
-			<limit effort="200.0" velocity="1.0" lower="${-(1+reflect_front)*5*PI/36-(1-reflect_front)*7*PI/36-reflect_front*hfe_pos0}" upper="${(1-reflect_front)*5*PI/36+(1+reflect_front)*7*PI/36-reflect_front*hfe_pos0}"/>
+			<limit effort="150.0" velocity="12.0" lower="${-(1+reflect_front)*5*PI/36-(1-reflect_front)*7*PI/36-reflect_front*hfe_pos0}" upper="${(1-reflect_front)*5*PI/36+(1+reflect_front)*7*PI/36-reflect_front*hfe_pos0}"/>
 			<axis xyz="0 0 1"/>
 			<dynamics damping="0.1" friction="0" />
@@ -41,5 +41,5 @@
 			<parent link="${name}_upper_leg"/>
 			<child  link="${name}_lower_leg"/>
-			<limit effort="200.0" velocity="1.0" lower="${-(1+reflect_front)*7*PI/18+(1-reflect_front)*PI/18-reflect_front*kfe_pos0}" upper="${(1-reflect_front)*7*PI/18-(1+reflect_front)*PI/18-reflect_front*kfe_pos0}"/>
+			<limit effort="150.0" velocity="12.0" lower="${-(1+reflect_front)*7*PI/18+(1-reflect_front)*PI/18-reflect_front*kfe_pos0}" upper="${(1-reflect_front)*7*PI/18-(1+reflect_front)*PI/18-reflect_front*kfe_pos0}"/>
 			<axis xyz="0 0 1"/>
 			<dynamics damping="0.1" friction="0" />
