Commit message: Removed the old trunk files and changed to the new one that contains the protection frames

File: hyq_description/urdfs/trunk/trunk.urdf.xacro (robot description, xacro)
@@ -12,16 +12,4 @@
 			<parent link="${name}_link"/>
 			<child link="trunk"/>
-		</joint>
-		<!-- Front Frame Joint -->
-		<joint name="front_frame" type="fixed">
-			<origin xyz="0.5 0.0 0.085" rpy="0.0 0.0 0.0"/>
-			<parent link="trunk"/>
-			<child link="front_frame"/>
-		</joint>
-		<!-- Hip Frame Joint -->
-		<joint name="hip_frame" type="fixed">
-			<origin xyz="-0.5 0.0 0.085" rpy="0.0 0.0 0.0"/>
-			<parent link="trunk"/>
-			<child link="hip_frame"/>
 		</joint>
 		<!-- Links -->
@@ -46,5 +34,5 @@
 			<collision>
 				<geometry>
-					<mesh filename="package://hyq_description/meshes/trunk/trunk.dae" scale="1 1 1"/>
+					<mesh filename="package://hyq_description/meshes/trunk/trunk_frame.dae" scale="1 1 1"/>
 				</geometry>
 			</collision>
@@ -52,51 +40,5 @@
 				<origin xyz="0 0 0" rpy="0 0 0" />
 				<geometry>
-					<mesh filename="package://hyq_description/meshes/trunk/trunk.dae" scale="1 1 1"/>
-				</geometry>
-					<material name="white">
-				<color rgba="1 1 1 1"/>
-				</material>
-			</visual>
-		</link>
-		<!-- Front Frame link -->
-		<link name="front_frame">
-			<inertial>
-				<origin xyz="0 0 0"/>
-				<mass value="0.01"/>
-				<inertia ixx="0.01" iyy="0.01" izz="0.01" ixy="0.0" ixz="0.0" iyz="0.0"/>
-			</inertial>
-			<collision>
-				<origin xyz="0 0 0" rpy="0 0 3.1416" />
-				<geometry>
-					<mesh filename="package://hyq_description/meshes/trunk/frame.dae" scale="1 1 1"/>
-				</geometry>
-			</collision>
-			<visual>
-				<origin xyz="0 0 0" rpy="0 0 ${PI}" />
-				<geometry>
-					<mesh filename="package://hyq_description/meshes/trunk/frame.dae" scale="1 1 1"/>
-				</geometry>
-					<material name="white">
-				<color rgba="1 1 1 1"/>
-				</material>
-			</visual>
-		</link>
-		<!-- Hip Frame link -->
-		<link name="hip_frame">
-			<inertial>
-				<origin xyz="0 0 0"/>
-				<mass value="0.01"/>
-				<inertia ixx="0.01" iyy="0.01" izz="0.01" ixy="0.0" ixz="0.0" iyz="0.0"/>
-			</inertial>
-			<collision>
-				<origin xyz="0 0 0" rpy="0 0 0" />
-				<geometry>
-					<mesh filename="package://hyq_description/meshes/trunk/frame.dae" scale="1 1 1"/>
-				</geometry>
-			</collision>
-			<visual>
-				<origin xyz="0 0 0" rpy="0 0 0" />
-				<geometry>
-					<mesh filename="package://hyq_description/meshes/trunk/frame.dae" scale="1 1 1"/>
+					<mesh filename="package://hyq_description/meshes/trunk/trunk_frame.dae" scale="1 1 1"/>
 				</geometry>
 					<material name="white">

Commit message: No comments

File: hyq_description/urdfs/trunk/trunk.urdf.xacro (robot description, xacro)
@@ -42,6 +42,6 @@
 					<mesh filename="package://hyq_description/meshes/trunk/trunk_frame.dae" scale="1 1 1"/>
 				</geometry>
-					<material name="white">
-				<color rgba="1 1 1 1"/>
+				<material name="white">
+					<color rgba="1 1 1 1"/>
 				</material>
 			</visual>

Commit message: Changed the floating joint to fixed one; this is necessary for Gazebo

File: hyq_description/urdfs/trunk/trunk.urdf.xacro (robot description, xacro)
@@ -7,5 +7,5 @@
 	<xacro:macro name="hyq_trunk" params="name">
 		<!-- Floating-base Joint -->
-		<joint name="floating_base" type="floating">
+		<joint name="floating_base" type="fixed">
 			<origin xyz="0 0 0" rpy="0 0 0"/>
 			<parent link="${name}_link"/>
