Commit message: Added the hyq_environments and hyq_gazebo packages. Modified the files in order to make simulations in Gazebo. Improved the launch files for making simulations or real experiments in HyQ.

File: hyq_description/gazebo/gazebo.urdf.xacro (robot description, xacro)
@@ -6,10 +6,10 @@
 			<controlPeriod>0.001</controlPeriod>
 		</plugin>
-    <plugin filename="libgazebo_ros_p3d.so" name="gazebo_ros_p3d">
-      <bodyName>base_link</bodyName>
-      <topicName>ground_truth_odom</topicName>
-      <alwaysOn>true</alwaysOn>
-      <updateRate>200.0</updateRate>
-    </plugin>
+		<plugin filename="libgazebo_ros_p3d.so" name="gazebo_ros_p3d">
+		 	<bodyName>base_link</bodyName>
+			<topicName>ground_truth_odom</topicName>
+			<alwaysOn>true</alwaysOn>
+			<updateRate>200.0</updateRate>
+		</plugin>
 	</gazebo>
 </robot>

File: hyq_description/robots/hyq.urdf.xacro (robot description, xacro)
@@ -74,12 +74,18 @@
 		<origin xyz="0.3 0 0.095" rpy="0 ${-PI} 0"/>
 	</xacro:microstrain_3dmgx325_imu>
+	<!-- PTU unit -->
+	<xacro:ptu_d46
+		name="ptu"
+		parent="trunk">
+		<origin xyz="0.693327 -0.015447 0.119533" rpy="-0.013127 0.574478 -0.007748"/>
+	</xacro:ptu_d46>
 	<!-- Asus Xtion Pro -->
+	<!-- The vertical offset between the middle of xtion and the middle of bumblebee is 5 cm-->
+	<!-- but since bumblebee_mount_link is computed in the middle of the camera and the xtion on its base instead -->
+	<!-- we have 5 cm - 3.5 cm (vertical distance between xtion optical frame and base) = 1.5 cm -->
 	<xacro:asus_xtion_camera
 		name="head_mount"
 		parent="ptu_mount_link">
 		<origin xyz="0.0 0 0.015" rpy="0 0 0"/>
-<!-- The vertical offset between the middle of xtion and the middle of bumblebee is 5 cm-->
-<!-- but since bumblebee_mount_link is computed in the middle of the camera and the xtion on its base instead -->
-<!-- we have 5 cm - 3.5 cm (vertical distance between xtion optical frame and base) = 1.5 cm -->
 	</xacro:asus_xtion_camera>
 	<!-- Velodyne -->
@@ -95,10 +101,4 @@
 		<origin xyz="0.63 0 0.095" rpy="0 0 0"/>
 	</xacro:kinect_camera-->
-	<!-- PTU unit -->
-	<xacro:ptu_d46
-		name="ptu"
-		parent="trunk">
-		<origin xyz="0.693327 -0.015447 0.119533" rpy="-0.013127 0.574478 -0.007748"/>
-	</xacro:ptu_d46>
 	<!-- Bumblebee -->
 	<xacro:bumblebee_97

File: hyq_description/robots/hyq_gazebo.urdf.xacro (robot description, xacro)
@@ -65,5 +65,5 @@
 		<origin xyz="${-d_fh/2} ${-d_lr/2} 0" rpy="0 ${PI/2} 0"/>
 	</xacro:hyq_leg>
-	<!-- IMU runk -->
+	<!-- IMU trunk -->
 	<xacro:microstrain_3dmgx325_imu
 		parent="trunk"
@@ -75,34 +75,37 @@
 	</xacro:microstrain_3dmgx325_imu>
 	<!-- PTU unit -->
-<!--	<xacro:ptu_d46
+	<xacro:ptu_d46
 		name="ptu"
 		parent="trunk">
-		<origin xyz="0.63 0 0.095" rpy="0 0 0"/>
-	</xacro:ptu_d46>-->
+		<origin xyz="0.693327 -0.015447 0.119533" rpy="-0.013127 0.574478 -0.007748"/>
+	</xacro:ptu_d46>
 	<!-- Asus Xtion Pro -->
+	<!-- The vertical offset between the middle of xtion and the middle of bumblebee is 5 cm-->
+	<!-- but since bumblebee_mount_link is computed in the middle of the camera and the xtion on its base instead -->
+	<!-- we have 5 cm - 3.5 cm (vertical distance between xtion optical frame and base) = 1.5 cm -->
 	<xacro:asus_xtion_camera
-		name="head_mount"
-		parent="trunk">
-		<origin xyz="0.63 0 0.095" rpy="0 ${PI/6} 0"/>
-	</xacro:asus_xtion_camera> <!-- <origin xyz="0.63 0 0.095" rpy="0 ${PI/6} 0"/> --> <!-- ptu_mount_link -->
+		name="head_mount_asus_xtion"
+		parent="ptu_mount_link">
+		<origin xyz="0.0 0 0.015" rpy="0 0 0"/>
+	</xacro:asus_xtion_camera>
 	<!-- Velodyne -->
-<!--	<xacro:velodyne
+	<!--<xacro:velodyne
 		name="trunk_mount"
 		parent="trunk">
 		<origin xyz="0.39 0 0.269" rpy="0 0 0"/>
-	</xacro:velodyne>-->
-	<!-- Kinect mount -->
-<!--	<xacro:kinect_camera
+	</xacro:velodyne-->
+	<!-- Kinect --> <!-- is no more used, but we keep it for compatibilty -->
+	<!--<xacro:kinect_camera
 		name="head_mount"
 		parent="trunk">
 		<origin xyz="0.63 0 0.095" rpy="0 0 0"/>
-	</xacro:kinect_camera>-->
+	</xacro:kinect_camera-->
 	<!-- Bumblebee -->
-<!--	<xacro:bumblebee_66
+	<!--<xacro:bumblebee_97
 		parent_link="ptu_mount_link"
 		xyz="0 0 0"
-		rpy="${PI/2} 0 ${PI/2}"
+		rpy="0 0 0"
 		ns="bumblebee"
 		frame_prefix="bumblebee_"
-		high_res="false"/>--> <!-- xyz="0.63 0 0.095" rpy="0 0 0" -->
+		high_res="false"/>-->
 </robot>

File: hyq_description/urdfs/common_gazebo.xacro (robot description, xacro)
@@ -8,5 +8,5 @@
 	<property name="d_p1p2" value="0.35"/>
 	<!-- Initial joint positions -->
-	<property name="haa_pos0" value="-0.8"/>
+	<property name="haa_pos0" value="-0.3"/>
 	<property name="hfe_pos0" value="0.6"/>
 	<property name="kfe_pos0" value="-1.4"/>

File: hyq_description/urdfs/leg/leg.urdf.xacro (robot description, xacro)
@@ -8,21 +8,21 @@
 	<xacro:macro name="hyq_leg" params="name parent *origin reflect_hip reflect_upper reflect_front">
 		<!-- Joints -->
-		<!-- Fake joint
-		<joint name="${name}_haa_fake_joint" type="fixed">
+		<!-- Hip assembly joint -->
+		<joint name="${name}_haa_assembly_joint" type="fixed">
 			<insert_block name="origin"/>
 			<parent link="${parent}"/>
-			<child  link="${name}_haa_fake"/>
-		</joint>-->
+			<child  link="${name}_assembly"/>
+		</joint>
 		<!-- Hip joint assembly -->
 		<joint name="${name}_haa_joint" type="revolute">
-			<!--<origin xyz="0.0 0.0 0.0" rpy="0.0 0.0 ${haa_pos0}"/>
-			<parent link="${name}_haa_fake"/>-->
-			<insert_block name="origin"/>
-			<parent link="${parent}"/>
+			<origin xyz="0.0 0.0 0.0" rpy="0.0 0.0 ${haa_pos0}"/>
+			<parent link="${name}_assembly"/>
+			<!--<insert_block name="origin"/>-->
+			<!--<parent link="${parent}"/>-->
 			<child  link="${name}_hip_assembly"/>
 			<limit effort="200.0" velocity="1000.0" lower="${-PI/2-haa_pos0}" upper="${PI/6-haa_pos0}"/>
 			<axis xyz="0 0 1"/>
-     <dynamics damping="0.1" friction="0" />
-     <safety_controller k_position="100" k_velocity="100" soft_lower_limit="-10" soft_upper_limit="12.45" />
+			<dynamics damping="0.1" friction="0" />
+			<safety_controller k_position="100" k_velocity="100" soft_lower_limit="-10" soft_upper_limit="12.45" />
 		</joint>
 		<!-- Upper leg joint -->
@@ -33,6 +33,6 @@
 			<limit effort="200.0" velocity="1.0" lower="${-(1+reflect_front)*5*PI/36-(1-reflect_front)*7*PI/36-reflect_front*hfe_pos0}" upper="${(1-reflect_front)*5*PI/36+(1+reflect_front)*7*PI/36-reflect_front*hfe_pos0}"/>
 			<axis xyz="0 0 1"/>
-     <dynamics damping="0.1" friction="0" />
-     <safety_controller k_position="100" k_velocity="100" soft_lower_limit="-10" soft_upper_limit="12.45" />
+			<dynamics damping="0.1" friction="0" />
+			<safety_controller k_position="100" k_velocity="100" soft_lower_limit="-10" soft_upper_limit="12.45" />
 		</joint>
 		<!-- Lower leg joint -->
@@ -43,6 +43,6 @@
 			<limit effort="200.0" velocity="1.0" lower="${-(1+reflect_front)*7*PI/18+(1-reflect_front)*PI/18-reflect_front*kfe_pos0}" upper="${(1-reflect_front)*7*PI/18-(1+reflect_front)*PI/18-reflect_front*kfe_pos0}"/>
 			<axis xyz="0 0 1"/>
-     <dynamics damping="0.1" friction="0" />
-     <safety_controller k_position="100" k_velocity="100" soft_lower_limit="-10" soft_upper_limit="12.45" />
+			<dynamics damping="0.1" friction="0" />
+			<safety_controller k_position="100" k_velocity="100" soft_lower_limit="-10" soft_upper_limit="12.45" />
 		<!-- Foot joint -->
 		</joint>
@@ -53,6 +53,6 @@
 		</joint>
 		<!-- Links -->
-		<!-- Fake hip assembly link
-		<link name="${name}_haa_fake">
+		<!-- Hip assembly link -->
+		<link name="${name}_assembly">
 			<inertial>
 				<origin xyz="0.0 0.0 0.0"/>
@@ -61,5 +61,4 @@
 			</inertial>
 		</link>
-		-->
 		<!-- Hip assembly link -->
 		<link name="${name}_hip_assembly">
@@ -74,8 +73,7 @@
 					<mesh filename="package://hyq_description/meshes/leg/hip.dae" scale="1 1 1"/>
 				</geometry>
-				<material name="white"/>
 			</visual>
 			<collision>
-				<origin xyz="0.0 0.0 0.0" rpy="${(1-reflect_hip)*PI/2} 0.0 0.0"/>
+				<origin xyz="0.0 0.0 0.0" rpy="${(1+reflect_hip)*PI/2} ${-reflect_hip*PI/2} 0.0"/>
 				<geometry>
 					<mesh filename="package://hyq_description/meshes/leg/hip.dae" scale="1 1 1"/>
@@ -95,8 +93,7 @@
 					<mesh filename="package://hyq_description/meshes/leg/upper.dae" scale="1 1 1"/>
 				</geometry>
-				<material name="white"/>
 			</visual>
 			<collision>
-				<origin xyz="0.0 0.0 0.0" rpy="${(1-reflect_front)*PI/2} 0.0 0.0"/>
+				<origin xyz="0.0 0.0 0.0" rpy="${(1+reflect_front)*PI/2} 0.0 0.0"/>
 				<geometry>
 					<mesh filename="package://hyq_description/meshes/leg/upper.dae" scale="1 1 1"/>

File: hyq_description/urdfs/sensors/asus_xtion.urdf.xacro (robot description, xacro)
@@ -9,32 +9,32 @@
 			<insert_block name="origin"/>
 			<parent link="${parent}"/>
-			<child link="${name}_asus_xtion_link"/>
+			<child link="${name}_link"/>
 		</joint>
 		<!-- asus ir sensor physical attachment -->
-		<joint name="${name}_asus_xtion_depth_joint" type="fixed">
+		<joint name="${name}_depth_joint" type="fixed">
 			<origin xyz="${asus_xtion_x} ${asus_xtion_depth_y} ${asus_xtion_z}" rpy="0.0 0.0 0.0"/>
-			<parent link="${name}_asus_xtion_link"/>
-			<child link="${name}_asus_xtion_depth_frame"/>
+			<parent link="${name}_link"/>
+			<child link="${name}_depth_frame"/>
 		</joint>
 		<!-- asus xtion ir sensor frame -->
-		<joint name="${name}_asus_xtion_depth_optical_frame_joint" type="fixed">
+		<joint name="${name}_depth_optical_frame_joint" type="fixed">
 			<origin xyz="0 0 0"	rpy="${asus_xtion_roll} ${asus_xtion_pitch} ${asus_xtion_yaw}"/>
-			<parent link="${name}_asus_xtion_depth_frame"/>
-			<child link="${name}_asus_xtion_depth_optical_frame"/>
+			<parent link="${name}_depth_frame"/>
+			<child link="${name}_depth_optical_frame"/>
 		</joint>
 		<!-- asus_xtion rgb sensor physical attachment -->
-		<joint name="${name}_asus_xtion_rgb_joint" type="fixed">
+		<joint name="${name}_rgb_joint" type="fixed">
 			<origin xyz="${asus_xtion_x} ${asus_xtion_rgb_y} ${asus_xtion_z}" rpy="0.0 0.0 0.0"/>
-			<parent link="${name}_asus_xtion_link"/>
-			<child link="${name}_asus_xtion_rgb_frame"/>
+			<parent link="${name}_link"/>
+			<child link="${name}_rgb_frame"/>
 		</joint>
 		<!-- asus xtion rgb sensor frame -->
-		<joint name="${name}_asus_xtion_rgb_optical_frame_joint" type="fixed">
+		<joint name="${name}_rgb_optical_frame_joint" type="fixed">
 			<origin xyz="0 0 0"	rpy="${asus_xtion_roll} ${asus_xtion_pitch} ${asus_xtion_yaw}"/>
-			<parent link="${name}_asus_xtion_rgb_frame"/>
-			<child link="${name}_asus_xtion_rgb_optical_frame"/>
+			<parent link="${name}_rgb_frame"/>
+			<child link="${name}_rgb_optical_frame"/>
 		</joint>
 		<!-- Links -->
-		<link name="${name}_asus_xtion_link">
+		<link name="${name}_link">
 			<inertial>
 				<mass value="0.1"/>
@@ -59,5 +59,5 @@
 		</link>
 		<!-- ir sensor link -->
-		<link name="${name}_asus_xtion_depth_frame">
+		<link name="${name}_depth_frame">
 			<inertial>
 				<mass value="0.1" />
@@ -79,7 +79,7 @@
 		</link>
 		<!-- ir optical sensor link -->
-		<link name="${name}_asus_xtion_depth_optical_frame"/>
+		<link name="${name}_depth_optical_frame"/>
 		<!-- rgb sensor link -->
-		<link name="${name}_asus_xtion_rgb_frame" >
+		<link name="${name}_rgb_frame" >
 			<inertial>
 				<mass value="0.1" />
@@ -101,8 +101,8 @@
 		</link>
 		<!-- rgb optical sensor link -->
-		<link name="${name}_asus_xtion_rgb_optical_frame"/>
+		<link name="${name}_rgb_optical_frame"/>
 	<!-- gazebo extensions -->
-	<xacro:asus_xtion_depth_sensor link_name="${name}_asus_xtion_depth_frame" frame_name="${name}_asus_xtion_depth_optical_frame" camera_name="${name}_asus_xtion" />
-	<xacro:asus_xtion_rgb_sensor link_name="${name}_asus_xtion_rgb_frame" frame_name="${name}_asus_xtion_rgb_optical_frame" camera_name="${name}_asus_xtion" />
+	<xacro:asus_xtion_depth_sensor link_name="${name}_depth_frame" frame_name="${name}_depth_optical_frame" camera_name="${name}" />
+	<xacro:asus_xtion_rgb_sensor link_name="${name}_rgb_frame" frame_name="${name}_rgb_optical_frame" camera_name="${name}" />
 	</xacro:macro>
 </root>

File: hyq_description/urdfs/sensors/ptu_d46.urdf.xacro (robot description, xacro)
@@ -52,27 +52,5 @@
 	</xacro:macro>
 	<xacro:macro name="ptu_d46" params="name parent *origin">
-		<d46_stepper_module ptu_name="${name}" joint_name="pan" />
-		<d46_stepper_module ptu_name="${name}" joint_name="tilt" />
-		<link name="${name}_base_link">
-			<inertial>
-				<origin xyz="0.0 0.0 0.0"/>
-				<mass value="0.01"/>
-				<inertia ixx="0.0" iyy="0.0" izz="0.0" ixy="0.0" ixz="0.0" iyz="0.0"/>
-			</inertial>
-		</link>
-		<link name="${name}_tilted_link">
-			<inertial>
-				<origin xyz="0.0 0.0 0.0"/>
-				<mass value="0.01"/>
-				<inertia ixx="0.0" iyy="0.0" izz="0.0" ixy="0.0" ixz="0.0" iyz="0.0"/>
-			</inertial>
-		</link>
-		<link name="${name}_mount_link">
-			<inertial>
-				<origin xyz="0.0 0.0 0.0"/>
-				<mass value="0.01"/>
-				<inertia ixx="0.0" iyy="0.0" izz="0.0" ixy="0.0" ixz="0.0" iyz="0.0"/>
-			</inertial>
-		</link>
+		<!-- Joints -->
 		<joint name="${name}_joint" type="fixed">
 			<insert_block name="origin"/>
@@ -88,18 +66,17 @@
 		</joint>
 		<!-- The pan joint -->
-		<joint name="${name}_pan" type="revolute">
+		<joint name="${name}_pan" type="fixed">
 			<origin xyz="0 0 0.066" rpy="-${PI/2} 0 0"/>
 			<parent link="${name}_pan_link"/>
-			<!--<parent link="${name}_base_link"/>-->
 			<child link="${name}_tilt_link"/>
-			<axis xyz="0 -1 0" rpy="0 0 0"/>
+			<axis xyz="0 -1 0"/>
 			<limit lower="${-pan_range}" upper="${pan_range}" effort="${joint_effort}" velocity="${pan_velocity}"/>
 		</joint>
 		<!-- The tilt joint -->
-		<joint name="${name}_tilt" type="revolute">
+		<joint name="${name}_tilt" type="fixed">
+			<origin xyz="0 0 0" rpy="-${PI/2} 0 0"/>
 			<parent link="${name}_tilt_link"/>
-			<origin xyz="0 0 0" rpy="-${PI/2} 0 0"/>
 			<child link="${name}_tilted_link"/>
-			<axis xyz="0 1 0"/> <!-- 0 1 0-->
+			<axis xyz="0 1 0"/>
 			<limit lower="${-tilt_down_range}" upper="${tilt_up_range}" effort="${joint_effort}" velocity="${tilt_velocity}"/>
 		</joint>
@@ -110,6 +87,66 @@
 			<child link="${name}_mount_link"/>
 		</joint>
+		<!-- Links -->
+		<d46_stepper_module ptu_name="${name}" joint_name="pan" />
+		<d46_stepper_module ptu_name="${name}" joint_name="tilt" />
+		<link name="${name}_base_link">
+			<inertial>
+				<origin xyz="0.0 0.0 0.0"/>
+				<mass value="0.01"/>
+				<inertia ixx="0.0" iyy="0.0" izz="0.0" ixy="0.0" ixz="0.0" iyz="0.0"/>
+			</inertial>
+			<visual>
+				<geometry>
+					<box size="0.001 0.001 0.001"/>
+				</geometry>
+				<origin xyz="0 0 0"/>
+			</visual>
+			<collision>
+				<geometry>
+					<box size="0.001 0.001 0.001"/>
+				</geometry>
+				<origin xyz="0 0 0"/>
+			</collision>
+		</link>
+		<link name="${name}_tilted_link">
+			<inertial>
+				<origin xyz="0.0 0.0 0.0"/>
+				<mass value="0.01"/>
+				<inertia ixx="0.0" iyy="0.0" izz="0.0" ixy="0.0" ixz="0.0" iyz="0.0"/>
+			</inertial>
+			<visual>
+				<geometry>
+					<box size="0.001 0.001 0.001"/>
+				</geometry>
+				<origin xyz="0 0 0"/>
+			</visual>
+			<collision>
+				<geometry>
+					<box size="0.001 0.001 0.001"/>
+				</geometry>
+				<origin xyz="0 0 0"/>
+			</collision>
+		</link>
+		<link name="${name}_mount_link">
+			<inertial>
+				<origin xyz="0.0 0.0 0.0"/>
+				<mass value="0.01"/>
+				<inertia ixx="0.0" iyy="0.0" izz="0.0" ixy="0.0" ixz="0.0" iyz="0.0"/>
+			</inertial>
+			<visual>
+				<geometry>
+					<box size="0.001 0.001 0.001"/>
+				</geometry>
+				<origin xyz="0 0 0"/>
+			</visual>
+			<collision>
+				<geometry>
+					<box size="0.001 0.001 0.001"/>
+				</geometry>
+				<origin xyz="0 0 0"/>
+			</collision>
+		</link>
 		<!-- Extensions -->
-		<xacro:ptu_transmission name="${name}"/>
+		<!--<xacro:ptu_transmission name="${name}"/>-->
 	</xacro:macro>
 </robot>
