Commit message: Removed the Simulation tag for having one urdf file. Updated the inertia parameters with new model of HyQ-Sylver. Cleaned the repository.

File: hyq_description/gazebo/gazebo.urdf.xacro (robot description, xacro)
@@ -4,9 +4,14 @@
 		<plugin name="gazebo_ros_controller_manager" filename="libgazebo_ros_control.so">
 			<robotNamespace>/hyq</robotNamespace>
-			<controlPeriod>0.001</controlPeriod>
+			<controlPeriod>0.005</controlPeriod>
 		</plugin>
 		<plugin filename="libgazebo_ros_p3d.so" name="gazebo_ros_p3d">
+			<robotNamespace>/hyq</robotNamespace>
 		 	<bodyName>base_link</bodyName>
 			<topicName>ground_truth_odom</topicName>
+			<frameName>world</frameName>
+			<xyzOffsets>0 0 0</xyzOffsets>
+			<rpyOffsets>0 0 0</rpyOffsets>
+			<gaussianNoise>0</gaussianNoise>
 			<alwaysOn>true</alwaysOn>
 			<updateRate>200.0</updateRate>

File: hyq_description/urdfs/common.xacro (robot description, xacro)
@@ -7,41 +7,49 @@
 	<property name="d_tbb" value="0.082"/>
 	<property name="d_p1p2" value="0.35"/>
-	<!-- Initial joint positions -->
-	<property name="haa_pos0" value="0"/>
-	<property name="hfe_pos0" value="0"/>
-	<property name="kfe_pos0" value="0"/>
 	<!-- Inertial values -->
 	<!-- Trunk with hydraulic system -->
-	<property name="m_trunk" value="53.0"/>
-	<property name="ixx_trunk" value="1.26"/>
-	<property name="iyy_trunk" value="6.56"/>
-	<property name="izz_trunk" value="6.69"/>
-	<property name="ixy_trunk" value="0.03"/>
-	<property name="ixz_trunk" value="-0.06"/>
-	<property name="iyz_trunk" value="-0.03"/>
+	<property name="xcom_trunk" value="0.027222"/>
+	<property name="ycom_trunk" value="-0.0000235"/>
+	<property name="zcom_trunk" value="0.042224"/>
+	<property name="m_trunk" value="64.862"/>
+	<property name="ixx_trunk" value="1.688238"/>
+	<property name="iyy_trunk" value="8.665299"/>
+	<property name="izz_trunk" value="9.243560"/>
+	<property name="ixy_trunk" value="-0.028789"/>
+	<property name="ixz_trunk" value="0.277694"/>
+	<property name="iyz_trunk" value="0.003820"/>
 	<!-- Hip assembly -->
-	<property name="m_hip" value="2.482"/>
-	<property name="ixx_hip" value="0.0956126"/>
-	<property name="iyy_hip" value="0.1012626"/>
-	<property name="izz_hip" value="6.758E-4"/>
-	<property name="ixy_hip" value="0.0"/>
-	<property name="ixz_hip" value="0.011"/>
-	<property name="iyz_hip" value="0.0"/>
+	<property name="xcom_hipassembly" value="0.04263"/>
+	<property name="ycom_hipassembly" value="0.0"/>
+	<property name="zcom_hipassembly" value="0.16931"/>
+	<property name="m_hipassembly" value="2.93"/>
+	<property name="ixx_hipassembly" value="0.134705"/>
+	<property name="iyy_hipassembly" value="0.144171"/>
+	<property name="izz_hipassembly" value="0.011033"/>
+	<property name="ixy_hipassembly" value="0.000036"/>
+	<property name="ixz_hipassembly" value="0.022734"/>
+	<property name="iyz_hipassembly" value="0.000051"/>
 	<!-- Upper leg -->
-	<property name="m_upper" value="2.16"/>
-	<property name="ixx_upper" value="0.004785"/>
-	<property name="iyy_upper" value="0.076166"/>
-	<property name="izz_upper" value="0.078576"/>
-	<property name="ixy_upper" value="0.0071588"/>
-	<property name="ixz_upper" value="0.0"/>
-	<property name="iyz_upper" value="0.0"/>
+	<property name="xcom_upperleg" value="0.15074"/>
+	<property name="ycom_upperleg" value="0.02625"/>
+	<property name="zcom_upperleg" value="0.0"/>
+	<property name="m_upperleg" value="2.638"/>
+	<property name="ixx_upperleg" value="0.005495"/>
+	<property name="iyy_upperleg" value="0.087136"/>
+	<property name="izz_upperleg" value="0.089871"/>
+	<property name="ixy_upperleg" value="-0.007418"/>
+	<property name="ixz_upperleg" value="-0.000102"/>
+	<property name="iyz_upperleg" value="-0.000021"/>
 	<!-- Lower leg -->
-	<property name="m_lower" value="1.8717"/>
-	<property name="ixx_lower" value="9.0E-4"/>
-	<property name="iyy_lower" value="0.0777"/>
-	<property name="izz_lower" value="0.0775"/>
-	<property name="ixy_lower" value="-0.0"/>
-	<property name="ixz_lower" value="-0.0"/>
-	<property name="iyz_lower" value="0.0"/>
+	<property name="xcom_lowerleg" value="0.1254"/>
+	<property name="ycom_lowerleg" value="0.00005"/>
+	<property name="zcom_lowerleg" value="-0.0001"/>
+	<property name="m_lowerleg" value="0.881"/>
+	<property name="ixx_lowerleg" value="0.000468"/>
+	<property name="iyy_lowerleg" value="0.026409"/>
+	<property name="izz_lowerleg" value="0.026181"/>
+	<property name="ixy_lowerleg" value="0.0"/>
+	<property name="ixz_lowerleg" value="0.0"/>
+	<property name="iyz_lowerleg" value="0.0"/>
 	<!-- PTU unit -->
 	<property name="pan_velocity" value="1.0" />

File: hyq_description/urdfs/leg/leg.gazebo.xacro (robot description, xacro)
@@ -2,5 +2,5 @@
 <robot xmlns:xacro="http://www.ros.org/wiki/xacro">
 	<xacro:macro name="leg_gazebo" params="name">
-		<gazebo reference="${name}_lower_leg">
+		<gazebo reference="${name}_lowerleg">
 			<kp>1000000.0</kp>
 			<kd>100.0</kd>

File: hyq_description/urdfs/leg/leg.urdf.xacro (robot description, xacro)
@@ -9,67 +9,61 @@
 		<!-- Joints -->
 		<!-- Hip assembly joint -->
-		<joint name="${name}_haa_assembly_joint" type="fixed">
+		<joint name="${name}_haa_joint" type="revolute">
 			<insert_block name="origin"/>
 			<parent link="${parent}"/>
-			<child  link="${name}_assembly"/>
-		</joint>
-		<!-- Hip joint assembly -->
-		<joint name="${name}_haa_joint" type="revolute">
-			<origin xyz="0 0 0" rpy="0 0 ${haa_pos0}"/>
-			<parent link="${name}_assembly"/>
-			<!--<insert_block name="origin"/>-->
-			<!--<parent link="${parent}"/>-->
-			<child  link="${name}_hip_assembly"/>
-			<limit effort="150.0" velocity="12.0" lower="${-PI/2-haa_pos0}" upper="${PI/6-haa_pos0}"/>
+			<child  link="${name}_hipassembly"/>
 			<axis xyz="0 0 1"/>
+			<limit effort="150.0" velocity="12.0" lower="${-7*PI/18}" upper="${PI/6}"/>
 			<dynamics damping="0.1" friction="0" />
-			<safety_controller k_position="100" k_velocity="100" soft_lower_limit="-10" soft_upper_limit="12.45" />
+			<safety_controller k_position="100" k_velocity="100"
+							   soft_lower_limit="-10" soft_upper_limit="12.45" />
 		</joint>
 		<!-- Upper leg joint -->
 		<joint name="${name}_hfe_joint" type="revolute">
-			<origin xyz="${d_tbb} 0.0 0.0" rpy="${reflect_upper*PI/2} ${-reflect_hip*hfe_pos0} 0.0"/>
-			<parent link="${name}_hip_assembly"/>
-			<child  link="${name}_upper_leg"/>
-			<limit effort="150.0" velocity="12.0" lower="${-(1+reflect_front)*5*PI/36-(1-reflect_front)*7*PI/36-reflect_front*hfe_pos0}" upper="${(1-reflect_front)*5*PI/36+(1+reflect_front)*7*PI/36-reflect_front*hfe_pos0}"/>
+			<origin xyz="${d_tbb} 0 0" rpy="${reflect_upper*PI/2} 0 0"/>
+			<parent link="${name}_hipassembly"/>
+			<child  link="${name}_upperleg"/>
 			<axis xyz="0 0 1"/>
+			<limit effort="150.0" velocity="12.0"
+				   lower="${-(1+reflect_front)*5*PI/36-(1-reflect_front)*7*PI/36}"
+				   upper="${(1-reflect_front)*5*PI/36+(1+reflect_front)*7*PI/36}"/>
 			<dynamics damping="0.1" friction="0" />
-			<safety_controller k_position="100" k_velocity="100" soft_lower_limit="-10" soft_upper_limit="12.45" />
+			<safety_controller k_position="100" k_velocity="100"
+							   soft_lower_limit="-10" soft_upper_limit="12.45" />
 		</joint>
 		<!-- Lower leg joint -->
 		<joint name="${name}_kfe_joint" type="revolute">
-			<origin xyz="${d_p1p2} 0 0" rpy="0 0 ${reflect_front*kfe_pos0}"/>
-			<parent link="${name}_upper_leg"/>
-			<child  link="${name}_lower_leg"/>
-			<limit effort="150.0" velocity="12.0" lower="${-(1+reflect_front)*7*PI/18+(1-reflect_front)*PI/18-reflect_front*kfe_pos0}" upper="${(1-reflect_front)*7*PI/18-(1+reflect_front)*PI/18-reflect_front*kfe_pos0}"/>
+			<origin xyz="${d_p1p2} 0 0" rpy="0 0 0"/>
+			<parent link="${name}_upperleg"/>
+			<child  link="${name}_lowerleg"/>
 			<axis xyz="0 0 1"/>
+			<limit effort="150.0" velocity="12.0"
+				   lower="${-(1+reflect_front)*7*PI/18+(1-reflect_front)*PI/18}"
+				   upper="${(1-reflect_front)*7*PI/18-(1+reflect_front)*PI/18}"/>
 			<dynamics damping="0.1" friction="0" />
-			<safety_controller k_position="100" k_velocity="100" soft_lower_limit="-10" soft_upper_limit="12.45" />
+			<safety_controller k_position="100" k_velocity="100"
+							   soft_lower_limit="-10" soft_upper_limit="12.45" />
 		<!-- Foot joint -->
 		</joint>
 		<joint name="${name}_foot_joint" type="fixed">
-			<origin xyz="0.34 0 0" rpy="${PI/2} 0 ${-PI/2}"/>
-			<parent link="${name}_lower_leg"/>
+			<origin xyz="0.35 0 0" rpy="${PI/2} 0 ${-PI/2}"/>
+			<parent link="${name}_lowerleg"/>
 			<child  link="${name}_foot"/>
 		</joint>
 		<!-- Links -->
 		<!-- Hip assembly link -->
-		<link name="${name}_assembly">
+		<link name="${name}_hipassembly">
 			<inertial>
-				<origin xyz="0 0 0"/>
-				<mass value="0.01"/>
-				<inertia ixx="0.01" iyy="0.01" izz="0.01" ixy="0.0" ixz="0.0" iyz="0.0"/>
-			</inertial>
-		</link>
-		<!-- Hip assembly link -->
-		<link name="${name}_hip_assembly">
-			<inertial>
-				<origin xyz="0.01310 ${reflect_hip*0.00010} ${reflect_hip*0.05730}"/>
-				<mass value="${m_hip}"/>
-				<inertia ixx="${ixx_hip}" iyy="${iyy_hip}" izz="${izz_hip}" ixy="${ixy_hip}" ixz="${-reflect_hip*ixz_hip}" iyz="${iyz_hip}"/>
+				<origin xyz="${xcom_hipassembly}
+							 ${reflect_hip*ycom_hipassembly}
+							 ${reflect_hip*zcom_hipassembly}"/>
+				<mass value="${m_hipassembly}"/>
+				<inertia ixx="${ixx_hipassembly}" iyy="${iyy_hipassembly}" izz="${izz_hipassembly}"
+						 ixy="${reflect_hip*reflect_front*ixy_hipassembly}" ixz="${reflect_hip*reflect_front*ixz_hipassembly}" iyz="${iyz_hipassembly}"/>
 			</inertial>
 			<visual>
 				<origin xyz="0 0 0" rpy="${(1-reflect_hip)*PI/2} 0 0"/>
 				<geometry>
-					<mesh filename="package://hyq_description/meshes/leg/hip.dae" scale="1 1 1"/>
+					<mesh filename="package://hyq_description/meshes/leg/hipassembly.dae" scale="1 1 1"/>
 				</geometry>
 			</visual>
@@ -77,19 +71,20 @@
 				<origin xyz="0 0 0" rpy="${(1-reflect_hip)*PI/2} 0 0"/>
 				<geometry>
-					<mesh filename="package://hyq_description/meshes/leg/hip.dae" scale="1 1 1"/>
+					<mesh filename="package://hyq_description/meshes/leg/hipassembly.dae" scale="1 1 1"/>
 				</geometry>
 			</collision>
 		</link>
 		<!-- Upper leg link -->
-		<link name="${name}_upper_leg">
+		<link name="${name}_upperleg">
 			<inertial>
-				<origin xyz="0.14796 ${reflect_upper*0.02958} 0"/>
-				<mass value="${m_upper}"/>
-				<inertia ixx="${ixx_upper}" iyy="${iyy_upper}" izz="${izz_upper}" ixy="${ixy_upper}" ixz="${ixz_upper}" iyz="${iyz_upper}"/>
+				<origin xyz="${xcom_upperleg} ${reflect_upper*ycom_upperleg} ${zcom_upperleg}"/>
+				<mass value="${m_upperleg}"/>
+				<inertia ixx="${ixx_upperleg}" iyy="${iyy_upperleg}" izz="${izz_upperleg}"
+						 ixy="${reflect_front*ixy_upperleg}" ixz="${reflect_front*ixz_upperleg}" iyz="${iyz_upperleg}"/>
 			</inertial>
 			<visual>
 				<origin xyz="0 0 0" rpy="${(1-reflect_front)*PI/2} 0 0"/>
 				<geometry>
-					<mesh filename="package://hyq_description/meshes/leg/upper.dae" scale="1 1 1"/>
+					<mesh filename="package://hyq_description/meshes/leg/upperleg.dae" scale="1 1 1"/>
 				</geometry>
 			</visual>
@@ -97,18 +92,19 @@
 				<origin xyz="0 0 0" rpy="${(1-reflect_front)*PI/2} 0 0"/>
 				<geometry>
-					<mesh filename="package://hyq_description/meshes/leg/upper.dae" scale="1 1 1"/>
+					<mesh filename="package://hyq_description/meshes/leg/upperleg.dae" scale="1 1 1"/>
 				</geometry>
 			</collision>
 		</link>
 		<!-- Lower leg link -->
-		<link name="${name}_lower_leg">
+		<link name="${name}_lowerleg">
 			<inertial>
-				<origin xyz=" 0.17830  0.00030 -0.00010"/>
-				<mass value="${m_lower}"/>
-				<inertia ixx="${ixx_lower}" iyy="${iyy_lower}" izz="${izz_lower}" ixy="${ixy_lower}" ixz="${ixz_lower}" iyz="${iyz_lower}"/>
+				<origin xyz="${xcom_lowerleg} ${ycom_lowerleg} ${zcom_lowerleg}"/>
+				<mass value="${m_lowerleg}"/>
+				<inertia ixx="${ixx_lowerleg}" iyy="${iyy_lowerleg}" izz="${izz_lowerleg}"
+						 ixy="${ixy_lowerleg}" ixz="${ixz_lowerleg}" iyz="${iyz_lowerleg}"/>
 			</inertial>
 			<visual>
 				<geometry>
-					<mesh filename="package://hyq_description/meshes/leg/lower.dae" scale="1 1 1"/>
+					<mesh filename="package://hyq_description/meshes/leg/lowerleg.dae" scale="1 1 1"/>
 				</geometry>
 				<material name="white"/>
@@ -116,5 +112,5 @@
 			<collision>
 				<geometry>
-					<mesh filename="package://hyq_description/meshes/leg/lower.dae" scale="1 1 1"/>
+					<mesh filename="package://hyq_description/meshes/leg/lowerleg.dae" scale="1 1 1"/>
 				</geometry>
 			</collision>

File: hyq_description/urdfs/trunk/trunk.urdf.xacro (robot description, xacro)
@@ -24,19 +24,19 @@
 		<link name="trunk">
 			<inertial>
-				<origin xyz="-0.00020  0.00010  0.00110"/>
+				<origin xyz="${xcom_trunk} ${ycom_trunk} ${zcom_trunk}"/>
 				<mass value="${m_trunk}"/>
-				<inertia ixx="${ixx_trunk}" iyy="${iyy_trunk}" izz="${izz_trunk}" ixy="${ixy_trunk}" ixz="${ixz_trunk}" iyz="${iyz_trunk}"/>
+				<inertia ixx="${ixx_trunk}" iyy="${iyy_trunk}" izz="${izz_trunk}"
+						 ixy="${ixy_trunk}" ixz="${ixz_trunk}" iyz="${iyz_trunk}"/>
 			</inertial>
+			<visual>
+				<geometry>
+					<mesh filename="package://hyq_description/meshes/trunk/trunk.dae" scale="1 1 1"/>
+				</geometry>
+			</visual>
 			<collision>
 				<geometry>
-					<mesh filename="package://hyq_description/meshes/trunk/trunk_frame.dae" scale="1 1 1"/>
+					<mesh filename="package://hyq_description/meshes/trunk/trunk.dae" scale="1 1 1"/>
 				</geometry>
 			</collision>
-			<visual>
-				<origin xyz="0 0 0" rpy="0 0 0" />
-				<geometry>
-					<mesh filename="package://hyq_description/meshes/trunk/trunk_frame.dae" scale="1 1 1"/>
-				</geometry>
-			</visual>
 		</link>
 		<!-- Extensions -->
