Commit message: Cosmetic changes

File: urdfs/sensors/hokuyo_laser.urdf.xacro (robot description, xacro)
@@ -1,41 +1,40 @@
 <?xml version="1.0"?>
 <robot xmlns:xacro="http://ros.org/wiki/xacro">
-    <xacro:property name="M_PI" value="3.1415926535897931" />
-  <xacro:macro name="hokuyo_laser" params="name parent *origin ros_topic update_rate min_angle max_angle range">
-    <joint name="${name}_joint" type="fixed">
-      <axis xyz="0 0 0" />
-      <insert_block name="origin" />
-      <parent link="${parent}"/>
-      <child link="${name}_mount_link"/>
-    </joint>
-    <link name="${name}_mount_link">
-      <inertial>
-        <mass value="0.001" />
-        <origin xyz="0 0 0" rpy="0 0 0" />
-        <inertia ixx="0.0001" ixy="0" ixz="0" iyy="0.000001" iyz="0" izz="0.0001" />
-      </inertial>
-      <visual>
-        <origin xyz="0 0 0" rpy="0 0 0" />
-        <geometry>
-          <mesh filename="package://hyq_description/meshes/sensors/hokuyo.dae" scale="0.0254 0.0254 0.0254" />
-        </geometry>
-      </visual>
-      <!-- ignore the collision element -->
-    </link>
-    <!-- go from the base of the laser to the actual sensor location -->
-    <joint name="${name}_laser_joint" type="fixed">
-      <origin xyz="0 0 0.058" />
-      <parent link="${name}_mount_link"/>
-      <child link="${name}"/>
-    </joint>
-    <link name="${name}" type="laser">
-      <inertial>
-        <mass value="0.001" />
-        <origin xyz="0 0 0" rpy="0 0 0" />
-        <inertia ixx="0.0001" ixy="0" ixz="0" iyy="0.000001" iyz="0" izz="0.0001" />
-      </inertial>
-    </link>
-    <!-- gazebo extensions -->
-    <xacro:hokuyo_laser_gazebo name="${name}_laser" ros_topic="${ros_topic}" update_rate="${update_rate}" min_angle="${min_angle}" max_angle="${max_angle}" range="${range}"/>
+	<xacro:macro name="hokuyo_laser" params="name parent *origin ros_topic update_rate min_angle max_angle range">
+		<joint name="${name}_joint" type="fixed">
+			<axis xyz="0 0 0" />
+			<insert_block name="origin" />
+			<parent link="${parent}"/>
+			<child link="${name}_mount_link"/>
+		</joint>
+		<!-- go from the base of the laser to the actual sensor location -->
+		<joint name="${name}_laser_joint" type="fixed">
+			<origin xyz="0 0 0.058" />
+			<parent link="${name}_mount_link"/>
+			<child link="${name}"/>
+		</joint>
+		<link name="${name}_mount_link">
+			<inertial>
+				<mass value="0.001" />
+				<origin xyz="0 0 0" rpy="0 0 0" />
+				<inertia ixx="0.0001" ixy="0" ixz="0" iyy="0.000001" iyz="0" izz="0.0001" />
+			</inertial>
+			<visual>
+				<origin xyz="0 0 0" rpy="0 0 0" />
+				<geometry>
+					<mesh filename="package://hyq_description/meshes/sensors/hokuyo.dae" scale="0.0254 0.0254 0.0254" />
+				</geometry>
+			</visual>
+			<!-- ignore the collision element -->
+		</link>
+		<link name="${name}" type="laser">
+			<inertial>
+				<mass value="0.001" />
+				<origin xyz="0 0 0" rpy="0 0 0" />
+				<inertia ixx="0.0001" ixy="0" ixz="0" iyy="0.000001" iyz="0" izz="0.0001" />
+			</inertial>
+		</link>
+		<!-- gazebo extensions -->
+		<xacro:hokuyo_laser_gazebo name="${name}_laser" ros_topic="${ros_topic}" update_rate="${update_rate}" min_angle="${min_angle}" max_angle="${max_angle}" range="${range}"/>
     </xacro:macro>
 </robot>
