Commit message: Stephane turn-off the gazebo plugin of the asus-xtion camera. I reintroduced it with the new Stephane's names

File: urdfs/sensors/asus_xtion.urdf.xacro (robot description, xacro)
@@ -12,21 +12,22 @@
 		</joint>
 		<!-- asus ir sensor physical attachment -->
-		<!--joint name="${name}_depth_joint" type="fixed">
+		<joint name="${name}_depth_joint" type="fixed">
 			<origin xyz="${asus_xtion_x} ${asus_xtion_depth_y} ${asus_xtion_z}" rpy="0 0 0"/>
 			<parent link="${name}_mount_link"/>
 			<child link="${name}_depth_frame"/>
-		</joint-->
+		</joint>
 		<!-- asus xtion ir sensor frame -->
 		<joint name="${name}_depth_optical_frame_joint" type="fixed">
-			<origin xyz="${asus_xtion_x} ${asus_xtion_depth_y} ${asus_xtion_z}"	rpy="${asus_xtion_roll} ${asus_xtion_pitch} ${asus_xtion_yaw}"/>
+			<origin xyz="${asus_xtion_x} ${asus_xtion_depth_y} ${asus_xtion_z}"
+					rpy="${asus_xtion_roll} ${asus_xtion_pitch} ${asus_xtion_yaw}"/>
 			<parent link="${name}_mount_link"/>
 			<child link="${name}_depth_optical_frame"/>
 		</joint>
 		<!-- asus_xtion rgb sensor physical attachment -->
-		<!--joint name="${name}_rgb_joint" type="fixed">
+		<joint name="${name}_rgb_joint" type="fixed">
 			<origin xyz="${asus_xtion_x} ${asus_xtion_rgb_y} ${asus_xtion_z}" rpy="0 0 0"/>
 			<parent link="${name}_mount_link"/>
 			<child link="${name}_rgb_frame"/>
-		</joint-->
+		</joint>
 		<!-- asus xtion rgb sensor frame -->
 		<joint name="${name}_rgb_optical_frame_joint" type="fixed">
@@ -59,5 +60,5 @@
 		</link>
 		<!-- ir sensor link -->
-		<!--link name="${name}_depth_frame">
+		<link name="${name}_depth_frame">
 			<inertial>
 				<mass value="0.1" />
@@ -77,9 +78,9 @@
 				</geometry>
 			</collision>
-		</link-->
+		</link>
 		<!-- ir optical sensor link -->
 		<link name="${name}_depth_optical_frame"/>
 		<!-- rgb sensor link -->
-		<!--link name="${name}_rgb_frame" >
+		<link name="${name}_rgb_frame" >
 			<inertial>
 				<mass value="0.1" />
@@ -99,10 +100,10 @@
 				</geometry>
 			</collision>
-		</link-->
+		</link>
 		<!-- rgb optical sensor link -->
 		<link name="${name}_rgb_optical_frame"/>
 	<!-- gazebo extensions -->
-	<!--xacro:asus_xtion_depth_sensor link_name="${name}_depth_frame" frame_name="${name}_depth_optical_frame" camera_name="${name}" /-->
-	<!--xacro:asus_xtion_rgb_sensor link_name="${name}_rgb_frame" frame_name="${name}_rgb_optical_frame" camera_name="${name}" /-->
+	<xacro:asus_xtion_depth_sensor link_name="${name}_depth_frame" frame_name="${name}_depth_optical_frame" camera_name="${name}"/>
+	<xacro:asus_xtion_rgb_sensor link_name="${name}_rgb_frame" frame_name="${name}_rgb_optical_frame" camera_name="${name}"/>
 	</xacro:macro>
 </root>
