Commit message: Updated IMU box model

File: urdfs/sensors/microstrain_3dmgx425_imu.urdf.xacro (robot description, xacro)
@@ -22,6 +22,9 @@
 				<origin xyz="0 0 0" rpy="0 0 0"/>
 				<geometry>
-					<box size="0.02 0.02 0.02" />
+					<box size="0.0329 0.0244 0.0111" />
 				</geometry>
+				<material name="black">
+					<color rgba="0 0 0 0.9"/>
+				</material>
 			</visual>
 		</link>

Commit message: Updated imu visual origin

File: urdfs/sensors/microstrain_3dmgx425_imu.urdf.xacro (robot description, xacro)
@@ -20,5 +20,5 @@
 			</inertial>
 			<visual>
-				<origin xyz="0 0 0" rpy="0 0 0"/>
+				<origin xyz="0.00485 0 -0.0105" rpy="0 0 0"/>
 				<geometry>
 					<box size="0.0329 0.0244 0.0111" />

Commit message: updated again visual origin

File: urdfs/sensors/microstrain_3dmgx425_imu.urdf.xacro (robot description, xacro)
@@ -20,5 +20,5 @@
 			</inertial>
 			<visual>
-				<origin xyz="0.00485 0 -0.0105" rpy="0 0 0"/>
+				<origin xyz="0.00485 0 -0.00105" rpy="0 0 0"/>
 				<geometry>
 					<box size="0.0329 0.0244 0.0111" />
