Commit message: changed angle and min intensity of teraranger

File: urdfs/sensors/teraranger_range.gazebo.xacro (robot description, xacro)
@@ -35,5 +35,5 @@
 					<topicName>/${ros_topic}</topicName>
 					<frameName>${frame_name}</frameName>
-					<hokuyoMinIntensity>101</hokuyoMinIntensity>
+					<hokuyoMinIntensity>102</hokuyoMinIntensity>
 				</plugin>
 			</sensor>

File: urdfs/sensors/teraranger_range.urdf.xacro (robot description, xacro)
@@ -12,5 +12,5 @@
 		<!-- go from the base of the laser to the actual sensor location -->
 		<joint name="${name}_laser_joint" type="fixed">
-			<origin xyz="0 0 0.058" rpy="0 0 0"/>
+			<origin xyz="0 0 0.058" rpy="0 0.25 0"/>
 			<parent link="${name}_mount_link"/>
 			<child link="${name}"/>
