Commit message: Updated IMU position and model

File: robots/hyq_model.urdf.xacro (robot description, xacro)
@@ -59,9 +59,9 @@
 	</xacro:hyq_leg>
 	<!-- IMU trunk -->
-	<xacro:microstrain_3dmgx325_imu
+	<xacro:microstrain_3dmgx425_imu
 		parent="trunk"
 		imu_name="imu"
 		imu_topic="trunk_imu/data"
-		update_rate="1000"
+		update_rate="250"
 		rate_mean="0"
 		rate_stddev="2e-4"
@@ -72,5 +72,5 @@
 		accel_bias_mean="0.002"
 		accel_bias_stddev="0.001">
-		<origin xyz="0.4825 0.006 0.0905" rpy="0 ${-PI} 0"/>
-	</xacro:microstrain_3dmgx325_imu>
+		<origin xyz="0.290 0.000 0.0999214" rpy="0 ${-PI} 0"/>
+	</xacro:microstrain_3dmgx425_imu>
 </robot>
