Commit message: changed no sensor file

File: robots/hyq_no_sensors.urdf.xacro (robot description, xacro)
@@ -12,4 +12,5 @@
 	<!-- generic simulator_gazebo plugins for starting mechanism control, ros time -->
 	<xacro:include filename="$(find hyq_description)/gazebo/gazebo.urdf.xacro"/>
+	<xacro:include filename="$(find hyq_description)/urdfs/sensors/teraranger_range.urdf.xacro"/>
 	<!-- Now we can start using the macros included above to define the actual HyQ -->
 	<!-- The first use of a macro. This one was defined in trunk.urdf.xacro above.
@@ -77,3 +78,12 @@
 		<origin xyz="0.290 0.000 0.0999214" rpy="0 ${-PI} 0"/>
 	</xacro:microstrain_3dmgx425_imu>
+		<!-- teraranger -->
+    <xacro:teraranger_range
+		name="rf_ranger"
+		parent="rf_lowerleg"
+		ros_topic="rf_terarangerone"
+		update_rate="400"
+		range="4.0">
+		<origin xyz="0.12 0.0 0.0" rpy = "${PI/2} 0.0 0.0"/>
+	</xacro:teraranger_range>
 </robot>

File: urdfs/sensors/teraranger_range.urdf.xacro (robot description, xacro)
@@ -25,5 +25,5 @@
 				<origin xyz="0 0 0" rpy="0 0 0" />
 				<geometry>
-					<mesh filename="package://hyq_description/meshes/sensors/hokuyo.dae" scale="0.0254 0.0254 0.0254" />
+					<mesh filename="package://sensors_description/meshes/sensors/hokuyo.dae" scale="0.0254 0.0254 0.0254" />
 				</geometry>
 			</visual>

Commit message: removed no sensors teraranger

File: robots/hyq_no_sensors.urdf.xacro (robot description, xacro)
@@ -78,12 +78,3 @@
 		<origin xyz="0.290 0.000 0.0999214" rpy="0 ${-PI} 0"/>
 	</xacro:microstrain_3dmgx425_imu>
-		<!-- teraranger -->
-    <xacro:teraranger_range
-		name="rf_ranger"
-		parent="rf_lowerleg"
-		ros_topic="rf_terarangerone"
-		update_rate="400"
-		range="4.0">
-		<origin xyz="0.12 0.0 0.0" rpy = "${PI/2} 0.0 0.0"/>
-	</xacro:teraranger_range>
 </robot>

Commit message: Compliance with new xacro standard (kinetic)

File: robots/hyq_no_sensors.urdf.xacro (robot description, xacro)
@@ -1,4 +1,4 @@
 <?xml version="1.0"?>
-<robot name="hyq" xmlns:xacro="http://www.ros.org/wiki/xacro">
+<robot name="hyq" xmlns:xacro="http://ros.org/wiki/xacro">
 	<!-- This argument allows us to load joint sensors that measure the internal wrenches -->
 	<xacro:arg name="load_force_sensors" default="false"/>
@@ -21,9 +21,9 @@
 (e.g., base_link). The included origin block is also an argument to the macro. By convention,
 the origin block defines where the component is w.r.t its parent (in this case the parent
-is the world frame). For more, see http://www.ros.org/wiki/xacro -->
+is the world frame). For more, see http://ros.org/wiki/xacro -->
 	<!-- body -->
 	<!-- trunk -->
 	<xacro:hyq_trunk name="base">
-		<origin xyz="-0.443 -0.191 -0.276" rpy="0 0 0"/>
+		<!--origin xyz="-0.443 -0.191 -0.276" rpy="0 0 0"/-->
 	</xacro:hyq_trunk>
 	<!-- LF leg -->

File: urdfs/common.xacro (robot description, xacro)
@@ -1,55 +1,55 @@
 <?xml version="1.0"?>
-<robot>
-	<property name="PI" value="3.1415926535897931"/>
+<robot xmlns:xacro="http://ros.org/wiki/xacro">
+	<xacro:property name="PI" value="3.1415926535897931"/>
 	<!-- standard distances -->
-	<property name="d_lr" value="0.414"/>
-	<property name="d_fh" value="0.747"/>
-	<property name="d_p0p1" value="0.08"/>
-	<property name="d_p1p2" value="0.35"/>
-	<property name="d_p2p3" value="0.346"/>
+	<xacro:property name="d_lr" value="0.414"/>
+	<xacro:property name="d_fh" value="0.747"/>
+	<xacro:property name="hipassembly_length" value="0.08"/>
+	<xacro:property name="upperleg_length" value="0.35"/>
+	<xacro:property name="lowerleg_length" value="0.346"/>
 	<!-- Inertial values -->
 	<!-- Trunk with hydraulic system -->
-	<property name="xcom_trunk" value="0.056"/>
-	<property name="ycom_trunk" value="0.0215"/>
-	<property name="zcom_trunk" value="0.00358"/>
-	<property name="m_trunk" value="60.96"/>
-	<property name="ixx_trunk" value="1.5725937"/>
-	<property name="iyy_trunk" value="8.5015928"/>
-	<property name="izz_trunk" value="9.1954911"/>
-	<property name="ixy_trunk" value="0.028375"/>
-	<property name="ixz_trunk" value="-0.203139"/>
-	<property name="iyz_trunk" value="-0.004462"/>
+	<xacro:property name="xcom_trunk" value="0.056"/>
+	<xacro:property name="ycom_trunk" value="0.0215"/>
+	<xacro:property name="zcom_trunk" value="0.00358"/>
+	<xacro:property name="m_trunk" value="60.96"/>
+	<xacro:property name="ixx_trunk" value="1.5725937"/>
+	<xacro:property name="iyy_trunk" value="8.5015928"/>
+	<xacro:property name="izz_trunk" value="9.1954911"/>
+	<xacro:property name="ixy_trunk" value="0.028375"/>
+	<xacro:property name="ixz_trunk" value="-0.203139"/>
+	<xacro:property name="iyz_trunk" value="-0.004462"/>
 	<!-- Hip assembly -->
-	<property name="xcom_hipassembly" value="0.04263"/>
-	<property name="ycom_hipassembly" value="0.0"/>
-	<property name="zcom_hipassembly" value="0.16931"/>
-	<property name="m_hipassembly" value="2.93"/>
-	<property name="ixx_hipassembly" value="0.05071"/>
-	<property name="iyy_hipassembly" value="0.05486"/>
-	<property name="izz_hipassembly" value="0.00571"/>
-	<property name="ixy_hipassembly" value="-0.00004"/>
-	<property name="ixz_hipassembly" value="-0.00159"/>
-	<property name="iyz_hipassembly" value="-0.00005"/>
+	<xacro:property name="xcom_hipassembly" value="0.04263"/>
+	<xacro:property name="ycom_hipassembly" value="0.0"/>
+	<xacro:property name="zcom_hipassembly" value="0.16931"/>
+	<xacro:property name="m_hipassembly" value="2.93"/>
+	<xacro:property name="ixx_hipassembly" value="0.05071"/>
+	<xacro:property name="iyy_hipassembly" value="0.05486"/>
+	<xacro:property name="izz_hipassembly" value="0.00571"/>
+	<xacro:property name="ixy_hipassembly" value="-0.00004"/>
+	<xacro:property name="ixz_hipassembly" value="-0.00159"/>
+	<xacro:property name="iyz_hipassembly" value="-0.00005"/>
 	<!-- Upper leg -->
-	<property name="xcom_upperleg" value="0.15074"/>
-	<property name="ycom_upperleg" value="0.02625"/>
-	<property name="zcom_upperleg" value="0.0"/>
-	<property name="m_upperleg" value="2.638"/>
-	<property name="ixx_upperleg" value="0.00368"/>
-	<property name="iyy_upperleg" value="0.02719"/>
-	<property name="izz_upperleg" value="0.02811"/>
-	<property name="ixy_upperleg" value="-0.00302"/>
-	<property name="ixz_upperleg" value="0.0001"/>
-	<property name="iyz_upperleg" value="0.00002"/>
+	<xacro:property name="xcom_upperleg" value="0.15074"/>
+	<xacro:property name="ycom_upperleg" value="0.02625"/>
+	<xacro:property name="zcom_upperleg" value="0.0"/>
+	<xacro:property name="m_upperleg" value="2.638"/>
+	<xacro:property name="ixx_upperleg" value="0.00368"/>
+	<xacro:property name="iyy_upperleg" value="0.02719"/>
+	<xacro:property name="izz_upperleg" value="0.02811"/>
+	<xacro:property name="ixy_upperleg" value="-0.00302"/>
+	<xacro:property name="ixz_upperleg" value="0.0001"/>
+	<xacro:property name="iyz_upperleg" value="0.00002"/>
 	<!-- Lower leg -->
-	<property name="xcom_lowerleg" value="0.1254"/>
-	<property name="ycom_lowerleg" value="0.00004"/>
-	<property name="zcom_lowerleg" value="-0.0001"/>
-	<property name="m_lowerleg" value="0.881"/>
-	<property name="ixx_lowerleg" value="0.00047"/>
-	<property name="iyy_lowerleg" value="0.01256"/>
-	<property name="izz_lowerleg" value="0.01233"/>
-	<property name="ixy_lowerleg" value="0.00006"/>
-	<property name="ixz_lowerleg" value="-0.00001"/>
-	<property name="iyz_lowerleg" value="-0.0"/>
+	<xacro:property name="xcom_lowerleg" value="0.1254"/>
+	<xacro:property name="ycom_lowerleg" value="0.00004"/>
+	<xacro:property name="zcom_lowerleg" value="-0.0001"/>
+	<xacro:property name="m_lowerleg" value="0.881"/>
+	<xacro:property name="ixx_lowerleg" value="0.00047"/>
+	<xacro:property name="iyy_lowerleg" value="0.01256"/>
+	<xacro:property name="izz_lowerleg" value="0.01233"/>
+	<xacro:property name="ixy_lowerleg" value="0.00006"/>
+	<xacro:property name="ixz_lowerleg" value="-0.00001"/>
+	<xacro:property name="iyz_lowerleg" value="-0.0"/>
 </robot>

File: urdfs/leg/leg.gazebo.xacro (robot description, xacro)
@@ -1,4 +1,4 @@
 <?xml version="1.0"?>
-<robot xmlns:xacro="http://www.ros.org/wiki/xacro">
+<robot xmlns:xacro="http://ros.org/wiki/xacro">
 	<xacro:macro name="leg_gazebo" params="name load_force_sensors">
 		<gazebo reference="${name}_haa_joint">
@@ -64,5 +64,5 @@
 				<update_rate>1000.0</update_rate>
 				<contact>
-					<collision>${name}_foot_collision</collision>
+					<collision>${name}_lowerleg_fixed_joint_lump__${name}_foot_collision_1</collision>
 				</contact>
 				<plugin name="${name}_foot_bumper" filename="libgazebo_ros_bumper.so">

Commit message: fixes for kinetic

File: robots/hyq_no_sensors.urdf.xacro (robot description, xacro)
@@ -25,5 +25,5 @@
 	<!-- trunk -->
 	<xacro:hyq_trunk name="base">
-		<origin xyz="-0.443 -0.191 -0.276" rpy="0 0 0"/>
+		<!--origin xyz="-0.443 -0.191 -0.276" rpy="0 0 0"/-->
 	</xacro:hyq_trunk>
 	<!-- LF leg -->

File: urdfs/common.xacro (robot description, xacro)
@@ -1,22 +1,22 @@
 <?xml version="1.0"?>
 <robot xmlns:xacro="http://ros.org/wiki/xacro">
-	<property name="PI" value="3.1415926535897931"/>
+	<xacro:property name="PI" value="3.1415926535897931"/>
     <!-- kin limits (sign ref is RH leg)-->
-    <property name="haa_max" value="25"/>
-    <property name="haa_min" value="-70"/>
-    <property name="hfe_max" value="50"/>
-    <property name="hfe_min" value="-70"/>
-    <property name="kfe_max" value="140"/>
-    <property name="kfe_min" value="20"/>
+    <xacro:property name="haa_max" value="25"/>
+    <xacro:property name="haa_min" value="-70"/>
+    <xacro:property name="hfe_max" value="50"/>
+    <xacro:property name="hfe_min" value="-70"/>
+    <xacro:property name="kfe_max" value="140"/>
+    <xacro:property name="kfe_min" value="20"/>
     <!-- torque limits 120-->
-    <property name="haa_limit" value="150"/>
-    <property name="hfe_limit" value="150"/>
-    <property name="kfe_limit" value="150"/>
+    <xacro:property name="haa_limit" value="150"/>
+    <xacro:property name="hfe_limit" value="150"/>
+    <xacro:property name="kfe_limit" value="150"/>
 	<!-- standard distances -->
-	<property name="d_lr" value="0.414"/>
-	<property name="d_fh" value="0.747"/>
-	<property name="hipassembly_length" value="0.08"/>
-	<property name="upperleg_length" value="0.35"/>
-	<property name="lowerleg_length" value="0.346"/>
+	<xacro:property name="d_lr" value="0.414"/>
+	<xacro:property name="d_fh" value="0.747"/>
+	<xacro:property name="hipassembly_length" value="0.08"/>
+	<xacro:property name="upperleg_length" value="0.35"/>
+	<xacro:property name="lowerleg_length" value="0.346"/>
 	<!-- Inertial values -->
 	<!-- Trunk with hydraulic system -->

Commit message: Added leg backward option

File: robots/hyq_no_sensors.urdf.xacro (robot description, xacro)
@@ -34,4 +34,5 @@
 		reflect_upper="1"
 		reflect_front="1"
+		knee_bent_backward="1"
 		load_force_sensors="$(arg load_force_sensors)">
 		<origin xyz="${d_fh/2} ${d_lr/2} 0" rpy="0 ${PI/2} ${PI}"/>
@@ -44,4 +45,5 @@
 		reflect_upper="-1"
 		reflect_front="1"
+		knee_bent_backward ="1"
 		load_force_sensors="$(arg load_force_sensors)">
 		<origin xyz="${d_fh/2} ${-d_lr/2} 0" rpy="0 ${PI/2} 0"/>
@@ -54,4 +56,5 @@
 		reflect_upper="1"
 		reflect_front="-1"
+		knee_bent_backward="0"
 		load_force_sensors="$(arg load_force_sensors)">
 		<origin xyz="${-d_fh/2} ${d_lr/2} 0" rpy="0 ${PI/2} ${PI}"/>
@@ -64,4 +67,5 @@
 		reflect_upper="-1"
 		reflect_front="-1"
+		knee_bent_backward="0"
 		load_force_sensors="$(arg load_force_sensors)">
 		<origin xyz="${-d_fh/2} ${-d_lr/2} 0" rpy="0 ${PI/2} 0"/>

File: urdfs/common.xacro (robot description, xacro)
@@ -2,4 +2,15 @@
 <robot xmlns:xacro="http://ros.org/wiki/xacro">
 	<xacro:property name="PI" value="3.1415926535897931"/>
+    <!-- kin limits (sign ref is RH leg)-->
+    <xacro:property name="haa_max" value="25"/>
+    <xacro:property name="haa_min" value="-70"/>
+    <xacro:property name="hfe_max" value="50"/>
+    <xacro:property name="hfe_min" value="-70"/>
+    <xacro:property name="kfe_max" value="140"/>
+    <xacro:property name="kfe_min" value="20"/>
+    <!-- torque limits 120-->
+    <xacro:property name="haa_limit" value="150"/>
+    <xacro:property name="hfe_limit" value="150"/>
+    <xacro:property name="kfe_limit" value="150"/>
 	<!-- standard distances -->
 	<xacro:property name="d_lr" value="0.414"/>

File: urdfs/leg/leg.urdf.xacro (robot description, xacro)
@@ -6,5 +6,5 @@
 	<!-- ================================== Leg ================================== -->
 	<!-- The xacro macro xacro:hyq_leg contains: hip assembly, upper and lower leg -->
-	<xacro:macro name="hyq_leg" params="name parent *origin reflect_hip reflect_upper reflect_front load_force_sensors">
+	<xacro:macro name="hyq_leg" params="name parent *origin reflect_hip reflect_upper reflect_front knee_bent_backward load_force_sensors">
 		<!-- Joints -->
 		<!-- Hip assembly joint -->
@@ -14,40 +14,40 @@
 			<child  link="${name}_hipassembly"/>
 			<axis xyz="0 0 1"/>
-			<limit effort="150.0" velocity="12.0" lower="${-7*PI/18}" upper="${5*PI/36}"/>
+			<limit effort="${haa_limit}" velocity="12.0" lower="${haa_min*PI/180}" upper="${haa_max*PI/180}" />
 			<dynamics damping="0.1" friction="0" />
-			<safety_controller k_position="100" k_velocity="100"
-							   soft_lower_limit="${-7*PI/18}" soft_upper_limit="${5*PI/36}" />
+			<safety_controller k_position="50" k_velocity="10"
+							   soft_lower_limit="${haa_min*PI/180}" soft_upper_limit="${haa_max*PI/180}" />
 		</joint>
 		<!-- Upper leg joint -->
 		<joint name="${name}_hfe_joint" type="revolute">
-			<origin xyz="${d_p0p1} 0 0" rpy="${reflect_upper*PI/2} 0 0"/>
+			<origin xyz="${hipassembly_length} 0 0" rpy="${reflect_upper*PI/2} 0 0"/>
 			<parent link="${name}_hipassembly"/>
 			<child  link="${name}_upperleg"/>
 			<axis xyz="0 0 1"/>
-			<limit effort="150.0" velocity="12.0"
-				   lower="${-(1+reflect_front)*5*PI/36-(1-reflect_front)*7*PI/36}"
-				   upper="${(1-reflect_front)*5*PI/36+(1+reflect_front)*7*PI/36}"/>
+			<limit effort="${hfe_limit}" velocity="12.0"
+                  lower="${(1-knee_bent_backward)*(hfe_min)*PI/180 + (knee_bent_backward)*(-hfe_max)*PI/180}"
+                  upper="${(1-knee_bent_backward)*(hfe_max)*PI/180 + (knee_bent_backward)*(-hfe_min)*PI/180}"/>
 			<dynamics damping="0.1" friction="0" />
-			<safety_controller k_position="100" k_velocity="100"
-							   soft_lower_limit="${-(1+reflect_front)*5*PI/36-(1-reflect_front)*7*PI/36}"
-							   soft_upper_limit="${(1-reflect_front)*5*PI/36+(1+reflect_front)*7*PI/36}" />
+			<safety_controller k_position="50" k_velocity="10"
+                  soft_lower_limit="${(1-knee_bent_backward)*(hfe_min)*PI/180 + (knee_bent_backward)*(-hfe_max)*PI/180}"
+                  soft_upper_limit="${(1-knee_bent_backward)*(hfe_max)*PI/180 + (knee_bent_backward)*(-hfe_min)*PI/180}"/>
 		</joint>
 		<!-- Lower leg joint -->
 		<joint name="${name}_kfe_joint" type="revolute">
-			<origin xyz="${d_p1p2} 0 0" rpy="0 0 0"/>
+			<origin xyz="${upperleg_length} 0 0" rpy="0 0 0"/>
 			<parent link="${name}_upperleg"/>
 			<child  link="${name}_lowerleg"/>
 			<axis xyz="0 0 1"/>
-			<limit effort="150.0" velocity="12.0"
-				   lower="${-(1+reflect_front)*7*PI/18+(1-reflect_front)*PI/18}"
-				   upper="${(1-reflect_front)*7*PI/18-(1+reflect_front)*PI/18}"/>
+			<limit effort="${kfe_limit}" velocity="12.0"
+                  lower="${(1-knee_bent_backward)*(kfe_min)*PI/180 + (knee_bent_backward)*(-kfe_max)*PI/180}"
+                  upper="${(1-knee_bent_backward)*(kfe_max)*PI/180 + (knee_bent_backward)*(-kfe_min)*PI/180}"/>
 			<dynamics damping="0.1" friction="0" />
-			<safety_controller k_position="100" k_velocity="100"
-							   soft_lower_limit="${-(1+reflect_front)*7*PI/18+(1-reflect_front)*PI/18}"
-							   soft_upper_limit="${(1-reflect_front)*7*PI/18-(1+reflect_front)*PI/18}" />
+			<safety_controller k_position="50" k_velocity="10"
+                  soft_lower_limit="${(1-knee_bent_backward)*(kfe_min)*PI/180 + (knee_bent_backward)*(-kfe_max)*PI/180}"
+                  soft_upper_limit="${(1-knee_bent_backward)*(kfe_max)*PI/180 + (knee_bent_backward)*(-kfe_min)*PI/180}"/>
 		<!-- Foot joint -->
 		</joint>
 		<joint name="${name}_foot_joint" type="fixed">
-			<origin xyz="${d_p2p3} 0 0" rpy="${PI/2} 0 ${-PI/2}"/>
+			<origin xyz="${lowerleg_length} 0 0" rpy="${PI/2} 0 ${-PI/2}"/>
 			<parent link="${name}_lowerleg"/>
 			<child  link="${name}_foot"/>
@@ -113,6 +113,7 @@
 			</visual>
 			<collision>
+			    <origin xyz="${lowerleg_length/2.0} 0 0" rpy="0 ${-PI/2}  0"/>
 				<geometry>
-					<mesh filename="package://hyq_description/meshes/leg/lowerleg.dae" scale="1 1 1"/>
+					<cylinder length="${lowerleg_length}"  radius="0.02"/>
 				</geometry>
 			</collision>
