Commit message: Add arm for hyq [skip ci]

File: robots/hyq.srdf.xacro (robot description, xacro)
@@ -1,4 +1,53 @@
 <?xml version="1.0" ?>
 <robot name="hyq" xmlns:xacro="http://ros.org/wiki/xacro">
+<xacro:arg name="arm" default="false"/>
+<xacro:if value="$(arg arm)">
+  <group name="base">
+    <link name="base_link"/>
+    <link name="teleop_link0"/>
+  </group>
+  <group name="arm">
+       <chain base_link="teleop_link0" tip_link="TCP"/>
+  </group>
+  <group name="lf">
+    <chain base_link="trunk" tip_link="lf_foot"/>
+  </group>
+  <group name="rf">
+    <chain base_link="trunk" tip_link="rf_foot"/>
+  </group>
+  <group name="lh">
+    <chain base_link="trunk" tip_link="lh_foot"/>
+  </group>
+  <group name="rh">
+    <chain base_link="trunk" tip_link="rh_foot"/>
+  </group>
+  <group name="chains">
+    <group name="lf"/>
+    <group name="rf"/>
+    <group name="lh"/>
+    <group name="rh"/>
+    <group name="arm"/>
+  </group>
+  <group_state group="chains" name="home">
+    <joint name="lf_haa_joint" value="-0.2"/>
+    <joint name="lf_hfe_joint" value="0.75"/>
+    <joint name="lf_kfe_joint" value="-1.5"/>
+    <joint name="rf_haa_joint" value="-0.2"/>
+    <joint name="rf_hfe_joint" value="0.75"/>
+    <joint name="rf_kfe_joint" value="-1.5"/>
+    <joint name="lh_haa_joint" value="-0.2"/>
+    <joint name="lh_hfe_joint" value="-0.75"/>
+    <joint name="lh_kfe_joint" value="1.5"/>
+    <joint name="rh_haa_joint" value="-0.2"/>
+    <joint name="rh_hfe_joint" value="-0.75"/>
+    <joint name="rh_kfe_joint" value="1.5"/>
+    <joint name="joint1" value="0.0"/>
+    <joint name="joint2" value="1.0"/>
+    <joint name="joint3" value="1.0"/>
+    <joint name="joint4" value="0.0"/>
+    <joint name="joint5" value="0.0"/>
+  </group_state>
+</xacro:if>
+<xacro:unless value="$(arg arm)">
   <group name="base">
     <link name="base_link"/>
@@ -36,3 +85,4 @@
     <joint name="rh_kfe_joint" value="1.5"/>
   </group_state>
+</xacro:unless>
 </robot>

File: robots/hyq.urdf.xacro (robot description, xacro)
@@ -1,6 +1,7 @@
 <?xml version="1.0"?>
 <robot name="hyq" xmlns:xacro="http://ros.org/wiki/xacro">
-<xacro:arg name="task_period" default="0.004"/>
-<xacro:arg name="sensors" default="true"/>
+	<xacro:arg name="task_period" default="0.004"/>
+	<xacro:arg name="sensors" default="true"/>
+	<xacro:arg name="arm" default="false"/>
 	<!-- This argument allows us to load joint sensors that measure the internal wrenches -->
 	<xacro:arg name="load_force_sensors" default="false"/>
@@ -82,4 +83,19 @@
 		<origin xyz="${-d_fh/2} ${-d_lr/2} 0" rpy="0 ${PI/2} 0"/>
 	</xacro:hyq_leg>
+<xacro:if value="$(arg arm)">
+	<joint name="joint_base_robots" type="fixed">
+	    	<parent link="base_link"/>
+	    	<child link="teleop_link0"/>
+   	 	<origin xyz="0.59 0 0" rpy="0 0 0"/>
+    	</joint>
+	<!-- SELECTION OF KINEMATICS CHAINS IS HANDLED INSIDE THE FILES -->
+	<xacro:include filename="$(find teleop_urdf)/urdf/teleop.urdf.xacro" />
+        <xacro:include filename="$(find hyq_description)/urdfs/arm/arm.transmission.xacro"/>
+        <xacro:arm_transmission name="joint1"/>
+        <xacro:arm_transmission name="joint2"/>
+        <xacro:arm_transmission name="joint3"/>
+        <xacro:arm_transmission name="joint4"/>
+        <xacro:arm_transmission name="joint5"/>
+</xacro:if>
 <xacro:if value="$(arg sensors)">
 	<!-- IMU trunk -->
