Commit message: Improved the position of the bumblebee mount link. Improved the transformation between tilted frame and ptu mount frame.

File: robots/hyq.urdf.xacro (robot description, xacro)
@@ -105,5 +105,5 @@
 	<xacro:bumblebee_97
 		parent_link="ptu_mount_link"
-		xyz="0 0 0.018"
+		xyz="0 0 0"
 		rpy="0 0 0"
 		ns="bumblebee"

File: urdfs/sensors/bumblebee.urdf.xacro (robot description, xacro)
@@ -14,9 +14,9 @@
 			<child link="${frame_prefix}optical_frame"/>
 			<!--<origin xyz="0 0 0" rpy="0 0 0"/>-->
-			<origin xyz="0 -0.06 0" rpy="-${PI/2} 0 -${PI/2}"/>
+			<origin xyz="0 -0.06 0.018" rpy="-${PI/2} 0 -${PI/2}"/>
 		</joint>
 		<link name="${frame_prefix}mount_link">
 			<visual>
-				<origin xyz="0 0 0" rpy="${PI/2} 0 ${PI/2}"/>
+				<origin xyz="0 0 0.018" rpy="${PI/2} 0 ${PI/2}"/>
 				<geometry>
 					<mesh filename="package://hyq_description/meshes/sensors/bumblebee.dae"/>
@@ -24,5 +24,5 @@
 			</visual>
 			<collision>
-				<origin xyz="0 0 0" rpy="${PI/2} 0 ${PI/2}"/>
+				<origin xyz="0 0 0.018" rpy="${PI/2} 0 ${PI/2}"/>
 				<geometry>
 					<mesh filename="package://hyq_description/meshes/sensors/bumblebee.dae"/>

File: urdfs/sensors/ptu_d46.urdf.xacro (robot description, xacro)
@@ -86,5 +86,5 @@
 		<!-- Fixed joint to provide a convenient attachment point for accessories. -->
 		<joint name="${name}_mount" type="fixed">
-			<origin xyz="0 0 -0.03912" rpy="${PI} 0 0"/>
+			<origin xyz="0 0 -0.039116" rpy="${PI} 0 0"/>
 			<parent link="${name}_tilted_link"/>
 			<child link="${name}_mount_link"/>

Commit message: Changed the values of the PTU transforms

File: robots/hyq.urdf.xacro (robot description, xacro)
@@ -85,5 +85,6 @@
 		name="ptu"
 		parent="trunk">
-		<origin xyz="0.657353 0.015447 0.119533" rpy="-0.013127 0.569257 -0.007748"/>
+		<origin xyz="0.677 0.004 0.111" rpy="0.011 0.485 0.015"/>
+<!--		<origin xyz="0.657353 0.015447 0.119533" rpy="-0.013127 0.569257 -0.007748"/>-->
 <!--		<origin xyz="0.667353 -0.010101 0.160544" rpy="0.043239 0.569257 0.041771"/>-->
 	</xacro:ptu_d46>

File: urdfs/sensors/ptu_d46.urdf.xacro (robot description, xacro)
@@ -64,5 +64,5 @@
         	 the overall device, which is between the mounting screws on its base. -->
 		<joint name="${name}_base" type="fixed">
-			<origin xyz="0 -0.011 0.022" rpy="0 0 0"/>
+			<origin xyz="0 -0.0127254 0.022" rpy="0 0 0"/>
 			<parent link="${name}_base_link"/>
 			<child link="${name}_pan_link"/>
@@ -78,5 +78,5 @@
 		<!-- The tilt joint -->
 		<joint name="${name}_tilt" type="revolute">
-			<origin xyz="0 0 0" rpy="-${PI/2} 0 0"/>
+			<origin xyz="0 -0.002424 0" rpy="-${PI/2} 0 0"/>
 			<parent link="${name}_tilt_link"/>
 			<child link="${name}_tilted_link"/>

Commit message: Update xacro file to remove useless links. This provides a minimalistic version of hyq urdf which is easier to use for the identification of the inertial parameters of the robot.

File: robots/hyq.urdf.xacro (robot description, xacro)
@@ -9,10 +9,4 @@
 	<!-- HyQ sensors -->
 	<xacro:include filename="$(find hyq_description)/urdfs/sensors/microstrain_3dmgx325_imu.urdf.xacro"/>
-	<xacro:include filename="$(find hyq_description)/urdfs/sensors/asus_xtion.urdf.xacro"/>
-	<xacro:include filename="$(find hyq_description)/urdfs/sensors/velodyne.urdf.xacro"/>
-	<xacro:include filename="$(find hyq_description)/urdfs/sensors/kinect.urdf.xacro"/>
-	<xacro:include filename="$(find hyq_description)/urdfs/sensors/ptu_d46.urdf.xacro"/>
-	<xacro:include filename="$(find hyq_description)/urdfs/sensors/bumblebee.urdf.xacro"/>
-	<xacro:include filename="$(find hyq_description)/urdfs/sensors/vislab_3dve.urdf.xacro"/>
 	<!-- generic simulator_gazebo plugins for starting mechanism control, ros time -->
 	<xacro:include filename="$(find hyq_description)/gazebo/gazebo.urdf.xacro"/>
@@ -75,44 +69,3 @@
 		<origin xyz="0.3 0 0.095" rpy="0 ${-PI} 0"/>
 	</xacro:microstrain_3dmgx325_imu>
-	<!-- Velodyne -->
-	<xacro:velodyne
-		name="trunk_mount"
-		parent="trunk">
-		<origin xyz="0.39 0 0.269" rpy="0 0 0"/>
-	</xacro:velodyne>
-	<!-- PTU unit -->
-	<xacro:ptu_d46
-		name="ptu"
-		parent="trunk">
-		<origin xyz="0.657353 0.015447 0.119533" rpy="-0.013127 0.569257 -0.007748"/>
-<!--		<origin xyz="0.667353 -0.010101 0.160544" rpy="0.043239 0.569257 0.041771"/>-->
-	</xacro:ptu_d46>
-	<!-- Asus Xtion Pro -->
-	<!--<origin xyz="0 0.005 0.036" rpy="0 0 0"/> with Bumblebee setup -->
-	<!--<origin xyz="0 0 0.04397" rpy="0 0 0"/> with Vislab setup -->
-	<xacro:asus_xtion_camera
-		name="head_mount"
-		parent="ptu_mount_link">
-		<origin xyz="0 0.005 0.036" rpy="0 0 0"/>
-	</xacro:asus_xtion_camera>
-	<!-- Kinect --> <!-- is no more used, but we keep it for compatibilty -->
-	<!--xacro:kinect_camera
-		name="head_mount"
-		parent="trunk">
-		<origin xyz="0.63 0 0.095" rpy="0 0 0"/>
-	</xacro:kinect_camera-->
-	<!-- Bumblebee -->
-	<xacro:bumblebee_97
-		parent_link="ptu_mount_link"
-		xyz="0 0 0.018"
-		rpy="0 0 0"
-		ns="bumblebee"
-		frame_prefix="bumblebee_"
-		high_res="false"/>
-<!--	<xacro:vislab_3dve_72
-		name="vislab_3dve"
-		parent="ptu_mount_link"
-		xyz="0 0 0.025"
-		rpy="0 0 0"
-		high_res="false"/>-->
 </robot>

Commit message: Reintroduced setup for velodyne and added Hokuyo
Conflicts:
	meshes/trunk/trunk.dae

File: robots/hyq.urdf.xacro (robot description, xacro)
@@ -15,4 +15,5 @@
 	<xacro:include filename="$(find hyq_description)/urdfs/sensors/bumblebee.urdf.xacro"/>
 	<xacro:include filename="$(find hyq_description)/urdfs/sensors/vislab_3dve.urdf.xacro"/>
+	<xacro:include filename="$(find hyq_description)/urdfs/sensors/hokuyo_laser.urdf.xacro"/>
 	<!-- generic simulator_gazebo plugins for starting mechanism control, ros time -->
 	<xacro:include filename="$(find hyq_description)/gazebo/gazebo.urdf.xacro"/>
@@ -69,5 +70,5 @@
 	<xacro:microstrain_3dmgx325_imu
 		parent="trunk"
-		imu_name="3dmgx325_trunk_imu"
+		imu_name="imu"
 		imu_topic="trunk_imu/data"
 		update_rate="1000"
@@ -84,8 +85,36 @@
 	<!-- Velodyne -->
 	<xacro:velodyne
-		name="trunk_mount"
+		name="velodyne"
 		parent="trunk">
-		<origin xyz="0.39 0 0.269" rpy="0 0 0"/>
+		<!--origin xyz="0.39 0 0.269" rpy="0 0 3.14"/-->
+		<!--origin xyz="0.39 0.0 0.269" rpy="0 0.0 3.10"/-->
+		<origin xyz="0.39 0.0 0.271" rpy="0.0084 -0.0169 3.14371"/>
 	</xacro:velodyne>
+	<!-- Hokuyo -->
+	<xacro:hokuyo_laser
+		name="laser"
+		parent="trunk"
+		ros_topic="scan"
+		update_rate="10"
+		min_angle="-5"
+		max_angle="5"
+		range="4.0">
+	<origin xyz="0.475 0.0 -0.08823" rpy="3.14 0.0 0"/>
+    <!--origin xyz="0 -${0.5*INCH_TO_M} ${7*INCH_TO_M}" rpy="${M_PI/2} ${M_PI/2} 0" /-->
+	</xacro:hokuyo_laser>
+		<!-- Hokuyo -->
+	<!--xacro:hokuyo_utm30lx
+		name="laser"
+		parent="trunk"
+		ros_topic="scan"
+		update_rate="10"
+		ray_count="1"
+		min_angle="-5"
+		max_angle="5">
+		<origin xyz="0.475 0.0 -0.133" rpy="3.14 0.0 0"/>
+	</xacro:hokuyo_utm30lx-->
+	<!--xacro:hokuyo_mount name="nav_hokuyo" parent="front_left_vertical_beam" length="${SENSOR_BEAM_LENGTH*INCH_TO_M}" ros_topic="scan" update_rate="10" min_angle="${-(5 * M_PI)/12}" max_angle="${(5 * M_PI)/12}" range="4.0">
+    <origin xyz="0 -${0.5*INCH_TO_M} ${7*INCH_TO_M}" rpy="${M_PI/2} ${M_PI/2} 0" />
+  </xacro:hokuyo_mount-->
 	<!-- PTU unit -->
 	<xacro:ptu_d46
@@ -99,5 +128,5 @@
 	<!--<origin xyz="0 0 0.04397" rpy="0 0 0"/> with Vislab setup -->
 	<xacro:asus_xtion_camera
-		name="head_mount"
+		name="asus"
 		parent="ptu_mount_link">
 		<origin xyz="0 0.005 0.036" rpy="0 0 0"/>

Commit message: Reintroduced setup for velodyne and added Hokuyo
Conflicts:
	meshes/trunk/trunk.dae

File: robots/hyq.urdf.xacro (robot description, xacro)
@@ -15,4 +15,5 @@
 	<xacro:include filename="$(find hyq_description)/urdfs/sensors/bumblebee.urdf.xacro"/>
 	<xacro:include filename="$(find hyq_description)/urdfs/sensors/vislab_3dve.urdf.xacro"/>
+	<xacro:include filename="$(find hyq_description)/urdfs/sensors/hokuyo_laser.urdf.xacro"/>
 	<!-- generic simulator_gazebo plugins for starting mechanism control, ros time -->
 	<xacro:include filename="$(find hyq_description)/gazebo/gazebo.urdf.xacro"/>
@@ -69,5 +70,5 @@
 	<xacro:microstrain_3dmgx325_imu
 		parent="trunk"
-		imu_name="3dmgx325_trunk_imu"
+		imu_name="imu"
 		imu_topic="trunk_imu/data"
 		update_rate="100.0"
@@ -77,8 +78,36 @@
 	<!-- Velodyne -->
 	<xacro:velodyne
-		name="trunk_mount"
+		name="velodyne"
 		parent="trunk">
-		<origin xyz="0.39 0 0.269" rpy="0 0 0"/>
+		<!--origin xyz="0.39 0 0.269" rpy="0 0 3.14"/-->
+		<!--origin xyz="0.39 0.0 0.269" rpy="0 0.0 3.10"/-->
+		<origin xyz="0.39 0.0 0.271" rpy="0.0084 -0.0169 3.14371"/>
 	</xacro:velodyne>
+	<!-- Hokuyo -->
+	<xacro:hokuyo_laser
+		name="laser"
+		parent="trunk"
+		ros_topic="scan"
+		update_rate="10"
+		min_angle="-5"
+		max_angle="5"
+		range="4.0">
+	<origin xyz="0.475 0.0 -0.08823" rpy="3.14 0.0 0"/>
+    <!--origin xyz="0 -${0.5*INCH_TO_M} ${7*INCH_TO_M}" rpy="${M_PI/2} ${M_PI/2} 0" /-->
+	</xacro:hokuyo_laser>
+		<!-- Hokuyo -->
+	<!--xacro:hokuyo_utm30lx
+		name="laser"
+		parent="trunk"
+		ros_topic="scan"
+		update_rate="10"
+		ray_count="1"
+		min_angle="-5"
+		max_angle="5">
+		<origin xyz="0.475 0.0 -0.133" rpy="3.14 0.0 0"/>
+	</xacro:hokuyo_utm30lx-->
+	<!--xacro:hokuyo_mount name="nav_hokuyo" parent="front_left_vertical_beam" length="${SENSOR_BEAM_LENGTH*INCH_TO_M}" ros_topic="scan" update_rate="10" min_angle="${-(5 * M_PI)/12}" max_angle="${(5 * M_PI)/12}" range="4.0">
+    <origin xyz="0 -${0.5*INCH_TO_M} ${7*INCH_TO_M}" rpy="${M_PI/2} ${M_PI/2} 0" />
+  </xacro:hokuyo_mount-->
 	<!-- PTU unit -->
 	<xacro:ptu_d46
@@ -92,5 +121,5 @@
 	<!--<origin xyz="0 0 0.04397" rpy="0 0 0"/> with Vislab setup -->
 	<xacro:asus_xtion_camera
-		name="head_mount"
+		name="asus"
 		parent="ptu_mount_link">
 		<origin xyz="0 0.005 0.036" rpy="0 0 0"/>

File: urdfs/sensors/asus_xtion.urdf.xacro (robot description, xacro)
@@ -9,32 +9,32 @@
 			<insert_block name="origin"/>
 			<parent link="${parent}"/>
-			<child link="${name}_asus_xtion_mount_link"/>
+			<child link="${name}_mount_link"/>
 		</joint>
 		<!-- asus ir sensor physical attachment -->
-		<joint name="${name}_asus_xtion_depth_joint" type="fixed">
+		<!--joint name="${name}_depth_joint" type="fixed">
 			<origin xyz="${asus_xtion_x} ${asus_xtion_depth_y} ${asus_xtion_z}" rpy="0 0 0"/>
-			<parent link="${name}_asus_xtion_mount_link"/>
-			<child link="${name}_asus_xtion_depth_frame"/>
-		</joint>
+			<parent link="${name}_mount_link"/>
+			<child link="${name}_depth_frame"/>
+		</joint-->
 		<!-- asus xtion ir sensor frame -->
-		<joint name="${name}_asus_xtion_depth_optical_frame_joint" type="fixed">
-			<origin xyz="0 0 0"	rpy="${asus_xtion_roll} ${asus_xtion_pitch} ${asus_xtion_yaw}"/>
-			<parent link="${name}_asus_xtion_depth_frame"/>
-			<child link="${name}_asus_xtion_depth_optical_frame"/>
+		<joint name="${name}_depth_optical_frame_joint" type="fixed">
+			<origin xyz="${asus_xtion_x} ${asus_xtion_depth_y} ${asus_xtion_z}"	rpy="${asus_xtion_roll} ${asus_xtion_pitch} ${asus_xtion_yaw}"/>
+			<parent link="${name}_mount_link"/>
+			<child link="${name}_depth_optical_frame"/>
 		</joint>
 		<!-- asus_xtion rgb sensor physical attachment -->
-		<joint name="${name}_asus_xtion_rgb_joint" type="fixed">
+		<!--joint name="${name}_rgb_joint" type="fixed">
 			<origin xyz="${asus_xtion_x} ${asus_xtion_rgb_y} ${asus_xtion_z}" rpy="0 0 0"/>
-			<parent link="${name}_asus_xtion_mount_link"/>
-			<child link="${name}_asus_xtion_rgb_frame"/>
-		</joint>
+			<parent link="${name}_mount_link"/>
+			<child link="${name}_rgb_frame"/>
+		</joint-->
 		<!-- asus xtion rgb sensor frame -->
-		<joint name="${name}_asus_xtion_rgb_optical_frame_joint" type="fixed">
-			<origin xyz="0 0 0"	rpy="${asus_xtion_roll} ${asus_xtion_pitch} ${asus_xtion_yaw}"/>
-			<parent link="${name}_asus_xtion_rgb_frame"/>
-			<child link="${name}_asus_xtion_rgb_optical_frame"/>
+		<joint name="${name}_rgb_optical_frame_joint" type="fixed">
+			<origin xyz="${asus_xtion_x} ${asus_xtion_rgb_y} ${asus_xtion_z}"	rpy="${asus_xtion_roll} ${asus_xtion_pitch} ${asus_xtion_yaw}"/>
+			<parent link="${name}_mount_link"/>
+			<child link="${name}_rgb_optical_frame"/>
 		</joint>
 		<!-- Links -->
-		<link name="${name}_asus_xtion_mount_link">
+		<link name="${name}_mount_link">
 			<inertial>
 				<mass value="0.1"/>
@@ -59,5 +59,5 @@
 		</link>
 		<!-- ir sensor link -->
-		<link name="${name}_asus_xtion_depth_frame">
+		<!--link name="${name}_depth_frame">
 			<inertial>
 				<mass value="0.1" />
@@ -77,9 +77,9 @@
 				</geometry>
 			</collision>
-		</link>
+		</link-->
 		<!-- ir optical sensor link -->
-		<link name="${name}_asus_xtion_depth_optical_frame"/>
+		<link name="${name}_depth_optical_frame"/>
 		<!-- rgb sensor link -->
-		<link name="${name}_asus_xtion_rgb_frame" >
+		<!--link name="${name}_rgb_frame" >
 			<inertial>
 				<mass value="0.1" />
@@ -99,10 +99,10 @@
 				</geometry>
 			</collision>
-		</link>
+		</link-->
 		<!-- rgb optical sensor link -->
-		<link name="${name}_asus_xtion_rgb_optical_frame"/>
+		<link name="${name}_rgb_optical_frame"/>
 	<!-- gazebo extensions -->
-	<xacro:asus_xtion_depth_sensor link_name="${name}_asus_xtion_depth_frame" frame_name="${name}_asus_xtion_depth_optical_frame" camera_name="${name}_asus_xtion" />
-	<xacro:asus_xtion_rgb_sensor link_name="${name}_asus_xtion_rgb_frame" frame_name="${name}_asus_xtion_rgb_optical_frame" camera_name="${name}_asus_xtion" />
+	<!--xacro:asus_xtion_depth_sensor link_name="${name}_depth_frame" frame_name="${name}_depth_optical_frame" camera_name="${name}" /-->
+	<!--xacro:asus_xtion_rgb_sensor link_name="${name}_rgb_frame" frame_name="${name}_rgb_optical_frame" camera_name="${name}" /-->
 	</xacro:macro>
 </root>

File: urdfs/sensors/velodyne.urdf.xacro (robot description, xacro)
@@ -6,17 +6,17 @@
 	<xacro:macro name="velodyne" params="name parent *origin">
 		<!-- Joints -->
-		<joint name="${name}_velodyne_joint" type="fixed">
+		<joint name="${name}_joint" type="fixed">
 			<insert_block name="origin"/>
 			<parent link="${parent}"/>
-			<child link="${name}_velodyne_frame"/>
+			<child link="${name}_mount_link"/>
 		</joint>
 		<!-- velodyne sensor optical frame -->
-		<joint name="${name}_velodyne_optical_frame_joint" type="fixed">
+		<joint name="${name}_optical_frame_joint" type="fixed">
 			<origin xyz="${velodyne_x} ${velodyne_y} ${velodyne_z}" rpy="0.0 0.0 0.0"/>
-			<parent link="${name}_velodyne_frame"/>
-			<child link="${name}_velodyne_optical_frame"/>
+			<parent link="${name}_mount_link"/>
+			<child link="${name}"/>
 		</joint>
 		<!-- Links -->
-		<link name="${name}_velodyne_frame">
+		<link name="${name}_mount_link">
 			<inertial>
 				<mass value="0.1"/>
@@ -41,5 +41,5 @@
 		</link>
 		<!-- rgb optical sensor link -->
-		<link name="${name}_velodyne_optical_frame">
+		<link name="${name}">
 			<inertial>
 				<mass value="0.1"/>
@@ -49,5 +49,5 @@
 		</link>
 		<!-- gazebo extensions -->
-		<xacro:velodyne_sensor link_name="${name}_velodyne_optical_frame" frame_name="${name}_velodyne_frame" lidar_name="${name}_velodyne" />
+		<xacro:velodyne_sensor link_name="${name}_optical_frame" frame_name="${name}_frame" lidar_name="${name}" />
 	</xacro:macro>
 </robot>

Commit message: Upgraded the imu sensor files

File: robots/hyq.urdf.xacro (robot description, xacro)
@@ -71,7 +71,14 @@
 		imu_name="3dmgx325_trunk_imu"
 		imu_topic="trunk_imu/data"
-		update_rate="100.0"
-		stdev="0.00017">
-		<origin xyz="0.3 0 0.095" rpy="0 ${-PI} 0"/>
+		update_rate="1000"
+		rate_mean="0"
+		rate_stddev="2e-4"
+		rate_bias_mean="0.00087"
+		rate_bias_stddev="0.0000008"
+		accel_mean="0"
+		accel_stddev="1.7e-2"
+		accel_bias_mean="0.002"
+		accel_bias_stddev="0.001">
+		<origin xyz="0.4825 0.006 0.0905" rpy="0 ${-PI} 0"/>
 	</xacro:microstrain_3dmgx325_imu>
 	<!-- Velodyne -->
@@ -85,6 +92,5 @@
 		name="ptu"
 		parent="trunk">
-		<origin xyz="0.677 0.004 0.111" rpy="0.011 0.485 0.015"/>
-<!--		<origin xyz="0.657353 0.015447 0.119533" rpy="-0.013127 0.569257 -0.007748"/>-->
+		<origin xyz="0.657353 0.015447 0.119533" rpy="-0.013127 0.569257 -0.007748"/>
 <!--		<origin xyz="0.667353 -0.010101 0.160544" rpy="0.043239 0.569257 0.041771"/>-->
 	</xacro:ptu_d46>
@@ -106,5 +112,5 @@
 	<xacro:bumblebee_97
 		parent_link="ptu_mount_link"
-		xyz="0 0 0"
+		xyz="0 0 0.018"
 		rpy="0 0 0"
 		ns="bumblebee"

File: urdfs/sensors/microstrain_3dmgx325_imu.gazebo.xacro (robot description, xacro)
@@ -1,5 +1,6 @@
 <?xml version="1.0"?>
 <robot xmlns:xacro="http://ros.org/wiki/xacro">
-	<xacro:macro name="microstrain_3dmgx325_imu_sensor" params="imu_name imu_topic update_rate stdev">
+	<xacro:macro name="microstrain_3dmgx325_imu_sensor" params="imu_name imu_topic update_rate
+		rate_mean rate_stddev rate_bias_mean rate_bias_stddev accel_mean accel_stddev accel_bias_mean accel_bias_stddev">
 		<gazebo>
 			<plugin name="${imu_name}_controller" filename="libgazebo_ros_imu.so">
@@ -8,5 +9,5 @@
 				<bodyName>${imu_name}</bodyName>
 				<topicName>${imu_topic}</topicName>
-				<gaussianNoise>${stdev*stdev}</gaussianNoise>
+				<gaussianNoise>${rate_stddev*rate_stddev}</gaussianNoise>
 				<xyzOffset>0 0 0</xyzOffset>
 				<rpyOffset>0 0 0</rpyOffset>
@@ -14,4 +15,28 @@
 			</plugin>
 		</gazebo>
+		<!-- Imu definition required for hardware interface of ros control -->
+		<gazebo reference="${imu_name}">
+			<sensor name="trunk_imu" type="imu">
+				<always_on>1</always_on>
+				<update_rate>${update_rate}</update_rate>
+				<imu>
+					<noise>
+						<type>gaussian</type>
+						<rate>
+							<mean>${rate_mean}</mean>
+							<stddev>${rate_stddev}</stddev>
+							<bias_mean>${rate_bias_mean}</bias_mean>
+							<bias_stddev>${rate_bias_stddev}</bias_stddev>
+						</rate>
+						<accel>
+							<mean>${accel_mean}</mean>
+							<stddev>${accel_stddev}</stddev>
+							<bias_mean>${accel_bias_mean}</bias_mean>
+							<bias_stddev>${accel_bias_stddev}</bias_stddev>
+						</accel>
+					</noise>
+				</imu>
+			</sensor>
+		</gazebo>
 	</xacro:macro>
 </robot>

Commit message: From one of the merging with lost the Stephane last values of PTU and Bumblebee. I updated to the last one, as you can see in the commits 60e8cc280a4c8ea937c2b4e038d3b84f49d6527c and eb34616cefd15f41f3af360e0aea437871d77f7b

File: robots/hyq.urdf.xacro (robot description, xacro)
@@ -121,6 +121,6 @@
 		name="ptu"
 		parent="trunk">
-		<origin xyz="0.657353 0.015447 0.119533" rpy="-0.013127 0.569257 -0.007748"/>
-<!--		<origin xyz="0.667353 -0.010101 0.160544" rpy="0.043239 0.569257 0.041771"/>-->
+		<origin xyz="0.677 0.004 0.111"
+				rpy="-0.013127 0.569257 -0.007748"/>
 	</xacro:ptu_d46>
 	<!-- Asus Xtion Pro -->

File: urdfs/sensors/bumblebee.urdf.xacro (robot description, xacro)
@@ -13,10 +13,9 @@
 			<parent link="${frame_prefix}mount_link"/>
 			<child link="${frame_prefix}optical_frame"/>
-			<!--<origin xyz="0 0 0" rpy="0 0 0"/>-->
-			<origin xyz="0 -0.06 0" rpy="-${PI/2} 0 -${PI/2}"/>
+			<origin xyz="0 -0.06 0.018" rpy="-${PI/2} 0 -${PI/2}"/>
 		</joint>
 		<link name="${frame_prefix}mount_link">
 			<visual>
-				<origin xyz="0 0 0" rpy="${PI/2} 0 ${PI/2}"/>
+				<origin xyz="0 0 0.018" rpy="${PI/2} 0 ${PI/2}"/>
 				<geometry>
 					<mesh filename="package://hyq_description/meshes/sensors/bumblebee.dae"/>
@@ -24,5 +23,5 @@
 			</visual>
 			<collision>
-				<origin xyz="0 0 0" rpy="${PI/2} 0 ${PI/2}"/>
+				<origin xyz="0 0 0.018" rpy="${PI/2} 0 ${PI/2}"/>
 				<geometry>
 					<mesh filename="package://hyq_description/meshes/sensors/bumblebee.dae"/>
@@ -34,5 +33,5 @@
 						 iyy="${1/12*b2mass*(b2lx*b2lx + b2lz*b2lz)}" iyz="0"
 						 izz="${1/12*b2mass*(b2lx*b2lx + b2ly*b2ly)}" />
-				</inertial>
+			</inertial>
 		</link>
 		<link name="${frame_prefix}optical_frame">

File: urdfs/sensors/ptu_d46.urdf.xacro (robot description, xacro)
@@ -64,5 +64,5 @@
         	 the overall device, which is between the mounting screws on its base. -->
 		<joint name="${name}_base" type="fixed">
-			<origin xyz="0 -0.011 0.022" rpy="0 0 0"/>
+			<origin xyz="0 -0.0127254 0.022" rpy="0 0 0"/>
 			<parent link="${name}_base_link"/>
 			<child link="${name}_pan_link"/>
@@ -78,5 +78,5 @@
 		<!-- The tilt joint -->
 		<joint name="${name}_tilt" type="revolute">
-			<origin xyz="0 0 0" rpy="-${PI/2} 0 0"/>
+			<origin xyz="0 -0.002424 0" rpy="-${PI/2} 0 0"/>
 			<parent link="${name}_tilt_link"/>
 			<child link="${name}_tilted_link"/>
@@ -86,5 +86,5 @@
 		<!-- Fixed joint to provide a convenient attachment point for accessories. -->
 		<joint name="${name}_mount" type="fixed">
-			<origin xyz="0 0 -0.03912" rpy="${PI} 0 0"/>
+			<origin xyz="0 0 -0.039116" rpy="${PI} 0 0"/>
 			<parent link="${name}_tilted_link"/>
 			<child link="${name}_mount_link"/>

Commit message: Updated IMU position and model
Updated IMU position and model after mounting plastic support

File: robots/hyq.urdf.xacro (robot description, xacro)
@@ -8,5 +8,5 @@
 	<xacro:include filename="$(find hyq_description)/urdfs/leg/leg.urdf.xacro"/>
 	<!-- HyQ sensors -->
-	<xacro:include filename="$(find hyq_description)/urdfs/sensors/microstrain_3dmgx325_imu.urdf.xacro"/>
+	<xacro:include filename="$(find hyq_description)/urdfs/sensors/microstrain_3dmgx425_imu.urdf.xacro"/>
 	<xacro:include filename="$(find hyq_description)/urdfs/sensors/asus_xtion.urdf.xacro"/>
 	<xacro:include filename="$(find hyq_description)/urdfs/sensors/velodyne.urdf.xacro"/>
@@ -68,9 +68,9 @@
 	</xacro:hyq_leg>
 	<!-- IMU trunk -->
-	<xacro:microstrain_3dmgx325_imu
+	<xacro:microstrain_3dmgx425_imu
 		parent="trunk"
 		imu_name="imu"
 		imu_topic="trunk_imu/data"
-		update_rate="1000"
+		update_rate="250"
 		rate_mean="0"
 		rate_stddev="2e-4"
@@ -81,6 +81,6 @@
 		accel_bias_mean="0.002"
 		accel_bias_stddev="0.001">
-		<origin xyz="0.4825 0.006 0.0905" rpy="0 ${-PI} 0"/>
-	</xacro:microstrain_3dmgx325_imu>
+		<origin xyz="0.290 0.000 0.0999214" rpy="0 ${-PI} 0"/>
+	</xacro:microstrain_3dmgx425_imu>
 	<!-- Velodyne -->
 	<xacro:velodyne
