Commit message: Added the vicon marker to the model

File: robots/hyq.urdf.xacro (robot description, xacro)
@@ -16,4 +16,5 @@
 	<xacro:include filename="$(find hyq_description)/urdfs/sensors/vislab_3dve.urdf.xacro"/>
 	<xacro:include filename="$(find hyq_description)/urdfs/sensors/hokuyo_laser.urdf.xacro"/>
+        <xacro:include filename="$(find hyq_description)/urdfs/sensors/vicon.urdf.xacro" />
 	<!-- generic simulator_gazebo plugins for starting mechanism control, ros time -->
 	<xacro:include filename="$(find hyq_description)/gazebo/gazebo.urdf.xacro"/>
@@ -83,4 +84,8 @@
 		<origin xyz="0.290 0.000 0.0999214" rpy="0 ${-PI} 0"/>
 	</xacro:microstrain_3dmgx425_imu>
+        <!-- See vicon_bridge and Vicon doc to know what subject and segment mean -->
+        <xacro:vicon subject="hyq_green" segment="body" parent="trunk">
+               <origin xyz="0.455864 -0.231012 0.104193" rpy="-1.70031 0.0 -3.00989"/>
+        </xacro:vicon>
 	<!-- Velodyne -->
 	<xacro:velodyne

File: urdfs/sensors/vicon.urdf.xacro (robot description, xacro)
@@ -1,36 +1,27 @@
 <?xml version="1.0"?>
-<robot xmlns:xacro="http://www.ros.org/wiki/xacro">
-	<!-- ======================================= VICON MARKER ====================================== -->
-	<!-- The xacro macro xacro:vicon_marker contains: vicon marker link -->
-	<xacro:macro name="vicon" params="child *origin">
-		<!-- Joints -->
-		<joint name="vicon_maker_joint" type="floating">
-			<insert_block name="origin"/>
-			<parent link="vicon_marker_link"/>
-			<child link="${child}"/>
+<robot xmlns:xacro="http://ros.org/wiki/xacro">
+	<xacro:macro name="vicon" params="subject segment parent *origin">
+		<joint name="${subject}_joint" type="fixed">
+			<axis xyz="0 0 0" />
+			<insert_block name="origin" />
+			<parent link="${parent}"/>
+			<child link="vicon/${subject}/${segment}"/>
 		</joint>
-		<!-- Links -->
-		<link name="vicon_marker_link">
+		<link name="vicon/${subject}/${segment}">
 			<inertial>
-				<mass value="0.001"/>
-				<origin xyz="0 0 0" rpy="0 0 0"/>
-				<inertia ixx="0.01" ixy="0.0" ixz="0.0" iyy="0.01" iyz="0.0" izz="0.01"/>
+				<mass value="0.001" />
+				<origin xyz="0 0 0" rpy="0 0 0" />
+				<inertia ixx="0.0001" ixy="0" ixz="0" iyy="0.000001" iyz="0" izz="0.0001" />
 			</inertial>
 			<visual>
-				<origin xyz="0 0 0" rpy="0 0 0"/>
-				<geometry>
-					<sphere radius="0.005" />
-				</geometry>
-				<material name="gray">
-					<color rgba="0.5 0.5 0.5 1"/>
-				</material>
-			</visual>
-			<collision>
 				<origin xyz="0 0 0" rpy="0 0 0" />
 				<geometry>
-					<sphere radius="0.005" />
+                                    <sphere radius="0.007"/>
 				</geometry>
-			</collision>
+                                <material name="silver">
+                                    <color rgba="0.95 0.95 0.95 1.0"/>
+                                </material>
+			</visual>
 		</link>
-	</xacro:macro>
+        </xacro:macro>
 </robot>

Commit message: Corrected vicon marker. After all, it was better as father of base_link and not vice versa

File: robots/hyq.urdf.xacro (robot description, xacro)
@@ -85,6 +85,8 @@
 	</xacro:microstrain_3dmgx425_imu>
         <!-- See vicon_bridge and Vicon doc to know what subject and segment mean -->
-        <xacro:vicon subject="hyq_green" segment="body" parent="trunk">
-               <origin xyz="0.455864 -0.231012 0.104193" rpy="-1.70031 0.0 -3.00989"/>
+        <xacro:vicon subject="hyq_green" segment="body" target_frame="base_link">
+               <!--origin xyz="0.455864 -0.231012 0.104193" rpy="-1.70031 0.0 -3.00989"/-->
+               <!--origin xyz="0.455864 -0.231012 0.104193" rpy="${PI/2} ${-PI/2} 0.0"/-->
+<origin xyz="-0.104392 0.454994 -0.23086" rpy="-1.57252 -0.00346852 -1.57112"/>
         </xacro:vicon>
 	<!-- Velodyne -->

File: urdfs/sensors/vicon.urdf.xacro (robot description, xacro)
@@ -1,17 +1,12 @@
 <?xml version="1.0"?>
 <robot xmlns:xacro="http://ros.org/wiki/xacro">
-	<xacro:macro name="vicon" params="subject segment parent *origin">
+	<xacro:macro name="vicon" params="subject segment target_frame *origin">
 		<joint name="${subject}_joint" type="fixed">
 			<axis xyz="0 0 0" />
 			<insert_block name="origin" />
-			<parent link="${parent}"/>
-			<child link="vicon/${subject}/${segment}"/>
+			<parent link="vicon/${subject}/${segment}"/>
+			<child link="${target_frame}"/>
 		</joint>
 		<link name="vicon/${subject}/${segment}">
-			<inertial>
-				<mass value="0.001" />
-				<origin xyz="0 0 0" rpy="0 0 0" />
-				<inertia ixx="0.0001" ixy="0" ixz="0" iyy="0.000001" iyz="0" izz="0.0001" />
-			</inertial>
 			<visual>
 				<origin xyz="0 0 0" rpy="0 0 0" />

Commit message: hyq teraranger addition

File: robots/hyq.urdf.xacro (robot description, xacro)
@@ -16,4 +16,5 @@
 	<xacro:include filename="$(find hyq_description)/urdfs/sensors/vislab_3dve.urdf.xacro"/>
 	<xacro:include filename="$(find hyq_description)/urdfs/sensors/hokuyo_laser.urdf.xacro"/>
+	<xacro:include filename="$(find hyq_description)/urdfs/sensors/teraranger_range.urdf.xacro"/>
 	<!-- generic simulator_gazebo plugins for starting mechanism control, ros time -->
 	<xacro:include filename="$(find hyq_description)/gazebo/gazebo.urdf.xacro"/>
@@ -84,23 +85,33 @@
 	</xacro:microstrain_3dmgx425_imu>
 	<!-- Velodyne -->
+	<!--
 	<xacro:velodyne
 		name="velodyne"
 		parent="trunk">
-		<!--origin xyz="0.39 0 0.269" rpy="0 0 3.14"/-->
-		<!--origin xyz="0.39 0.0 0.269" rpy="0 0.0 3.10"/-->
 		<origin xyz="0.39 0.0 0.271" rpy="0.0084 -0.0169 3.14371"/>
 	</xacro:velodyne>
+	-->
+	<!--origin xyz="0.39 0 0.269" rpy="0 0 3.14"/-->
+	<!--origin xyz="0.39 0.0 0.269" rpy="0 0.0 3.10"/-->
 	<!-- Hokuyo -->
 	<xacro:hokuyo_laser
 		name="laser"
-		parent="trunk"
+		parent="rf_lowerleg"
 		ros_topic="scan"
-		update_rate="10"
+		update_rate="100"
 		min_angle="-5"
 		max_angle="5"
 		range="4.0">
-	<origin xyz="0.475 0.0 -0.08823" rpy="3.14 0.0 0"/>
-    <!--origin xyz="0 -${0.5*INCH_TO_M} ${7*INCH_TO_M}" rpy="${M_PI/2} ${M_PI/2} 0" /-->
+		<origin xyz="0.12 0.0 0.0" rpy = "${PI/2} 0.0 0.0"/>
 	</xacro:hokuyo_laser>
+	<!-- teraranger -->
+    <xacro:teraranger_range
+		name="ranger"
+		parent="rf_lowerleg"
+		ros_topic="terarange"
+		update_rate="250"
+		range="4.0">
+		<origin xyz="0.12 0.0 0.0" rpy = "${PI/2} 0.0 0.0"/>
+	</xacro:teraranger_range>
 		<!-- Hokuyo -->
 	<!--xacro:hokuyo_utm30lx
@@ -114,4 +125,6 @@
 		<origin xyz="0.475 0.0 -0.133" rpy="3.14 0.0 0"/>
 	</xacro:hokuyo_utm30lx-->
+	<!-- <origin xyz="0.475 0.0 -0.08823" rpy="3.14 0.0 0"/>  -->
+    <!--origin xyz="0 -${0.5*INCH_TO_M} ${7*INCH_TO_M}" rpy="${M_PI/2} ${M_PI/2} 0" /-->
 	<!--xacro:hokuyo_mount name="nav_hokuyo" parent="front_left_vertical_beam" length="${SENSOR_BEAM_LENGTH*INCH_TO_M}" ros_topic="scan" update_rate="10" min_angle="${-(5 * M_PI)/12}" max_angle="${(5 * M_PI)/12}" range="4.0">
     <origin xyz="0 -${0.5*INCH_TO_M} ${7*INCH_TO_M}" rpy="${M_PI/2} ${M_PI/2} 0" />

File: urdfs/sensors/hokuyo_laser.gazebo.xacro (robot description, xacro)
@@ -1,28 +1,28 @@
 <?xml version="1.0"?>
 <root xmlns:xacro="http://ros.org/wiki/xacro">
-	<xacro:macro name="velodyne_sensor" params="link_name frame_name lidar_name">
+	<xacro:macro name="hokuyo_laser_gazebo" params="link_name frame_name ros_topic update_rate min_angle max_angle range">
 		<gazebo reference="${link_name}">
-			<sensor name="${link_name}_velodyne_sensor" type="ray">
+			<sensor name="${link_name}_laser_sensor" type="ray">
 				<always_on>true</always_on>
-				<update_rate>1.0</update_rate>
+				<update_rate>${update_rate}</update_rate>
 				<pose>0 0 0 0 0 0</pose>
 				<ray>
 					<scan>
 						<horizontal>
-							<samples>300</samples>
+							<samples>2</samples>
 							<resolution>1</resolution>
-							<min_angle>${-PI}</min_angle>
-							<max_angle>${PI}</max_angle>
+							<min_angle>${-1 * PI / 180}</min_angle>
+							<max_angle>${1 * PI / 180}</max_angle>
 						</horizontal>
 						<vertical>
-							<samples>32</samples>
+							<samples>2</samples>
 							<resolution>1</resolution>
-							<min_angle>${-30.67*PI/180}</min_angle>
-							<max_angle>${10.67*PI/180}</max_angle>
+							<min_angle>${-1*PI/180}</min_angle>
+							<max_angle>${1*PI/180}</max_angle>
 						</vertical>
 					</scan>
 					<range>
-						<min>1.0</min>
-						<max>20.0</max>
+						<min>0.2</min>
+						<max>${range}</max>
 						<resolution>0.02</resolution>
 					</range>
@@ -32,6 +32,6 @@
 					<gaussianNoise>0.005</gaussianNoise>
 					<alwaysOn>true</alwaysOn>
-					<updateRate>10</updateRate>
-					<topicName>/${lidar_name}/velodyne_pointcloud</topicName>
+					<updateRate>${update_rate}</updateRate>
+					<topicName>/${ros_topic}</topicName>
 					<frameName>${frame_name}</frameName>
 					<hokuyoMinIntensity>101</hokuyoMinIntensity>

File: urdfs/sensors/teraranger_range.gazebo.xacro (robot description, xacro)
@@ -1,37 +1,37 @@
 <?xml version="1.0"?>
 <root xmlns:xacro="http://ros.org/wiki/xacro">
-	<xacro:macro name="velodyne_sensor" params="link_name frame_name lidar_name">
+	<xacro:macro name="teraranger_range_gazebo" params="link_name frame_name ros_topic update_rate range">
 		<gazebo reference="${link_name}">
-			<sensor name="${link_name}_velodyne_sensor" type="ray">
+			<sensor name="${link_name}_sensor" type="ray">
 				<always_on>true</always_on>
-				<update_rate>1.0</update_rate>
+				<update_rate>${update_rate}</update_rate>
 				<pose>0 0 0 0 0 0</pose>
 				<ray>
 					<scan>
 						<horizontal>
-							<samples>300</samples>
+							<samples>2</samples>
 							<resolution>1</resolution>
-							<min_angle>${-PI}</min_angle>
-							<max_angle>${PI}</max_angle>
+							<min_angle>${-1 * PI / 180}</min_angle>
+							<max_angle>${1 * PI / 180}</max_angle>
 						</horizontal>
 						<vertical>
-							<samples>32</samples>
+							<samples>2</samples>
 							<resolution>1</resolution>
-							<min_angle>${-30.67*PI/180}</min_angle>
-							<max_angle>${10.67*PI/180}</max_angle>
+							<min_angle>${-1*PI/180}</min_angle>
+							<max_angle>${1*PI/180}</max_angle>
 						</vertical>
 					</scan>
 					<range>
-						<min>1.0</min>
-						<max>20.0</max>
+						<min>0.2</min>
+						<max>${range}</max>
 						<resolution>0.02</resolution>
 					</range>
 				</ray>
 				<!-- test plugin -->
-				<plugin name="${link_name}_controller" filename="libgazebo_ros_block_laser.so">
+				<plugin name="${link_name}_controller" filename="libgazebo_ros_range.so">
 					<gaussianNoise>0.005</gaussianNoise>
 					<alwaysOn>true</alwaysOn>
-					<updateRate>10</updateRate>
-					<topicName>/${lidar_name}/velodyne_pointcloud</topicName>
+					<updateRate>${update_rate}</updateRate>
+					<topicName>/${ros_topic}</topicName>
 					<frameName>${frame_name}</frameName>
 					<hokuyoMinIntensity>101</hokuyoMinIntensity>

File: urdfs/sensors/teraranger_range.urdf.xacro (robot description, xacro)
@@ -2,6 +2,6 @@
 <robot xmlns:xacro="http://ros.org/wiki/xacro">
 	<!-- dima -->
-	<xacro:include filename="$(find hyq_description)/urdfs/sensors/hokuyo_laser.gazebo.xacro" />
-	<xacro:macro name="hokuyo_laser" params="name parent *origin ros_topic update_rate min_angle max_angle range">
+	<xacro:include filename="$(find hyq_description)/urdfs/sensors/teraranger_range.gazebo.xacro" />
+	<xacro:macro name="teraranger_range" params="name parent *origin ros_topic update_rate range">
 		<joint name="${name}_joint" type="fixed">
 			<axis xyz="0 0 0" />
@@ -38,5 +38,5 @@
 		</link>
 		<!-- gazebo extensions -->
-		<xacro:hokuyo_laser_gazebo link_name="${name}" frame_name="${name}" ros_topic="${ros_topic}" update_rate="${update_rate}" min_angle="${min_angle}" max_angle="${max_angle}" range="${range}"/>
+		<xacro:teraranger_range_gazebo link_name="${name}" frame_name="${name}" ros_topic="${ros_topic}" update_rate="${update_rate}" range="${range}"/>
     </xacro:macro>
 </robot>

Commit message: First introduction of the multisense

File: robots/hyq.urdf.xacro (robot description, xacro)
@@ -17,4 +17,5 @@
 	<xacro:include filename="$(find hyq_description)/urdfs/sensors/vislab_3dve.urdf.xacro"/>
 	<xacro:include filename="$(find hyq_description)/urdfs/sensors/hokuyo_laser.urdf.xacro"/>
+        <xacro:include filename="$(find hyq_description)/urdfs/sensors/multisense_sl.urdf.xacro" />
 	<!-- generic simulator_gazebo plugins for starting mechanism control, ros time -->
 	<xacro:include filename="$(find hyq_description)/gazebo/gazebo.urdf.xacro"/>
@@ -85,11 +86,4 @@
 	</xacro:microstrain_3dmgx425_imu>
 	<!-- Velodyne -->
-	<xacro:velodyne
-		name="velodyne"
-		parent="trunk">
-		<!--origin xyz="0.39 0 0.269" rpy="0 0 3.14"/-->
-		<!--origin xyz="0.39 0.0 0.269" rpy="0 0.0 3.10"/-->
-		<origin xyz="0.39 0.0 0.271" rpy="0.0084 -0.0169 3.14371"/>
-	</xacro:velodyne>
 	<!-- Hokuyo -->
 	<xacro:hokuyo_laser
@@ -102,54 +96,10 @@
 		range="4.0">
 	<origin xyz="0.475 0.0 -0.08823" rpy="3.14 0.0 0"/>
-    <!--origin xyz="0 -${0.5*INCH_TO_M} ${7*INCH_TO_M}" rpy="${M_PI/2} ${M_PI/2} 0" /-->
 	</xacro:hokuyo_laser>
-		<!-- Hokuyo -->
-	<!--xacro:hokuyo_utm30lx
-		name="laser"
-		parent="trunk"
-		ros_topic="scan"
-		update_rate="10"
-		ray_count="1"
-		min_angle="-5"
-		max_angle="5">
-		<origin xyz="0.475 0.0 -0.133" rpy="3.14 0.0 0"/>
-	</xacro:hokuyo_utm30lx-->
-	<!--xacro:hokuyo_mount name="nav_hokuyo" parent="front_left_vertical_beam" length="${SENSOR_BEAM_LENGTH*INCH_TO_M}" ros_topic="scan" update_rate="10" min_angle="${-(5 * M_PI)/12}" max_angle="${(5 * M_PI)/12}" range="4.0">
-    <origin xyz="0 -${0.5*INCH_TO_M} ${7*INCH_TO_M}" rpy="${M_PI/2} ${M_PI/2} 0" />
-  </xacro:hokuyo_mount-->
-	<!-- PTU unit -->
-	<xacro:ptu_d46
-		name="ptu"
-		parent="trunk">
-		<origin xyz="0.677 0.004 0.111"
-				rpy="-0.013127 0.569257 -0.007748"/>
-	</xacro:ptu_d46>
+        <xacro:multisense_sl parent="trunk">
+                <origin xyz="0.741737 0.0191395 0.143229" rpy="-0.0241345 0.446222 -0.0347202"/>
+        </xacro:multisense_sl>
 	<!-- Asus Xtion Pro -->
 	<!--<origin xyz="0 0.005 0.036" rpy="0 0 0"/> with Bumblebee setup -->
 	<!--<origin xyz="0 0 0.04397" rpy="0 0 0"/> with Vislab setup -->
-	<xacro:asus_xtion_camera
-		name="asus"
-		parent="ptu_mount_link">
-		<origin xyz="0 0.005 0.036" rpy="0 0 0"/>
-	</xacro:asus_xtion_camera>
-	<!-- Kinect --> <!-- is no more used, but we keep it for compatibilty -->
-	<!--xacro:kinect_camera
-		name="head_mount"
-		parent="trunk">
-		<origin xyz="0.63 0 0.095" rpy="0 0 0"/>
-	</xacro:kinect_camera-->
-	<!-- Bumblebee -->
-	<xacro:bumblebee_97
-		parent_link="ptu_mount_link"
-                xyz= "0 0 0"
-		rpy="0 0 0"
-		ns="bumblebee"
-		frame_prefix="bumblebee_"
-		high_res="false"/>
-<!--	<xacro:vislab_3dve_72
-		name="vislab_3dve"
-		parent="ptu_mount_link"
-		xyz="0 0 0.025"
-		rpy="0 0 0"
-		high_res="false"/>-->
 </robot>

Commit message: prefix is now parametric for multisense

File: robots/hyq.urdf.xacro (robot description, xacro)
@@ -97,5 +97,5 @@
 	<origin xyz="0.475 0.0 -0.08823" rpy="3.14 0.0 0"/>
 	</xacro:hokuyo_laser>
-        <xacro:multisense_sl parent="trunk">
+        <xacro:multisense_sl parent="trunk" prefix="hyq">
                 <origin xyz="0.741737 0.0191395 0.143229" rpy="-0.0241345 0.446222 -0.0347202"/>
         </xacro:multisense_sl>

File: urdfs/sensors/multisense_sl.urdf.xacro (robot description, xacro)
@@ -1,5 +1,5 @@
 <?xml version="1.0" ?>
 <robot xmlns:xacro="http://ros.org/wiki/xacro">
-<xacro:macro name="multisense_sl" params="parent *origin" >
+<xacro:macro name="multisense_sl" params="parent *origin prefix" >
   <joint name="${parent}_head_root_joint" type="fixed">
     <insert_block name="origin"/>
@@ -36,19 +36,19 @@
   </link>
   <joint name="left_camera_optical_joint" type="continuous">
-    <parent link="left_camera_optical_frame" />
-    <child link="motor" />
+    <parent link="${prefix}/left_camera_optical_frame" />
+    <child link="${prefix}/motor" />
   </joint>
-  <link name="motor"/>
-  <link name="spindle"/>
+  <link name="${prefix}/motor"/>
+  <link name="${prefix}/spindle"/>
   <joint name="motor_joint" type="continuous">
-    <parent link="motor" />
-    <child link="spindle" />
+    <parent link="${prefix}/motor" />
+    <child link="${prefix}/spindle" />
     <axis xyz="0 0 1" />
   </joint>
   <joint name="spindle_joint" type="continuous">
-    <parent link="spindle" />
-    <child link="hokuyo_link" />
+    <parent link="${prefix}/spindle" />
+    <child link="${prefix}/hokuyo_link" />
   </joint>
-  <link name="hokuyo_link">
+  <link name="${prefix}/hokuyo_link">
     <inertial>
       <origin xyz="0.012428 0.0004084 -0.0041835" rpy="0 0 0" />
@@ -72,5 +72,5 @@
   </collision>
   </link>
-  <link name="head_hokuyo_frame"/>
+  <link name="${prefix}/head_hokuyo_frame"/>
   <joint name="head_hokuyo_frame_joint" type="fixed">
     <!--
@@ -81,6 +81,6 @@
      -->
     <origin xyz="0 0 0" rpy="-1.57079632679 -1.57079632679 0.0" />
-    <parent link="hokuyo_link" />
-    <child link="head_hokuyo_frame"/>
+    <parent link="${prefix}/hokuyo_link" />
+    <child link="${prefix}/head_hokuyo_frame"/>
   </joint>
   <!-- Stereo Camera -->
@@ -101,7 +101,7 @@
     <origin xyz="0 0 0" rpy="-1.57079632679 0.0 -1.57079632679" />
     <parent link="left_camera_frame" />
-    <child link="left_camera_optical_frame"/>
+    <child link="${prefix}/left_camera_optical_frame"/>
   </joint>
-  <link name="left_camera_optical_frame"/>
+  <link name="${prefix}/left_camera_optical_frame"/>
   <joint name="right_camera_frame_joint" type="fixed">
     <origin xyz="0.0 -0.035 -0.002"/>

Commit message: added xtion in its new position

File: robots/hyq.urdf.xacro (robot description, xacro)
@@ -103,3 +103,6 @@
 	<!--<origin xyz="0 0.005 0.036" rpy="0 0 0"/> with Bumblebee setup -->
 	<!--<origin xyz="0 0 0.04397" rpy="0 0 0"/> with Vislab setup -->
+<xacro:asus_xtion_camera name="asus" parent="trunk">
+	<origin xyz="0.66489 0.0016545 0.0380496" rpy="0.00740313 0.479116 0.0244919"/>
+</xacro:asus_xtion_camera>
 </robot>
