Commit message: Multisense laser and camera working in sim, still needs a lot of work and testing

File: robots/hyq.urdf.xacro (robot description, xacro)
@@ -17,5 +17,5 @@
 	<xacro:include filename="$(find hyq_description)/urdfs/sensors/vislab_3dve.urdf.xacro"/>
 	<xacro:include filename="$(find hyq_description)/urdfs/sensors/hokuyo_laser.urdf.xacro"/>
-        <xacro:include filename="$(find hyq_description)/urdfs/sensors/multisense_sl.urdf.xacro" />
+	<xacro:include filename="$(find hyq_description)/urdfs/sensors/multisense_sl.urdf.xacro" />
 	<!-- generic simulator_gazebo plugins for starting mechanism control, ros time -->
 	<xacro:include filename="$(find hyq_description)/gazebo/gazebo.urdf.xacro"/>
@@ -97,7 +97,8 @@
 	<origin xyz="0.475 0.0 -0.08823" rpy="3.14 0.0 0"/>
 	</xacro:hokuyo_laser>
-        <xacro:multisense_sl parent="trunk" prefix="hyq">
-                <origin xyz="0.741737 0.0191395 0.143229" rpy="-0.0241345 0.446222 -0.0347202"/>
-        </xacro:multisense_sl>
+    <xacro:multisense_sl parent="trunk" prefix="hyq">
+            <!-- <origin xyz="0.741737 0.0191395 0.143229" rpy="-0.0241345 0.446222 -0.0347202"/> -->
+            <origin xyz="0.741737 0.0 0.143229" rpy="-0.0241345 0.446222 -0.0347202"/>
+    </xacro:multisense_sl>
 	<!-- Asus Xtion Pro -->
 	<!--<origin xyz="0 0.005 0.036" rpy="0 0 0"/> with Bumblebee setup -->

File: urdfs/sensors/multisense_sl.urdf.xacro (robot description, xacro)
@@ -1,4 +1,5 @@
 <?xml version="1.0" ?>
 <robot xmlns:xacro="http://ros.org/wiki/xacro">
+<xacro:include filename="$(find hyq_description)/urdfs/sensors/multisense_sl.gazebo.xacro"/>
 <xacro:macro name="multisense_sl" params="parent *origin prefix" >
   <joint name="${parent}_head_root_joint" type="fixed">
@@ -35,20 +36,27 @@
   </collision>
   </link>
-  <joint name="left_camera_optical_joint" type="continuous">
-    <parent link="${prefix}/left_camera_optical_frame" />
-    <child link="${prefix}/motor" />
-  </joint>
-  <link name="${prefix}/motor"/>
-  <link name="${prefix}/spindle"/>
-  <joint name="motor_joint" type="continuous">
-    <parent link="${prefix}/motor" />
-    <child link="${prefix}/spindle" />
-    <axis xyz="0 0 1" />
-  </joint>
-  <joint name="spindle_joint" type="continuous">
-    <parent link="${prefix}/spindle" />
-    <child link="${prefix}/hokuyo_link" />
-  </joint>
-  <link name="${prefix}/hokuyo_link">
+  <joint name="hokuyo_joint" type="continuous">
+    <origin xyz="-0.0446 0 0.0880" rpy="0 0 0" />
+    <parent link="head" />
+    <child link="hokuyo_link" />
+    <axis xyz="1 0 0" />
+    <dynamics damping="0.01" friction="0"/>
+  </joint>
+  <!-- Hokuyo Laser -->
+  <joint name="head_hokuyo_joint" type="fixed">
+    <axis xyz="0 1 0" />
+    <origin xyz="0.03 0 0.015" rpy="0 0 0"/>
+    <parent link="hokuyo_link"/>
+    <child link="head_hokuyo_frame"/>
+  </joint>
+  <link name="head_hokuyo_frame">
+    <inertial>
+      <mass value="1e-5" />
+      <!-- collocate with parent link and remove mass from it -->
+      <origin xyz="0.042428 0.0004084 0.0108165" rpy="0 0 0"/>
+      <inertia ixx="1e-6" ixy="0" ixz="0" iyy="1e-6" iyz="0" izz="1e-6" />
+    </inertial>
+  </link>
+  <link name="hokuyo_link">
     <inertial>
       <origin xyz="0.012428 0.0004084 -0.0041835" rpy="0 0 0" />
@@ -72,16 +80,4 @@
   </collision>
   </link>
-  <link name="${prefix}/head_hokuyo_frame"/>
-  <joint name="head_hokuyo_frame_joint" type="fixed">
-    <!--
-     This transform accounts for the fact ROS expects laser data in the x forward,
-     y left, z up frame and the calibraton has the data in x left, y up, z forward.
-     Thus a roll of -90 * a pitch of -90 will make the appropriate transform. Note
-     Roll and pitch are both with respect to the origional x left, y up, z forward frame
-     -->
-    <origin xyz="0 0 0" rpy="-1.57079632679 -1.57079632679 0.0" />
-    <parent link="${prefix}/hokuyo_link" />
-    <child link="${prefix}/head_hokuyo_frame"/>
-  </joint>
   <!-- Stereo Camera -->
   <joint name="left_camera_frame_joint" type="fixed">
@@ -101,7 +97,7 @@
     <origin xyz="0 0 0" rpy="-1.57079632679 0.0 -1.57079632679" />
     <parent link="left_camera_frame" />
-    <child link="${prefix}/left_camera_optical_frame"/>
-  </joint>
-  <link name="${prefix}/left_camera_optical_frame"/>
+    <child link="left_camera_optical_frame"/>
+  </joint>
+  <link name="left_camera_optical_frame"/>
   <joint name="right_camera_frame_joint" type="fixed">
     <origin xyz="0.0 -0.035 -0.002"/>
@@ -172,4 +168,27 @@
   <!-- IMU Frames, Mag/Accel and Gyro -->
   <!-- Include transfrom to the left_camera_frame (shift in -.035mm in X and -.002mm in Z) -->
+  <!-- imu link -->
+  <link name="head_imu_link">
+    <inertial>
+      <mass value="1e-5" />
+      <!-- collocate with parent link and remove mass from it -->
+      <origin xyz="-0.122993 0.035033383 0.02774" rpy="0 0 0" />
+      <inertia ixx="1e-6" ixy="0" ixz="0" iyy="1e-6" iyz="0" izz="1e-6" />
+    </inertial>
+    <visual>
+      <origin rpy="0 0 0" xyz="0 0 0"/>
+      <geometry>
+        <box size="0.01 0.01 0.01"/>
+      </geometry>
+    </visual>
+  </link>
+  <joint name="head_imu_joint" type="fixed">
+    <parent link="head"/>
+    <child link="head_imu_link"/>
+    <!-- putting it at the same z-level as the stereo -->
+    <origin xyz="-0.0475 0.035 0.0" rpy="0 0 0"/>
+  </joint>
+  <xacro:multisense_sl_sensor prefix="hyq"/>
+      <!-- IMU definition -->
   <link name="accel"/>
   <joint name="accel_joint" type="fixed">

Commit message: removed ptu and velodyne, and added multisenseto default model

File: robots/hyq.urdf.xacro (robot description, xacro)
@@ -18,4 +18,5 @@
 	<xacro:include filename="$(find sensors_description)/urdfs/sensors/vislab_3dve.urdf.xacro"/>
 	<xacro:include filename="$(find sensors_description)/urdfs/sensors/hokuyo_laser.urdf.xacro"/>
+	<xacro:include filename="$(find sensors_description)/urdfs/sensors/multisense_sl.urdf.xacro"/>
 	<!-- generic simulator_gazebo plugins for starting mechanism control, ros time -->
 	<xacro:include filename="$(find hyq_description)/gazebo/gazebo.urdf.xacro"/>
@@ -86,11 +87,4 @@
 	</xacro:microstrain_3dmgx425_imu>
 	<!-- Velodyne -->
-	<xacro:velodyne
-		name="velodyne"
-		parent="trunk">
-		<!--origin xyz="0.39 0 0.269" rpy="0 0 3.14"/-->
-		<!--origin xyz="0.39 0.0 0.269" rpy="0 0.0 3.10"/-->
-		<origin xyz="0.39 0.0 0.271" rpy="0.0084 -0.0169 3.14371"/>
-	</xacro:velodyne>
 	<!-- Hokuyo -->
 	<xacro:hokuyo_laser
@@ -103,54 +97,14 @@
 		range="4.0">
 	<origin xyz="0.475 0.0 -0.08823" rpy="3.14 0.0 0"/>
-    <!--origin xyz="0 -${0.5*INCH_TO_M} ${7*INCH_TO_M}" rpy="${M_PI/2} ${M_PI/2} 0" /-->
 	</xacro:hokuyo_laser>
-		<!-- Hokuyo -->
-	<!--xacro:hokuyo_utm30lx
-		name="laser"
-		parent="trunk"
-		ros_topic="scan"
-		update_rate="10"
-		ray_count="1"
-		min_angle="-5"
-		max_angle="5">
-		<origin xyz="0.475 0.0 -0.133" rpy="3.14 0.0 0"/>
-	</xacro:hokuyo_utm30lx-->
-	<!--xacro:hokuyo_mount name="nav_hokuyo" parent="front_left_vertical_beam" length="${SENSOR_BEAM_LENGTH*INCH_TO_M}" ros_topic="scan" update_rate="10" min_angle="${-(5 * M_PI)/12}" max_angle="${(5 * M_PI)/12}" range="4.0">
-    <origin xyz="0 -${0.5*INCH_TO_M} ${7*INCH_TO_M}" rpy="${M_PI/2} ${M_PI/2} 0" />
-  </xacro:hokuyo_mount-->
-	<!-- PTU unit -->
-	<xacro:ptu_d46
-		name="ptu"
-		parent="trunk">
-		<origin xyz="0.677 0.004 0.111"
-				rpy="-0.013127 0.569257 -0.007748"/>
-	</xacro:ptu_d46>
+    <xacro:multisense_sl parent="trunk" prefix="hyq">
+            <!-- <origin xyz="0.741737 0.0191395 0.143229" rpy="-0.0241345 0.446222 -0.0347202"/> -->
+            <origin xyz="0.741737 0.0 0.143229" rpy="-0.0241345 0.446222 -0.0347202"/>
+    </xacro:multisense_sl>
 	<!-- Asus Xtion Pro -->
 	<!--<origin xyz="0 0.005 0.036" rpy="0 0 0"/> with Bumblebee setup -->
 	<!--<origin xyz="0 0 0.04397" rpy="0 0 0"/> with Vislab setup -->
-	<xacro:asus_xtion_camera
-		name="asus"
-		parent="ptu_mount_link">
-		<origin xyz="0 0.005 0.036" rpy="0 0 0"/>
-	</xacro:asus_xtion_camera>
-	<!-- Kinect --> <!-- is no more used, but we keep it for compatibilty -->
-	<!--xacro:kinect_camera
-		name="head_mount"
-		parent="trunk">
-		<origin xyz="0.63 0 0.095" rpy="0 0 0"/>
-	</xacro:kinect_camera-->
-	<!-- Bumblebee -->
-	<xacro:bumblebee_97
-		parent_link="ptu_mount_link"
-                xyz= "0 0 0"
-		rpy="0 0 0"
-		ns="bumblebee"
-		frame_prefix="bumblebee_"
-		high_res="false"/>
-<!--	<xacro:vislab_3dve_72
-		name="vislab_3dve"
-		parent="ptu_mount_link"
-		xyz="0 0 0.025"
-		rpy="0 0 0"
-		high_res="false"/>-->
+<xacro:asus_xtion_camera name="asus" parent="trunk">
+	<origin xyz="0.66489 0.0016545 0.0380496" rpy="0.00740313 0.479116 0.0244919"/>
+</xacro:asus_xtion_camera>
 </robot>

Commit message: Fixing inconsistencies with the master merging

File: robots/hyq.urdf.xacro (robot description, xacro)
@@ -86,10 +86,4 @@
 		<origin xyz="0.290 0.000 0.0999214" rpy="0 ${-PI} 0"/>
 	</xacro:microstrain_3dmgx425_imu>
-        <!-- See vicon_bridge and Vicon doc to know what subject and segment mean -->
-        <xacro:vicon subject="hyq_green" segment="body" target_frame="base_link">
-               <!--origin xyz="0.455864 -0.231012 0.104193" rpy="-1.70031 0.0 -3.00989"/-->
-               <!--origin xyz="0.455864 -0.231012 0.104193" rpy="${PI/2} ${-PI/2} 0.0"/-->
-<origin xyz="-0.104392 0.454994 -0.23086" rpy="-1.57252 -0.00346852 -1.57112"/>
-        </xacro:vicon>
 	<!-- Velodyne -->
 	<!-- Hokuyo -->

Commit message: [cleanup] Removed some empty lines

File: robots/hyq.urdf.xacro (robot description, xacro)
@@ -86,5 +86,4 @@
 		<origin xyz="0.290 0.000 0.0999214" rpy="0 ${-PI} 0"/>
 	</xacro:microstrain_3dmgx425_imu>
-	<!-- Velodyne -->
 	<!-- Hokuyo -->
 	<xacro:hokuyo_laser
@@ -105,6 +104,6 @@
 	<!--<origin xyz="0 0.005 0.036" rpy="0 0 0"/> with Bumblebee setup -->
 	<!--<origin xyz="0 0 0.04397" rpy="0 0 0"/> with Vislab setup -->
-<xacro:asus_xtion_camera name="asus" parent="trunk">
-	<origin xyz="0.66489 0.0016545 0.0380496" rpy="0.00740313 0.479116 0.0244919"/>
-</xacro:asus_xtion_camera>
+	<xacro:asus_xtion_camera name="asus" parent="trunk">
+		<origin xyz="0.66489 0.0016545 0.0380496" rpy="0.00740313 0.479116 0.0244919"/>
+	</xacro:asus_xtion_camera>
 </robot>

Commit message: changed name to rf_terarangerone

File: robots/hyq.urdf.xacro (robot description, xacro)
@@ -110,5 +110,5 @@
 		name="rf_ranger"
 		parent="rf_lowerleg"
-		ros_topic="terarangerone_rf"
+		ros_topic="rf_terarangerone"
 		update_rate="400"
 		range="4.0">

File: robots/hyq_model.urdf.xacro (robot description, xacro)
@@ -10,4 +10,6 @@
 	<xacro:include filename="$(find hyq_description)/gazebo/gazebo.urdf.xacro"/>
 	<!-- Now we can start using the macros included above to define the actual HyQ -->
+	<xacro:include filename="$(find hyq_description)/urdfs/sensors/microstrain_3dmgx425_imu.urdf.xacro"/>
+	<xacro:include filename="$(find hyq_description)/urdfs/sensors/teraranger_range.urdf.xacro"/>
 	<!-- The first use of a macro. This one was defined in trunk.urdf.xacro above.
 A macro like this will expand to a set of link and joint definitions, and to additional
@@ -74,3 +76,12 @@
 		<origin xyz="0.290 0.000 0.0999214" rpy="0 ${-PI} 0"/>
 	</xacro:microstrain_3dmgx425_imu>
+		<!-- teraranger -->
+    <xacro:teraranger_range
+		name="rf_ranger"
+		parent="rf_lowerleg"
+		ros_topic="rf_terarangerone"
+		update_rate="400"
+		range="4.0">
+		<origin xyz="0.12 0.0 0.0" rpy = "${PI/2} 0.0 0.0"/>
+	</xacro:teraranger_range>
 </robot>

Commit message: [config] Changed the pitch angle for the Asus. This angle could change during time

File: robots/hyq.urdf.xacro (robot description, xacro)
@@ -105,5 +105,6 @@
 	<!--<origin xyz="0 0 0.04397" rpy="0 0 0"/> with Vislab setup -->
 	<xacro:asus_xtion_camera name="asus" parent="trunk">
-		<origin xyz="0.66489 0.0016545 0.0380496" rpy="0.00740313 0.479116 0.0244919"/>
+		<origin xyz="0.66489 0.0016545 0.0380496" rpy="0.00740313 1.2 0.0244919"/>
+<!--		<origin xyz="0.66489 0.0016545 0.0380496" rpy="0.00740313 0.479116 0.0244919"/>-->
 	</xacro:asus_xtion_camera>
 </robot>

Commit message: multi sence debug

File: robots/hyq.urdf.xacro (robot description, xacro)
@@ -106,13 +106,3 @@
 		<origin xyz="0.12 0.0 0.0" rpy = "${PI/2} 0.0 0.0"/>
 	</xacro:teraranger_range>
-    <xacro:multisense_sl parent="trunk" prefix="hyq">
-            <!-- <origin xyz="0.741737 0.0191395 0.143229" rpy="-0.0241345 0.446222 -0.0347202"/> -->
-            <origin xyz="0.741737 0.0 0.143229" rpy="-0.0241345 0.446222 -0.0347202"/>
-    </xacro:multisense_sl>
-	<!-- Asus Xtion Pro -->
-	<!--<origin xyz="0 0.005 0.036" rpy="0 0 0"/> with Bumblebee setup -->
-	<!--<origin xyz="0 0 0.04397" rpy="0 0 0"/> with Vislab setup -->
-	<xacro:asus_xtion_camera name="asus" parent="trunk">
-		<origin xyz="0.66489 0.0016545 0.0380496" rpy="0.00740313 0.479116 0.0244919"/>
-	</xacro:asus_xtion_camera>
 </robot>

Commit message: freq put to 600, inclination to -0.15

File: robots/hyq.urdf.xacro (robot description, xacro)
@@ -92,5 +92,5 @@
 		parent="rf_lowerleg"
 		ros_topic="scan"
-		update_rate="200"
+		update_rate="0"
 		min_angle="-5"
 		max_angle="5"
@@ -103,5 +103,5 @@
 		parent="rf_lowerleg"
 		ros_topic="rf_terarangerone"
-		update_rate="400"
+		update_rate="600"
 		range="4.0">
 		<origin xyz="0.12 0.0 0.0" rpy = "${PI/2} 0.0 0.0"/>

File: urdfs/sensors/teraranger_range.urdf.xacro (robot description, xacro)
@@ -10,7 +10,7 @@
 			<child link="${name}_mount_link"/>
 		</joint>
-		<!-- go from the base of the laser to the actual sensor location -->
+		<!-- go from the base of the laser to the actual sensor location -0.15 -->
 		<joint name="${name}_laser_joint" type="fixed">
-			<origin xyz="0 0 0.058" rpy="0 0.25 0"/>
+			<origin xyz="0 0 0.058" rpy="0 -0.15 0"/>
 			<parent link="${name}_mount_link"/>
 			<child link="${name}"/>

Commit message: [feature] Defined an argument for loading the force joint sensors
Conflicts:
	urdfs/leg/leg.gazebo.xacro

File: robots/hyq.urdf.xacro (robot description, xacro)
@@ -1,4 +1,6 @@
 <?xml version="1.0"?>
 <robot name="hyq" xmlns:xacro="http://www.ros.org/wiki/xacro">
+	<!-- This argument allows us to load joint sensors that measure the internal wrenches -->
+	<xacro:arg name="load_force_sensors" default="false"/>
 	<!-- The following included files set up definitions of parts of the robot body -->
 	<xacro:include filename="$(find hyq_description)/urdfs/common.xacro"/>
@@ -40,5 +42,6 @@
 		reflect_hip="1"
 		reflect_upper="1"
-		reflect_front="1">
+		reflect_front="1"
+		load_force_sensors="$(arg load_force_sensors)">
 		<origin xyz="${d_fh/2} ${d_lr/2} 0" rpy="0 ${PI/2} ${PI}"/>
 	</xacro:hyq_leg>
@@ -49,5 +52,6 @@
 		reflect_hip="-1"
 		reflect_upper="-1"
-		reflect_front="1">
+		reflect_front="1"
+		load_force_sensors="$(arg load_force_sensors)">
 		<origin xyz="${d_fh/2} ${-d_lr/2} 0" rpy="0 ${PI/2} 0"/>
 	</xacro:hyq_leg>
@@ -58,5 +62,6 @@
 		reflect_hip="-1"
 		reflect_upper="1"
-		reflect_front="-1">
+		reflect_front="-1"
+		load_force_sensors="$(arg load_force_sensors)">
 		<origin xyz="${-d_fh/2} ${d_lr/2} 0" rpy="0 ${PI/2} ${PI}"/>
 	</xacro:hyq_leg>
@@ -67,5 +72,6 @@
 		reflect_hip="1"
 		reflect_upper="-1"
-		reflect_front="-1">
+		reflect_front="-1"
+		load_force_sensors="$(arg load_force_sensors)">
 		<origin xyz="${-d_fh/2} ${-d_lr/2} 0" rpy="0 ${PI/2} 0"/>
 	</xacro:hyq_leg>

File: urdfs/leg/leg.gazebo.xacro (robot description, xacro)
@@ -1,38 +1,44 @@
 <?xml version="1.0"?>
 <robot xmlns:xacro="http://www.ros.org/wiki/xacro">
-	<xacro:macro name="leg_gazebo" params="name">
+	<xacro:macro name="leg_gazebo" params="name load_force_sensors">
 		<gazebo reference="${name}_haa_joint">
 			<provideFeedback>true</provideFeedback>
 		</gazebo>
-		<gazebo>
-			<plugin name="${name}_haa_sensor" filename="libgazebo_ros_ft_sensor.so">
-				<robotNamespace>/hyq/internal_wrench/</robotNamespace>
-				<updateRate>100.0</updateRate>
-				<topicName>${name}_haa_joint</topicName>
-				<jointName>${name}_haa_joint</jointName>
-			</plugin>
-		</gazebo>
+		<xacro:if value="${load_force_sensors}">
+			<gazebo>
+				<plugin name="${name}_haa_sensor" filename="libgazebo_ros_ft_sensor.so">
+					<robotNamespace>/hyq/internal_wrench/</robotNamespace>
+					<updateRate>100.0</updateRate>
+					<topicName>${name}_haa_joint</topicName>
+					<jointName>${name}_haa_joint</jointName>
+				</plugin>
+			</gazebo>
+		</xacro:if>
 		<gazebo reference="${name}_kfe_joint">
 			<provideFeedback>true</provideFeedback>
 		</gazebo>
-		<gazebo>
-			<plugin name="${name}_kfe_sensor" filename="libgazebo_ros_ft_sensor.so">
-				<robotNamespace>/hyq/internal_wrench/</robotNamespace>
-				<updateRate>100.0</updateRate>
-				<topicName>${name}_kfe_joint</topicName>
-				<jointName>${name}_kfe_joint</jointName>
-			</plugin>
-		</gazebo>
+		<xacro:if value="${load_force_sensors}">
+			<gazebo>
+				<plugin name="${name}_kfe_sensor" filename="libgazebo_ros_ft_sensor.so">
+					<robotNamespace>/hyq/internal_wrench/</robotNamespace>
+					<updateRate>100.0</updateRate>
+					<topicName>${name}_kfe_joint</topicName>
+					<jointName>${name}_kfe_joint</jointName>
+				</plugin>
+			</gazebo>
+		</xacro:if>
 		<gazebo reference="${name}_hfe_joint">
 			<provideFeedback>true</provideFeedback>
 		</gazebo>
-		<gazebo>
-			<plugin name="${name}_hfe_sensor" filename="libgazebo_ros_ft_sensor.so">
-				<robotNamespace>/hyq/internal_wrench/</robotNamespace>
-				<updateRate>100.0</updateRate>
-				<topicName>${name}_hfe_joint</topicName>
-				<jointName>${name}_hfe_joint</jointName>
-			</plugin>
-		</gazebo>
+		<xacro:if value="${load_force_sensors}">
+			<gazebo>
+				<plugin name="${name}_hfe_sensor" filename="libgazebo_ros_ft_sensor.so">
+					<robotNamespace>/hyq/internal_wrench/</robotNamespace>
+					<updateRate>100.0</updateRate>
+					<topicName>${name}_hfe_joint</topicName>
+					<jointName>${name}_hfe_joint</jointName>
+				</plugin>
+			</gazebo>
+		</xacro:if>
 		<gazebo reference="${name}_upperleg">
 			<kp>1000000.0</kp>
