Commit message: [feature] Defined an argument for loading the force joint sensors

File: robots/hyq.urdf.xacro (robot description, xacro)
@@ -1,4 +1,6 @@
 <?xml version="1.0"?>
 <robot name="hyq" xmlns:xacro="http://www.ros.org/wiki/xacro">
+	<!-- This argument allows us to load joint sensors that measure the internal wrenches -->
+	<xacro:arg name="load_force_sensors" default="false"/>
 	<!-- The following included files set up definitions of parts of the robot body -->
 	<xacro:include filename="$(find hyq_description)/urdfs/common.xacro"/>
@@ -40,5 +42,6 @@
 		reflect_hip="1"
 		reflect_upper="1"
-		reflect_front="1">
+		reflect_front="1"
+		load_force_sensors="$(arg load_force_sensors)">
 		<origin xyz="${d_fh/2} ${d_lr/2} 0" rpy="0 ${PI/2} ${PI}"/>
 	</xacro:hyq_leg>
@@ -49,5 +52,6 @@
 		reflect_hip="-1"
 		reflect_upper="-1"
-		reflect_front="1">
+		reflect_front="1"
+		load_force_sensors="$(arg load_force_sensors)">
 		<origin xyz="${d_fh/2} ${-d_lr/2} 0" rpy="0 ${PI/2} 0"/>
 	</xacro:hyq_leg>
@@ -58,5 +62,6 @@
 		reflect_hip="-1"
 		reflect_upper="1"
-		reflect_front="-1">
+		reflect_front="-1"
+		load_force_sensors="$(arg load_force_sensors)">
 		<origin xyz="${-d_fh/2} ${d_lr/2} 0" rpy="0 ${PI/2} ${PI}"/>
 	</xacro:hyq_leg>
@@ -67,5 +72,6 @@
 		reflect_hip="1"
 		reflect_upper="-1"
-		reflect_front="-1">
+		reflect_front="-1"
+		load_force_sensors="$(arg load_force_sensors)">
 		<origin xyz="${-d_fh/2} ${-d_lr/2} 0" rpy="0 ${PI/2} 0"/>
 	</xacro:hyq_leg>

File: robots/hyq_model.urdf.xacro (robot description, xacro)
@@ -28,5 +28,6 @@
 		reflect_hip="1"
 		reflect_upper="1"
-		reflect_front="1">
+		reflect_front="1"
+		load_force_sensors="false">
 		<origin xyz="${d_fh/2} ${d_lr/2} 0" rpy="0 ${PI/2} ${PI}"/>
 	</xacro:hyq_leg>
@@ -37,5 +38,6 @@
 		reflect_hip="-1"
 		reflect_upper="-1"
-		reflect_front="1">
+		reflect_front="1"
+		load_force_sensors="false">
 		<origin xyz="${d_fh/2} ${-d_lr/2} 0" rpy="0 ${PI/2} 0"/>
 	</xacro:hyq_leg>
@@ -46,5 +48,6 @@
 		reflect_hip="-1"
 		reflect_upper="1"
-		reflect_front="-1">
+		reflect_front="-1"
+		load_force_sensors="false">
 		<origin xyz="${-d_fh/2} ${d_lr/2} 0" rpy="0 ${PI/2} ${PI}"/>
 	</xacro:hyq_leg>
@@ -55,5 +58,6 @@
 		reflect_hip="1"
 		reflect_upper="-1"
-		reflect_front="-1">
+		reflect_front="-1"
+		load_force_sensors="false">
 		<origin xyz="${-d_fh/2} ${-d_lr/2} 0" rpy="0 ${PI/2} 0"/>
 	</xacro:hyq_leg>

File: robots/hyq_no_sensors.urdf.xacro (robot description, xacro)
@@ -1,4 +1,6 @@
 <?xml version="1.0"?>
 <robot name="hyq" xmlns:xacro="http://www.ros.org/wiki/xacro">
+	<!-- This argument allows us to load joint sensors that measure the internal wrenches -->
+	<xacro:arg name="load_force_sensors" default="false"/>
 	<!-- The following included files set up definitions of parts of the robot body -->
 	<xacro:include filename="$(find hyq_description)/urdfs/common.xacro"/>
@@ -31,5 +33,6 @@
 		reflect_hip="1"
 		reflect_upper="1"
-		reflect_front="1">
+		reflect_front="1"
+		load_force_sensors="$(arg load_force_sensors)">
 		<origin xyz="${d_fh/2} ${d_lr/2} 0" rpy="0 ${PI/2} ${PI}"/>
 	</xacro:hyq_leg>
@@ -40,5 +43,6 @@
 		reflect_hip="-1"
 		reflect_upper="-1"
-		reflect_front="1">
+		reflect_front="1"
+		load_force_sensors="$(arg load_force_sensors)">
 		<origin xyz="${d_fh/2} ${-d_lr/2} 0" rpy="0 ${PI/2} 0"/>
 	</xacro:hyq_leg>
@@ -49,5 +53,6 @@
 		reflect_hip="-1"
 		reflect_upper="1"
-		reflect_front="-1">
+		reflect_front="-1"
+		load_force_sensors="$(arg load_force_sensors)">
 		<origin xyz="${-d_fh/2} ${d_lr/2} 0" rpy="0 ${PI/2} ${PI}"/>
 	</xacro:hyq_leg>
@@ -58,5 +63,6 @@
 		reflect_hip="1"
 		reflect_upper="-1"
-		reflect_front="-1">
+		reflect_front="-1"
+		load_force_sensors="$(arg load_force_sensors)">
 		<origin xyz="${-d_fh/2} ${-d_lr/2} 0" rpy="0 ${PI/2} 0"/>
 	</xacro:hyq_leg>

File: urdfs/leg/leg.gazebo.xacro (robot description, xacro)
@@ -1,38 +1,44 @@
 <?xml version="1.0"?>
 <robot xmlns:xacro="http://www.ros.org/wiki/xacro">
-	<xacro:macro name="leg_gazebo" params="name">
+	<xacro:macro name="leg_gazebo" params="name load_force_sensors">
 		<gazebo reference="${name}_haa_joint">
 			<provideFeedback>true</provideFeedback>
 		</gazebo>
-		<gazebo>
-			<plugin name="${name}_haa_sensor" filename="libgazebo_ros_ft_sensor.so">
-				<robotNamespace>/hyq/internal_wrench/</robotNamespace>
-				<updateRate>100.0</updateRate>
-				<topicName>${name}_haa_joint</topicName>
-				<jointName>${name}_haa_joint</jointName>
-			</plugin>
-		</gazebo>
+		<xacro:if value="${load_force_sensors}">
+			<gazebo>
+				<plugin name="${name}_haa_sensor" filename="libgazebo_ros_ft_sensor.so">
+					<robotNamespace>/hyq/internal_wrench/</robotNamespace>
+					<updateRate>100.0</updateRate>
+					<topicName>${name}_haa_joint</topicName>
+					<jointName>${name}_haa_joint</jointName>
+				</plugin>
+			</gazebo>
+		</xacro:if>
 		<gazebo reference="${name}_kfe_joint">
 			<provideFeedback>true</provideFeedback>
 		</gazebo>
-		<gazebo>
-			<plugin name="${name}_kfe_sensor" filename="libgazebo_ros_ft_sensor.so">
-				<robotNamespace>/hyq/internal_wrench/</robotNamespace>
-				<updateRate>100.0</updateRate>
-				<topicName>${name}_kfe_joint</topicName>
-				<jointName>${name}_kfe_joint</jointName>
-			</plugin>
-		</gazebo>
+		<xacro:if value="${load_force_sensors}">
+			<gazebo>
+				<plugin name="${name}_kfe_sensor" filename="libgazebo_ros_ft_sensor.so">
+					<robotNamespace>/hyq/internal_wrench/</robotNamespace>
+					<updateRate>100.0</updateRate>
+					<topicName>${name}_kfe_joint</topicName>
+					<jointName>${name}_kfe_joint</jointName>
+				</plugin>
+			</gazebo>
+		</xacro:if>
 		<gazebo reference="${name}_hfe_joint">
 			<provideFeedback>true</provideFeedback>
 		</gazebo>
-		<gazebo>
-			<plugin name="${name}_hfe_sensor" filename="libgazebo_ros_ft_sensor.so">
-				<robotNamespace>/hyq/internal_wrench/</robotNamespace>
-				<updateRate>100.0</updateRate>
-				<topicName>${name}_hfe_joint</topicName>
-				<jointName>${name}_hfe_joint</jointName>
-			</plugin>
-		</gazebo>
+		<xacro:if value="${load_force_sensors}">
+			<gazebo>
+				<plugin name="${name}_hfe_sensor" filename="libgazebo_ros_ft_sensor.so">
+					<robotNamespace>/hyq/internal_wrench/</robotNamespace>
+					<updateRate>100.0</updateRate>
+					<topicName>${name}_hfe_joint</topicName>
+					<jointName>${name}_hfe_joint</jointName>
+				</plugin>
+			</gazebo>
+		</xacro:if>
 		<gazebo reference="${name}_upperleg">
 			<kp>1000000.0</kp>

File: urdfs/leg/leg.urdf.xacro (robot description, xacro)
@@ -6,5 +6,5 @@
 	<!-- ================================== Leg ================================== -->
 	<!-- The xacro macro xacro:hyq_leg contains: hip assembly, upper and lower leg -->
-	<xacro:macro name="hyq_leg" params="name parent *origin reflect_hip reflect_upper reflect_front">
+	<xacro:macro name="hyq_leg" params="name parent *origin reflect_hip reflect_upper reflect_front load_force_sensors">
 		<!-- Joints -->
 		<!-- Hip assembly joint -->
@@ -134,5 +134,5 @@
 		<!-- Extensions -->
 		<xacro:leg_transmission name="${name}"/>
-		<xacro:leg_gazebo name="${name}"/>
+		<xacro:leg_gazebo name="${name}" load_force_sensors="${load_force_sensors}"/>
 	</xacro:macro>
 </robot>

Commit message: removed multisense

File: robots/hyq.urdf.xacro (robot description, xacro)
@@ -103,8 +103,8 @@
 	<origin xyz="0.475 0.0 -0.08823" rpy="3.14 0.0 0"/>
 	</xacro:hokuyo_laser>
-    <xacro:multisense_sl parent="trunk" prefix="hyq">
+    <!--<xacro:multisense_sl parent="trunk" prefix="hyq">-->
             <!-- <origin xyz="0.741737 0.0191395 0.143229" rpy="-0.0241345 0.446222 -0.0347202"/> -->
-            <origin xyz="0.741737 0.0 0.143229" rpy="-0.0241345 0.446222 -0.0347202"/>
-    </xacro:multisense_sl>
+            <!--<origin xyz="0.741737 0.0 0.143229" rpy="-0.0241345 0.446222 -0.0347202"/>
+    </xacro:multisense_sl>-->
 	<!-- Asus Xtion Pro -->
 	<!--<origin xyz="0 0.005 0.036" rpy="0 0 0"/> with Bumblebee setup -->

Commit message: Added kvh 1775 to hyq green

File: robots/hyq.urdf.xacro (robot description, xacro)
@@ -12,4 +12,5 @@
 	<!-- HyQ sensors -->
 	<xacro:include filename="$(find sensors_description)/urdfs/sensors/microstrain_3dmgx425_imu.urdf.xacro"/>
+    <xacro:include filename="$(find sensors_description)/urdfs/sensors/kvh_1775_imu.urdf.xacro"/>
 	<xacro:include filename="$(find sensors_description)/urdfs/sensors/asus_xtion.urdf.xacro"/>
 	<!-- Velodyne disabled because it takes too long to load-up -->
@@ -92,4 +93,22 @@
 		<origin xyz="0.290 0.000 0.0999214" rpy="0 ${-PI} 0"/>
 	</xacro:microstrain_3dmgx425_imu>
+    <!-- IMU trunk -->
+    <xacro:kvh_1775_imu
+        parent="trunk"
+        imu_name="kvh_imu"
+        imu_topic="trunk_imu/data"
+        update_rate="250"
+        rate_mean="0"
+        rate_stddev="2e-4"
+        rate_bias_mean="0.00087"
+        rate_bias_stddev="0.0000008"
+        accel_mean="0"
+        accel_stddev="1.7e-2"
+        accel_bias_mean="0.002"
+        accel_bias_stddev="0.001">
+        <!--origin xyz="0.331545 0.000 0.0887678" rpy="0 0 0"/-->
+        <!--origin xyz="0.310245 0.0029 0.1271678" rpy="0 ${-PI} 0"/-->
+        <origin xyz="0.352845 0.0029 0.0503678" rpy="0 ${-PI} 0"/>
+    </xacro:kvh_1775_imu>
 	<!-- Hokuyo -->
 	<xacro:hokuyo_laser
@@ -101,5 +120,5 @@
 		max_angle="5"
 		range="4.0">
-	<origin xyz="0.475 0.0 -0.08823" rpy="3.14 0.0 0"/>
+    <origin xyz="0.475 0.0 -0.08823" rpy="${PI} 0.0 0"/>
 	</xacro:hokuyo_laser>
     <xacro:multisense_sl parent="trunk" prefix="hyq">

Commit message: [upd] Updated the orientation of the Asus

File: robots/hyq.urdf.xacro (robot description, xacro)
@@ -108,12 +108,10 @@
 	</xacro:hokuyo_laser>
     <xacro:multisense_sl parent="trunk" prefix="hyq">
-            <!-- <origin xyz="0.741737 0.0191395 0.143229" rpy="-0.0241345 0.446222 -0.0347202"/> -->
-            <origin xyz="0.741737 0.0 0.143229" rpy="-0.0241345 0.446222 -0.0347202"/>
+		<!-- <origin xyz="0.741737 0.0191395 0.143229" rpy="-0.0241345 0.446222 -0.0347202"/> -->
+		<origin xyz="0.741737 0.0 0.143229" rpy="-0.0241345 0.446222 -0.0347202"/>
     </xacro:multisense_sl>
 	<!-- Asus Xtion Pro -->
-	<!--<origin xyz="0 0.005 0.036" rpy="0 0 0"/> with Bumblebee setup -->
-	<!--<origin xyz="0 0 0.04397" rpy="0 0 0"/> with Vislab setup -->
 	<xacro:asus_xtion_camera name="asus" parent="trunk">
-		<origin xyz="0.66489 0.0016545 0.0380496" rpy="0.00740313 0.479116 0.0244919"/>
+		<origin xyz="0.66489 0.0016545 0.0380496" rpy="0.00740313 0.516618 0.0244919"/>
 	</xacro:asus_xtion_camera>
 </robot>

Commit message: [config] Recalibrated the Asus and Multisense cameras

File: robots/hyq.urdf.xacro (robot description, xacro)
@@ -109,9 +109,9 @@
     <xacro:multisense_sl parent="trunk" prefix="multisense">
 		<!-- <origin xyz="0.741737 0.0191395 0.143229" rpy="-0.0241345 0.446222 -0.0347202"/> -->
-		<origin xyz="0.741737 0.0 0.143229" rpy="-0.0241345 0.446222 -0.0347202"/>
+		<origin xyz="0.761 0.005 0.127" rpy="-0.028 0.515 -0.013"/>
     </xacro:multisense_sl>
 	<!-- Asus Xtion Pro -->
 	<xacro:asus_xtion_camera name="asus" parent="trunk">
-		<origin xyz="0.66489 0.0016545 0.0380496" rpy="0.00740313 0.516618 0.0244919"/>
+		<origin xyz="0.624 -0.013 0.061" rpy="0.018 0.535 0.057"/>
 	</xacro:asus_xtion_camera>
 </robot>

Commit message: Compliance with new xacro standard (kinetic)

File: robots/hyq.urdf.xacro (robot description, xacro)
@@ -1,4 +1,4 @@
 <?xml version="1.0"?>
-<robot name="hyq" xmlns:xacro="http://www.ros.org/wiki/xacro">
+<robot name="hyq" xmlns:xacro="http://ros.org/wiki/xacro">
 	<!-- This argument allows us to load joint sensors that measure the internal wrenches -->
 	<xacro:arg name="load_force_sensors" default="false"/>
@@ -31,9 +31,9 @@
 (e.g., base_link). The included origin block is also an argument to the macro. By convention,
 the origin block defines where the component is w.r.t its parent (in this case the parent
-is the world frame). For more, see http://www.ros.org/wiki/xacro -->
+is the world frame). For more, see http://ros.org/wiki/xacro -->
 	<!-- body -->
 	<!-- trunk -->
 	<xacro:hyq_trunk name="base">
-		<origin xyz="-0.443 -0.191 -0.276" rpy="0 0 0"/>
+		<!--origin xyz="-0.443 -0.191 -0.276" rpy="0 0 0"/-->
 	</xacro:hyq_trunk>
 	<!-- LF leg -->

File: robots/hyq_model.urdf.xacro (robot description, xacro)
@@ -1,4 +1,4 @@
 <?xml version="1.0"?>
-<robot name="hyq" xmlns:xacro="http://www.ros.org/wiki/xacro">
+<robot name="hyq" xmlns:xacro="http://ros.org/wiki/xacro">
 	<!-- The following included files set up definitions of parts of the robot body -->
 	<xacro:include filename="$(find hyq_description)/urdfs/common.xacro"/>
@@ -9,4 +9,5 @@
 	<!-- generic simulator_gazebo plugins for starting mechanism control, ros time -->
 	<xacro:include filename="$(find hyq_description)/gazebo/gazebo.urdf.xacro"/>
+        <xacro:include filename="$(find sensors_description)/urdfs/sensors/microstrain_3dmgx425_imu.urdf.xacro"/>
 	<!-- Now we can start using the macros included above to define the actual HyQ -->
 	<!-- The first use of a macro. This one was defined in trunk.urdf.xacro above.
@@ -16,9 +17,9 @@
 (e.g., base_link). The included origin block is also an argument to the macro. By convention,
 the origin block defines where the component is w.r.t its parent (in this case the parent
-is the world frame). For more, see http://www.ros.org/wiki/xacro -->
+is the world frame). For more, see http://ros.org/wiki/xacro -->
 	<!-- body -->
 	<!-- trunk -->
 	<xacro:hyq_trunk name="base">
-		<origin xyz="-0.443 -0.191 -0.276" rpy="0 0 0"/>
+		<!--origin xyz="-0.443 -0.191 -0.276" rpy="0 0 0"/-->
 	</xacro:hyq_trunk>
 	<!-- LF leg -->

File: robots/hyq_no_sensors.urdf.xacro (robot description, xacro)
@@ -1,4 +1,4 @@
 <?xml version="1.0"?>
-<robot name="hyq" xmlns:xacro="http://www.ros.org/wiki/xacro">
+<robot name="hyq" xmlns:xacro="http://ros.org/wiki/xacro">
 	<!-- This argument allows us to load joint sensors that measure the internal wrenches -->
 	<xacro:arg name="load_force_sensors" default="false"/>
@@ -21,5 +21,5 @@
 (e.g., base_link). The included origin block is also an argument to the macro. By convention,
 the origin block defines where the component is w.r.t its parent (in this case the parent
-is the world frame). For more, see http://www.ros.org/wiki/xacro -->
+is the world frame). For more, see http://ros.org/wiki/xacro -->
 	<!-- body -->
 	<!-- trunk -->

File: urdfs/common.xacro (robot description, xacro)
@@ -1,55 +1,55 @@
 <?xml version="1.0"?>
-<robot>
-	<property name="PI" value="3.1415926535897931"/>
+<robot xmlns:xacro="http://ros.org/wiki/xacro">
+	<xacro:property name="PI" value="3.1415926535897931"/>
 	<!-- standard distances -->
-	<property name="d_lr" value="0.414"/>
-	<property name="d_fh" value="0.747"/>
-	<property name="d_p0p1" value="0.08"/>
-	<property name="d_p1p2" value="0.35"/>
-	<property name="d_p2p3" value="0.346"/>
+	<xacro:property name="d_lr" value="0.414"/>
+	<xacro:property name="d_fh" value="0.747"/>
+	<xacro:property name="d_p0p1" value="0.08"/>
+	<xacro:property name="d_p1p2" value="0.35"/>
+	<xacro:property name="d_p2p3" value="0.346"/>
 	<!-- Inertial values -->
 	<!-- Trunk with hydraulic system -->
-	<property name="xcom_trunk" value="0.056"/>
-	<property name="ycom_trunk" value="0.0215"/>
-	<property name="zcom_trunk" value="0.00358"/>
-	<property name="m_trunk" value="60.96"/>
-	<property name="ixx_trunk" value="1.5725937"/>
-	<property name="iyy_trunk" value="8.5015928"/>
-	<property name="izz_trunk" value="9.1954911"/>
-	<property name="ixy_trunk" value="0.028375"/>
-	<property name="ixz_trunk" value="-0.203139"/>
-	<property name="iyz_trunk" value="-0.004462"/>
+	<xacro:property name="xcom_trunk" value="0.056"/>
+	<xacro:property name="ycom_trunk" value="0.0215"/>
+	<xacro:property name="zcom_trunk" value="0.00358"/>
+	<xacro:property name="m_trunk" value="60.96"/>
+	<xacro:property name="ixx_trunk" value="1.5725937"/>
+	<xacro:property name="iyy_trunk" value="8.5015928"/>
+	<xacro:property name="izz_trunk" value="9.1954911"/>
+	<xacro:property name="ixy_trunk" value="0.028375"/>
+	<xacro:property name="ixz_trunk" value="-0.203139"/>
+	<xacro:property name="iyz_trunk" value="-0.004462"/>
 	<!-- Hip assembly -->
-	<property name="xcom_hipassembly" value="0.04263"/>
-	<property name="ycom_hipassembly" value="0.0"/>
-	<property name="zcom_hipassembly" value="0.16931"/>
-	<property name="m_hipassembly" value="2.93"/>
-	<property name="ixx_hipassembly" value="0.05071"/>
-	<property name="iyy_hipassembly" value="0.05486"/>
-	<property name="izz_hipassembly" value="0.00571"/>
-	<property name="ixy_hipassembly" value="-0.00004"/>
-	<property name="ixz_hipassembly" value="-0.00159"/>
-	<property name="iyz_hipassembly" value="-0.00005"/>
+	<xacro:property name="xcom_hipassembly" value="0.04263"/>
+	<xacro:property name="ycom_hipassembly" value="0.0"/>
+	<xacro:property name="zcom_hipassembly" value="0.16931"/>
+	<xacro:property name="m_hipassembly" value="2.93"/>
+	<xacro:property name="ixx_hipassembly" value="0.05071"/>
+	<xacro:property name="iyy_hipassembly" value="0.05486"/>
+	<xacro:property name="izz_hipassembly" value="0.00571"/>
+	<xacro:property name="ixy_hipassembly" value="-0.00004"/>
+	<xacro:property name="ixz_hipassembly" value="-0.00159"/>
+	<xacro:property name="iyz_hipassembly" value="-0.00005"/>
 	<!-- Upper leg -->
-	<property name="xcom_upperleg" value="0.15074"/>
-	<property name="ycom_upperleg" value="0.02625"/>
-	<property name="zcom_upperleg" value="0.0"/>
-	<property name="m_upperleg" value="2.638"/>
-	<property name="ixx_upperleg" value="0.00368"/>
-	<property name="iyy_upperleg" value="0.02719"/>
-	<property name="izz_upperleg" value="0.02811"/>
-	<property name="ixy_upperleg" value="-0.00302"/>
-	<property name="ixz_upperleg" value="0.0001"/>
-	<property name="iyz_upperleg" value="0.00002"/>
+	<xacro:property name="xcom_upperleg" value="0.15074"/>
+	<xacro:property name="ycom_upperleg" value="0.02625"/>
+	<xacro:property name="zcom_upperleg" value="0.0"/>
+	<xacro:property name="m_upperleg" value="2.638"/>
+	<xacro:property name="ixx_upperleg" value="0.00368"/>
+	<xacro:property name="iyy_upperleg" value="0.02719"/>
+	<xacro:property name="izz_upperleg" value="0.02811"/>
+	<xacro:property name="ixy_upperleg" value="-0.00302"/>
+	<xacro:property name="ixz_upperleg" value="0.0001"/>
+	<xacro:property name="iyz_upperleg" value="0.00002"/>
 	<!-- Lower leg -->
-	<property name="xcom_lowerleg" value="0.1254"/>
-	<property name="ycom_lowerleg" value="0.00004"/>
-	<property name="zcom_lowerleg" value="-0.0001"/>
-	<property name="m_lowerleg" value="0.881"/>
-	<property name="ixx_lowerleg" value="0.00047"/>
-	<property name="iyy_lowerleg" value="0.01256"/>
-	<property name="izz_lowerleg" value="0.01233"/>
-	<property name="ixy_lowerleg" value="0.00006"/>
-	<property name="ixz_lowerleg" value="-0.00001"/>
-	<property name="iyz_lowerleg" value="-0.0"/>
+	<xacro:property name="xcom_lowerleg" value="0.1254"/>
+	<xacro:property name="ycom_lowerleg" value="0.00004"/>
+	<xacro:property name="zcom_lowerleg" value="-0.0001"/>
+	<xacro:property name="m_lowerleg" value="0.881"/>
+	<xacro:property name="ixx_lowerleg" value="0.00047"/>
+	<xacro:property name="iyy_lowerleg" value="0.01256"/>
+	<xacro:property name="izz_lowerleg" value="0.01233"/>
+	<xacro:property name="ixy_lowerleg" value="0.00006"/>
+	<xacro:property name="ixz_lowerleg" value="-0.00001"/>
+	<xacro:property name="iyz_lowerleg" value="-0.0"/>
 </robot>

File: urdfs/leg/leg.gazebo.xacro (robot description, xacro)
@@ -1,4 +1,4 @@
 <?xml version="1.0"?>
-<robot xmlns:xacro="http://www.ros.org/wiki/xacro">
+<robot xmlns:xacro="http://ros.org/wiki/xacro">
 	<xacro:macro name="leg_gazebo" params="name load_force_sensors">
 		<gazebo reference="${name}_haa_joint">

File: urdfs/leg/leg.urdf.xacro (robot description, xacro)
@@ -1,4 +1,4 @@
 <?xml version="1.0"?>
-<robot xmlns:xacro="http://www.ros.org/wiki/xacro">
+<robot xmlns:xacro="http://ros.org/wiki/xacro">
 	<!-- Things that are needed only for Gazebo (not the physical robot). These include sensor and controller plugin specifications -->
 	<xacro:include filename="$(find hyq_description)/urdfs/leg/leg.transmission.xacro"/>
@@ -10,5 +10,5 @@
 		<!-- Hip assembly joint -->
 		<joint name="${name}_haa_joint" type="revolute">
-			<insert_block name="origin"/>
+			<xacro:insert_block name="origin"/>
 			<parent link="${parent}"/>
 			<child  link="${name}_hipassembly"/>

File: urdfs/trunk/trunk.urdf.xacro (robot description, xacro)
@@ -1,4 +1,4 @@
 <?xml version="1.0"?>
-<robot xmlns:xacro="http://www.ros.org/wiki/xacro">
+<robot xmlns:xacro="http://ros.org/wiki/xacro">
 	<!-- Things that are needed only for Gazebo (not the physical robot). These include sensor and controller plugin specifications -->
 	<xacro:include filename="$(find hyq_description)/urdfs/trunk/trunk.gazebo.xacro"/>

File: urdfs/trunk/trunk_model.urdf.xacro (robot description, xacro)
@@ -1,4 +1,4 @@
 <?xml version="1.0"?>
-<robot xmlns:xacro="http://www.ros.org/wiki/xacro">
+<robot xmlns:xacro="http://ros.org/wiki/xacro">
 	<!-- Things that are needed only for Gazebo (not the physical robot). These include sensor and controller plugin specifications -->
 	<xacro:include filename="$(find hyq_description)/urdfs/trunk/trunk.gazebo.xacro"/>
