Commit message: Modified shin collision and added leg backward option

File: robots/hyq.urdf.xacro (robot description, xacro)
@@ -44,4 +44,5 @@
 		reflect_upper="1"
 		reflect_front="1"
+		knee_bent_backward="1"
 		load_force_sensors="$(arg load_force_sensors)">
 		<origin xyz="${d_fh/2} ${d_lr/2} 0" rpy="0 ${PI/2} ${PI}"/>
@@ -54,4 +55,5 @@
 		reflect_upper="-1"
 		reflect_front="1"
+		knee_bent_backward="1"
 		load_force_sensors="$(arg load_force_sensors)">
 		<origin xyz="${d_fh/2} ${-d_lr/2} 0" rpy="0 ${PI/2} 0"/>
@@ -64,4 +66,5 @@
 		reflect_upper="1"
 		reflect_front="-1"
+		knee_bent_backward="0"
 		load_force_sensors="$(arg load_force_sensors)">
 		<origin xyz="${-d_fh/2} ${d_lr/2} 0" rpy="0 ${PI/2} ${PI}"/>
@@ -74,4 +77,5 @@
 		reflect_upper="-1"
 		reflect_front="-1"
+		knee_bent_backward="0"
 		load_force_sensors="$(arg load_force_sensors)">
 		<origin xyz="${-d_fh/2} ${-d_lr/2} 0" rpy="0 ${PI/2} 0"/>

File: robots/hyq_model.urdf.xacro (robot description, xacro)
@@ -30,4 +30,5 @@
 		reflect_upper="1"
 		reflect_front="1"
+		knee_bent_backward="1"
 		load_force_sensors="false">
 		<origin xyz="${d_fh/2} ${d_lr/2} 0" rpy="0 ${PI/2} ${PI}"/>
@@ -40,4 +41,5 @@
 		reflect_upper="-1"
 		reflect_front="1"
+		knee_bent_backward="1"
 		load_force_sensors="false">
 		<origin xyz="${d_fh/2} ${-d_lr/2} 0" rpy="0 ${PI/2} 0"/>
@@ -50,4 +52,5 @@
 		reflect_upper="1"
 		reflect_front="-1"
+		knee_bent_backward="0"
 		load_force_sensors="false">
 		<origin xyz="${-d_fh/2} ${d_lr/2} 0" rpy="0 ${PI/2} ${PI}"/>
@@ -60,4 +63,5 @@
 		reflect_upper="-1"
 		reflect_front="-1"
+		knee_bent_backward="0"
 		load_force_sensors="false">
 		<origin xyz="${-d_fh/2} ${-d_lr/2} 0" rpy="0 ${PI/2} 0"/>

File: robots/hyq_no_sensors.urdf.xacro (robot description, xacro)
@@ -34,4 +34,5 @@
 		reflect_upper="1"
 		reflect_front="1"
+		knee_bent_backward="1"
 		load_force_sensors="$(arg load_force_sensors)">
 		<origin xyz="${d_fh/2} ${d_lr/2} 0" rpy="0 ${PI/2} ${PI}"/>
@@ -44,4 +45,5 @@
 		reflect_upper="-1"
 		reflect_front="1"
+		knee_bent_backward ="1"
 		load_force_sensors="$(arg load_force_sensors)">
 		<origin xyz="${d_fh/2} ${-d_lr/2} 0" rpy="0 ${PI/2} 0"/>
@@ -54,4 +56,5 @@
 		reflect_upper="1"
 		reflect_front="-1"
+		knee_bent_backward="0"
 		load_force_sensors="$(arg load_force_sensors)">
 		<origin xyz="${-d_fh/2} ${d_lr/2} 0" rpy="0 ${PI/2} ${PI}"/>
@@ -64,4 +67,5 @@
 		reflect_upper="-1"
 		reflect_front="-1"
+		knee_bent_backward="0"
 		load_force_sensors="$(arg load_force_sensors)">
 		<origin xyz="${-d_fh/2} ${-d_lr/2} 0" rpy="0 ${PI/2} 0"/>

File: urdfs/common.xacro (robot description, xacro)
@@ -1,11 +1,22 @@
 <?xml version="1.0"?>
 <robot xmlns:xacro="http://ros.org/wiki/xacro">
-	<xacro:property name="PI" value="3.1415926535897931"/>
+	<property name="PI" value="3.1415926535897931"/>
+    <!-- kin limits (sign ref is RH leg)-->
+    <property name="haa_max" value="25"/>
+    <property name="haa_min" value="-70"/>
+    <property name="hfe_max" value="50"/>
+    <property name="hfe_min" value="-70"/>
+    <property name="kfe_max" value="140"/>
+    <property name="kfe_min" value="20"/>
+    <!-- torque limits 120-->
+    <property name="haa_limit" value="150"/>
+    <property name="hfe_limit" value="150"/>
+    <property name="kfe_limit" value="150"/>
 	<!-- standard distances -->
-	<xacro:property name="d_lr" value="0.414"/>
-	<xacro:property name="d_fh" value="0.747"/>
-	<xacro:property name="d_p0p1" value="0.08"/>
-	<xacro:property name="d_p1p2" value="0.35"/>
-	<xacro:property name="d_p2p3" value="0.346"/>
+	<property name="d_lr" value="0.414"/>
+	<property name="d_fh" value="0.747"/>
+	<property name="hipassembly_length" value="0.08"/>
+	<property name="upperleg_length" value="0.35"/>
+	<property name="lowerleg_length" value="0.346"/>
 	<!-- Inertial values -->
 	<!-- Trunk with hydraulic system -->

File: urdfs/leg/leg.gazebo.xacro (robot description, xacro)
@@ -58,4 +58,14 @@
 			<maxVel>1.0</maxVel>
 			<minDepth>0.00</minDepth>
+			<sensor name="${name}_shin_contact_sensor" type="contact">
+                <always_on>true</always_on>
+                <update_rate>250.0</update_rate>
+                <contact>
+                  <collision>${name}_lowerleg_collision</collision>
+                </contact>
+                <plugin name="${name}_shin_bumper" filename="libgazebo_ros_bumper.so">
+                  <bumperTopicName>/${name}_shin_sensor</bumperTopicName>
+                </plugin>
+            </sensor>
 		</gazebo>
 		<gazebo reference="${name}_foot">

File: urdfs/leg/leg.urdf.xacro (robot description, xacro)
@@ -6,5 +6,5 @@
 	<!-- ================================== Leg ================================== -->
 	<!-- The xacro macro xacro:hyq_leg contains: hip assembly, upper and lower leg -->
-	<xacro:macro name="hyq_leg" params="name parent *origin reflect_hip reflect_upper reflect_front load_force_sensors">
+	<xacro:macro name="hyq_leg" params="name parent *origin reflect_hip reflect_upper reflect_front knee_bent_backward load_force_sensors">
 		<!-- Joints -->
 		<!-- Hip assembly joint -->
@@ -14,40 +14,40 @@
 			<child  link="${name}_hipassembly"/>
 			<axis xyz="0 0 1"/>
-			<limit effort="150.0" velocity="12.0" lower="${-7*PI/18}" upper="${5*PI/36}"/>
+			<limit effort="${haa_limit}" velocity="12.0" lower="${haa_min*PI/180}" upper="${haa_max*PI/180}" />
 			<dynamics damping="0.1" friction="0" />
-			<safety_controller k_position="100" k_velocity="100"
-							   soft_lower_limit="${-7*PI/18}" soft_upper_limit="${5*PI/36}" />
+			<safety_controller k_position="50" k_velocity="10"
+							   soft_lower_limit="${haa_min*PI/180}" soft_upper_limit="${haa_max*PI/180}" />
 		</joint>
 		<!-- Upper leg joint -->
 		<joint name="${name}_hfe_joint" type="revolute">
-			<origin xyz="${d_p0p1} 0 0" rpy="${reflect_upper*PI/2} 0 0"/>
+			<origin xyz="${hipassembly_length} 0 0" rpy="${reflect_upper*PI/2} 0 0"/>
 			<parent link="${name}_hipassembly"/>
 			<child  link="${name}_upperleg"/>
 			<axis xyz="0 0 1"/>
-			<limit effort="150.0" velocity="12.0"
-				   lower="${-(1+reflect_front)*5*PI/36-(1-reflect_front)*7*PI/36}"
-				   upper="${(1-reflect_front)*5*PI/36+(1+reflect_front)*7*PI/36}"/>
+			<limit effort="${hfe_limit}" velocity="12.0"
+                  lower="${(1-knee_bent_backward)*(hfe_min)*PI/180 + (knee_bent_backward)*(-hfe_max)*PI/180}"
+                  upper="${(1-knee_bent_backward)*(hfe_max)*PI/180 + (knee_bent_backward)*(-hfe_min)*PI/180}"/>
 			<dynamics damping="0.1" friction="0" />
-			<safety_controller k_position="100" k_velocity="100"
-							   soft_lower_limit="${-(1+reflect_front)*5*PI/36-(1-reflect_front)*7*PI/36}"
-							   soft_upper_limit="${(1-reflect_front)*5*PI/36+(1+reflect_front)*7*PI/36}" />
+			<safety_controller k_position="50" k_velocity="10"
+                  soft_lower_limit="${(1-knee_bent_backward)*(hfe_min)*PI/180 + (knee_bent_backward)*(-hfe_max)*PI/180}"
+                  soft_upper_limit="${(1-knee_bent_backward)*(hfe_max)*PI/180 + (knee_bent_backward)*(-hfe_min)*PI/180}"/>
 		</joint>
 		<!-- Lower leg joint -->
 		<joint name="${name}_kfe_joint" type="revolute">
-			<origin xyz="${d_p1p2} 0 0" rpy="0 0 0"/>
+			<origin xyz="${upperleg_length} 0 0" rpy="0 0 0"/>
 			<parent link="${name}_upperleg"/>
 			<child  link="${name}_lowerleg"/>
 			<axis xyz="0 0 1"/>
-			<limit effort="150.0" velocity="12.0"
-				   lower="${-(1+reflect_front)*7*PI/18+(1-reflect_front)*PI/18}"
-				   upper="${(1-reflect_front)*7*PI/18-(1+reflect_front)*PI/18}"/>
+			<limit effort="${kfe_limit}" velocity="12.0"
+                  lower="${(1-knee_bent_backward)*(kfe_min)*PI/180 + (knee_bent_backward)*(-kfe_max)*PI/180}"
+                  upper="${(1-knee_bent_backward)*(kfe_max)*PI/180 + (knee_bent_backward)*(-kfe_min)*PI/180}"/>
 			<dynamics damping="0.1" friction="0" />
-			<safety_controller k_position="100" k_velocity="100"
-							   soft_lower_limit="${-(1+reflect_front)*7*PI/18+(1-reflect_front)*PI/18}"
-							   soft_upper_limit="${(1-reflect_front)*7*PI/18-(1+reflect_front)*PI/18}" />
+			<safety_controller k_position="50" k_velocity="10"
+                  soft_lower_limit="${(1-knee_bent_backward)*(kfe_min)*PI/180 + (knee_bent_backward)*(-kfe_max)*PI/180}"
+                  soft_upper_limit="${(1-knee_bent_backward)*(kfe_max)*PI/180 + (knee_bent_backward)*(-kfe_min)*PI/180}"/>
 		<!-- Foot joint -->
 		</joint>
 		<joint name="${name}_foot_joint" type="fixed">
-			<origin xyz="${d_p2p3} 0 0" rpy="${PI/2} 0 ${-PI/2}"/>
+			<origin xyz="${lowerleg_length} 0 0" rpy="${PI/2} 0 ${-PI/2}"/>
 			<parent link="${name}_lowerleg"/>
 			<child  link="${name}_foot"/>
@@ -113,6 +113,7 @@
 			</visual>
 			<collision>
+			    <origin xyz="${lowerleg_length/2.0} 0 0" rpy="0 ${-PI/2}  0"/>
 				<geometry>
-					<mesh filename="package://hyq_description/meshes/leg/lowerleg.dae" scale="1 1 1"/>
+					<cylinder length="${lowerleg_length}"  radius="0.02"/>
 				</geometry>
 			</collision>

Commit message: Removal of unused sensor and adding of KVH again

File: robots/hyq.urdf.xacro (robot description, xacro)
@@ -12,13 +12,8 @@
 	<!-- HyQ sensors -->
 	<xacro:include filename="$(find sensors_description)/urdfs/sensors/microstrain_3dmgx425_imu.urdf.xacro"/>
-    <xacro:include filename="$(find sensors_description)/urdfs/sensors/kvh_1775_imu.urdf.xacro"/>
+        <xacro:include filename="$(find sensors_description)/urdfs/sensors/kvh_1775_imu.urdf.xacro"/>
 	<xacro:include filename="$(find sensors_description)/urdfs/sensors/asus_xtion.urdf.xacro"/>
-	<!-- Velodyne disabled because it takes too long to load-up -->
-	<!-- <xacro:include filename="$(find sensors_description)/urdfs/sensors/velodyne.urdf.xacro"/> -->
-	<xacro:include filename="$(find sensors_description)/urdfs/sensors/kinect.urdf.xacro"/>
-	<xacro:include filename="$(find sensors_description)/urdfs/sensors/ptu_d46.urdf.xacro"/>
-	<xacro:include filename="$(find sensors_description)/urdfs/sensors/bumblebee.urdf.xacro"/>
-	<xacro:include filename="$(find sensors_description)/urdfs/sensors/vislab_3dve.urdf.xacro"/>
-	<xacro:include filename="$(find sensors_description)/urdfs/sensors/hokuyo_laser.urdf.xacro"/>
+        <!-- we may mount the hokuyo again in the future -->
+	<!--xacro:include filename="$(find sensors_description)/urdfs/sensors/hokuyo_laser.urdf.xacro"/-->
 	<xacro:include filename="$(find sensors_description)/urdfs/sensors/multisense_sl.urdf.xacro"/>
 	<!-- generic simulator_gazebo plugins for starting mechanism control, ros time -->
@@ -89,17 +84,16 @@
 		<origin xyz="0.290 0.000 0.0999214" rpy="0 ${-PI} 0"/>
 	</xacro:microstrain_3dmgx425_imu>
-    <!-- IMU trunk -->
-<!-- TODO We have to substitute the microstrain IMU with this one. Note that the imu_name has to be
-trunk_imu because the DLS HW interfaces hardcoded that name
+        <!-- IMU trunk -->
+        <!-- TODO We have to substitute the microstrain IMU with this one. Note that the imu_name has to be
+                  trunk_imu because the DLS HW interfaces hardcoded that name -->
     	<xacro:kvh_1775_imu
-        parent="trunk"
-        imu_name="trunk_imu"
-        imu_topic="trunk_imu_2/data"
-        update_rate="250">
-        <origin xyz="0.352845 0.0029 0.0503678" rpy="0 ${-PI} 0"/>
-    </xacro:kvh_1775_imu>
--->
+                parent="trunk"
+                imu_name="kvh_imu"
+                imu_topic="kvh_imu/data"
+                update_rate="250">
+            <origin xyz="0.352845 0.0029 0.0503678" rpy="0 ${-PI} 0"/>
+        </xacro:kvh_1775_imu>
 	<!-- Hokuyo -->
-	<xacro:hokuyo_laser
+	<!--xacro:hokuyo_laser
 		name="laser"
 		parent="trunk"
@@ -109,13 +103,13 @@
 		max_angle="5"
 		range="4.0">
-    <origin xyz="0.475 0.0 -0.08823" rpy="${PI} 0.0 0"/>
-	</xacro:hokuyo_laser>
-    <xacro:multisense_sl parent="trunk" prefix="multisense">
-		<!-- <origin xyz="0.741737 0.0191395 0.143229" rpy="-0.0241345 0.446222 -0.0347202"/> -->
-		<origin xyz="0.761 0.005 0.127" rpy="-0.028 0.515 -0.013"/>
-    </xacro:multisense_sl>
+            <origin xyz="0.475 0.0 -0.08823" rpy="${PI} 0.0 0"/>
+	</xacro:hokuyo_laser-->
+        <xacro:multisense_sl parent="trunk" prefix="multisense">
+	    <!-- <origin xyz="0.741737 0.0191395 0.143229" rpy="-0.0241345 0.446222 -0.0347202"/> -->
+            <origin xyz="0.761 0.005 0.127" rpy="-0.028 0.515 -0.013"/>
+        </xacro:multisense_sl>
 	<!-- Asus Xtion Pro -->
 	<xacro:asus_xtion_camera name="asus" parent="trunk">
-		<origin xyz="0.624 -0.013 0.061" rpy="0.018 0.535 0.057"/>
+	    <origin xyz="0.624 -0.013 0.061" rpy="0.018 0.535 0.057"/>
 	</xacro:asus_xtion_camera>
 </robot>

Commit message: added cart (commented)

File: robots/hyq.urdf.xacro (robot description, xacro)
@@ -10,4 +10,6 @@
 	<!-- HyQ legs -->
 	<xacro:include filename="$(find hyq_description)/urdfs/leg/leg.urdf.xacro"/>
+	<!-- cart -->
+    <xacro:include filename="$(find hyq_description)/urdfs/cart/cart.urdf.xacro"/>
 	<!-- HyQ sensors -->
 	<xacro:include filename="$(find sensors_description)/urdfs/sensors/microstrain_3dmgx425_imu.urdf.xacro"/>
@@ -32,4 +34,7 @@
 		<!--origin xyz="-0.443 -0.191 -0.276" rpy="0 0 0"/-->
 	</xacro:hyq_trunk>
+    <!-- <xacro:cart   parent="trunk">
+        <origin xyz="-0.6 0 0" rpy="0 0 0"/>
+    </xacro:cart>-->
 	<!-- LF leg -->
 	<xacro:hyq_leg

Commit message: added cart (commented)

File: robots/hyq.urdf.xacro (robot description, xacro)
@@ -10,4 +10,6 @@
 	<!-- HyQ legs -->
 	<xacro:include filename="$(find hyq_description)/urdfs/leg/leg.urdf.xacro"/>
+	<!-- cart -->
+    <xacro:include filename="$(find hyq_description)/urdfs/cart/cart.urdf.xacro"/>
 	<!-- HyQ sensors -->
 	<xacro:include filename="$(find sensors_description)/urdfs/sensors/microstrain_3dmgx425_imu.urdf.xacro"/>
@@ -32,4 +34,7 @@
 		<!--origin xyz="-0.443 -0.191 -0.276" rpy="0 0 0"/-->
 	</xacro:hyq_trunk>
+    <!-- <xacro:cart   parent="trunk">
+        <origin xyz="-0.6 0 0" rpy="0 0 0"/>
+    </xacro:cart>-->
 	<!-- LF leg -->
 	<xacro:hyq_leg

File: robots/hyq_no_sensors.urdf.xacro (robot description, xacro)
@@ -10,4 +10,6 @@
 	<!-- HyQ legs -->
 	<xacro:include filename="$(find hyq_description)/urdfs/leg/leg.urdf.xacro"/>
+	<!-- cart -->
+    <xacro:include filename="$(find hyq_description)/urdfs/cart/cart.urdf.xacro"/>
 	<!-- HyQ sensors -->
 	<xacro:include filename="$(find sensors_description)/urdfs/sensors/microstrain_3dmgx425_imu.urdf.xacro"/>
@@ -27,4 +29,7 @@
 		<!--origin xyz="-0.443 -0.191 -0.276" rpy="0 0 0"/-->
 	</xacro:hyq_trunk>
+    <!--<xacro:cart   parent="trunk">
+        <origin xyz="-0.6 0 0" rpy="0 0 0"/>
+    </xacro:cart>-->
 	<!-- LF leg -->
 	<xacro:hyq_leg

Commit message: Updated sensor location values for Asus-Xtion after calibration

File: robots/hyq.urdf.xacro (robot description, xacro)
@@ -116,5 +116,5 @@
 	<!-- Asus Xtion Pro -->
 	<xacro:asus_xtion_camera name="asus" parent="trunk">
-	    <origin xyz="0.624 -0.013 0.061" rpy="0.018 0.535 0.057"/>
+	    <origin xyz="0.672 -0.013 0.039" rpy="0.014 1.0 0.053"/>
 	</xacro:asus_xtion_camera>
 </robot>

Commit message: [Important] updated ASUS position with manual calibration

File: robots/hyq.urdf.xacro (robot description, xacro)
@@ -107,9 +107,10 @@
         <xacro:multisense_sl parent="trunk" prefix="multisense">
 	    <!-- <origin xyz="0.741737 0.0191395 0.143229" rpy="-0.0241345 0.446222 -0.0347202"/> -->
-            <origin xyz="0.761 0.005 0.127" rpy="-0.028 0.515 -0.013"/>
+            <origin xyz="0.661 0.00 0.112" rpy="0 0.515 0"/>
         </xacro:multisense_sl>
 	<!-- Asus Xtion Pro -->
 	<xacro:asus_xtion_camera name="asus" parent="trunk">
-	    <origin xyz="0.624 -0.013 0.061" rpy="0.018 0.535 0.057"/>
+	    <!--<origin xyz="0.722 -0.013 0.039" rpy="0.014 1.0 0.053"/>-->
+	       <origin xyz="0.62 0.0 0.024" rpy="0.0 1.0 0.0"/>
 	</xacro:asus_xtion_camera>
 </robot>
