Commit message: [stl] Added argument that allows us to load the STL files instead of DAE ones
By default the DAE file are loaded as is current defined (i.e.
stl=false).

File: robots/hyq.urdf.xacro (robot description, xacro)
@@ -3,4 +3,6 @@
 	<!-- This argument allows us to load joint sensors that measure the internal wrenches -->
 	<xacro:arg name="load_force_sensors" default="false"/>
+	<!-- This argument allows us to load STL mesh files instead of DAE ones -->
+	<xacro:arg name="stl" default="false"/>
 	<!-- The following included files set up definitions of parts of the robot body -->
 	<xacro:include filename="$(find hyq_description)/urdfs/common.xacro"/>
@@ -34,5 +36,6 @@
 	<!-- body -->
 	<!-- trunk -->
-	<xacro:hyq_trunk name="base">
+	<xacro:hyq_trunk name="base"
+		stl="$(arg stl)">
 		<origin xyz="-0.443 -0.191 -0.276" rpy="0 0 0"/>
 	</xacro:hyq_trunk>
@@ -44,5 +47,6 @@
 		reflect_upper="1"
 		reflect_front="1"
-		load_force_sensors="$(arg load_force_sensors)">
+		load_force_sensors="$(arg load_force_sensors)"
+		stl="$(arg stl)">
 		<origin xyz="${d_fh/2} ${d_lr/2} 0" rpy="0 ${PI/2} ${PI}"/>
 	</xacro:hyq_leg>
@@ -54,5 +58,6 @@
 		reflect_upper="-1"
 		reflect_front="1"
-		load_force_sensors="$(arg load_force_sensors)">
+		load_force_sensors="$(arg load_force_sensors)"
+		stl="$(arg stl)">
 		<origin xyz="${d_fh/2} ${-d_lr/2} 0" rpy="0 ${PI/2} 0"/>
 	</xacro:hyq_leg>
@@ -64,5 +69,6 @@
 		reflect_upper="1"
 		reflect_front="-1"
-		load_force_sensors="$(arg load_force_sensors)">
+		load_force_sensors="$(arg load_force_sensors)"
+		stl="$(arg stl)">
 		<origin xyz="${-d_fh/2} ${d_lr/2} 0" rpy="0 ${PI/2} ${PI}"/>
 	</xacro:hyq_leg>
@@ -74,5 +80,6 @@
 		reflect_upper="-1"
 		reflect_front="-1"
-		load_force_sensors="$(arg load_force_sensors)">
+		load_force_sensors="$(arg load_force_sensors)"
+		stl="$(arg stl)">
 		<origin xyz="${-d_fh/2} ${-d_lr/2} 0" rpy="0 ${PI/2} 0"/>
 	</xacro:hyq_leg>

File: robots/hyq_model.urdf.xacro (robot description, xacro)
@@ -29,5 +29,6 @@
 		reflect_upper="1"
 		reflect_front="1"
-		load_force_sensors="false">
+		load_force_sensors="false"
+		stl="false">
 		<origin xyz="${d_fh/2} ${d_lr/2} 0" rpy="0 ${PI/2} ${PI}"/>
 	</xacro:hyq_leg>
@@ -39,5 +40,6 @@
 		reflect_upper="-1"
 		reflect_front="1"
-		load_force_sensors="false">
+		load_force_sensors="false"
+		stl="false">
 		<origin xyz="${d_fh/2} ${-d_lr/2} 0" rpy="0 ${PI/2} 0"/>
 	</xacro:hyq_leg>
@@ -49,5 +51,6 @@
 		reflect_upper="1"
 		reflect_front="-1"
-		load_force_sensors="false">
+		load_force_sensors="false"
+		stl="false">
 		<origin xyz="${-d_fh/2} ${d_lr/2} 0" rpy="0 ${PI/2} ${PI}"/>
 	</xacro:hyq_leg>
@@ -59,5 +62,6 @@
 		reflect_upper="-1"
 		reflect_front="-1"
-		load_force_sensors="false">
+		load_force_sensors="false"
+		stl="false">
 		<origin xyz="${-d_fh/2} ${-d_lr/2} 0" rpy="0 ${PI/2} 0"/>
 	</xacro:hyq_leg>

File: robots/hyq_no_sensors.urdf.xacro (robot description, xacro)
@@ -3,4 +3,6 @@
 	<!-- This argument allows us to load joint sensors that measure the internal wrenches -->
 	<xacro:arg name="load_force_sensors" default="false"/>
+	<!-- This argument allows us to load STL mesh files instead of DAE ones -->
+	<xacro:arg name="stl" default="false"/>
 	<!-- The following included files set up definitions of parts of the robot body -->
 	<xacro:include filename="$(find hyq_description)/urdfs/common.xacro"/>
@@ -24,5 +26,6 @@
 	<!-- body -->
 	<!-- trunk -->
-	<xacro:hyq_trunk name="base">
+	<xacro:hyq_trunk name="base"
+		stl="$(arg stl)">
 		<origin xyz="-0.443 -0.191 -0.276" rpy="0 0 0"/>
 	</xacro:hyq_trunk>
@@ -34,5 +37,6 @@
 		reflect_upper="1"
 		reflect_front="1"
-		load_force_sensors="$(arg load_force_sensors)">
+		load_force_sensors="$(arg load_force_sensors)"
+		stl="$(arg stl)">
 		<origin xyz="${d_fh/2} ${d_lr/2} 0" rpy="0 ${PI/2} ${PI}"/>
 	</xacro:hyq_leg>
@@ -44,5 +48,6 @@
 		reflect_upper="-1"
 		reflect_front="1"
-		load_force_sensors="$(arg load_force_sensors)">
+		load_force_sensors="$(arg load_force_sensors)"
+		stl="$(arg stl)">
 		<origin xyz="${d_fh/2} ${-d_lr/2} 0" rpy="0 ${PI/2} 0"/>
 	</xacro:hyq_leg>
@@ -54,5 +59,6 @@
 		reflect_upper="1"
 		reflect_front="-1"
-		load_force_sensors="$(arg load_force_sensors)">
+		load_force_sensors="$(arg load_force_sensors)"
+		stl="$(arg stl)">
 		<origin xyz="${-d_fh/2} ${d_lr/2} 0" rpy="0 ${PI/2} ${PI}"/>
 	</xacro:hyq_leg>
@@ -64,5 +70,6 @@
 		reflect_upper="-1"
 		reflect_front="-1"
-		load_force_sensors="$(arg load_force_sensors)">
+		load_force_sensors="$(arg load_force_sensors)"
+		stl="$(arg stl)">
 		<origin xyz="${-d_fh/2} ${-d_lr/2} 0" rpy="0 ${PI/2} 0"/>
 	</xacro:hyq_leg>

File: urdfs/leg/leg.urdf.xacro (robot description, xacro)
@@ -6,5 +6,5 @@
 	<!-- ================================== Leg ================================== -->
 	<!-- The xacro macro xacro:hyq_leg contains: hip assembly, upper and lower leg -->
-	<xacro:macro name="hyq_leg" params="name parent *origin reflect_hip reflect_upper reflect_front load_force_sensors">
+	<xacro:macro name="hyq_leg" params="name parent *origin reflect_hip reflect_upper reflect_front load_force_sensors stl">
 		<!-- Joints -->
 		<!-- Hip assembly joint -->
@@ -67,5 +67,10 @@
 				<origin xyz="0 0 0" rpy="${(1-reflect_hip)*PI/2} 0 0"/>
 				<geometry>
-					<mesh filename="package://hyq_description/meshes/leg/hipassembly.dae" scale="1 1 1"/>
+					<xacro:if value="${stl}">
+						<mesh filename="package://hyq_description/meshes/leg/hipassembly.stl" scale="1 1 1"/>
+					</xacro:if>
+					<xacro:unless value="${stl}">
+						<mesh filename="package://hyq_description/meshes/leg/hipassembly.dae" scale="1 1 1"/>
+					</xacro:unless>
 				</geometry>
 				<material name="grey"/>
@@ -74,5 +79,10 @@
 				<origin xyz="0 0 0" rpy="${(1-reflect_hip)*PI/2} 0 0"/>
 				<geometry>
-					<mesh filename="package://hyq_description/meshes/leg/hipassembly.dae" scale="1 1 1"/>
+					<xacro:if value="${stl}">
+						<mesh filename="package://hyq_description/meshes/leg/hipassembly.stl" scale="1 1 1"/>
+					</xacro:if>
+					<xacro:unless value="${stl}">
+						<mesh filename="package://hyq_description/meshes/leg/hipassembly.dae" scale="1 1 1"/>
+					</xacro:unless>
 				</geometry>
 			</collision>
@@ -89,5 +99,10 @@
 				<origin xyz="0 0 0" rpy="${(1-reflect_front)*PI/2} 0 0"/>
 				<geometry>
-					<mesh filename="package://hyq_description/meshes/leg/upperleg.dae" scale="1 1 1"/>
+					<xacro:if value="${stl}">
+						<mesh filename="package://hyq_description/meshes/leg/upperleg.stl" scale="1 1 1"/>
+					</xacro:if>
+					<xacro:unless value="${stl}">
+						<mesh filename="package://hyq_description/meshes/leg/upperleg.dae" scale="1 1 1"/>
+					</xacro:unless>
 				</geometry>
 				<material name="grey"/>
@@ -96,5 +111,10 @@
 				<origin xyz="0 0 0" rpy="${(1-reflect_front)*PI/2} 0 0"/>
 				<geometry>
-					<mesh filename="package://hyq_description/meshes/leg/upperleg.dae" scale="1 1 1"/>
+					<xacro:if value="${stl}">
+						<mesh filename="package://hyq_description/meshes/leg/upperleg.stl" scale="1 1 1"/>
+					</xacro:if>
+					<xacro:unless value="${stl}">
+						<mesh filename="package://hyq_description/meshes/leg/upperleg.dae" scale="1 1 1"/>
+					</xacro:unless>
 				</geometry>
 			</collision>
@@ -110,5 +130,10 @@
 			<visual>
 				<geometry>
-					<mesh filename="package://hyq_description/meshes/leg/lowerleg.dae" scale="1 1 1"/>
+					<xacro:if value="${stl}">
+						<mesh filename="package://hyq_description/meshes/leg/lowerleg.stl" scale="1 1 1"/>
+					</xacro:if>
+					<xacro:unless value="${stl}">
+						<mesh filename="package://hyq_description/meshes/leg/lowerleg.dae" scale="1 1 1"/>
+					</xacro:unless>
 				</geometry>
 				<material name="grey"/>
@@ -116,5 +141,10 @@
 			<collision>
 				<geometry>
-					<mesh filename="package://hyq_description/meshes/leg/lowerleg.dae" scale="1 1 1"/>
+					<xacro:if value="${stl}">
+						<mesh filename="package://hyq_description/meshes/leg/lowerleg.stl" scale="1 1 1"/>
+					</xacro:if>
+					<xacro:unless value="${stl}">
+						<mesh filename="package://hyq_description/meshes/leg/lowerleg.dae" scale="1 1 1"/>
+					</xacro:unless>
 				</geometry>
 			</collision>

File: urdfs/trunk/trunk.urdf.xacro (robot description, xacro)
@@ -5,5 +5,5 @@
 	<!-- ================================ Trunk ================================ -->
 	<!-- The xacro macro xacro:hyq_base contains: base and trunk -->
-	<xacro:macro name="hyq_trunk" params="name">
+	<xacro:macro name="hyq_trunk" params="name stl">
 		<!-- Floating-base Joint -->
 		<joint name="floating_base" type="fixed">
@@ -31,5 +31,10 @@
 			<visual>
 				<geometry>
-					<mesh filename="package://hyq_description/meshes/trunk/trunk.dae" scale="1 1 1"/>
+					<xacro:if value="${stl}">
+						<mesh filename="package://hyq_description/meshes/trunk/trunk.stl" scale="1 1 1"/>
+					</xacro:if>
+					<xacro:unless value="${stl}">
+						<mesh filename="package://hyq_description/meshes/trunk/trunk.dae" scale="1 1 1"/>
+					</xacro:unless>
 				</geometry>
 				<material name="green"/>
@@ -37,5 +42,10 @@
 			<collision>
 				<geometry>
-					<mesh filename="package://hyq_description/meshes/trunk/trunk.dae" scale="1 1 1"/>
+					<xacro:if value="${stl}">
+						<mesh filename="package://hyq_description/meshes/trunk/trunk.stl" scale="1 1 1"/>
+					</xacro:if>
+					<xacro:unless value="${stl}">
+						<mesh filename="package://hyq_description/meshes/trunk/trunk.dae" scale="1 1 1"/>
+					</xacro:unless>
 				</geometry>
 			</collision>

Commit message: added calibration plate to robot description

File: robots/hyq.urdf.xacro (robot description, xacro)
@@ -14,4 +14,6 @@
         <xacro:include filename="$(find sensors_description)/urdfs/sensors/kvh_1775_imu.urdf.xacro"/>
 	<xacro:include filename="$(find sensors_description)/urdfs/sensors/asus_xtion.urdf.xacro"/>
+	<!-- HyQ leg mount (for camera calibration) -->
+	<xacro:include filename="$(find hyq_description)/urdfs/calibration_plate.urdf.xacro"/>
         <!-- we may mount the hokuyo again in the future -->
 	<!--xacro:include filename="$(find sensors_description)/urdfs/sensors/hokuyo_laser.urdf.xacro"/-->
@@ -105,4 +107,7 @@
             <origin xyz="0.475 0.0 -0.08823" rpy="${PI} 0.0 0"/>
 	</xacro:hokuyo_laser-->
+    	<xacro:calibration_plate_xacro>
+            <origin xyz="0.0 0.0 0.0" rpy="0 0 0"/>
+        </xacro:calibration_plate_xacro>
         <xacro:multisense_sl parent="trunk" prefix="multisense">
 	    <!-- <origin xyz="0.741737 0.0191395 0.143229" rpy="-0.0241345 0.446222 -0.0347202"/> -->

Commit message: modified location of the plate according to the lowerleg frame from CAD
also moved the file into leg subfolder

File: robots/hyq.urdf.xacro (robot description, xacro)
@@ -15,5 +15,5 @@
 	<xacro:include filename="$(find sensors_description)/urdfs/sensors/asus_xtion.urdf.xacro"/>
 	<!-- HyQ leg mount (for camera calibration) -->
-	<xacro:include filename="$(find hyq_description)/urdfs/calibration_plate.urdf.xacro"/>
+	<xacro:include filename="$(find hyq_description)/urdfs/leg/calibration_plate.urdf.xacro"/>
         <!-- we may mount the hokuyo again in the future -->
 	<!--xacro:include filename="$(find sensors_description)/urdfs/sensors/hokuyo_laser.urdf.xacro"/-->
@@ -107,7 +107,4 @@
             <origin xyz="0.475 0.0 -0.08823" rpy="${PI} 0.0 0"/>
 	</xacro:hokuyo_laser-->
-    	<xacro:calibration_plate_xacro>
-            <origin xyz="0.0 0.0 0.0" rpy="0 0 0"/>
-        </xacro:calibration_plate_xacro>
         <xacro:multisense_sl parent="trunk" prefix="multisense">
 	    <!-- <origin xyz="0.741737 0.0191395 0.143229" rpy="-0.0241345 0.446222 -0.0347202"/> -->
@@ -119,3 +116,6 @@
 	       <origin xyz="0.62 0.0 0.024" rpy="0.0 1.0 0.0"/>
 	</xacro:asus_xtion_camera>
+    	<xacro:calibration_plate_xacro parent="lf_lowerleg">
+            <origin xyz="0.393 -0.023 -0.1" rpy="${PI/2} 0 0"/>
+        </xacro:calibration_plate_xacro>
 </robot>

File: urdfs/leg/calibration_plate.urdf.xacro (robot description, xacro)
@@ -1,8 +1,8 @@
 <?xml version="1.0"?>
 <robot xmlns:xacro="http://ros.org/wiki/xacro">
-	<xacro:macro name="calibration_plate_xacro" params="*origin">
+	<xacro:macro name="calibration_plate_xacro" params="*origin parent">
 	<joint name="lf_foot_calibration_plate_joint" type="fixed">
 		<xacro:insert_block name="origin"/>
-		<parent link="lf_foot"/>
+		<parent link="${parent}"/>
 		<child link="calibration_plate_head"/>
 	</joint>
@@ -14,5 +14,5 @@
 		</inertial>
 		<visual>
-			<origin xyz="0.02 0.0 -0.135" rpy="1.57 -1.57 0" />
+			<origin xyz="0.1 0.1 -0.0035" rpy="${PI/2.0} ${PI} 0" />
 			<geometry>
 				<mesh filename="package://hyq_description/meshes/calibration_plate.dae" scale="0.001 0.001 0.001" />
@@ -23,5 +23,5 @@
 		</visual>
 		<collision>
-			<origin xyz="0 0 0" rpy="1.57 -1.57 0" />
+			<origin xyz="0 0 0" rpy="${PI/2.0} ${-PI/2.0} 0.0" />
 			<geometry>
 				<mesh filename="package://hyq_description/meshes/calibration_plate.dae" />

Commit message: Ultimate values got with oneshot calibration AFTER encoder calibration

File: robots/hyq.urdf.xacro (robot description, xacro)
@@ -108,11 +108,11 @@
 	</xacro:hokuyo_laser-->
         <xacro:multisense_sl parent="trunk" prefix="multisense">
-	    <!-- <origin xyz="0.741737 0.0191395 0.143229" rpy="-0.0241345 0.446222 -0.0347202"/> -->
-            <origin xyz="0.661 0.00 0.112" rpy="0 0.515 0"/>
+		<!-- taken from head calibration (with vicon) -->
+		<!--origin xyz="0.761 -0.013 0.127" rpy="-0.002799508 0.514994302 -0.013000958" /-->
+		<origin xyz="0.775883 0.000304069 0.147268" rpy="-0.0145379 0.52898 0.0107014"/>
         </xacro:multisense_sl>
 	<!-- Asus Xtion Pro -->
 	<xacro:asus_xtion_camera name="asus" parent="trunk">
-	    <!--<origin xyz="0.722 -0.013 0.039" rpy="0.014 1.0 0.053"/>-->
-	       <origin xyz="0.62 0.0 0.024" rpy="0.0 1.0 0.0"/>
+		<origin xyz="0.660678 -0.00571526 0.0705706" rpy="0.0364271 1.00115 0.0827391"/>
 	</xacro:asus_xtion_camera>
     	<xacro:calibration_plate_xacro parent="lf_lowerleg">

Commit message: Ultimate values got with oneshot calibration AFTER encoder calibration

File: robots/hyq.urdf.xacro (robot description, xacro)
@@ -118,11 +118,11 @@
 	</xacro:hokuyo_laser-->
         <xacro:multisense_sl parent="trunk" prefix="multisense">
-	    <!-- <origin xyz="0.741737 0.0191395 0.143229" rpy="-0.0241345 0.446222 -0.0347202"/> -->
-            <origin xyz="0.661 0.00 0.112" rpy="0 0.515 0"/>
+		<!-- taken from head calibration (with vicon) -->
+		<!--origin xyz="0.761 -0.013 0.127" rpy="-0.002799508 0.514994302 -0.013000958" /-->
+		<origin xyz="0.775883 0.000304069 0.147268" rpy="-0.0145379 0.52898 0.0107014"/>
         </xacro:multisense_sl>
 	<!-- Asus Xtion Pro -->
 	<xacro:asus_xtion_camera name="asus" parent="trunk">
-	    <!--<origin xyz="0.722 -0.013 0.039" rpy="0.014 1.0 0.053"/>-->
-	       <origin xyz="0.62 0.0 0.024" rpy="0.0 1.0 0.0"/>
+		<origin xyz="0.660678 -0.00571526 0.0705706" rpy="0.0364271 1.00115 0.0827391"/>
 	</xacro:asus_xtion_camera>
 </robot>

Commit message: using new URDF for the IMUs, with correct frames of reference

File: robots/hyq.urdf.xacro (robot description, xacro)
@@ -77,11 +77,16 @@
 	</xacro:hyq_leg>
 	<!-- IMU trunk -->
-	<xacro:microstrain_3dmgx425_imu
+        <xacro:microstrain_3dmgx425_imu
 		parent="trunk"
 		imu_name="trunk_imu"
 		imu_topic="trunk_imu_1/data"
 		update_rate="250">
-		<origin xyz="0.290 0.000 0.0999214" rpy="0 ${-PI} 0"/>
-	</xacro:microstrain_3dmgx425_imu>
+		<!-- old URDF -->
+		<!--origin xyz="0.290 0.000 0.0999214" rpy="0 ${-PI} 0"/ -->
+		<!-- new URDF with ideal values from CAD -->
+                <!--origin xyz="0.28525 0.000 0.0967678" rpy="0 0 0"/-->
+		<!-- new URDF, REAL values manually measured from the edge of the robot -->
+                <origin xyz="0.27025 0.000 0.0967678" rpy="0 0 0"/>
+        </xacro:microstrain_3dmgx425_imu>
         <!-- IMU trunk -->
         <!-- TODO We have to substitute the microstrain IMU with this one. Note that the imu_name has to be
@@ -92,5 +97,12 @@
                 imu_topic="kvh_imu/data"
                 update_rate="250">
-            <origin xyz="0.352845 0.0029 0.0503678" rpy="0 ${-PI} 0"/>
+	    <!-- OLD URDF with manually created cylinder -->
+            <!--origin xyz="0.352845 0.0029 0.0503678" rpy="0 ${-PI} 0"/-->
+            <!-- NEW URDF with mesh, ideal values from CAD -->
+            <!--origin xyz="0.36347 0.00 0.0887678" rpy="0 ${PI} ${PI/4}"/-->
+	    	<!-- NEW URDF with mesh, REAL values measured from the edge of the robot -->
+		<!-- x = (500 - 153 - 61.77/2) / 1000	-->
+		<!-- y = from CAD -->
+		<origin xyz="0.316115 0.00 0.0887678" rpy="0 ${PI} ${PI/4}"/>
         </xacro:kvh_1775_imu>
 	<!-- Hokuyo -->
