Commit message: rename links prepending ext_
removed unused carts

File: robots/hyq.urdf.xacro (robot description, xacro)
@@ -34,7 +34,7 @@
 		<!--origin xyz="-0.443 -0.191 -0.276" rpy="0 0 0"/-->
 	</xacro:hyq_trunk>
-        <xacro:cart   parent="trunk">
+        <xacro:ext_cart   parent="trunk">
         <origin xyz="-0.6 0 0" rpy="0 0 0"/>
-        </xacro:cart>
+        </xacro:ext_cart>
 	<!-- LF leg -->
 	<xacro:hyq_leg

File: urdfs/cart/car.urdf.xacro (robot description, xacro)
@@ -14,10 +14,10 @@
             <insert_block name="origin"/>
             <parent link="${parent}"/>
-            <child link="fake_link1"/>
+            <child link="ext_fake_link1"/>
             <origin xyz="0 0 0" rpy="0 0 0"/>
             <axis xyz="0 0 1 "/>
             <limit effort="150" velocity="12.0" lower="${-70*PI/180}" upper="${70*PI/180}"/>
       </joint>
-  	     <link name="fake_link1">
+             <link name="ext_fake_link1">
             <inertial>
             <mass value="1"/>
@@ -26,11 +26,11 @@
         </link>
       <joint name="pitch_robot_joint" type="revolute">
-            <parent link="fake_link1"/>
-            <child link="fake_link2"/>
+            <parent link="ext_fake_link1"/>
+            <child link="ext_fake_link2"/>
             <axis xyz="0 0 1 "/>
             <origin xyz="0 0 0" rpy="-1.57 0 0"/>
              <limit effort="150" velocity="12.0" lower="${-70*PI/180}" upper="${70*PI/180}" />
       </joint>
-        <link name="fake_link2">
+        <link name="ext_fake_link2">
             <inertial>
             <mass value="1"/>
@@ -39,11 +39,11 @@
         </link>
    		<joint name="roll_robot_joint" type="revolute">
-            <parent link="fake_link2"/>
-            <child link="link1"/>
+            <parent link="ext_fake_link2"/>
+            <child link="ext_link1"/>
             <axis xyz="0 0 1 "/>
             <origin xyz="0 0 0" rpy=" 0 -1.57 0"/>
              <limit effort="150" velocity="12.0" lower="${-70*PI/180}" upper="${70*PI/180}" />
       </joint>
-       <link name="link1">
+       <link name="ext_link1">
             <inertial>
             <mass value="1"/>
@@ -60,11 +60,11 @@
         <!--NB convention of subsequent rotations is YPR , the translation should be applied before in the previous parent frame-->
       <joint name="pitch_cart_joint" type="revolute">
-            <parent link="link1"/>
-            <child link="fake_link3"/>
+            <parent link="ext_link1"/>
+            <child link="ext_fake_link3"/>
             <axis xyz="0 0 1 "/>
             <origin xyz="0 0 1.0" rpy="0 1.57 0"/>
              <limit effort="150" velocity="12.0" lower="${-70*PI/180}" upper="${70*PI/180}"/>
       </joint>
-            <link name="fake_link3">
+            <link name="ext_fake_link3">
             <inertial>
             <mass value="1"/>
@@ -73,11 +73,11 @@
         </link>
         <joint name="yaw_cart_joint" type="revolute">
-            <parent link="fake_link3"/>
-            <child link="fake_link4"/>
+            <parent link="ext_fake_link3"/>
+            <child link="ext_fake_link4"/>
             <axis xyz="0 0 1 "/>
             <origin xyz="0 0 0.0" rpy="1.57 0  0"/>
              <limit effort="150" velocity="12.0" lower="${-70*PI/180}" upper="${70*PI/180}"/>
        </joint>
-          <link name="fake_link4">
+          <link name="ext_fake_link4">
             <inertial>
             <mass value="1"/>
@@ -87,9 +87,9 @@
         <!-- the fixed frames are merged with the cart-->
                  <joint name="cart_attach" type="fixed">
-            <parent link="fake_link4"/>
-            <child link="cart"/>
+            <parent link="ext_fake_link4"/>
+            <child link="ext_cart"/>
             <origin rpy="0.0 0 0 " xyz="0 0 0.0 "/>
       </joint>
-       <link name="cart">
+       <link name="ext_cart">
             <inertial>
            <origin xyz="-0.5 0 0.0"/>
@@ -105,14 +105,14 @@
        </visual>
      </link>
-        <gazebo reference="cart">
+        <gazebo reference="ext_cart">
             <material>Gazebo/Black</material>
         </gazebo>
      <joint name="right_wheel_joint" type="continuous">
-        <parent link="cart"/>
-        <child link="right_wheel"/>
+        <parent link="ext_cart"/>
+        <child link="ext_right_wheel"/>
         <origin rpy="1.57 0 0" xyz=" 0 -0.5 -0.25"/>
          <axis xyz="0 0 1 "/>
       </joint>
-     <link name="right_wheel">
+     <link name="ext_right_wheel">
                 <inertial>
             <mass value="2"/>
@@ -133,5 +133,5 @@
     </collision>
   </link>
-          <gazebo reference="right_wheel">
+          <gazebo reference="ext_right_wheel">
             <material>Gazebo/Blue</material>
             <!-- kp and kd for rubber -->
@@ -145,10 +145,10 @@
         </gazebo>
   <joint name="left_wheel_joint" type="continuous">
-    <parent link="cart"/>
-    <child link="left_wheel"/>
+    <parent link="ext_cart"/>
+    <child link="ext_left_wheel"/>
     <origin rpy="-1.57 0 0" xyz=" 0 0.5 -0.25"/>
      <axis xyz="0 0 1 "/>
   </joint>
-  <link name="left_wheel">
+  <link name="ext_left_wheel">
              <inertial>
             <mass value="2"/>
@@ -169,5 +169,5 @@
     </collision>
   </link>
-        <gazebo reference="left_wheel">
+        <gazebo reference="ext_left_wheel">
             <material>Gazebo/Blue</material>
             <!-- kp and kd for rubber -->
@@ -181,10 +181,10 @@
        </gazebo>
 <joint name="left_bwheel_joint" type="continuous">
-    <parent link="cart"/>
-    <child link="left_bwheel"/>
+    <parent link="ext_cart"/>
+    <child link="ext_left_bwheel"/>
     <origin rpy="-1.57 0 0" xyz=" -1 0.5 -0.25"/>
      <axis xyz="0 0 1 "/>
   </joint>
-  <link name="left_bwheel">
+  <link name="ext_left_bwheel">
              <inertial>
             <mass value="2"/>
@@ -205,5 +205,5 @@
     </collision>
   </link>
-        <gazebo reference="left_bwheel">
+        <gazebo reference="ext_left_bwheel">
             <material>Gazebo/Red</material>
             <!-- kp and kd for rubber -->
@@ -222,5 +222,5 @@
      <axis xyz="0 0 1 "/>
   </joint>
-  <link name="right_bwheel">
+  <link name="ext_right_bwheel">
              <inertial>
             <mass value="2"/>
@@ -241,5 +241,5 @@
     </collision>
   </link>
-        <gazebo reference="right_bwheel">
+        <gazebo reference="ext_right_bwheel">
             <material>Gazebo/Red</material>
             <!-- kp and kd for rubber -->

File: urdfs/cart/cart.urdf.xacro (robot description, xacro)
@@ -2,5 +2,5 @@
 <robot xmlns:xacro="http://ros.org/wiki/xacro">
 <xacro:include filename="$(find hyq_description)/urdfs/cart/cart.transmission.xacro"/>
-<xacro:macro name="cart" params="parent *origin">
+<xacro:macro name="ext_cart" params="parent *origin">
 <material name="blue">
    <color rgba="0 0 0.8 1"/>
@@ -16,11 +16,11 @@
             <insert_block name="origin"/>
             <parent link="${parent}"/>
-            <child link="fake_link1"/>
+            <child link="ext_fake_link1"/>
             <axis xyz="0 0 1 "/>
             <limit effort="150" velocity="12.0" lower="${-70*PI/180}" upper="${70*PI/180}"/>
       </joint>
       <joint name="pitch_robot_joint" type="revolute">
-            <parent link="fake_link1"/>
-            <child link="fake_link2"/>
+            <parent link="ext_fake_link1"/>
+            <child link="ext_fake_link2"/>
             <axis xyz="0 0 1 "/>
             <origin xyz="0 0 0" rpy="-1.57 0 0"/>
@@ -28,11 +28,11 @@
       </joint>
       <joint name="roll_robot_joint" type="revolute">
-            <parent link="fake_link2"/>
-            <child link="link1"/>
+            <parent link="ext_fake_link2"/>
+            <child link="ext_link1"/>
             <axis xyz="0 0 1 "/>
             <origin xyz="0 0 0" rpy="0 -1.57 0"/>
              <limit effort="150" velocity="12.0" lower="${-70*PI/180}" upper="${70*PI/180}" />
       </joint>
-       <link name="fake_link1">
+       <link name="ext_fake_link1">
             <inertial>
             <mass value="1"/>
@@ -40,5 +40,5 @@
           </inertial>
         </link>
-        <link name="fake_link2">
+        <link name="ext_fake_link2">
             <inertial>
             <mass value="1"/>
@@ -46,5 +46,5 @@
           </inertial>
         </link>
-       <link name="link1">
+       <link name="ext_link1">
             <inertial>
             <mass value="1"/>
@@ -62,9 +62,9 @@
         <!-- the fixed frames are merged with the cart-->
         <joint name="cart_attach" type="fixed">
-            <parent link="link1"/>
-            <child link="cart"/>
+            <parent link="ext_link1"/>
+            <child link="ext_cart"/>
             <origin rpy="0 1.57 -1.57" xyz="0 0 0.5 "/>
       </joint>
-       <link name="cart">
+       <link name="ext_cart">
                   <inertial>
             <mass value="20"/>
@@ -86,14 +86,14 @@
        </collision>
      </link>
-        <gazebo reference="cart">
+        <gazebo reference="ext_cart">
             <material>Gazebo/Black</material>
         </gazebo>
      <joint name="right_wheel_joint" type="continuous">
-        <parent link="cart"/>
-        <child link="right_wheel"/>
+        <parent link="ext_cart"/>
+        <child link="ext_right_wheel"/>
         <origin rpy="1.57 0 0" xyz=" -0.5 -0.5 -0.25"/>
          <axis xyz="0 0 1 "/>
       </joint>
-     <link name="right_wheel">
+     <link name="ext_right_wheel">
                 <inertial>
             <mass value="2"/>
@@ -114,14 +114,14 @@
     </collision>
   </link>
-          <gazebo reference="right_wheel">
+          <gazebo reference="ext_right_wheel">
             <material>Gazebo/Blue</material>
         </gazebo>
   <joint name="left_wheel_joint" type="continuous">
-    <parent link="cart"/>
-    <child link="left_wheel"/>
+    <parent link="ext_cart"/>
+    <child link="ext_left_wheel"/>
     <origin rpy="-1.57 0 0" xyz=" -0.5 0.5 -0.25"/>
      <axis xyz="0 0 1 "/>
   </joint>
-  <link name="left_wheel">
+  <link name="ext_left_wheel">
              <inertial>
             <mass value="2"/>
@@ -142,8 +142,8 @@
     </collision>
   </link>
-        <gazebo reference="left_wheel">
+        <gazebo reference="ext_left_wheel">
             <material>Gazebo/Blue</material>
         </gazebo>
-<xacro:cart_transmission name="cart"/>
+<xacro:cart_transmission name="ext_cart"/>
 </xacro:macro>
 </robot>

Commit message: added car transmission and fixed car joints

File: robots/hyq.urdf.xacro (robot description, xacro)
@@ -12,4 +12,6 @@
 	<!-- cart -->
         <xacro:include filename="$(find hyq_description)/urdfs/cart/cart.urdf.xacro"/>
+        <!-- car -->
+        <xacro:include filename="$(find hyq_description)/urdfs/cart/car.urdf.xacro"/>
 	<!-- HyQ sensors -->
 	<xacro:include filename="$(find sensors_description)/urdfs/sensors/microstrain_3dmgx425_imu.urdf.xacro"/>

File: urdfs/cart/car.transmission.xacro (robot description, xacro)
@@ -1,5 +1,5 @@
 <?xml version="1.0"?>
 <robot xmlns:xacro="http://ros.org/wiki/xacro">
-    <xacro:macro name="cart_transmission" params="name">
+    <xacro:macro name="car_transmission" params="name">
                 <transmission name="yaw_robot_trans">
 			<type>transmission_interface/SimpleTransmission</type>
@@ -32,4 +32,24 @@
 			</actuator>
 		</transmission>
+                <transmission name="pitch_cart_trans">
+                        <type>transmission_interface/SimpleTransmission</type>
+                        <joint name="pitch_cart_joint">
+                                <hardwareInterface>EffortJointInterface</hardwareInterface>
+                        </joint>
+                        <actuator name="pitch_cart_motor">
+                                <hardwareInterface>EffortJointInterface</hardwareInterface>
+                                <mechanicalReduction>1</mechanicalReduction>
+                        </actuator>
+                </transmission>
+                <transmission name="yaw_cart_trans">
+                        <type>transmission_interface/SimpleTransmission</type>
+                        <joint name="yaw_cart_joint">
+                                <hardwareInterface>EffortJointInterface</hardwareInterface>
+                        </joint>
+                        <actuator name="yaw_cart_motor">
+                                <hardwareInterface>EffortJointInterface</hardwareInterface>
+                                <mechanicalReduction>1</mechanicalReduction>
+                        </actuator>
+                </transmission>
                 <transmission name="right_wheel_trans">
                         <type>transmission_interface/SimpleTransmission</type>
@@ -52,4 +72,24 @@
                         </actuator>
                 </transmission>
+                <transmission name="right_bwheel_trans">
+                        <type>transmission_interface/SimpleTransmission</type>
+                        <joint name="right_bwheel_joint">
+                                <hardwareInterface>EffortJointInterface</hardwareInterface>
+                        </joint>
+                        <actuator name="right_bwheel_motor">
+                                <hardwareInterface>EffortJointInterface</hardwareInterface>
+                                <mechanicalReduction>1</mechanicalReduction>
+                        </actuator>
+                </transmission>
+                <transmission name="left_bwheel_trans">
+                        <type>transmission_interface/SimpleTransmission</type>
+                        <joint name="left_bwheel_joint">
+                                <hardwareInterface>EffortJointInterface</hardwareInterface>
+                        </joint>
+                        <actuator name="left_bwheel_motor">
+                                <hardwareInterface>EffortJointInterface</hardwareInterface>
+                                <mechanicalReduction>1</mechanicalReduction>
+                        </actuator>
+                </transmission>
 	</xacro:macro>
 </robot>

File: urdfs/cart/car.urdf.xacro (robot description, xacro)
@@ -1,4 +1,5 @@
 <?xml version="1.0" encoding="UTF-8"?><robot xmlns:xacro="http://www.ros.org/wiki/xacro">
-<xacro:macro name="car" params="parent *origin">
+<xacro:include filename="$(find hyq_description)/urdfs/cart/car.transmission.xacro"/>
+<xacro:macro name="ext_car" params="parent *origin">
 <material name="blue">
    <color rgba="0 0 0.8 1"/>
@@ -94,5 +95,5 @@
             <inertial>
            <origin xyz="-0.5 0 0.0"/>
-            <mass value="200"/>
+            <mass value="400"/>
             <inertia ixx="1" ixy="0" ixz="0" iyy="1" iyz="0" izz="1"/>
           </inertial>
@@ -217,6 +218,6 @@
        </gazebo>
 <joint name="right_bwheel_joint" type="continuous">
-    <parent link="cart"/>
-    <child link="right_bwheel"/>
+    <parent link="ext_cart"/>
+    <child link="ext_right_bwheel"/>
     <origin rpy="-1.57 0 0" xyz=" -1 -0.5 -0.25"/>
      <axis xyz="0 0 1 "/>
@@ -252,4 +253,5 @@
             <minDepth>0.00</minDepth>
        </gazebo>
+<xacro:car_transmission name="ext_car"/>
 </xacro:macro>
 </robot>

Commit message: Add realsense

File: robots/hyq.urdf.xacro (robot description, xacro)
@@ -15,6 +15,7 @@
 	<xacro:include filename="$(find sensors_description)/urdfs/sensors/asus_xtion.urdf.xacro"/>
         <!-- we may mount the hokuyo again in the future -->
-	<!--xacro:include filename="$(find sensors_description)/urdfs/sensors/hokuyo_laser.urdf.xacro"/-->
+	<!-- xacro:include filename="$(find sensors_description)/urdfs/sensors/hokuyo_laser.urdf.xacro"/> -->
 	<xacro:include filename="$(find sensors_description)/urdfs/sensors/multisense_sl.urdf.xacro"/>
+	<xacro:include filename="$(find sensors_description)/urdfs/sensors/realsense.urdf.xacro"/>
 	<!-- generic simulator_gazebo plugins for starting mechanism control, ros time -->
 	<xacro:include filename="$(find hyq_description)/gazebo/gazebo.urdf.xacro"/>
@@ -122,4 +123,7 @@
 		<origin xyz="0.775883 0.000304069 0.147268" rpy="-0.0145379 0.52898 0.0107014"/>
         </xacro:multisense_sl>
+        <xacro:sensor_r430 parent="trunk" prefix="realsense">
+		<origin xyz="0.775883 0.000304069 0.147268" rpy="-0.0145379 0.52898 0.0107014"/>
+        </xacro:sensor_r430>
 	<!-- Asus Xtion Pro -->
 	<xacro:asus_xtion_camera name="asus" parent="trunk">

Commit message: Add second realsense to hyq

File: robots/hyq.urdf.xacro (robot description, xacro)
@@ -123,6 +123,9 @@
 		<origin xyz="0.775883 0.000304069 0.147268" rpy="-0.0145379 0.52898 0.0107014"/>
         </xacro:multisense_sl>
-        <xacro:sensor_r430 parent="trunk" prefix="realsense">
-		<origin xyz="0.775883 0.000304069 0.147268" rpy="-0.0145379 0.52898 0.0107014"/>
+        <xacro:sensor_r430 parent="trunk" prefix="front">
+		<origin xyz="0.775883 0.000304069 0.147268" rpy="0 0.5 0"/>
+        </xacro:sensor_r430>
+        <xacro:sensor_r430 parent="trunk" prefix="back">
+		<origin xyz="-0.775883 0.000304069 0.147268" rpy="0 0.5 3.14159"/>
         </xacro:sensor_r430>
 	<!-- Asus Xtion Pro -->

Commit message: corrected attachment point of cart

File: robots/hyq.urdf.xacro (robot description, xacro)
@@ -37,5 +37,5 @@
 	</xacro:hyq_trunk>
         <xacro:ext_cart   parent="trunk">
-        <origin xyz="-0.6 0 0" rpy="0 0 0"/>
+        <origin xyz="-0.6 0 0.08" rpy="0 0 0"/>
         </xacro:ext_cart>
 	<!-- LF leg -->

Commit message: Update launch files for realsense

File: robots/hyq.urdf.xacro (robot description, xacro)
@@ -3,4 +3,9 @@
 	<!-- This argument allows us to load joint sensors that measure the internal wrenches -->
 	<xacro:arg name="load_force_sensors" default="false"/>
+	<xacro:arg name="multisense" default="false"/>
+	<xacro:arg name="realsense" default="false"/>
+	<xacro:arg name="asus" default="false"/>
+	<xacro:arg name="multirealsense" default="false"/>
+	<xacro:arg name="hokuyo" default="false"/>
 	<!-- The following included files set up definitions of parts of the robot body -->
 	<xacro:include filename="$(find hyq_description)/urdfs/common.xacro"/>
@@ -13,9 +18,16 @@
 	<xacro:include filename="$(find sensors_description)/urdfs/sensors/microstrain_3dmgx425_imu.urdf.xacro"/>
         <xacro:include filename="$(find sensors_description)/urdfs/sensors/kvh_1775_imu.urdf.xacro"/>
-	<xacro:include filename="$(find sensors_description)/urdfs/sensors/asus_xtion.urdf.xacro"/>
-        <!-- we may mount the hokuyo again in the future -->
-	<!-- xacro:include filename="$(find sensors_description)/urdfs/sensors/hokuyo_laser.urdf.xacro"/> -->
-	<xacro:include filename="$(find sensors_description)/urdfs/sensors/multisense_sl.urdf.xacro"/>
-	<xacro:include filename="$(find sensors_description)/urdfs/sensors/realsense.urdf.xacro"/>
+	<xacro:if value="false"> <!-- "$(arg asus)" -->
+		<xacro:include filename="$(find sensors_description)/urdfs/sensors/asus_xtion.urdf.xacro"/>
+	</xacro:if>
+	<xacro:if value="false"> <!-- "$(arg hokuyo)" -->
+		<xacro:include filename="$(find sensors_description)/urdfs/sensors/hokuyo_laser.urdf.xacro"/>
+	</xacro:if> -->
+	<xacro:if value="false">  <!-- "$(arg multisense)" -->
+		<xacro:include filename="$(find sensors_description)/urdfs/sensors/multisense_sl.urdf.xacro"/>
+	</xacro:if>
+	<xacro:if value="true">  <!-- "$(arg realsense)" -->
+		<xacro:include filename="$(find sensors_description)/urdfs/sensors/realsense.urdf.xacro"/>
+	</xacro:if>
 	<!-- generic simulator_gazebo plugins for starting mechanism control, ros time -->
 	<xacro:include filename="$(find hyq_description)/gazebo/gazebo.urdf.xacro"/>
@@ -107,29 +119,30 @@
 		<origin xyz="0.316115 0.00 0.0887678" rpy="0 ${PI} ${PI/4}"/>
         </xacro:kvh_1775_imu>
-	<!-- Hokuyo -->
-	<!--xacro:hokuyo_laser
-		name="laser"
-		parent="trunk"
-		ros_topic="scan"
-		update_rate="10"
-		min_angle="-5"
-		max_angle="5"
-		range="4.0">
-            <origin xyz="0.475 0.0 -0.08823" rpy="${PI} 0.0 0"/>
-	</xacro:hokuyo_laser-->
-        <xacro:multisense_sl parent="trunk" prefix="multisense">
-		<!-- taken from head calibration (with vicon) -->
-		<!--origin xyz="0.761 -0.013 0.127" rpy="-0.002799508 0.514994302 -0.013000958" /-->
-		<origin xyz="0.775883 0.000304069 0.147268" rpy="-0.0145379 0.52898 0.0107014"/>
-        </xacro:multisense_sl>
-        <xacro:sensor_r430 parent="trunk" prefix="front">
-		<origin xyz="0.775883 0.000304069 0.147268" rpy="0 0.5 0"/>
-        </xacro:sensor_r430>
-        <xacro:sensor_r430 parent="trunk" prefix="back">
-		<origin xyz="-0.775883 0.000304069 0.147268" rpy="0 0.5 3.14159"/>
-        </xacro:sensor_r430>
-	<!-- Asus Xtion Pro -->
-	<xacro:asus_xtion_camera name="asus" parent="trunk">
-		<origin xyz="0.660678 -0.00571526 0.0705706" rpy="0.0364271 1.00115 0.0827391"/>
-	</xacro:asus_xtion_camera>
+	<xacro:if value="false"> <!-- "$(arg hokuyo)" -->
+		<xacro:hokuyo_laser name="laser" parent="trunk" ros_topic="scan" update_rate="10" min_angle="-5" max_angle="5" range="4.0">
+		    <origin xyz="0.475 0.0 -0.08823" rpy="${PI} 0.0 0"/>
+		</xacro:hokuyo_laser>
+	</xacro:if>
+	<xacro:if value="false"> <!-- "$(arg multisense)" -->
+		<xacro:multisense_sl parent="trunk" prefix="multisense">
+			<!-- taken from head calibration (with vicon) -->
+			<!--origin xyz="0.761 -0.013 0.127" rpy="-0.002799508 0.514994302 -0.013000958" /-->
+			<origin xyz="0.775883 0.000304069 0.147268" rpy="-0.0145379 0.52898 0.0107014"/>
+		</xacro:multisense_sl>
+	</xacro:if>
+	<xacro:if value="true"> <!-- "$(arg realsense)" -->
+		<xacro:sensor_r430 parent="trunk" prefix="front">
+			<origin xyz="0.775883 0.000304069 0.147268" rpy="0 0.5 0"/>
+		</xacro:sensor_r430>
+		<xacro:if value="true"> <!-- "$(arg multirealsense)" -->
+			<xacro:sensor_r430 parent="trunk" prefix="back">
+				<origin xyz="-0.775883 0.000304069 0.147268" rpy="0 0.5 3.14159"/>
+			</xacro:sensor_r430>
+		</xacro:if>
+	</xacro:if>
+	<xacro:if value="false"> <!-- "$(arg asus)" -->
+		<xacro:asus_xtion_camera name="asus" parent="trunk">
+			<origin xyz="0.660678 -0.00571526 0.0705706" rpy="0.0364271 1.00115 0.0827391"/>
+		</xacro:asus_xtion_camera>
+	</xacro:if>
 </robot>
