Commit message: Update IMUs with frame name, remove multisense

File: robots/hyq.urdf.xacro (robot description, xacro)
@@ -81,5 +81,7 @@
 		imu_name="trunk_imu"
 		imu_topic="trunk_imu_1/data"
-		update_rate="250">
+                update_rate="250"
+                frame_name="trunk_imu"
+                >
 		<!-- old URDF -->
 		<!--origin xyz="0.290 0.000 0.0999214" rpy="0 ${-PI} 0"/ -->
@@ -94,7 +96,9 @@
     	<xacro:kvh_1775_imu
                 parent="trunk"
-                imu_name="kvh_imu"
-                imu_topic="kvh_imu/data"
-                update_rate="250">
+                imu_name="trunk_imu2"
+                imu_topic="trunk_imu_2/data"
+                update_rate="250"
+                frame_name="trunk_imu2"
+                >
 	    <!-- OLD URDF with manually created cylinder -->
             <!--origin xyz="0.352845 0.0029 0.0503678" rpy="0 ${-PI} 0"/-->
@@ -117,9 +121,9 @@
             <origin xyz="0.475 0.0 -0.08823" rpy="${PI} 0.0 0"/>
 	</xacro:hokuyo_laser-->
-        <xacro:multisense_sl parent="trunk" prefix="multisense">
+        <!-- <xacro:multisense_sl parent="trunk" prefix="multisense"> -->
 		<!-- taken from head calibration (with vicon) -->
 		<!--origin xyz="0.761 -0.013 0.127" rpy="-0.002799508 0.514994302 -0.013000958" /-->
-		<origin xyz="0.775883 0.000304069 0.147268" rpy="-0.0145379 0.52898 0.0107014"/>
-        </xacro:multisense_sl>
+                <!-- <origin xyz="0.775883 0.000304069 0.147268" rpy="-0.0145379 0.52898 0.0107014"/>  -->
+        <!-- </xacro:multisense_sl> -->
 	<!-- Asus Xtion Pro -->
 	<xacro:asus_xtion_camera name="asus" parent="trunk">

File: robots/hyq_model.urdf.xacro (robot description, xacro)
@@ -72,4 +72,5 @@
 		imu_name="trunk_imu"
 		imu_topic="trunk_imu/data"
+                frame_name="trunk_imu"
 		update_rate="250">
 		<origin xyz="0.290 0.000 0.0999214" rpy="0 ${-PI} 0"/>

File: robots/hyq_model_ordered.urdf.xacro (robot description, xacro)
@@ -83,5 +83,7 @@
 		imu_name="trunk_imu"
 		imu_topic="trunk_imu/data"
-		update_rate="250">
+                update_rate="250"
+                frame_name="trunk_imu"
+                >
 		<origin xyz="0.290 0.000 0.0999214" rpy="0 ${-PI} 0"/>
 	</xacro:microstrain_3dmgx425_imu>

Commit message: parametrized arm position
removed duplicate (wrong) call to semantic description

File: robots/hyq.urdf.xacro (robot description, xacro)
@@ -84,9 +84,9 @@
 	</xacro:hyq_leg>
 <xacro:if value="$(arg arm)">
-	<joint name="joint_base_robots" type="fixed">
-	    	<parent link="base_link"/>
-	    	<child link="teleop_link0"/>
-   	 	<origin xyz="0.59 0 0" rpy="0 0 0"/>
-    	</joint>
+        <joint name="joint_base_robots" type="fixed">
+                <parent link="base_link"/>
+                <child link="teleop_link0"/>
+                <origin xyz="${x_arm} 0 ${z_arm}" rpy="0 ${pitch_arm} 0"/>
+        </joint>
 	<!-- SELECTION OF KINEMATICS CHAINS IS HANDLED INSIDE THE FILES -->
 	<xacro:include filename="$(find teleop_urdf)/urdf/teleop.urdf.xacro" />

File: urdfs/common.xacro (robot description, xacro)
@@ -64,3 +64,7 @@
 	<xacro:property name="ixz_lowerleg" value="-0.00001"/>
 	<xacro:property name="iyz_lowerleg" value="-0.0"/>
+        <!-- arm position-->
+        <xacro:property name="x_arm" value="0.66"/>
+        <xacro:property name="z_arm" value="0.1"/>
+        <xacro:property name="pitch_arm" value="0.17"/>
 </robot>

Commit message: commented multisense!

File: robots/hyq.urdf.xacro (robot description, xacro)
@@ -140,9 +140,4 @@
             <origin xyz="0.475 0.0 -0.08823" rpy="${PI} 0.0 0"/>
 	</xacro:hokuyo_laser-->
-        <xacro:multisense_sl parent="trunk" prefix="multisense">
-		<!-- taken from head calibration (with vicon) -->
-		<!--origin xyz="0.761 -0.013 0.127" rpy="-0.002799508 0.514994302 -0.013000958" /-->
-		<origin xyz="0.775883 0.000304069 0.147268" rpy="-0.0145379 0.52898 0.0107014"/>
-        </xacro:multisense_sl>
 	<!-- Asus Xtion Pro -->
 	<xacro:asus_xtion_camera name="asus" parent="trunk">

Commit message: Merge with develop

File: robots/hyq.urdf.xacro (robot description, xacro)
@@ -1,4 +1,7 @@
 <?xml version="1.0"?>
 <robot name="hyq" xmlns:xacro="http://ros.org/wiki/xacro">
+	<xacro:arg name="task_period" default="0.004"/>
+	<xacro:arg name="sensors" default="true"/>
+	<xacro:arg name="arm" default="false"/>
 	<!-- This argument allows us to load joint sensors that measure the internal wrenches -->
 	<xacro:arg name="load_force_sensors" default="false"/>
@@ -11,12 +14,16 @@
 	<xacro:include filename="$(find hyq_description)/urdfs/leg/leg.urdf.xacro"/>
 	<!-- HyQ sensors -->
-	<xacro:include filename="$(find sensors_description)/urdfs/sensors/microstrain_3dmgx425_imu.urdf.xacro"/>
-        <xacro:include filename="$(find sensors_description)/urdfs/sensors/kvh_1775_imu.urdf.xacro"/>
-	<xacro:include filename="$(find sensors_description)/urdfs/sensors/asus_xtion.urdf.xacro"/>
-        <!-- we may mount the hokuyo again in the future -->
-	<!--xacro:include filename="$(find sensors_description)/urdfs/sensors/hokuyo_laser.urdf.xacro"/-->
-	<xacro:include filename="$(find sensors_description)/urdfs/sensors/multisense_sl.urdf.xacro"/>
+        <xacro:if value="$(arg sensors)">
+            <xacro:include filename="$(find sensors_description)/urdfs/sensors/microstrain_3dmgx425_imu.urdf.xacro"/>
+            <xacro:include filename="$(find sensors_description)/urdfs/sensors/kvh_1775_imu.urdf.xacro"/>
+            <xacro:include filename="$(find sensors_description)/urdfs/sensors/asus_xtion.urdf.xacro"/>
+            <!-- we may mount the hokuyo again in the future -->
+            <!--xacro:include filename="$(find sensors_description)/urdfs/sensors/hokuyo_laser.urdf.xacro"/-->
+            <xacro:include filename="$(find sensors_description)/urdfs/sensors/multisense_sl.urdf.xacro"/>
+        </xacro:if>
 	<!-- generic simulator_gazebo plugins for starting mechanism control, ros time -->
-	<xacro:include filename="$(find hyq_description)/gazebo/gazebo.urdf.xacro"/>
+        <xacro:include filename="$(find hyq_description)/gazebo/gazebo.urdf.xacro">
+             <xacro:arg name="task_period" value="$(arg task_period)"/>
+        </xacro:include>
 	<!-- Now we can start using the macros included above to define the actual HyQ -->
 	<!-- The first use of a macro. This one was defined in trunk.urdf.xacro above.
@@ -76,4 +83,20 @@
 		<origin xyz="${-d_fh/2} ${-d_lr/2} 0" rpy="0 ${PI/2} 0"/>
 	</xacro:hyq_leg>
+<xacro:if value="$(arg arm)">
+        <joint name="joint_base_robots" type="fixed">
+                <parent link="base_link"/>
+                <child link="teleop_link0"/>
+                <origin xyz="${x_arm} 0 ${z_arm}" rpy="0 ${pitch_arm} 0"/>
+        </joint>
+	<!-- SELECTION OF KINEMATICS CHAINS IS HANDLED INSIDE THE FILES -->
+	<xacro:include filename="$(find teleop_urdf)/urdf/teleop.urdf.xacro" />
+        <xacro:include filename="$(find hyq_description)/urdfs/arm/arm.transmission.xacro"/>
+        <xacro:arm_transmission name="joint1"/>
+        <xacro:arm_transmission name="joint2"/>
+        <xacro:arm_transmission name="joint3"/>
+        <xacro:arm_transmission name="joint4"/>
+        <xacro:arm_transmission name="joint5"/>
+</xacro:if>
+<xacro:if value="$(arg sensors)">
 	<!-- IMU trunk -->
         <xacro:microstrain_3dmgx425_imu
@@ -121,12 +144,8 @@
             <origin xyz="0.475 0.0 -0.08823" rpy="${PI} 0.0 0"/>
 	</xacro:hokuyo_laser-->
-        <!-- <xacro:multisense_sl parent="trunk" prefix="multisense"> -->
-		<!-- taken from head calibration (with vicon) -->
-		<!--origin xyz="0.761 -0.013 0.127" rpy="-0.002799508 0.514994302 -0.013000958" /-->
-                <!-- <origin xyz="0.775883 0.000304069 0.147268" rpy="-0.0145379 0.52898 0.0107014"/>  -->
-        <!-- </xacro:multisense_sl> -->
 	<!-- Asus Xtion Pro -->
 	<xacro:asus_xtion_camera name="asus" parent="trunk">
 		<origin xyz="0.660678 -0.00571526 0.0705706" rpy="0.0364271 1.00115 0.0827391"/>
 	</xacro:asus_xtion_camera>
+    </xacro:if>
 </robot>

Commit message: Add calibration foot (commented out)

File: robots/hyq.urdf.xacro (robot description, xacro)
@@ -22,4 +22,5 @@
             <xacro:include filename="$(find sensors_description)/urdfs/sensors/multisense_sl.urdf.xacro"/>
         </xacro:if>
+	<xacro:include filename="$(find hyq_description)/urdfs/leg/calibration_plate.urdf.xacro"/>
 	<!-- generic simulator_gazebo plugins for starting mechanism control, ros time -->
         <xacro:include filename="$(find hyq_description)/gazebo/gazebo.urdf.xacro">
@@ -149,3 +150,6 @@
 	</xacro:asus_xtion_camera>
     </xacro:if>
+    <!--xacro:calibration_plate_xacro parent="lf_lowerleg">
+	<origin xyz="0.393 -0.023 -0.1" rpy="${PI/2} 0 0"/>
+    </xacro:calibration_plate_xacro-->
 </robot>

Commit message: First reslsense calibration

File: robots/hyq.urdf.xacro (robot description, xacro)
@@ -20,7 +20,8 @@
             <!-- we may mount the hokuyo again in the future -->
             <!--xacro:include filename="$(find sensors_description)/urdfs/sensors/hokuyo_laser.urdf.xacro"/-->
-            <xacro:include filename="$(find sensors_description)/urdfs/sensors/multisense_sl.urdf.xacro"/>
+            <!--xacro:include filename="$(find sensors_description)/urdfs/sensors/multisense_sl.urdf.xacro"/-->
+            <xacro:include filename="$(find sensors_description)/urdfs/sensors/d435_camera.urdf.xacro"/>
         </xacro:if>
-	<xacro:include filename="$(find hyq_description)/urdfs/leg/calibration_plate.urdf.xacro"/>
+        <xacro:include filename="$(find hyq_description)/urdfs/leg/new_calibration_plate.urdf.xacro"/>
 	<!-- generic simulator_gazebo plugins for starting mechanism control, ros time -->
         <xacro:include filename="$(find hyq_description)/gazebo/gazebo.urdf.xacro">
@@ -146,10 +147,22 @@
 	</xacro:hokuyo_laser-->
 	<!-- Asus Xtion Pro -->
-	<xacro:asus_xtion_camera name="asus" parent="trunk">
+        <!--xacro:asus_xtion_camera name="asus" parent="trunk">
 		<origin xyz="0.660678 -0.00571526 0.0705706" rpy="0.0364271 1.00115 0.0827391"/>
-	</xacro:asus_xtion_camera>
+        </xacro:asus_xtion_camera-->
+        <xacro:d435_camera parent="trunk" prefix="realsense/front">
+            <origin xyz="0.5 0.0 -0.10" rpy="0 ${PI/4} 0"/>
+            <!--origin xyz="0.542717 0.034674  -0.0778795" rpy=" rpy="-0.0594806 0.772105 0.0110605"/-->
+            <!--origin xyz="0.542967 0.0367956 -0.0775982" rpy=" rpy="-0.0738274 0.768856 0.0313372"/-->
+            <!--origin xyz="0.538659 0.0289166 -0.0814392" rpy=" rpy="-0.0497367 0.776145 0.0275152"/-->
+        </xacro:d435_camera>
+        <xacro:d435_camera parent="trunk" prefix="realsense/back">
+            <origin xyz="-0.5 -0.0 -0.10" rpy="0 ${PI/4} 3.14159"/>
+        </xacro:d435_camera>
     </xacro:if>
-    <!--xacro:calibration_plate_xacro parent="lf_lowerleg">
-	<origin xyz="0.393 -0.023 -0.1" rpy="${PI/2} 0 0"/>
-    </xacro:calibration_plate_xacro-->
+<!--xacro:new_calibration_plate_xacro parent="rh_lowerleg">
+    <origin xyz="0.39 -0.01 0.1" rpy="${-PI/2} 0 0"/>
+</xacro:new_calibration_plate_xacro-->
+    <!--xacro:new_calibration_plate_xacro parent="lf_lowerleg">
+        <origin xyz="0.39 0.01 -0.1" rpy="${PI/2} 0 0"/>
+    </xacro:new_calibration_plate_xacro-->
 </robot>

Commit message: Update urdf after calibrating cameras

File: robots/hyq.urdf.xacro (robot description, xacro)
@@ -151,18 +151,27 @@
         </xacro:asus_xtion_camera-->
         <xacro:d435_camera parent="trunk" prefix="realsense/front">
-            <origin xyz="0.5 0.0 -0.10" rpy="0 ${PI/4} 0"/>
-            <!--origin xyz="0.542717 0.034674  -0.0778795" rpy=" rpy="-0.0594806 0.772105 0.0110605"/-->
-            <!--origin xyz="0.542967 0.0367956 -0.0775982" rpy=" rpy="-0.0738274 0.768856 0.0313372"/-->
-            <!--origin xyz="0.538659 0.0289166 -0.0814392" rpy=" rpy="-0.0497367 0.776145 0.0275152"/-->
+            <!-- "Guess" of camera location -->
+            <!-- origin xyz="0.5 0.0 -0.10" rpy="0 ${PI/4} 0"/ -->
+            <!-- LF calibration trials using ipopt -->
+            <!-- origin xyz="0.556849 0.0275077 -0.0799648" rpy=" rpy="-0.0872665 0.791739 0.0872665"/>
+            <origin xyz="0.557156 0.0299427 -0.0775026" rpy=" rpy="-0.0327945 0.799206 -0.0252025"/>
+            <origin xyz="0.541865 0.0322597 -0.0730521" rpy=" rpy="-0.0447015 0.755414 -0.00943697"/>
+            <origin xyz="0.552173 0.0360462 -0.0749277" rpy=" rpy="-0.0640513 0.774692 0.0103402"/>
+            <origin xyz="0.55039 0.0327616 -0.0749135" rpy=" rpy="-0.0513261 0.773668 0.00448148"/ -->
+            <!-- Average of trials -->
+            <origin xyz="0.552 0.032 -0.076" rpy="-0.056 0.766 -0.007"/>
         </xacro:d435_camera>
         <xacro:d435_camera parent="trunk" prefix="realsense/back">
-            <origin xyz="-0.5 -0.0 -0.10" rpy="0 ${PI/4} 3.14159"/>
+            <!-- origin xyz="-0.5 -0.0 -0.10" rpy="0 ${PI/4} ${PI}"/ -->
+            <!-- Rear calibration failed, using approximate values from front camera -->
+            <origin xyz="-0.552 0.0 -0.076" rpy="0 ${PI/4} ${PI}"/>
         </xacro:d435_camera>
     </xacro:if>
-<!--xacro:new_calibration_plate_xacro parent="rh_lowerleg">
-    <origin xyz="0.39 -0.01 0.1" rpy="${-PI/2} 0 0"/>
-</xacro:new_calibration_plate_xacro-->
-    <!--xacro:new_calibration_plate_xacro parent="lf_lowerleg">
-        <origin xyz="0.39 0.01 -0.1" rpy="${PI/2} 0 0"/>
+    <!--xacro:new_calibration_plate_xacro parent="rh_lowerleg">
+        <origin xyz="0.39 -0.01 0.1" rpy="${-PI/2} 0 0"/>
     </xacro:new_calibration_plate_xacro-->
+    <!-- Numbers from Chundri Aug. 2019 -->
+    <!-- xacro:new_calibration_plate_xacro parent="lf_lowerleg">
+        <origin xyz="0.39415 0.00775 -0.1" rpy="${PI/2} 0 0"/>
+    </xacro:new_calibration_plate_xacro -->
 </robot>

Commit message: fix urdf error and python2 error

File: robots/hyq.urdf.xacro (robot description, xacro)
@@ -11,7 +11,7 @@
 	<xacro:include filename="$(find hyq_description)/urdfs/leg/leg.urdf.xacro"/>
 	<!-- generic simulator_gazebo plugins for starting mechanism control, ros time -->
-        <xacro:include filename="$(find hyq_description)/gazebo/gazebo.urdf.xacro">
-             <xacro:arg name="task_period" value="$(arg task_period)"/>
-        </xacro:include>
+    <xacro:include filename="$(find hyq_description)/gazebo/gazebo.urdf.xacro">
+        <xacro:arg name="task_period" value="$(arg task_period)"/>
+    </xacro:include>
 	<!-- Now we can start using the macros included above to define the actual HyQ -->
 	<!-- The first use of a macro. This one was defined in trunk.urdf.xacro above.

File: urdfs/common.xacro (robot description, xacro)
@@ -64,7 +64,7 @@
 	<xacro:property name="ixz_lowerleg" value="-0.00001"/>
 	<xacro:property name="iyz_lowerleg" value="-0.0"/>
-        <!-- arm position-->
-        <xacro:property name="x_arm" value="0.66"/>
-        <xacro:property name="z_arm" value="0.1"/>
-        <xacro:property name="pitch_arm" value="0.17"/>
+    <!-- arm position-->
+    <xacro:property name="x_arm" value="0.66"/>
+    <xacro:property name="z_arm" value="0.1"/>
+    <xacro:property name="pitch_arm" value="0.17"/>
 </robot>

File: urdfs/trunk/trunk.urdf.xacro (robot description, xacro)
@@ -6,18 +6,6 @@
 	<!-- The xacro macro xacro:hyq_base contains: base and trunk -->
 	<xacro:macro name="hyq_trunk" params="name">
-		  <!-- Floating-base Joint -->
-                <link name="world"/>
-                <joint name="floating_base_joint" type="floating">
-                  <origin rpy="0 0 0" xyz="0 0 0"/>
-                  <parent link="world"/>
-                  <child link="base_link"/>
-                </joint>
-                <joint name="floating_base" type="fixed">
-                  <origin rpy="0 0 0" xyz="0 0 0"/>
-                  <parent link="base_link"/>
-                  <child link="trunk"/>
-                </joint>
-		<!-- Links -->
 		<!-- Footprint link -->
+		<!-- inertial to avoid being ignore!-->
 		<link name="${name}_link">
 			<visual>
@@ -27,6 +15,13 @@
 			</visual>
 		</link>
-		<!-- Trunk link -->
+		<!-- Trunk link-->
+		<!-- value manually found with RVIZ to correctly align the trunk to the hip assemblies -->
 		<link name="trunk">
+			<visual>
+				<origin xyz="0 0 -0.0082" />
+				<geometry>
+					<mesh filename="package://hyq_description/meshes/trunk/trunk.dae" scale="1 1 1" />
+				</geometry>
+			</visual>
 			<inertial>
 				<origin xyz="${xcom_trunk} ${ycom_trunk} ${zcom_trunk}"/>
@@ -35,19 +30,16 @@
 						 ixy="${ixy_trunk}" ixz="${ixz_trunk}" iyz="${iyz_trunk}"/>
 			</inertial>
-			<visual>
-				<!-- value manually found with RVIZ to correctly align the trunk to the hip assemblies -->
-				<origin  xyz="0 0 -0.0082" />
+			<collision>
+				<origin xyz="0 0 -0.0082" />
 				<geometry>
-					<mesh filename="package://hyq_description/meshes/trunk/trunk.dae" scale="1 1 1"/>
-				</geometry>
-			</visual>
-			<collision>
-				<!-- value manually found with RVIZ to correctly align the trunk to the hip assemblies -->
-				<origin  xyz="0 0 -0.0082" />
-				<geometry>
-					<mesh filename="package://hyq_description/meshes/trunk/trunk.dae" scale="1 1 1"/>
+					<mesh filename="package://hyq_description/meshes/trunk/trunk.dae" scale="1 1 1" />
 				</geometry>
 			</collision>
 		</link>
+        <joint name="floating_base" type="fixed">
+            <origin rpy="0 0 0" xyz="0 0 0"/>
+            <parent link="base_link"/>
+            <child link="trunk"/>
+        </joint>
 		<!-- Extensions -->
 		<xacro:trunk_gazebo name="trunk"/>
