Commit message: setting proper contact values for shin and foot
Hi all I will summarize the results of our difficult and painful
debugging month

1) in  Gazebo 2.0

the properties of a fake link (e.g. the link_foot) were inherithing the
properties of the parent foot (e.g. the lowerleg)

in our case to have a proper contact behaviour we were setting the
contact stiffness to kp = 1000000 and the damping to kd= 100

in Gazebo 7.0 this does not happen anymore, so the stiffness and the
damping for the foot were not kp = 1000000 and the damping to kd= 100

anymore but were set to the MAXIMUM possible value screwing the
simulation (the robot glides...)

2) to have meaningful joint velocity readings we should set the
parameter <max_vel>1.0</max_vel>

otherwise it spits out crappy value (again this value was not set for
the foot and the joint velocities  were not meaningful)

File: urdfs/leg/leg.gazebo.xacro (robot description, xacro)
@@ -53,14 +53,19 @@
 			<kp>1000000.0</kp>
 			<kd>100.0</kd>
-			<mu1>1.5</mu1>
-			<mu2>1.5</mu2>
-			<fdir1>1 0 0</fdir1>
+			<mu1>1.0</mu1>
+			<mu2>1.0</mu2>
 			<maxVel>1.0</maxVel>
-			<minDepth>0.00</minDepth>
+			<maxContacts>1</maxContacts>
 		</gazebo>
 		<gazebo reference="${name}_foot">
+                        <kp>1000000.0</kp>
+                        <kd>100.0</kd>
+                        <mu1>1.0</mu1>
+                        <mu2>1.0</mu2>
+                        <maxVel>1.0</maxVel>
+			<maxContacts>1</maxContacts>
 			<sensor name="${name}_foot_contact_sensor" type="contact">
 				<always_on>true</always_on>
-				<update_rate>1000.0</update_rate>
+				<update_rate>250.0</update_rate>
 				<contact>
 					<collision>${name}_lowerleg_fixed_joint_lump__${name}_foot_collision_1</collision>
@@ -71,4 +76,5 @@
 				</plugin>
 			</sensor>
+			<material>Gazebo/Black</material>
 		</gazebo>
 	</xacro:macro>

File: urdfs/leg/leg.urdf.xacro (robot description, xacro)
@@ -120,16 +120,4 @@
 		<!-- Foot link -->
 		<link name="${name}_foot">
-			<inertial>
-				<origin xyz="0 0 0"/>
-				<mass value="0.0"/>
-				<inertia ixx="0.0" iyy="0.0" izz="0.0" ixy="0.0" ixz="0.0" iyz="0.0"/>
-			</inertial>
-			<visual>
-                <origin xyz="0 0 0" rpy="0 0 0"/>
-                <geometry>
-                    <sphere radius="0.02175"/>
-                </geometry>
-				<material name="black"/>
-            </visual>
 			<collision>
 				<origin xyz="0 0 0" rpy="0 0 0"/>
@@ -138,8 +126,11 @@
 				</geometry>
 			</collision>
+			<visual>
+				<geometry>
+					<sphere radius="0.02175" />
+				</geometry>
+				<material name="black" />
+			</visual>
 		</link>
-		<gazebo reference="${name}_foot">
-            <material>Gazebo/Black</material>
-        </gazebo>
 		<!-- Extensions -->
 		<xacro:leg_transmission name="${name}"/>

Commit message: setting proper contact values for shin and foot
Hi all I will summarize the results of our difficult and painful
debugging month

1) in  Gazebo 2.0

the properties of a fake link (e.g. the link_foot) were inherithing the
properties of the parent foot (e.g. the lowerleg)

in our case to have a proper contact behaviour we were setting the
contact stiffness to kp = 1000000 and the damping to kd= 100

in Gazebo 7.0 this does not happen anymore, so the stiffness and the
damping for the foot were not kp = 1000000 and the damping to kd= 100

anymore but were set to the MAXIMUM possible value screwing the
simulation (the robot glides...)

2) to have meaningful joint velocity readings we should set the
parameter <max_vel>1.0</max_vel>

otherwise it spits out crappy value (again this value was not set for
the foot and the joint velocities  were not meaningful)

File: urdfs/leg/leg.gazebo.xacro (robot description, xacro)
@@ -53,9 +53,7 @@
 			<kp>1000000.0</kp>
 			<kd>100.0</kd>
-			<mu1>1.5</mu1>
-			<mu2>1.5</mu2>
-			<fdir1>1 0 0</fdir1>
+			<mu1>1.0</mu1>
+			<mu2>1.0</mu2>
 			<maxVel>1.0</maxVel>
-			<minDepth>0.001</minDepth>
 			<maxContacts>1</maxContacts>
 			<sensor name="${name}_shin_contact_sensor" type="contact">
@@ -72,4 +70,10 @@
 		</gazebo>
 		<gazebo reference="${name}_foot">
+                        <kp>1000000.0</kp>
+                        <kd>100.0</kd>
+                        <mu1>1.0</mu1>
+                        <mu2>1.0</mu2>
+                        <maxVel>1.0</maxVel>
+			<maxContacts>1</maxContacts>
 			<sensor name="${name}_foot_contact_sensor" type="contact">
 				<always_on>true</always_on>
@@ -83,4 +87,5 @@
 				</plugin>
 			</sensor>
+			<material>Gazebo/Black</material>
 		</gazebo>
 	</xacro:macro>

File: urdfs/leg/leg.urdf.xacro (robot description, xacro)
@@ -121,9 +121,4 @@
 		<!-- Foot link -->
 		<link name="${name}_foot">
-			<inertial>
-				<origin xyz="0 0 0"/>
-				<mass value="0.07"/>
-				<inertia ixx="0.0000112" iyy="0.0000112" izz="0.0000112" ixy="0.0" ixz="0.0" iyz="0.0"/>
-			</inertial>
 			<collision>
 				<origin xyz="0 0 0" rpy="0 0 0"/>
@@ -139,13 +134,4 @@
 			</visual>
 		</link>
-		<gazebo reference="${name}_foot">
-                	<mu1>1</mu1>
-			<mu2>1</mu2>
-			<fdir1>1 0 0</fdir1>
-			<maxContacts>1</maxContacts>
-                        <minDepth>0.002</minDepth>
-                        <gravity>true</gravity>
-            	<material>Gazebo/Black</material>
-        	</gazebo>
 		<!-- Extensions -->
 		<xacro:leg_transmission name="${name}"/>

Commit message: bufix corrected name for collision of foot sensor

File: urdfs/leg/leg.gazebo.xacro (robot description, xacro)
@@ -80,5 +80,5 @@
 				<update_rate>250.0</update_rate>
 				<contact>
-					<collision>${name}_foot_collision</collision>
+					<collision>${name}_lowerleg_fixed_joint_lump__${name}_foot_collision_1</collision>
 				</contact>
 				<plugin name="${name}_foot_bumper" filename="libgazebo_ros_bumper.so">

Commit message: adding shin bumper sensor

File: urdfs/leg/leg.gazebo.xacro (robot description, xacro)
@@ -57,4 +57,15 @@
 			<maxVel>1.0</maxVel>
 			<maxContacts>1</maxContacts>
+			<sensor name="${name}_shin_contact_sensor" type="contact">
+                <always_on>true</always_on>
+                <update_rate>250.0</update_rate>
+                <contact>
+                  <collision>${name}_lowerleg_collision</collision>
+                </contact>
+                <plugin name="${name}_shin_bumper" filename="libgazebo_ros_bumper.so">
+                  <bumperTopicName>/hyq/${name}_shin_bumper</bumperTopicName>
+                  <frameName>base_link</frameName>
+                </plugin>
+            </sensor>
 		</gazebo>
 		<gazebo reference="${name}_foot">
@@ -72,6 +83,7 @@
 				</contact>
 				<plugin name="${name}_foot_bumper" filename="libgazebo_ros_bumper.so">
-					<bumperTopicName>/${name}_grf</bumperTopicName>
+					<bumperTopicName>/hyq/${name}_foot_bumper</bumperTopicName>
 					<frameName>base_link</frameName>
+					<robotNamespace>hyq</robotNamespace>
 				</plugin>
 			</sensor>
