Commit message: added ext_ prefix to see the plate

File: urdfs/leg/calibration_plate.urdf.xacro (robot description, xacro)
@@ -5,7 +5,7 @@
 		<xacro:insert_block name="origin"/>
 		<parent link="${parent}"/>
-		<child link="calibration_plate_head"/>
+		<child link="ext_calibration_plate_head"/>
 	</joint>
-	<link name="calibration_plate_head">
+	<link name="ext_calibration_plate_head">
 		<inertial>
 			<origin xyz="0 0 0" rpy="0 0 0" />
