Commit message: Removed the mass of the foot. Cleaned a bit the code

File: urdfs/leg/leg.urdf.xacro (robot description, xacro)
@@ -122,13 +122,7 @@
 			<inertial>
 				<origin xyz="0 0 0"/>
-				<mass value="0.01"/>
+				<mass value="0.0"/>
 				<inertia ixx="0.0" iyy="0.0" izz="0.0" ixy="0.0" ixz="0.0" iyz="0.0"/>
 			</inertial>
-			<!--<visual>
-				<origin xyz="0.0 0.0 0.0" rpy="0.0 0.0 0.0"/>
-				<geometry>
-					<sphere radius="0.021"/>
-				</geometry>
-			</visual>-->
 			<collision>
 				<origin xyz="0 0 0" rpy="0 0 0"/>

Commit message: added visualization for feet balls

File: urdfs/leg/leg.urdf.xacro (robot description, xacro)
@@ -125,4 +125,10 @@
 				<inertia ixx="0.0" iyy="0.0" izz="0.0" ixy="0.0" ixz="0.0" iyz="0.0"/>
 			</inertial>
+			<visual>
+                <origin xyz="0 0 0" rpy="0 0 0"/>
+                <geometry>
+                    <sphere radius="0.02175"/>
+                </geometry>
+            </visual>
 			<collision>
 				<origin xyz="0 0 0" rpy="0 0 0"/>
@@ -132,4 +138,7 @@
 			</collision>
 		</link>
+		<gazebo reference="${name}_foot">
+            <material>Gazebo/Black</material>
+        </gazebo>
 		<!-- Extensions -->
 		<xacro:leg_transmission name="${name}"/>

Commit message: [cleanup] Added the black color to the foot

File: urdfs/leg/leg.urdf.xacro (robot description, xacro)
@@ -130,4 +130,5 @@
                     <sphere radius="0.02175"/>
                 </geometry>
+				<material name="black"/>
             </visual>
 			<collision>

Commit message: Commented collision with perfect spheric feet because robot slips (probably the torsional friction cannot be set)

File: urdfs/leg/leg.urdf.xacro (robot description, xacro)
@@ -132,10 +132,10 @@
 				<material name="black"/>
             </visual>
-			<collision>
+			<!--collision>
 				<origin xyz="0 0 0" rpy="0 0 0"/>
 				<geometry>
 					<sphere radius="0.02175"/>
 				</geometry>
-			</collision>
+			</collision-->
 		</link>
 		<gazebo reference="${name}_foot">

Commit message: Fixed the slipping problem with robot feet

File: urdfs/leg/leg.urdf.xacro (robot description, xacro)
@@ -123,24 +123,29 @@
 			<inertial>
 				<origin xyz="0 0 0"/>
-				<mass value="0.0"/>
-				<inertia ixx="0.0" iyy="0.0" izz="0.0" ixy="0.0" ixz="0.0" iyz="0.0"/>
+				<mass value="0.07"/>
+				<inertia ixx="0.0000112" iyy="0.0000112" izz="0.0000112" ixy="0.0" ixz="0.0" iyz="0.0"/>
 			</inertial>
-			<visual>
-                <origin xyz="0 0 0" rpy="0 0 0"/>
-                <geometry>
-                    <sphere radius="0.02175"/>
-                </geometry>
-				<material name="black"/>
-            </visual>
-			<!--collision>
+			<collision>
 				<origin xyz="0 0 0" rpy="0 0 0"/>
 				<geometry>
 					<sphere radius="0.02175"/>
 				</geometry>
-			</collision-->
+			</collision>
+			<visual>
+				<geometry>
+					<sphere radius="0.02175" />
+				</geometry>
+				<material name="black" />
+			</visual>
 		</link>
 		<gazebo reference="${name}_foot">
-            <material>Gazebo/Black</material>
-        </gazebo>
+                	<mu1>1</mu1>
+			<mu2>1</mu2>
+			<fdir1>1 0 0</fdir1>
+			<maxContacts>1</maxContacts>
+                        <minDepth>0.005</minDepth>
+                        <gravity>true</gravity>
+            	<material>Gazebo/Black</material>
+        	</gazebo>
 		<!-- Extensions -->
 		<xacro:leg_transmission name="${name}"/>

Commit message: artificially making the lf heavier (testing model uncertanties)

File: urdfs/leg/leg.urdf.xacro (robot description, xacro)
@@ -101,6 +101,15 @@
 		<link name="${name}_lowerleg">
 			<inertial>
-				<origin xyz="${xcom_lowerleg} ${reflect_front*ycom_lowerleg} ${reflect_front*zcom_lowerleg}"/>
-				<mass value="${m_lowerleg}"/>
+				<!-- adding half kg to lf lowerleg -->
+				<xacro:property name="var" value="${name}"/>
+				<xacro:property name="mass" value="${m_lowerleg}"/>
+				<xacro:if value="${var == 'lf'}">
+					<origin xyz="${xcom_lowerleg+0.15} ${reflect_front*ycom_lowerleg} ${reflect_front*zcom_lowerleg}"/>
+					<mass value="${mass + 3}"/>
+				</xacro:if>
+				<xacro:unless value="${var == 'lf'}">
+					<origin xyz="${xcom_lowerleg} ${reflect_front*ycom_lowerleg} ${reflect_front*zcom_lowerleg}"/>
+					<mass value="${m_lowerleg}"/>
+				</xacro:unless>
 				<inertia ixx="${ixx_lowerleg}" iyy="${iyy_lowerleg}" izz="${izz_lowerleg}"
 						 ixy="${reflect_front*ixy_lowerleg}" ixz="${reflect_front*ixz_lowerleg}" iyz="${iyz_lowerleg}"/>

Commit message: fix roslaunch and urdf file, add urdf color, remove unnecessary in-order agument, fix launch file name

File: urdfs/leg/leg.urdf.xacro (robot description, xacro)
@@ -110,5 +110,7 @@
 					<mesh filename="package://hyq_description/meshes/leg/lowerleg.dae" scale="1 1 1"/>
 				</geometry>
-				<material name="white"/>
+				<material name="White">
+					<color rgba="1.0 1.0 1.0 1.0"/>
+				</material>
 			</visual>
 			<collision>
@@ -131,5 +133,7 @@
 					<sphere radius="0.02175" />
 				</geometry>
-				<material name="black" />
+				<material name="Black" >
+					<color rgba="0.0 0.0 0.0 1.0"/>
+				</material>
 			</visual>
 		</link>
