Commit message: changed mass of cart to 20 kg otherwise it leans too much fwd and reach singularity
removed unuseful files
added collision to cart

File: urdfs/cart/cart.urdf.xacro (robot description, xacro)
@@ -68,5 +68,5 @@
        <link name="cart">
                   <inertial>
-            <mass value="30"/>
+            <mass value="20"/>
             <inertia ixx="1" ixy="0" ixz="0" iyy="1" iyz="0" izz="1"/>
           </inertial>
@@ -78,4 +78,11 @@
          <origin rpy="0 0 0" xyz="-0.5 0 0 "/>
        </visual>
+       <collision>
+          <geometry>
+              <box size="1.0 1.0 0.5"/>
+         </geometry>
+         <material name="black"/>
+         <origin rpy="0 0 0" xyz="-0.5 0 0 "/>
+       </collision>
      </link>
         <gazebo reference="cart">

File: urdfs/common.xacro (robot description, xacro)
@@ -22,6 +22,6 @@
 	<!-- Trunk with hydraulic system -->
 	<xacro:property name="xcom_trunk" value="0.056"/>
-	<xacro:property name="ycom_trunk" value="0.0215"/>
-	<xacro:property name="zcom_trunk" value="0.00358"/>
+	<xacro:property name="ycom_trunk" value="0.0"/>
+	<xacro:property name="zcom_trunk" value="0.0"/>
 	<xacro:property name="m_trunk" value="60.96"/>
 	<xacro:property name="ixx_trunk" value="1.5725937"/>
