Commit message: added friction on joints [skip ci]

File: urdfs/cart/car.urdf.xacro (robot description, xacro)
@@ -113,5 +113,6 @@
         <child link="ext_right_wheel"/>
         <origin rpy="1.57 0 0" xyz=" 0 -0.5 -0.25"/>
-         <axis xyz="0 0 1 "/>
+        <axis xyz="0 0 1"/>
+        <dynamics damping="0.1" friction="0.0"/>
       </joint>
      <link name="ext_right_wheel">
@@ -149,5 +150,6 @@
     <child link="ext_left_wheel"/>
     <origin rpy="-1.57 0 0" xyz=" 0 0.5 -0.25"/>
-     <axis xyz="0 0 1 "/>
+    <axis xyz="0 0 1"/>
+    <dynamics damping="0.1" friction="0.0"/>
   </joint>
   <link name="ext_left_wheel">
@@ -185,5 +187,6 @@
     <child link="ext_left_bwheel"/>
     <origin rpy="-1.57 0 0" xyz=" -1 0.5 -0.25"/>
-     <axis xyz="0 0 1 "/>
+    <axis xyz="0 0 1"/>
+    <dynamics damping="0.1" friction="0.0"/>
   </joint>
   <link name="ext_left_bwheel">
@@ -221,6 +224,7 @@
     <child link="ext_right_bwheel"/>
     <origin rpy="-1.57 0 0" xyz=" -1 -0.5 -0.25"/>
-     <axis xyz="0 0 1 "/>
-  </joint>
+    <axis xyz="0 0 1"/>
+    <dynamics damping="1" friction="0.0"/>
+</joint>
   <link name="ext_right_bwheel">
              <inertial>
