Commit message: Fixed the CoM positions of the leg given Michele and Guido input

File: urdfs/common.xacro (robot description, xacro)
@@ -43,5 +43,5 @@
 	<!-- Lower leg -->
 	<property name="xcom_lowerleg" value="0.1254"/>
-	<property name="ycom_lowerleg" value="0.00005"/>
+	<property name="ycom_lowerleg" value="0.00004"/>
 	<property name="zcom_lowerleg" value="-0.0001"/>
 	<property name="m_lowerleg" value="0.881"/>

File: urdfs/leg/leg.urdf.xacro (robot description, xacro)
@@ -80,5 +80,5 @@
 		<link name="${name}_upperleg">
 			<inertial>
-				<origin xyz="${xcom_upperleg} ${reflect_upper*ycom_upperleg} ${zcom_upperleg}"/>
+				<origin xyz="${xcom_upperleg} ${-reflect_front*ycom_upperleg} ${zcom_upperleg}"/>
 				<mass value="${m_upperleg}"/>
 				<inertia ixx="${ixx_upperleg}" iyy="${iyy_upperleg}" izz="${izz_upperleg}"
@@ -101,5 +101,5 @@
 		<link name="${name}_lowerleg">
 			<inertial>
-				<origin xyz="${xcom_lowerleg} ${ycom_lowerleg} ${zcom_lowerleg}"/>
+				<origin xyz="${xcom_lowerleg} ${reflect_front*ycom_lowerleg} ${reflect_front*zcom_lowerleg}"/>
 				<mass value="${m_lowerleg}"/>
 				<inertia ixx="${ixx_lowerleg}" iyy="${iyy_lowerleg}" izz="${izz_lowerleg}"

Commit message: corrected trunk of inertia which was expressed in the base frame instead than in the com frame
corrected kinematics to be consistent with the standard document

File: urdfs/common.xacro (robot description, xacro)
@@ -5,18 +5,19 @@
 	<property name="d_lr" value="0.414"/>
 	<property name="d_fh" value="0.747"/>
-	<property name="d_tbb" value="0.082"/>
+	<property name="d_tbb" value="0.08"/>
 	<property name="d_p1p2" value="0.35"/>
+	<property name="d_p2p3" value="0.33"/>
 	<!-- Inertial values -->
 	<!-- Trunk with hydraulic system -->
-	<property name="xcom_trunk" value="-0.02758"/>
-	<property name="ycom_trunk" value="-0.000023319"/>
-	<property name="zcom_trunk" value="0.03103"/>
-	<property name="m_trunk" value="50.24"/>
-	<property name="ixx_trunk" value="0.97322"/>
-	<property name="iyy_trunk" value="5.0487"/>
-	<property name="izz_trunk" value="5.283"/>
-	<property name="ixy_trunk" value="-0.0067362"/>
-	<property name="ixz_trunk" value="0.1681"/>
-	<property name="iyz_trunk" value="-0.0060307"/>
+	<property name="xcom_trunk" value="0.02707"/>
+	<property name="ycom_trunk" value="0.0000"/>
+	<property name="zcom_trunk" value="0.03290"/>
+	<property name="m_trunk" value="71.75800"/>
+	<property name="ixx_trunk" value="1.61053"/>
+	<property name="iyy_trunk" value="8.53505"/>
+	<property name="izz_trunk" value="9.19102"/>
+	<property name="ixy_trunk" value="-0.02880"/>
+	<property name="ixz_trunk" value="0.34161"/>
+	<property name="iyz_trunk" value="0.00380"/>
 	<!-- Hip assembly -->
 	<property name="xcom_hipassembly" value="0.04263"/>

File: urdfs/leg/leg.urdf.xacro (robot description, xacro)
@@ -49,5 +49,5 @@
 		</joint>
 		<joint name="${name}_foot_joint" type="fixed">
-			<origin xyz="0.35 0 0" rpy="${PI/2} 0 ${-PI/2}"/>
+			<origin xyz="${d_p2p3} 0 0" rpy="${PI/2} 0 ${-PI/2}"/>
 			<parent link="${name}_lowerleg"/>
 			<child  link="${name}_foot"/>

Commit message: Updated the values according to the latest reference document (HyQV1LegV2_StandardDefinitions_v3.pdf).This was the changes: foot position, haa joint limits

File: urdfs/common.xacro (robot description, xacro)
@@ -5,7 +5,7 @@
 	<property name="d_lr" value="0.414"/>
 	<property name="d_fh" value="0.747"/>
-	<property name="d_tbb" value="0.08"/>
+	<property name="d_p0p1" value="0.08"/>
 	<property name="d_p1p2" value="0.35"/>
-	<property name="d_p2p3" value="0.33"/>
+	<property name="d_p2p3" value="0.341"/>
 	<!-- Inertial values -->
 	<!-- Trunk with hydraulic system -->

File: urdfs/leg/leg.urdf.xacro (robot description, xacro)
@@ -14,12 +14,12 @@
 			<child  link="${name}_hipassembly"/>
 			<axis xyz="0 0 1"/>
-			<limit effort="150.0" velocity="12.0" lower="${-7*PI/18}" upper="${PI/6}"/>
+			<limit effort="150.0" velocity="12.0" lower="${-7*PI/18}" upper="${5*PI/36}"/>
 			<dynamics damping="0.1" friction="0" />
 			<safety_controller k_position="100" k_velocity="100"
-							   soft_lower_limit="${-7*PI/18}" soft_upper_limit="${PI/6}" />
+							   soft_lower_limit="${-7*PI/18}" soft_upper_limit="${5*PI/36}" />
 		</joint>
 		<!-- Upper leg joint -->
 		<joint name="${name}_hfe_joint" type="revolute">
-			<origin xyz="${d_tbb} 0 0" rpy="${reflect_upper*PI/2} 0 0"/>
+			<origin xyz="${d_p0p1} 0 0" rpy="${reflect_upper*PI/2} 0 0"/>
 			<parent link="${name}_hipassembly"/>
 			<child  link="${name}_upperleg"/>

Commit message: [bullet] The missed material properties are needed for bullet engine

File: urdfs/common.xacro (robot description, xacro)
@@ -53,3 +53,13 @@
 	<property name="ixz_lowerleg" value="-0.00001"/>
 	<property name="iyz_lowerleg" value="-0.0"/>
+    <!-- Materials -->
+    <material name="black">
+      <color rgba="0 0 0 1"/>
+    </material>
+    <material name="grey">
+      <color rgba="0.45 0.45 0.45 1"/>
+    </material>
+    <material name="green">
+      <color rgba="0 0.75 0 1"/>
+    </material>
 </robot>

File: urdfs/leg/leg.urdf.xacro (robot description, xacro)
@@ -69,4 +69,5 @@
 					<mesh filename="package://hyq_description/meshes/leg/hipassembly.dae" scale="1 1 1"/>
 				</geometry>
+				<material name="grey"/>
 			</visual>
 			<collision>
@@ -90,4 +91,5 @@
 					<mesh filename="package://hyq_description/meshes/leg/upperleg.dae" scale="1 1 1"/>
 				</geometry>
+				<material name="grey"/>
 			</visual>
 			<collision>
@@ -110,5 +112,5 @@
 					<mesh filename="package://hyq_description/meshes/leg/lowerleg.dae" scale="1 1 1"/>
 				</geometry>
-				<material name="white"/>
+				<material name="grey"/>
 			</visual>
 			<collision>

File: urdfs/trunk/trunk.urdf.xacro (robot description, xacro)
@@ -33,4 +33,5 @@
 					<mesh filename="package://hyq_description/meshes/trunk/trunk.dae" scale="1 1 1"/>
 				</geometry>
+				<material name="green"/>
 			</visual>
 			<collision>

Commit message: [update] trunk mass and com after trying with experiments (now the multisense mass is accounted separately from the trunk)

File: urdfs/common.xacro (robot description, xacro)
@@ -21,8 +21,8 @@
 	<!-- Inertial values -->
 	<!-- Trunk with hydraulic system -->
-	<xacro:property name="xcom_trunk" value="0.056"/>
-	<xacro:property name="ycom_trunk" value="0.0215"/>
+	<xacro:property name="xcom_trunk" value="0.01"/>
+	<xacro:property name="ycom_trunk" value="0.0"/>
 	<xacro:property name="zcom_trunk" value="0.00358"/>
-	<xacro:property name="m_trunk" value="60.96"/>
+	<xacro:property name="m_trunk" value="58.96"/>
 	<xacro:property name="ixx_trunk" value="1.5725937"/>
 	<xacro:property name="iyy_trunk" value="8.5015928"/>

Commit message: [!important] updated lowerleg length after removing foot sensor

File: urdfs/common.xacro (robot description, xacro)
@@ -18,5 +18,5 @@
 	<xacro:property name="hipassembly_length" value="0.08"/>
 	<xacro:property name="upperleg_length" value="0.35"/>
-	<xacro:property name="lowerleg_length" value="0.346"/>
+        <xacro:property name="lowerleg_length" value="0.341"/>
 	<!-- Inertial values -->
 	<!-- Trunk with hydraulic system -->
