Commit message: bugfix align the trunk correctly

File: urdfs/trunk/trunk.urdf.xacro (robot description, xacro)
@@ -30,4 +30,6 @@
 			</inertial>
 			<visual>
+				<!-- value manually found with RVIZ to correctly align the trunk to the hip assemblies -->
+				<origin  xyz="0 0 -0.0082" />
 				<geometry>
 					<mesh filename="package://hyq_description/meshes/trunk/trunk.dae" scale="1 1 1"/>
@@ -35,4 +37,6 @@
 			</visual>
 			<collision>
+				<!-- value manually found with RVIZ to correctly align the trunk to the hip assemblies -->
+				<origin  xyz="0 0 -0.0082" />
 				<geometry>
 					<mesh filename="package://hyq_description/meshes/trunk/trunk.dae" scale="1 1 1"/>

Commit message: Hyq description modified to work with the wb controller

File: urdfs/trunk/trunk.urdf.xacro (robot description, xacro)
@@ -6,10 +6,16 @@
 	<!-- The xacro macro xacro:hyq_base contains: base and trunk -->
 	<xacro:macro name="hyq_trunk" params="name">
-		<!-- Floating-base Joint -->
-		<joint name="floating_base" type="fixed">
-			<origin xyz="0 0 0" rpy="0 0 0"/>
-			<parent link="${name}_link"/>
-			<child link="trunk"/>
-		</joint>
+		  <!-- Floating-base Joint -->
+                <link name="world"/>
+                <joint name="floating_base_joint" type="floating">
+                  <origin rpy="0 0 0" xyz="0 0 0"/>
+                  <parent link="world"/>
+                  <child link="base_link"/>
+                </joint>
+                <joint name="floating_base" type="fixed">
+                  <origin rpy="0 0 0" xyz="0 0 0"/>
+                  <parent link="base_link"/>
+                  <child link="trunk"/>
+                </joint>
 		<!-- Links -->
 		<!-- Footprint link -->
