Commit message: Changes to make code work with Hyq2Max interface

File: gazebo/gazebo.urdf.xacro (robot description, xacro)
@@ -4,5 +4,6 @@
 		<plugin name="gazebo_ros_controller_manager" filename="libgazebo_ros_control.so">
 			<robotNamespace>/hyq</robotNamespace>
-			<controlPeriod>0.001</controlPeriod>
+			<robotSimType>hyq2max_gazebo/HyQ2MaxHWSim</robotSimType>
+			<controlPeriod>0.005</controlPeriod>
 		</plugin>
 		<plugin filename="libgazebo_ros_p3d.so" name="gazebo_ros_p3d">

File: robots/hyq.urdf.xacro (robot description, xacro)
@@ -71,6 +71,13 @@
 		imu_name="3dmgx325_trunk_imu"
 		imu_topic="trunk_imu/data"
-		update_rate="100.0"
-		stdev="0.00017">
+		update_rate="1000"
+		rate_mean="0"
+		rate_stddev="2e-4"
+		rate_bias_mean="0.00087"
+		rate_bias_stddev="0.0000008"
+		accel_mean="0"
+		accel_stddev="1.7e-2"
+		accel_bias_mean="0.002"
+		accel_bias_stddev="0.001">
 		<origin xyz="0.4825 0.006 0.0905" rpy="0 ${-PI} 0"/>
 	</xacro:microstrain_3dmgx325_imu>

File: robots/hyq_model.urdf.xacro (robot description, xacro)
@@ -63,7 +63,14 @@
 		imu_name="3dmgx325_trunk_imu"
 		imu_topic="trunk_imu/data"
-		update_rate="100.0"
-		stdev="0.00017">
-		<origin xyz="0.3 0 0.095" rpy="0 ${-PI} 0"/>
+		update_rate="1000"
+		rate_mean="0"
+		rate_stddev="2e-4"
+		rate_bias_mean="0.00087"
+		rate_bias_stddev="0.0000008"
+		accel_mean="0"
+		accel_stddev="1.7e-2"
+		accel_bias_mean="0.002"
+		accel_bias_stddev="0.001">
+		<origin xyz="0.4825 0.006 0.0905" rpy="0 ${-PI} 0"/>
 	</xacro:microstrain_3dmgx325_imu>
 </robot>

File: urdfs/sensors/microstrain_3dmgx325_imu.gazebo.xacro (robot description, xacro)
@@ -1,5 +1,6 @@
 <?xml version="1.0"?>
 <robot xmlns:xacro="http://ros.org/wiki/xacro">
-	<xacro:macro name="microstrain_3dmgx325_imu_sensor" params="imu_name imu_topic update_rate stdev">
+	<xacro:macro name="microstrain_3dmgx325_imu_sensor" params="imu_name imu_topic update_rate
+		rate_mean rate_stddev rate_bias_mean rate_bias_stddev accel_mean accel_stddev accel_bias_mean accel_bias_stddev">
 		<gazebo>
 			<plugin name="${imu_name}_controller" filename="libgazebo_ros_imu.so">
@@ -8,5 +9,5 @@
 				<bodyName>${imu_name}</bodyName>
 				<topicName>${imu_topic}</topicName>
-				<gaussianNoise>${stdev*stdev}</gaussianNoise>
+				<gaussianNoise>${rate_stddev*rate_stddev}</gaussianNoise>
 				<xyzOffset>0 0 0</xyzOffset>
 				<rpyOffset>0 0 0</rpyOffset>
@@ -14,4 +15,28 @@
 			</plugin>
 		</gazebo>
+		<!-- Imu definition required for HyQ2Max hardware interface of ros control -->
+		<gazebo reference="${imu_name}">
+			<sensor name="trunk_imu" type="imu">
+				<always_on>1</always_on>
+				<update_rate>${update_rate}</update_rate>
+				<imu>
+					<noise>
+						<type>gaussian</type>
+						<rate>
+							<mean>${rate_mean}</mean>
+							<stddev>${rate_stddev}</stddev>
+							<bias_mean>${rate_bias_mean}</bias_mean>
+							<bias_stddev>${rate_bias_stddev}</bias_stddev>
+						</rate>
+						<accel>
+							<mean>${accel_mean}</mean>
+							<stddev>${accel_stddev}</stddev>
+							<bias_mean>${accel_bias_mean}</bias_mean>
+							<bias_stddev>${accel_bias_stddev}</bias_stddev>
+						</accel>
+					</noise>
+				</imu>
+			</sensor>
+		</gazebo>
 	</xacro:macro>
 </robot>

File: urdfs/sensors/microstrain_3dmgx325_imu.urdf.xacro (robot description, xacro)
@@ -4,5 +4,6 @@
 	<!-- ============================ IMU microstrain ============================== -->
 	<!-- The xacro macro xacro:microstrain_3dmgx325_imu: imu frame -->
-	<xacro:macro name="microstrain_3dmgx325_imu" params="parent *origin imu_name imu_topic update_rate stdev">
+	<xacro:macro name="microstrain_3dmgx325_imu" params="parent *origin imu_name imu_topic update_rate
+		rate_mean rate_stddev rate_bias_mean rate_bias_stddev accel_mean accel_stddev accel_bias_mean accel_bias_stddev">
 		<!-- Joint -->
 		<joint name="${imu_name}_joint" type="fixed">
@@ -26,5 +27,9 @@
 		</link>
 		<!-- IMU definition -->
-		<xacro:microstrain_3dmgx325_imu_sensor imu_name="${imu_name}" imu_topic="${imu_topic}" update_rate="${update_rate}" stdev="${stdev}"/>
+		<xacro:microstrain_3dmgx325_imu_sensor imu_name="${imu_name}" imu_topic="${imu_topic}"
+		 	update_rate="${update_rate}" rate_mean="${rate_mean}" rate_stddev="${rate_stddev}"
+		 	rate_bias_mean="${rate_bias_mean}" rate_bias_stddev="${rate_bias_stddev}"
+		 	accel_mean="${accel_mean}" accel_stddev="${accel_stddev}" accel_bias_mean="${accel_bias_mean}"
+		 	accel_bias_stddev="${accel_bias_stddev}"/>
 	</xacro:macro>
 </robot>

Commit message: modifications to make hyqdescription robot independent

File: gazebo/gazebo.urdf.xacro (robot description, xacro)
@@ -5,6 +5,7 @@
 		<plugin name="gazebo_ros_controller_manager" filename="libgazebo_ros_control.so">
 			<robotNamespace>/hyq</robotNamespace>
-			<robotSimType>dls_gazebo_interface/DlsRobotHwSim</robotSimType>
-                        <controlPeriod>$(arg task_period)</controlPeriod>
+			<robotSimType>gazebo_ros_control/DefaultRobotHWSim</robotSimType>
+			<legacyModeNS>true</legacyModeNS>
+            <controlPeriod>$(arg task_period)</controlPeriod>
 		</plugin>
 		<plugin filename="libgazebo_ros_p3d.so" name="gazebo_ros_p3d">

File: robots/hyq.urdf.xacro (robot description, xacro)
@@ -2,26 +2,12 @@
 <robot name="hyq" xmlns:xacro="http://ros.org/wiki/xacro">
 	<xacro:arg name="task_period" default="0.004"/>
-	<xacro:arg name="sensors" default="true"/>
-	<xacro:arg name="arm" default="false"/>
 	<!-- This argument allows us to load joint sensors that measure the internal wrenches -->
 	<xacro:arg name="load_force_sensors" default="false"/>
 	<!-- The following included files set up definitions of parts of the robot body -->
 	<xacro:include filename="$(find hyq_description)/urdfs/common.xacro"/>
-	<xacro:include filename="$(find sensors_description)/urdfs/common.xacro"/>
 	<!-- HyQ trunk -->
 	<xacro:include filename="$(find hyq_description)/urdfs/trunk/trunk.urdf.xacro"/>
 	<!-- HyQ legs -->
 	<xacro:include filename="$(find hyq_description)/urdfs/leg/leg.urdf.xacro"/>
-	<!-- HyQ sensors -->
-        <xacro:if value="$(arg sensors)">
-            <xacro:include filename="$(find sensors_description)/urdfs/sensors/microstrain_3dmgx425_imu.urdf.xacro"/>
-            <xacro:include filename="$(find sensors_description)/urdfs/sensors/kvh_1775_imu.urdf.xacro"/>
-            <!--xacro:include filename="$(find sensors_description)/urdfs/sensors/asus_xtion.urdf.xacro"/-->
-            <!-- we may mount the hokuyo again in the future -->
-            <!--xacro:include filename="$(find sensors_description)/urdfs/sensors/hokuyo_laser.urdf.xacro"/-->
-            <!--xacro:include filename="$(find sensors_description)/urdfs/sensors/multisense_sl.urdf.xacro"/-->
-            <xacro:include filename="$(find sensors_description)/urdfs/sensors/d435_camera.urdf.xacro"/>
-        </xacro:if>
-        <xacro:include filename="$(find hyq_description)/urdfs/leg/new_calibration_plate.urdf.xacro"/>
 	<!-- generic simulator_gazebo plugins for starting mechanism control, ros time -->
         <xacro:include filename="$(find hyq_description)/gazebo/gazebo.urdf.xacro">
@@ -85,93 +71,3 @@
 		<origin xyz="${-d_fh/2} ${-d_lr/2} 0" rpy="0 ${PI/2} 0"/>
 	</xacro:hyq_leg>
-<xacro:if value="$(arg arm)">
-        <joint name="joint_base_robots" type="fixed">
-                <parent link="base_link"/>
-                <child link="teleop_link0"/>
-                <origin xyz="${x_arm} 0 ${z_arm}" rpy="0 ${pitch_arm} 0"/>
-        </joint>
-	<!-- SELECTION OF KINEMATICS CHAINS IS HANDLED INSIDE THE FILES -->
-	<xacro:include filename="$(find teleop_urdf)/urdf/teleop.urdf.xacro" />
-        <xacro:include filename="$(find hyq_description)/urdfs/arm/arm.transmission.xacro"/>
-        <xacro:arm_transmission name="joint1"/>
-        <xacro:arm_transmission name="joint2"/>
-        <xacro:arm_transmission name="joint3"/>
-        <xacro:arm_transmission name="joint4"/>
-        <xacro:arm_transmission name="joint5"/>
-</xacro:if>
-<xacro:if value="$(arg sensors)">
-	<!-- IMU trunk -->
-        <xacro:microstrain_3dmgx425_imu
-		parent="trunk"
-		imu_name="trunk_imu"
-		imu_topic="trunk_imu_1/data"
-                update_rate="250"
-                frame_name="trunk_imu"
-                >
-		<!-- old URDF -->
-		<!--origin xyz="0.290 0.000 0.0999214" rpy="0 ${-PI} 0"/ -->
-		<!-- new URDF with ideal values from CAD -->
-                <!--origin xyz="0.28525 0.000 0.0967678" rpy="0 0 0"/-->
-		<!-- new URDF, REAL values manually measured from the edge of the robot -->
-                <origin xyz="0.27025 0.000 0.0967678" rpy="0 0 0"/>
-        </xacro:microstrain_3dmgx425_imu>
-        <!-- IMU trunk -->
-        <!-- TODO We have to substitute the microstrain IMU with this one. Note that the imu_name has to be
-                  trunk_imu because the DLS HW interfaces hardcoded that name -->
-    	<xacro:kvh_1775_imu
-                parent="trunk"
-                imu_name="trunk_imu2"
-                imu_topic="trunk_imu_2/data"
-                update_rate="250"
-                frame_name="trunk_imu2"
-                >
-	    <!-- OLD URDF with manually created cylinder -->
-            <!--origin xyz="0.352845 0.0029 0.0503678" rpy="0 ${-PI} 0"/-->
-            <!-- NEW URDF with mesh, ideal values from CAD -->
-            <!--origin xyz="0.36347 0.00 0.0887678" rpy="0 ${PI} ${PI/4}"/-->
-	    	<!-- NEW URDF with mesh, REAL values measured from the edge of the robot -->
-		<!-- x = (500 - 153 - 61.77/2) / 1000	-->
-		<!-- y = from CAD -->
-		<origin xyz="0.316115 0.00 0.0887678" rpy="0 ${PI} ${PI/4}"/>
-        </xacro:kvh_1775_imu>
-	<!-- Hokuyo -->
-	<!--xacro:hokuyo_laser
-		name="laser"
-		parent="trunk"
-		ros_topic="scan"
-		update_rate="10"
-		min_angle="-5"
-		max_angle="5"
-		range="4.0">
-            <origin xyz="0.475 0.0 -0.08823" rpy="${PI} 0.0 0"/>
-	</xacro:hokuyo_laser-->
-	<!-- Asus Xtion Pro -->
-        <!--xacro:asus_xtion_camera name="asus" parent="trunk">
-		<origin xyz="0.660678 -0.00571526 0.0705706" rpy="0.0364271 1.00115 0.0827391"/>
-        </xacro:asus_xtion_camera-->
-        <xacro:d435_camera parent="trunk" prefix="realsense/front">
-            <!-- "Guess" of camera location -->
-            <!-- origin xyz="0.5 0.0 -0.10" rpy="0 ${PI/4} 0"/ -->
-            <!-- LF calibration trials using ipopt -->
-            <!-- origin xyz="0.556849 0.0275077 -0.0799648" rpy=" rpy="-0.0872665 0.791739 0.0872665"/>
-            <origin xyz="0.557156 0.0299427 -0.0775026" rpy=" rpy="-0.0327945 0.799206 -0.0252025"/>
-            <origin xyz="0.541865 0.0322597 -0.0730521" rpy=" rpy="-0.0447015 0.755414 -0.00943697"/>
-            <origin xyz="0.552173 0.0360462 -0.0749277" rpy=" rpy="-0.0640513 0.774692 0.0103402"/>
-            <origin xyz="0.55039 0.0327616 -0.0749135" rpy=" rpy="-0.0513261 0.773668 0.00448148"/ -->
-            <!-- Average of trials -->
-            <origin xyz="0.552 0.032 -0.076" rpy="-0.056 0.766 -0.007"/>
-        </xacro:d435_camera>
-        <xacro:d435_camera parent="trunk" prefix="realsense/back">
-            <!-- origin xyz="-0.5 -0.0 -0.10" rpy="0 ${PI/4} ${PI}"/ -->
-            <!-- Rear calibration failed, using approximate values from front camera -->
-            <origin xyz="-0.552 0.0 -0.076" rpy="0 ${PI/4} ${PI}"/>
-        </xacro:d435_camera>
-    </xacro:if>
-    <!--xacro:new_calibration_plate_xacro parent="rh_lowerleg">
-        <origin xyz="0.39 -0.01 0.1" rpy="${-PI/2} 0 0"/>
-    </xacro:new_calibration_plate_xacro-->
-    <!-- Numbers from Chundri Aug. 2019 -->
-    <!-- xacro:new_calibration_plate_xacro parent="lf_lowerleg">
-        <origin xyz="0.39415 0.00775 -0.1" rpy="${PI/2} 0 0"/>
-    </xacro:new_calibration_plate_xacro -->
 </robot>

File: robots/hyq_model.urdf.xacro (robot description, xacro)
@@ -9,5 +9,4 @@
 	<!-- generic simulator_gazebo plugins for starting mechanism control, ros time -->
 	<xacro:include filename="$(find hyq_description)/gazebo/gazebo.urdf.xacro"/>
-        <xacro:include filename="$(find sensors_description)/urdfs/sensors/microstrain_3dmgx425_imu.urdf.xacro"/>
 	<!-- Now we can start using the macros included above to define the actual HyQ -->
 	<!-- The first use of a macro. This one was defined in trunk.urdf.xacro above.

File: robots/hyq_model_ordered.urdf.xacro (robot description, xacro)
@@ -12,5 +12,4 @@
 	<!-- generic simulator_gazebo plugins for starting mechanism control, ros time -->
 	<xacro:include filename="$(find hyq_description)/gazebo/gazebo.urdf.xacro"/>
-        <xacro:include filename="$(find sensors_description)/urdfs/sensors/microstrain_3dmgx425_imu.urdf.xacro"/>
 	<!-- Now we can start using the macros included above to define the actual HyQ -->
 	<!-- The first use of a macro. This one was defined in trunk.urdf.xacro above.
@@ -78,13 +77,3 @@
 		<origin xyz="${-d_fh/2} ${-d_lr/2} 0" rpy="0 ${PI/2} 0"/>
 	</xacro:hyq_leg>
-	<!-- IMU trunk -->
-	<xacro:microstrain_3dmgx425_imu
-		parent="trunk"
-		imu_name="trunk_imu"
-		imu_topic="trunk_imu/data"
-                update_rate="250"
-                frame_name="trunk_imu"
-                >
-		<origin xyz="0.290 0.000 0.0999214" rpy="0 ${-PI} 0"/>
-	</xacro:microstrain_3dmgx425_imu>
 </robot>
